File: hardware/beta/kicad/aqroot-beta/05_i2c_devices.kicad_sch (KiCad schematic)
At the start: 0 parts

Commit message: AQROOT Beta: capture I2C, audio, IR, and SPI-A subsystems
Reconciles the active KiCad project from OneDrive into the canonical
repository. The four subsystem sheets existed here only as 169-byte
empty stubs; the real schematic capture had been done in the OneDrive
working copy.

Sheets brought in:
  03_spi_a_display_sd.kicad_sch   stub ->  62136 bytes
  05_i2c_devices.kicad_sch        stub ->  59631 bytes
  06_audio.kicad_sch              stub ->  55263 bytes
  07_ir.kicad_sch                 stub ->  50216 bytes

Also updated: aqroot-Beta.kicad_sch (root sheet, now carrying the
child sheet instances) and aqroot-Beta.kicad_pro.

03_spi_a_display_sd instantiates AQROOT_Beta:ILI9341_FT6236_MODULE_-
PLACEHOLDER; its cached symbol matches libraries/AQROOT_Beta.kicad_sym
exactly (13 pins, blank footprint, on_board=no).

Deliberately not taken from OneDrive:
  - sym-lib-table / fp-lib-table. The OneDrive copies hard-code an
    absolute P:/ path to this repository's library; the versions kept
    here use ${KIPRJMOD} and stay portable.
  - aqroot-Beta.kicad_prl (local project state) and .history/
    (2388 editor-history files, 5.87 MB).

Sheets identical on both sides and therefore untouched: 01_power_tree,
02_mcu_core, 04_spi_b_radios_nfc, 08_buttons_expanders,
09_community_header, aqroot-Beta.kicad_pcb.

Every copied file was verified by SHA-256 against its source, and each
staged blob is byte-identical to the working-tree file: CRLF endings
are preserved per .gitattributes, with no EOL normalization or
reformatting.

Co-Authored-By: Claude Opus 5 <noreply@anthropic.com>
Parts:
- added C6, C7: 100nF, symbol Device:C
- added R18: 220R, symbol Device:R
- added R19, R20: 4.7k, symbol Device:R
- added TP3: GPIO3_STRAP_TEST, symbol Connector:TestPoint
- added TP4: I2C_SDA_TEST, symbol Connector:TestPoint
- added TP5: I2C_SCL_TEST, symbol Connector:TestPoint
- added U4: BMI270, AQROOT_Beta:Bosch_LGA-14_2.5x3.0mm_P0.5mm_BMI270, symbol AQROOT_Beta:BMI270
Connections:
- new net +3V3: C6.1, C7.1, R19.1, R20.1, U4.12 (CSB), U4.2 (ASDx), U4.3 (ASCx), U4.5 (VDDIO), U4.8 (VDD)
- new net BMI270_INT1_RAW: R18.1, U4.4 (INT1)
- new net BMI270_INT1_STRAP: R18.2, TP3.1
- new net GND: C6.2, C7.2, U4.1 (SDO), U4.6 (GNDIO), U4.7 (GND)
- new net I2C_SCL_INT: R20.2, U4.13 (SCx)
- new net I2C_SCL_TEST: TP5.1
- new net I2C_SDA_INT: R19.2, TP4.1, U4.14 (SDx)
- no-connect marks 0 -> 3
Other:
- note added: "GPIO3 STRAP PROTECTION INT1 SERIES RESISTOR: 220R NO FIXED PULL FITTED REQUIREMENT: DO NOT BURN ESP32-S3 STRAP_JTAG_SEL EFUSE WITHOUT REASSESSING THIS CIRCUIT VALIDATE COLD BOOT + BMI270 INTERRUPT ON BETA FOOTPRINT NOT FAB-APPROVED DO NOT ROUTE UNTIL BMI270 LAND PATTERN IS REVIEWED"
- note added: "INTERNAL I2C BUS SDA/SCL PULL-UPS: 4.7k TO +3V3 ONE INTENTIONAL INTERNAL PULL-UP PAIR ONLY REMOVE OR ACCOUNT FOR DUPLICATE MODULE PULL-UPS INITIAL BETA BRING-UP: 100 kHz VERIFY 400 kHz AFTER FULL BUS VALIDATION"
