File: hardware/beta/kicad/aqroot-beta/05_i2c_devices.kicad_sch (KiCad schematic)
At the start: 9 parts, among them U4 BMI270

Commit message: AQROOT Beta: correct I2C SCL test point
TP5 probed a dead net: its label read I2C_SCL_TEST, a name carried by
nothing else, so the net contained only TP5 and ERC raised
isolated_pin_label.

TP4 is the working reference - its Value property is I2C_SDA_TEST while the
label on its wire is I2C_SDA_INT, so the test point sits on the real bus.
TP5 now mirrors that exactly: the label on its wire becomes I2C_SCL_INT and
the Value property stays I2C_SCL_TEST, matching TP4's convention.

One label name changed. No symbol, wire, junction or property was touched;
TP5's own wire (198.12 76.2)-(198.12 80.01) already ran to the label
position, exactly as TP4's does.

Verified with kicad-cli:
  /I2C_SCL_INT gains TP5.1 and keeps R20.2, U1.38, U14.7, U16.2, U2.22,
  U3.22, U4.13 - no member lost.
  /05_I2C_DEVICES/I2C_SCL_TEST no longer exists (149 -> 148 nets).
  /I2C_SDA_INT unchanged and still distinct from /I2C_SCL_INT - no bus short.
  isolated_pin_label clears, no new violation. Real ERC 15 -> 14.

Co-Authored-By: Claude Opus 5 <noreply@anthropic.com>
Connections:
- net I2C_SCL_TEST is gone; now on net I2C_SCL_INT: TP5.1
Changed lines of the file:
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@@
 		)
 	)
-	(label "I2C_SCL_TEST"
+	(label "I2C_SCL_INT"
 		(at 198.12 80.01 270)
 		(effects

Commit message: AQROOT Beta: assign remaining test-point footprints
TP1-TP5 carried an empty Footprint property while TP6-TP12 all used
TestPoint:TestPoint_Pad_D1.0mm. They now match the project convention, so
every test point in the design has a footprint.

  TP1  02_mcu_core   /02_MCU_CORE/TEST_GPIO45
  TP2  02_mcu_core   /02_MCU_CORE/TEST_GPIO46
  TP3  05_i2c        /BMI270_INT1_STRAP
  TP4  05_i2c        /I2C_SDA_INT
  TP5  05_i2c        /I2C_SCL_INT

Property-value edit only - five lines. No symbol was moved, no pin
reconnected, no wire or label touched.

Verified with kicad-cli: netlist pin-to-net mapping byte-identical before
and after, each TP still on its original net. ERC unchanged: raw 48,
unique 24, excluded 24, real 0.

Co-Authored-By: Claude Opus 5 <noreply@anthropic.com>
Parts:
- TP3, TP4, TP5: footprint (none) -> TestPoint:TestPoint_Pad_D1.0mm
Changed lines of the file:
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@@
 			)
 		)
-		(property "Footprint" ""
+		(property "Footprint" "TestPoint:TestPoint_Pad_D1.0mm"
 			(at 97.79 128.27 0)
 			(hide yes)
@@
 			)
 		)
-		(property "Footprint" ""
+		(property "Footprint" "TestPoint:TestPoint_Pad_D1.0mm"
 			(at 153.67 77.47 0)
 			(hide yes)
@@
 			)
 		)
-		(property "Footprint" ""
+		(property "Footprint" "TestPoint:TestPoint_Pad_D1.0mm"
 			(at 203.2 76.2 0)
 			(hide yes)

Commit message: AQROOT Beta: assign standard passive footprints
Assigns footprints to 40 passives whose package is unambiguous from
existing project precedent. Property-value edits only - no symbol, wire,
label or net touched.

  28 resistors -> Resistor_SMD:R_0603_1608Metric
     R1 R2 R3-R17 R18 R19 R20 R21 R22 R23 R25 R26 R27 R28 R29
     Basis: all 39 already-assigned resistors in the project are 0603, and
     every one of these is signal-level (pull-ups, dividers, series
     termination, MOSFET gate network).

  12 capacitors -> Capacitor_SMD:C_0603_1608Metric
     C1 C2 C4 C5 C6 C7 C8 C9 C13 C14 C16 C17
     Basis: 100nF is 5/5 and 1uF is 4/4 for 0603 among already-assigned
     capacitors - unanimous.

DELIBERATELY NOT ASSIGNED - split precedent, needs a decision:
  C3, C15, C10  10uF   -> project uses BOTH C_1206 (x2) and C_0805 (x1)
  C11           4.7uF  -> single 0805 precedent, different subsystem
Bulk capacitors must not be blindly converted to 0603, and the existing
precedent does not settle 0805 vs 1206.

Also untouched per instruction: C12/R24/Q1 (TBD), C18/C19 (placeholder),
L1/L2, mechanical switches and connectors, and the four RF/module
placeholders.

Separately noted, NOT changed here: C24 is 22uF 25V X7R with
C_0603_1608Metric already assigned. A 22uF 25V X7R does not exist in 0603
and the project's other 22uF parts use 1206/0805 - this looks like a
pre-existing error and is flagged for the BOM pass, not silently altered.

Verified with kicad-cli: netlist pin-to-net mapping byte-identical before
and after. ERC unchanged: raw 48, unique 24, excluded 24, real 0.
Footprint coverage 97 -> 137 of 166 components.

Co-Authored-By: Claude Opus 5 <noreply@anthropic.com>
Parts:
- C6, C7: footprint (none) -> Capacitor_SMD:C_0603_1608Metric
- R18, R19, R20: footprint (none) -> Resistor_SMD:R_0603_1608Metric
Changed lines of the file:
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@@
 			)
 		)
-		(property "Footprint" ""
+		(property "Footprint" "Resistor_SMD:R_0603_1608Metric"
 			(at 136.652 78.74 90)
 			(hide yes)
@@
 			)
 		)
-		(property "Footprint" ""
+		(property "Footprint" "Capacitor_SMD:C_0603_1608Metric"
 			(at 105.1052 62.23 0)
 			(hide yes)
@@
 			)
 		)
-		(property "Footprint" ""
+		(property "Footprint" "Capacitor_SMD:C_0603_1608Metric"
 			(at 74.6252 62.23 0)
 			(hide yes)
@@
 			)
 		)
-		(property "Footprint" ""
+		(property "Footprint" "Resistor_SMD:R_0603_1608Metric"
 			(at 179.832 78.74 90)
 			(hide yes)
@@
 			)
 		)
-		(property "Footprint" ""
+		(property "Footprint" "Resistor_SMD:R_0603_1608Metric"
 			(at 68.072 127 90)
 			(hide yes)
