File: hardware/beta/kicad/aqroot-beta/09_community_header.kicad_sch (KiCad schematic)
At the start: 34 parts, among them J5 COMMUNITY_HEADER_2x13, U15 TPS22918, U16 TCA9517ADGK

Commit message: AQROOT Beta: complete community header architecture
Complete the 09_COMMUNITY_HEADER architecture by adding the WAKE and FAST_IO
protection paths, finishing the protected interface set for the J5 community
header.

Added:
- R66 330R 1% in series on WAKE_INT_N, with D7 (TPD2E009DBZR) IO1 tapped on the
  connector side: WAKE_INT_N -> R66 -> WAKE_ATTN_N_HDR -> J5.24.
- R67 470R 1% in series on FAST_IO_U0TXD_ROOTPROBE_CS, with D7 IO2 on the
  connector side: FAST_IO_U0TXD_ROOTPROBE_CS -> R67 -> FAST_IO_GPIO43_HDR ->
  J5.23.
- D7 pin 2 on board GND. D7 is SOT-23, Package_TO_SOT_SMD:SOT-23.

Verified with a scratch kicad-cli netlist export and ERC comparison against
3b17272:
- All 15 XGPIOx_HDR nets unique, each exactly three nodes (one J5 pin, one
  series resistor, one ESD channel) with header number matching the internal
  channel. No XGPIO lines shorted.
- No orphan and no duplicate _HDR nets.
- All ESD channels sit on the connector side of their series resistor and are
  leaves on their nets, so no channel is in series with a signal.
- Resistor values: R51-R65 100R 1%, R66 330R 1%, R67 470R 1%, R47/R48 22R 1%,
  R49/R50 4.7k DNP, R46 100k 1%.
- All 37 parts on the sheet have footprints assigned. All symbol references
  unique.
- Power/I2C blocks unchanged and correct: U15 VIN/VOUT/ON/GND, U16
  VCCA/VCCB/EN/SCLA/SDAA/GND, D2 I2C ESD on the external SDA/SCL, R49/R50
  external pull-ups to ACC_3V3_SW.
- J5: 26 pins mapped, 6 GND, +3V3 on pin 1, ACC_3V3_SW on pin 26.

ERC total 232 -> 229, label_dangling 26 -> 23, no other category changed.

Remaining work, not addressed here: the internal side of the 15 /XGPIOx nets and
of /FAST_IO_U0TXD_ROOTPROBE_CS is still unwired, each holding only its series
resistor pin, so the RootProbe placeholder remains incomplete. TP1-TP5 have no
footprints. Not ERC-clean. Not fabrication-ready.

Co-Authored-By: Claude Opus 5 <noreply@anthropic.com>
Parts:
- added D7: TPD2E009DBZR, Package_TO_SOT_SMD:SOT-23, symbol AQROOT_Beta:TPD2E009DBZR
- added R66: 330R 1%, Resistor_SMD:R_0603_1608Metric, symbol Device:R
- added R67: 470R 1%, Resistor_SMD:R_0603_1608Metric, symbol Device:R
Connections:
- net FAST_IO_GPIO43_HDR: now also D7.3 (IO2), R67.1
- net FAST_IO_U0TXD_ROOTPROBE_CS: now also R67.2
- net GND: now also D7.2 (GND)
- net WAKE_ATTN_N_HDR: now also D7.1 (IO1), R66.2
- net WAKE_INT_N: now also R66.1
Other:
- note added: "ROOTPROBE PHASE 2 CONNECTOR / PIN COUNT / MECHANICAL FORMAT NOT LOCKED NO FOOTPRINT DO NOT ROUTE"
- note added: "WAKE_ATTN_N OPEN-DRAIN ACCESSORY ONLY INTERNAL 10k PULL-UP NO PUSH-PULL DRIVE"

Commit message: AQROOT Beta: complete community-header hierarchy integration
Connects XGPIO0-14 between U3 (TCA9535 port expander, sheet 08) and the
100R series resistors R51-R65 on sheet 09, replacing the 15 sheet-local
/08_BUTTONS_EXPANDERS/XGPIOx fragments with root-level /XGPIOx nets.

Connects ACC_PWR_EN between U3 pin 20 (P17) and the accessory rail
control: U15 pin 3 (TPS22918 ON) and U16 pin 5 (TCA9517A EN), joining
the existing R17 100k pull-down on one root-level /ACC_PWR_EN net. The
accessory load switch and I2C buffer enable are now actually driven by
U3 rather than floating.

Adds the missing FAST_IO boot-log warning note to sheet 09: FAST_IO is
U0TXD and emits the UART boot log at reset, so it must not be connected
to power enables or high-current loads.

Root-level hierarchy wiring only, except for the documentation text.
No component, value, footprint or pin-map changes: the component set is
unchanged at 158 parts and the J5 pin map, XGPIO series/ESD circuitry,
WAKE circuitry and FAST_IO electrical circuitry are untouched. No child
sheet required a schematic change.

ERC improves from 229 to 167 violations. This is not ERC-clean and not
fabrication-ready.

Co-Authored-By: Claude Opus 5 <noreply@anthropic.com>
Other:
- note added: "FAST_IO / U0TXD EMITS UART BOOT LOG AT RESET DO NOT CONNECT TO POWER ENABLES OR HIGH-CURRENT LOADS"
Changed lines of the file:
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@@
+		)
+	)
+	(text "FAST_IO / U0TXD\nEMITS UART BOOT LOG AT RESET\nDO NOT CONNECT TO POWER ENABLES\nOR HIGH-CURRENT LOADS"
+		(exclude_from_sim no)
+		(at 245.364 46.228 0)
+		(effects
+			(font
+				(size 0.635 0.635)
+			)
 		)
 	)
