File: hardware/beta/kicad/aqroot-beta/06_audio.kicad_sch (KiCad schematic)
At the start: 0 parts

Commit message: AQROOT Beta: capture I2C, audio, IR, and SPI-A subsystems
Reconciles the active KiCad project from OneDrive into the canonical
repository. The four subsystem sheets existed here only as 169-byte
empty stubs; the real schematic capture had been done in the OneDrive
working copy.

Sheets brought in:
  03_spi_a_display_sd.kicad_sch   stub ->  62136 bytes
  05_i2c_devices.kicad_sch        stub ->  59631 bytes
  06_audio.kicad_sch              stub ->  55263 bytes
  07_ir.kicad_sch                 stub ->  50216 bytes

Also updated: aqroot-Beta.kicad_sch (root sheet, now carrying the
child sheet instances) and aqroot-Beta.kicad_pro.

03_spi_a_display_sd instantiates AQROOT_Beta:ILI9341_FT6236_MODULE_-
PLACEHOLDER; its cached symbol matches libraries/AQROOT_Beta.kicad_sym
exactly (13 pins, blank footprint, on_board=no).

Deliberately not taken from OneDrive:
  - sym-lib-table / fp-lib-table. The OneDrive copies hard-code an
    absolute P:/ path to this repository's library; the versions kept
    here use ${KIPRJMOD} and stay portable.
  - aqroot-Beta.kicad_prl (local project state) and .history/
    (2388 editor-history files, 5.87 MB).

Sheets identical on both sides and therefore untouched: 01_power_tree,
02_mcu_core, 04_spi_b_radios_nfc, 08_buttons_expanders,
09_community_header, aqroot-Beta.kicad_pcb.

Every copied file was verified by SHA-256 against its source, and each
staged blob is byte-identical to the working-tree file: CRLF endings
are preserved per .gitattributes, with no EOL normalization or
reformatting.

Co-Authored-By: Claude Opus 5 <noreply@anthropic.com>
Parts:
- added C10: 10uf, symbol Device:C
- added C8, C9: 100nF, symbol Device:C
- added LS1: 8ohm_SPEAKER, symbol Device:Speaker
- added MK1: ICS-43434, Sensor_Audio:InvenSense_ICS-43434-6_3.5x2.65mm, symbol Sensor_Audio:ICS-43434
- added U5: MAX98357A, Package_DFN_QFN:TQFN-16-1EP_3x3mm_P0.5mm_EP1.23x1.23mm, symbol Audio:MAX98357A
Connections:
- new net: LS1.2, U5.10 (OUTN)
- new net: LS1.1, U5.9 (OUTP)
- new net +3V3: C10.1, C8.1, C9.1, MK1.5 (VDD), U5.7 (VDD), U5.8 (VDD)
- new net AMP_SD_MODE: U5.4 (~{SD_MODE})
- new net GND: C10.2, C8.2, C9.2, MK1.2 (LR), MK1.3 (GND), U5.11 (GND), U5.15 (GND), U5.17 (PAD), U5.2 (GAIN_SLOT), U5.3 (GND)
- new net I2S_BCLK: MK1.4 (SCK), U5.16 (BCLK)
- new net I2S_LRCLK: MK1.1 (WS), U5.14 (LRCLK)
- new net I2S_MIC_DIN: MK1.6 (SD)
- new net I2S_SPK_DOUT: U5.1 (DIN)
Other:
- note added: "AUDIO ARCHITECTURE LOCKED ICS-43434: LEFT I2S SLOT - LR PIN TIED TO GND MAX98357A: 3.3V SUPPLY GAIN_SLOT TIED TO GND - 12 dB GAIN DIFFERENTIAL FILTERLESS SPEAKER OUTPUT SPEAKER PART / FOOTPRINT PENDING VERIFY OUTPUT LEVEL AND THERMALS ON BETA DO NOT ROUTE UNTIL SPEAKER IS SELECTED"

Commit message: AQROOT Beta: assign standard passive footprints
Assigns footprints to 40 passives whose package is unambiguous from
existing project precedent. Property-value edits only - no symbol, wire,
label or net touched.

  28 resistors -> Resistor_SMD:R_0603_1608Metric
     R1 R2 R3-R17 R18 R19 R20 R21 R22 R23 R25 R26 R27 R28 R29
     Basis: all 39 already-assigned resistors in the project are 0603, and
     every one of these is signal-level (pull-ups, dividers, series
     termination, MOSFET gate network).

  12 capacitors -> Capacitor_SMD:C_0603_1608Metric
     C1 C2 C4 C5 C6 C7 C8 C9 C13 C14 C16 C17
     Basis: 100nF is 5/5 and 1uF is 4/4 for 0603 among already-assigned
     capacitors - unanimous.

DELIBERATELY NOT ASSIGNED - split precedent, needs a decision:
  C3, C15, C10  10uF   -> project uses BOTH C_1206 (x2) and C_0805 (x1)
  C11           4.7uF  -> single 0805 precedent, different subsystem
Bulk capacitors must not be blindly converted to 0603, and the existing
precedent does not settle 0805 vs 1206.

Also untouched per instruction: C12/R24/Q1 (TBD), C18/C19 (placeholder),
L1/L2, mechanical switches and connectors, and the four RF/module
placeholders.

Separately noted, NOT changed here: C24 is 22uF 25V X7R with
C_0603_1608Metric already assigned. A 22uF 25V X7R does not exist in 0603
and the project's other 22uF parts use 1206/0805 - this looks like a
pre-existing error and is flagged for the BOM pass, not silently altered.

Verified with kicad-cli: netlist pin-to-net mapping byte-identical before
and after. ERC unchanged: raw 48, unique 24, excluded 24, real 0.
Footprint coverage 97 -> 137 of 166 components.

Co-Authored-By: Claude Opus 5 <noreply@anthropic.com>
Parts:
- C8, C9: footprint (none) -> Capacitor_SMD:C_0603_1608Metric
Changed lines of the file:
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@@
 			)
 		)
-		(property "Footprint" ""
+		(property "Footprint" "Capacitor_SMD:C_0603_1608Metric"
 			(at 153.3652 81.28 0)
 			(hide yes)
@@
 			)
 		)
-		(property "Footprint" ""
+		(property "Footprint" "Capacitor_SMD:C_0603_1608Metric"
 			(at 248.6152 100.33 0)
 			(hide yes)

Commit message: AQROOT Beta: assign remaining generic bulk-cap footprints
Assigns Capacitor_SMD:C_0805_2012Metric to the four bulk capacitors left
open by the standard-passive pass.

  C3   10uF   +3V3                  02_mcu_core     generic bulk decoupling
  C15  10uF   +3V3                  03_spi_a        generic bulk decoupling
  C10  10uF   +3V3                  06_audio        generic bulk decoupling
  C11  4.7uF  /07_IR/IR_RX_VS_LOCAL 07_ir           TSOP382 supply RC

Basis: these are NOT regulator input/output capacitors. The project's 1206
precedent (C26/C27 CIN, C29-C32 COUT) is a TPS63020-specific requirement -
the kicad README states '1206 preferred ... Close to VIN/PGND' for those
parts only, so it does not generalise. For generic 10uF/10V and 4.7uF/10V
bulk on a 3.3V rail, 0805 is adequate and is the project's generic
precedent (C33, C20). C11's role is documented at libraries/README.md:1264
as Vishay's TSOP382 application R1/C1 supply filter, paired with R21 100R.

Property-value edits only - four lines. No value, symbol, wire, label or
net touched.

Verified with kicad-cli: netlist pin-to-net mapping byte-identical before
and after. ERC unchanged: raw 48, unique 24, excluded 24, real 0.

Still open and deliberately untouched: exact MPNs and DC-bias derating for
these parts. A 10uF/10V 0805 X7R typically retains only ~60-70% of its
nominal capacitance at 3.3V, so effective capacitance must be confirmed at
the BOM pass - the package is locked here, the part is not.

Co-Authored-By: Claude Opus 5 <noreply@anthropic.com>
Parts:
- C10: footprint (none) -> Capacitor_SMD:C_0805_2012Metric
Changed lines of the file:
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@@
 			)
 		)
-		(property "Footprint" ""
+		(property "Footprint" "Capacitor_SMD:C_0805_2012Metric"
 			(at 272.7452 100.33 0)
 			(hide yes)

Commit message: AQROOT Beta: lock mechanical component selections
Records exact MPN / manufacturer / package metadata for the mechanical
parts. All four footprints stay BLANK - every one needs a vendor drawing.

  SW9  JS102011SAQN     C&K (Littelfuse)      right-angle SMD SPDT slide
  J2   5025700893       Molex                 SMT push-push microSD, 8 contacts
  LS1  CMS-1535-058SP   Same Sky (CUI)        15 mm round 8 ohm solder-pad
  J1   Adafruit 2770    Adafruit              2.8in 240x320 + FT6236U cap touch

SW9 - SYMBOL/PART CONFLICT FOUND, NOT PAPERED OVER:
JS102011SAQN is a 3-terminal SPDT, but this instance uses Switch:SW_SPST
which has only two pins (A,B). Any correct land pattern for this part has
three signal pads plus mounting tabs, so symbol and footprint cannot agree
as they stand. The locked electrical intent is SPST (VINA -> switch -> EN,
never switching GND) and wiring an SPDT as SPST is fine, but the symbol has
to expose the unused throw so it can carry a no-connect. Swapping the symbol
is an approval-gated change and was deliberately NOT made. Recorded in the
part's Note so it cannot be missed at footprint time.

J1 is recorded as a VENDOR SKU lock, not a production MPN lock - Adafruit
can change panel manufacturer while preserving compatibility. Its Note
marks it a critical PCB/enclosure dependency and lists what is still needed:
the current Adafruit mechanical/FPC drawing, verification of the 50-pin
0.5 mm FPC pinout against the existing sheet architecture, and selection of
the separate mating FPC connector. The ~69 x 50 x 4 mm figure is flagged
approximate.

SW1-SW8 were deliberately left without MPNs. The class is locked (compact
SMD tactile) but the enclosure doc specifies only that there are seven
controls - D-pad, A and B - with no top-push versus side-push actuation
requirement recorded, so no per-reference MPN could be justified without
inventing a mechanical decision.

No fabricated dimensions, land patterns or ratings. Electrical circuits,
signal ar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
Parts:
- LS1: MPN (none) -> CMS-1535-058SP; Manufacturer (none) -> Same Sky (CUI Devices); Note (none) -> Audio circuit unchanged - driven differentially from MAX983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; Package (none) -> 15 mm round solder-pad speaker, 8 ohm - part LOCKED. Footpr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
Changed lines of the file:
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@@
+			)
+		)
+		(property "Note" "Audio circuit unchanged - driven differentially from MAX98357A OUTP/OUTN. Enclosure cavity, grille and acoustic sealing are a mechanical-phase check. Exact body height, mounting method and pad geometry NOT recorded here; take them from the Same Sky datasheet."
+			(at 241.3 72.39 0)
+			(hide yes)
+			(show_name no)
+			(do_not_autoplace no)
+			(effects
+				(font
+					(size 1.27 1.27)
+				)
+			)
+		)
+		(property "Package" "15 mm round solder-pad speaker, 8 ohm - part LOCKED. Footprint BLOCKED: needs the official Same Sky mechanical drawing / land pattern."
+			(at 241.3 72.39 0)
+			(hide yes)
+			(show_name no)
+			(do_not_autoplace no)
+			(effects
+				(font
+					(size 1.27 1.27)
+				)
+			)
+		)
+		(property "Manufacturer" "Same Sky (CUI Devices)"
+			(at 241.3 72.39 0)
+			(hide yes)
+			(show_name no)
+			(do_not_autoplace no)
+			(effects
+				(font
+					(size 1.27 1.27)
+				)
+			)
+		)
+		(property "MPN" "CMS-1535-058SP"
+			(at 241.3 72.39 0)
+			(hide yes)
+			(show_name no)
+			(do_not_autoplace no)
+			(effects
+				(font
+					(size 1.27 1.27)
+				)
 			)
 		)
