File: hardware/beta/kicad/aqroot-beta/08_buttons_expanders.kicad_sch (KiCad schematic)
At the start: 26 parts, among them SW2 UP, SW3 DOWN, SW4 LEFT, SW5 RIGHT, SW6 A_SELECT, SW7 B_BACK, SW8 HOME, U2 TCA9535PWR, U3 TCA9535PWR

Commit message: AQROOT Beta: assign standard passive footprints
Assigns footprints to 40 passives whose package is unambiguous from
existing project precedent. Property-value edits only - no symbol, wire,
label or net touched.

  28 resistors -> Resistor_SMD:R_0603_1608Metric
     R1 R2 R3-R17 R18 R19 R20 R21 R22 R23 R25 R26 R27 R28 R29
     Basis: all 39 already-assigned resistors in the project are 0603, and
     every one of these is signal-level (pull-ups, dividers, series
     termination, MOSFET gate network).

  12 capacitors -> Capacitor_SMD:C_0603_1608Metric
     C1 C2 C4 C5 C6 C7 C8 C9 C13 C14 C16 C17
     Basis: 100nF is 5/5 and 1uF is 4/4 for 0603 among already-assigned
     capacitors - unanimous.

DELIBERATELY NOT ASSIGNED - split precedent, needs a decision:
  C3, C15, C10  10uF   -> project uses BOTH C_1206 (x2) and C_0805 (x1)
  C11           4.7uF  -> single 0805 precedent, different subsystem
Bulk capacitors must not be blindly converted to 0603, and the existing
precedent does not settle 0805 vs 1206.

Also untouched per instruction: C12/R24/Q1 (TBD), C18/C19 (placeholder),
L1/L2, mechanical switches and connectors, and the four RF/module
placeholders.

Separately noted, NOT changed here: C24 is 22uF 25V X7R with
C_0603_1608Metric already assigned. A 22uF 25V X7R does not exist in 0603
and the project's other 22uF parts use 1206/0805 - this looks like a
pre-existing error and is flagged for the BOM pass, not silently altered.

Verified with kicad-cli: netlist pin-to-net mapping byte-identical before
and after. ERC unchanged: raw 48, unique 24, excluded 24, real 0.
Footprint coverage 97 -> 137 of 166 components.

Co-Authored-By: Claude Opus 5 <noreply@anthropic.com>
Parts:
- C4, C5: footprint (none) -> Capacitor_SMD:C_0603_1608Metric
- R10, R11, R12, R13, R14, R15, R16, R17, R3, R4, R5, R6, R7, R8, R9: footprint (none) -> Resistor_SMD:R_0603_1608Metric
Changed lines of the file:
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@@
 			)
 		)
-		(property "Footprint" ""
+		(property "Footprint" "Resistor_SMD:R_0603_1608Metric"
 			(at 146.812 137.16 90)
 			(hide yes)
@@
 			)
 		)
-		(property "Footprint" ""
+		(property "Footprint" "Resistor_SMD:R_0603_1608Metric"
 			(at 123.952 137.16 90)
 			(hide yes)
@@
 			)
 		)
-		(property "Footprint" ""
+		(property "Footprint" "Capacitor_SMD:C_0603_1608Metric"
 			(at 121.6152 49.53 0)
 			(hide yes)
@@
 			)
 		)
-		(property "Footprint" ""
+		(property "Footprint" "Resistor_SMD:R_0603_1608Metric"
 			(at 80.772 137.16 90)
 			(hide yes)
@@
 			)
 		)
-		(property "Footprint" ""
+		(property "Footprint" "Capacitor_SMD:C_0603_1608Metric"
 			(at 205.4352 50.8 0)
 			(hide yes)
@@
 			)
 		)
-		(property "Footprint" ""
+		(property "Footprint" "Resistor_SMD:R_0603_1608Metric"
 			(at 46.228 81.28 90)
 			(hide yes)
@@
 			)
 		)
-		(property "Footprint" ""
+		(property "Footprint" "Resistor_SMD:R_0603_1608Metric"
 			(at 101.092 182.88 90)
 			(hide yes)
@@
 			)
 		)
-		(property "Footprint" ""
+		(property "Footprint" "Resistor_SMD:R_0603_1608Metric"
 			(at 146.812 182.88 90)
 			(hide yes)
@@
 			)
 		)
-		(property "Footprint" ""
+		(property "Footprint" "Resistor_SMD:R_0603_1608Metric"
 			(at 57.912 137.16 90)
 			(hide yes)
@@
 			)
 		)
-		(property "Footprint" ""
+		(property "Footprint" "Resistor_SMD:R_0603_1608Metric"
 			(at 57.912 182.88 90)
 			(hide yes)
@@
 			)
 		)
-		(property "Footprint" ""
+		(property "Footprint" "Resistor_SMD:R_0603_1608Metric"
 			(at 167.132 137.16 90)
 			(hide yes)
@@
 			)
 		)
-		(property "Footprint" ""
+		(property "Footprint" "Resistor_SMD:R_0603_1608Metric"
 			(at 123.952 182.88 90)
 			(hide yes)
@@
 			)
 		)
-		(property "Footprint" ""
+		(property "Footprint" "Resistor_SMD:R_0603_1608Metric"
 			(at 36.322 36.83 90)
 			(hide yes)
@@
 			)
 		)
-		(property "Footprint" ""
+		(property "Footprint" "Resistor_SMD:R_0603_1608Metric"
 			(at 80.772 182.88 90)
 			(hide yes)
@@
 			)
 		)
-		(property "Footprint" ""
+		(property "Footprint" "Resistor_SMD:R_0603_1608Metric"
 			(at 36.322 137.16 90)
 			(hide yes)
@@
 			)
 		)
-		(property "Footprint" ""
+		(property "Footprint" "Resistor_SMD:R_0603_1608Metric"
 			(at 36.322 182.88 90)
 			(hide yes)
@@
 			)
 		)
-		(property "Footprint" ""
+		(property "Footprint" "Resistor_SMD:R_0603_1608Metric"
 			(at 101.092 137.16 90)
 			(hide yes)

Commit message: AQROOT Beta: integrate E22 module and dedicate XGPIO14 to RX control
Atomic change across four files - root, sheet 04, sheet 08 and sheet 09 -
because the hierarchy reallocation and the module capture are electrically
coupled and neither is valid alone.

APPLIED TO U8, NOT U7. The schematic is authoritative: U8 is the SX1262 /
E22-900M22S at 915 MHz and U7 remains the CC1101 / E07-400M10S at 433 MHz. The
earlier blocker-register transposition is corrected and annotated in the log;
U7 is untouched and still a placeholder awaiting its own vendor audit.

U8 CAPTURE. The SX1262_MODULE_PLACEHOLDER is replaced by the physical 22-pin
E22-900M22S symbol on AQROOT_Beta:Ebyte_E22-900M22S. All 22 pads resolve, none
unconnected: the ten physical grounds - pins 1 to 5, 10, 11, 12, 20 and 22 - all
land on GND individually rather than being collapsed, pin 9 VCC is on +3V3, and
pins 13 to 19 carry SX1262_DIO1, SX1262_BUSY, SX1262_RST_N, SPI_B_MISO,
SPI_B_MOSI, SPI_B_SCK and SX1262_CS_N respectively. The seven existing
hierarchical labels were relocated onto the new pin stubs rather than
duplicated.

RF SWITCH. DIO2 on pin 8 is strapped locally to TXEN on pin 7, and the netlist
confirms DIO2_TXEN contains exactly those two nodes and nothing else, so no MCU
or expander pin is consumed for transmit control. Firmware must enable
SetDIO2AsRfSwitchCtrl or TXEN never asserts. Receive control comes from
SX1262_RXEN, which contains exactly U3 pin 19, U8 pin 6 and the new R74
pulldown.

XGPIO14 RETIRED. U3 pin 19 is reallocated from XGPIO14 to SX1262_RXEN across the
whole hierarchy - the sheet 08 hierarchical label, the sheet 08 sheet pin in the
root, and a new sheet 04 sheet pin plus root label. On sheet 09 the community
path is removed: R65 and its wires are deleted, the XGPIO14 hierarchical label
is gone, and both XGPIO14_HDR labels become RESERVED_NC, so J5 pin 19 no longer
advertises a GPIO. D6's now-spare ESD channel carries an explicit no_connect.
XGPIO0 to XGPIO13 are untouched and a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
Connections:
- net XGPIO14 renamed SX1262_RXEN
Changed lines of the file:
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@@
 		)
 	)
-	(hierarchical_label "XGPIO14"
+	(hierarchical_label "SX1262_RXEN"
 		(shape bidirectional)
 		(at 186.69 92.71 0)

Commit message: AQROOT Beta: lock final user-button footprints
SW1-SW8 assigned Button_Switch_SMD:SW_SPST_PTS645Sx43SMTR92.

Classification: VERIFIED_VENDOR_EXACT. Checked against the C&K / Littelfuse
PTS645 series datasheet (Revised VL 01/29/26), RECOMMENDED PCB LAYOUT panels,
rasterised to confirm which feature each dimension attaches to. The drawing
gives 9.5 outer-edge to outer-edge and 6.4 inner-edge to inner-edge in X, and
5.8 outer to 3.2 inner in Y, which yields pads 1.55 (X) x 1.30 (Y) on centres of
+/-3.975 (X) and +/-2.25 (Y). The KiCad footprint implements 1.55 x 1.30 at
(+/-3.98, +/-2.25): exact on pad size and on the Y centre, with a 0.005 mm
rounding on the X centre that is far inside any fabrication tolerance.

The ratified premise that straight-SMT PTS645 variants share one published land
pattern is confirmed rather than assumed: the identical 9.5 / 6.4 / 5.8 / 3.2
set is published for both the 4.3 mm SMT G Type and the 7.3 mm straight SMT
variants. That is why the footprint can be locked while the actuator-height
suffix is not.

Pad mapping verified: four physical pads; C&K numbers 1 and 2 on the top row and
3 and 4 on the bottom row with 1-2 tied and 3-4 tied, so the footprint's pad 1
covers the top pair and pad 2 the bottom pair, matching the 2-pin
Switch:SW_Push symbol. No phantom or missing pads.

BOM status is FOOTPRINT LOCKED / BOM SUFFIX VERIFY. MPN is recorded as the
approved family notation PTS645Sx SMTR92 LFS with 160gf TARGET, ~5mm ACTUATOR
TARGET, ~0.25 mm travel and 100,000 operation class marked as selection targets.
No actuator height, force suffix, package code, travel or lifecycle figure was
invented.

SCOPE NOTE - the eight footprintless switches are SW1 plus SW2-SW8. SW1 is the
ESP32 BOOT strap button on 02_mcu_core, not a user-facing game button; it takes
the same part and land pattern but receives no plastic cap. The seven
user-facing buttons are SW2-SW8. SW9, the power slide switch, already had its
own footprint and was not touched.

Enclosur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
Parts:
- SW2, SW3, SW4, SW5, SW6, SW7, SW8: footprint (none) -> Button_Switch_SMD:SW_SPST_PTS645Sx43SMTR92; BOM_Status (none) -> C&K / Littelfuse PTS645 family, 6 mm SMD, top-actuated. FIN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; Footprint_Provenance (none) -> Land pattern VERIFIED_VENDOR_EXACT against the C&K / Littel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; MPN (none) -> PTS645Sx SMTR92 LFS; Manufacturer (none) -> C&K / Littelfuse; Mounting (none) -> BOARD_MOUNTED; Note (none) -> User-facing button; receives an individual plastic cap. ENC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; Package (none) -> 6.0 x 6.0 mm tactile switch, straight SMT gull-wing, 4 term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
Other:
- note added: "USER BUTTONS - PTS645 FAMILY LOCKED C&K / Littelfuse PTS645, 6x6 mm SMD, top-actuated FOOTPRINT LOCKED (VERIFIED_VENDOR_EXACT vs C&K PCB LAYOUT) BOM SUFFIX VERIFY AT BOM LOCK SELECTION TARGETS: 160 gf, ~5 mm actuator, ~0.25 mm travel, 100k operation class ENCLOSURE DESIGN TARGETS (NOT SWITCH SPECS): individual plastic caps, no membrane for Beta 0.1-0.3 mm rest gap, no preload hard stop at ~0.3-0.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"
