File: hardware/beta/kicad/aqroot-beta/03_spi_a_display_sd.kicad_sch (KiCad schematic)
At the start: 18 parts, among them J1 CH280QV10-CT_50P, J2 Molex_5025700893, U17 TPS61169DCKR

Commit message: AQROOT Beta: set C56 to 1 uF for TI-compliant local CIN
C56 100 nF -> 1 uF, keeping ref, footprint, position (46.100, 82.500),
rotation 0, B.Cu side and nets (+3V3 / GND). No capacitor added.

TI SNVSA40B section 7.5.1 requires the input capacitor close to the VIN
and GND pins, and Recommended Operating Conditions give CI minimum 1 uF.
100 nF was useful HF bypassing but did not satisfy that literally. C43
4.7 uF remains the power-stage reservoir next to L3 at 2.37 mm; C56 is
now the local U17 VIN capacitor at 1.624 mm from pin 5.

BOM stays a multi-source commodity passive: 1 uF, 16 V, X7R, 0603, exact
MPN deferred to BOM verification, which must confirm the production part
keeps reasonable effective capacitance at 3.3 V DC bias.

Verified: schematic netlist topology byte-identical (174 nets, same node
sets); PCB footprint Value synchronised so parity gains nothing; DRC 0
errors, 234 warnings; ERC 116/58 excluded/58 live, zero delta; placement
188 footprints unchanged.

Co-Authored-By: Claude Opus 5 <noreply@anthropic.com>
Parts:
- C56: value 100nF -> 1uF; Note LOCAL VIN BYPASS for U17 TPS61169. Required by TI SNVSA40B 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 -> LOCAL CIN for U17 TPS61169. TI SNVSA40B section 7.5.1 requi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
Changed lines of the file:
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@@
 			)
 		)
-		(property "Value" "100nF"
+		(property "Value" "1uF"
 			(at 224.79 166.3699 0)
 			(show_name no)
@@
 			)
 		)
-		(property "Note" "LOCAL VIN BYPASS for U17 TPS61169. Required by TI SNVSA40B section 7.5.1: the input capacitor must be close to the VIN pin and GND pin. C43 4.7uF is the power-stage input capacitor and sits 9.39 mm from U17 pin 5 - correct for the C43->L3 power loop (2.37 mm) but too far to bypass VIN. Added 2026-08-11 during the Routing Pass 1 blocker correction. Place immediately beside U17 VIN/GND; NOT ROUTED in this pass."
+		(property "Note" "LOCAL CIN for U17 TPS61169. TI SNVSA40B section 7.5.1 requires the input capacitor close to the VIN pin and GND pin, and Recommended Operating Conditions give CI minimum 1 uF - so this part is 1 uF, not a 100 nF bypass, to satisfy that requirement literally. C43 4.7uF is the power-stage input capacitor and sits 9.39 mm from U17 pin 5 - correct for the C43->L3 power loop (2.37 mm) but too far to bypass VIN. Added 2026-08-11 during the Routing Pass 1 blocker correction. Place immediately beside U17 VIN/GND; NOT ROUTED in this pass."
 			(at 220.98 165.1 0)
 			(hide yes)
