File: hardware/beta/kicad/aqroot-beta/01_power_tree.kicad_sch (KiCad schematic)
At the start: 53 parts, among them J3 USB_C_Receptacle_USB2.0_16P, J4 JST-PH-2 BATTERY, SW9 SW_SPDT, U10 USBLC6-2SC6, U11 BQ25185, U12 TPS63020, U13 TPS61023, U14 MAX17048

Commit message: Close metadata drift on SW9, U7, U8, U9, J3; verify netlist and ERC unchanged
Five symbols carried metadata contradicting decisions already locked elsewhere
in the Design Decisions Log. No external vendor document was needed for any of
them - this propagates existing locks rather than selecting anything new.

SW9 - the Note still declared an unresolved SPST/SPDT symbol conflict and said
the symbol change "was NOT made here". That is stale: the instance is already
Switch:SW_SPDT with pins 1/2/3. Pole mapping is now VERIFIED 1:1 - the KiCad
symbol places pin 2 (name B) alone at (-5.08, 0), opposite throws 1 (A) and
3 (C), which is what makes it the pole, and C&K terminal 2 is likewise the
COMMON/POLE, so no cross-map is needed. Netlist confirms pin 2 to BQ25185_SYS,
pin 1 to U12 EN and TP13, pin 3 an unused throw carrying a no_connect.
Electrical intent unchanged, still SPST-in-practice. SW9 is no longer blocked on
symbol numbering - only on land-pattern geometry from the C&K layout drawing.

U7/U8 - both still read Manufacturer TBD, MPN TBD despite the RF plan locking
the Ebyte modules. U7 is now Ebyte E07-400M10S (433 MHz, CC1101) and U8 is Ebyte
E22-900M22S (915 MHz, SX1262). Their Package fields also record the standing
constraint that each module owns its matching network and presents a matched
50-ohm IPEX port, so no matching network and no separate U.FL test connector
belong on the main PCB. Footprints remain blocked pending Ebyte drawings.

U9 - MPN was still bare ST25R3916. The NFC package lock explicitly closed that
open question, so the suffix is now recorded: ST25R3916-AQET, VQFN-32 5x5 mm,
discrete and not a plug-on module. Footprint still blocked pending ST's outline.

J3 - had a GCT-specific footprint but no Manufacturer and no MPN property at
all. Added GCT and USB4105-GF-A-120, with the Package field stating plainly that
the family is locked while the variant suffix remains a CANDIDATE, unconfirmed
against the GCT drawing at the locked 1.6 mm board th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
Parts:
- J3: MPN (none) -> USB4105-GF-A-120; Manufacturer (none) -> GCT (Global Connector Technology); Package (none) -> 16-contact USB 2.0 Type-C receptacle, top-mount horizontal,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
- SW9: Note SYMBOL/PART CONFLICT - MUST BE RESOLVED BEFORE FOOTPRINT. J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 -> SYMBOL CONFLICT RESOLVED (2026-08-07). This instance is now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; Package Right-angle SMD SPDT slide switch - part LOCKED. Footprint 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 -> Right-angle SMD SPDT slide switch - part LOCKED, symbol con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
Changed lines of the file:
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@@
 			)
 		)
-		(property "Note" "SYMBOL/PART CONFLICT - MUST BE RESOLVED BEFORE FOOTPRINT. JS102011SAQN is a 3-terminal SPDT; this instance uses Switch:SW_SPST which has only 2 pins (A,B). Any correct JS102011SAQN land pattern has 3 signal pads plus mounting tabs, so symbol and footprint cannot agree as-is. The locked electrical intent is SPST (VINA -> switch -> EN, never switching GND); wiring an SPDT as SPST is fine, but the symbol must then expose the unused throw so it can carry a no-connect. Changing the symbol is an approval-gated change and was NOT made here. Actuator direction and travel also still require the enclosure mechanical review."
-			(at 190.5 63.5 0)
-			(hide yes)
-			(show_name no)
-			(do_not_autoplace no)
-			(effects
-				(font
-					(size 1.27 1.27)
-				)
-			)
-		)
-		(property "Package" "Right-angle SMD SPDT slide switch - part LOCKED. Footprint BLOCKED: needs the official C&K PCB layout drawing, and see the SYMBOL CONFLICT below."
+		(property "Note" "SYMBOL CONFLICT RESOLVED (2026-08-07). This instance is now Switch:SW_SPDT with pins 1/2/3, matching the 3-terminal JS102011SAQN. Pole mapping VERIFIED 1:1 - KiCad pin 2 (name 'B') is the pole, sitting alone on the opposite side of the symbol body from throws 1 ('A') and 3 ('C'), and C&K terminal 2 is likewise the COMMON/POLE. Wiring as built: pin 2 = BQ25185_SYS (source), pin 1 = U12 EN + TP13, pin 3 = unused throw carrying a no_connect. Electrical intent is unchanged and still SPST-in-practice (VINA -> switch -> EN, never switching GND). Actuator direction and travel still require the enclosure mechanical review."
+			(at 190.5 63.5 0)
+			(hide yes)
+			(show_name no)
+			(do_not_autoplace no)
+			(effects
+				(font
+					(size 1.27 1.27)
+				)
+			)
+		)
+		(property "Package" "Right-angle SMD SPDT slide switch - part LOCKED, symbol conflict RESOLVED. Footprint BLOCKED: needs the official C&K PCB layout drawing for the land pattern geometry only (3 signal pads plus mounting tabs). Symbol-to-terminal numbering is no longer a blocker - see Note."
 			(at 190.5 63.5 0)
 			(hide yes)
@@
 			(at 30.48 46.99 0)
 			(hide yes)
+			(show_name no)
+			(do_not_autoplace no)
+			(effects
+				(font
+					(size 1.27 1.27)
+				)
+			)
+		)
+		(property "Manufacturer" "GCT (Global Connector Technology)"
+			(at 30.48 46.99 0)
+			(hide yes)
+			(show_name no)
+			(do_not_autoplace no)
+			(effects
+				(font
+					(size 1.27 1.27)
+				)
+			)
+		)
+		(property "MPN" "USB4105-GF-A-120"
+			(at 30.48 46.99 0)
+			(hide yes)
+			(show_name no)
+			(do_not_autoplace no)
+			(effects
+				(font
+					(size 1.27 1.27)
+				)
+			)
+		)
+		(property "Package" "16-contact USB 2.0 Type-C receptacle, top-mount horizontal, SMD contacts with through-hole shell stakes. FAMILY LOCKED: GCT USB4105. Footprint cites GCT's own drawing. The variant suffix -GF-A-120 is a CANDIDATE and is NOT confirmed - the exact suffix, and whether it matches the intended shell-stake configuration at the locked 1.6 mm board thickness, must be VERIFIED against the GCT drawing before release."
+			(at 30.48 46.99 0)
+			(hide yes)

Commit message: Footprints: verify and assign C&K JS102011SAQN; lock L3 and touch-IRQ decisions
SW9 CLOSED. Assigns Button_Switch_SMD:SW_SPDT_CK_JS102011SAQN and classifies it
VERIFIED_VENDOR_EXACT. The C&K site returns 403, so the drawing was taken from
the octopart mirror of the C&K/ITT JS-series datasheet and page 4 rasterised to
read the leader lines on the RIGHT ANGLE SURFACE MOUNT / PCB MOUNT - HOLE
LAYOUT block for JS102011SAQN.

Verified exact against that drawing: terminal pitch 2.5 TYP matches the KiCad
lands at -2.5, 0 and +2.5; the two locating holes are diameter 0.9 with a 6.8
span, matching the footprint's non-plated holes at x = +/-3.4 exactly; and the
three SPDT lands match. One delta is documented rather than glossed: the KiCad
land is 1.25 wide against the drawing's 1.2 TYP, a 0.025 mm per-side solder
fillet allowance. The mechanically critical features - hole diameter, hole span
and pitch - are exact. Pole mapping is unchanged and was previously verified
1:1, KiCad pin 2 = C&K terminal 2 = COMMON. No electrical wiring changed; the
netlist is identical at 155 nets before and after.

TWO DECISIONS LOCKED. L3 stays as Coilcraft XFL4020-472MEC despite being
electrically oversized, because its land pattern is already vendor-verified and
shared with L1, so no new footprint verification is needed; it is not to be
replaced for optimisation alone, and size/cost work is deferred unless PCB
placement proves the 4x4 mm body is a real constraint. J1 pin 46 CTP_IRQ stays
NC for Beta with the rationale recorded verbatim: Beta touch uses I2C polling,
CTP_IRQ is intentionally not connected, and IRQ allocation is deferred unless
firmware testing demonstrates a need. It is carried by an explicit no_connect,
which is why it produces no ERC warning.

J3 VERIFIED AS NOT MISSING. It already carries the GCT USB4105 footprint with
MPN USB4105-GF-A-120. It remains UNVERIFIED because the variant suffix and
shell-stake configuration at 1.6 mm board thickness are unconfirmed, but
UNVERIFIED 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
Parts:
- SW9: footprint (none) -> Button_Switch_SMD:SW_SPDT_CK_JS102011SAQN; Package Right-angle SMD SPDT slide switch - part LOCKED, symbol con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 -> Right-angle SMD SPDT slide switch, C&K JS series. FOOTPRINT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
Changed lines of the file:
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@@
 			)
 		)
-		(property "Footprint" ""
+		(property "Footprint" "Button_Switch_SMD:SW_SPDT_CK_JS102011SAQN"
 			(at 190.5 63.5 0)
 			(hide yes)
@@
 			)
 		)
-		(property "Package" "Right-angle SMD SPDT slide switch - part LOCKED, symbol conflict RESOLVED. Footprint BLOCKED: needs the official C&K PCB layout drawing for the land pattern geometry only (3 signal pads plus mounting tabs). Symbol-to-terminal numbering is no longer a blocker - see Note."
+		(property "Package" "Right-angle SMD SPDT slide switch, C&K JS series. FOOTPRINT VERIFIED against the C&K JS-series drawing (octopart mirror of the C&K/ITT datasheet), page 4 'RIGHT ANGLE SURFACE MOUNT / PCB MOUNT - HOLE LAYOUT' for JS102011SAQN. Verified exact: terminal pitch 2.5 TYP; two locating holes dia 0.9 with 6.8 span, i.e. x = +/-3.4; three SPDT lands; body 9.0 x 3.6 + 2.0. Documented delta: KiCad land is 1.25 wide vs the drawing's 1.2 TYP, a 0.025 mm per-side solder-fillet allowance. Mechanically critical features (hole diameter, hole span, pitch) match exactly. Contact rating 6 VDC 0.3 A, 5000 cycles. Pole mapping unchanged and previously verified 1:1: KiCad pin 2 = C&K terminal 2 = COMMON."
 			(at 190.5 63.5 0)
 			(hide yes)

Commit message: Footprints: add verified TI TPS63020 DSJ package
Closes U12. Creates AQROOT_Beta:TI_TPS63020_DSJ and assigns it, classified
VERIFIED_VENDOR_EXACT for the signal lands and the thermal-pad envelope.

THE AMBIGUITY IS RESOLVED. The previous pass stalled on TI's 4X 0.20 features
at 0.46 spacing, unable to tell whether they were separate exposed pads or part
of the thermal pad, and the standing rule forbade inferring them from stencil
aperture counts. Rasterising TI's Example Board Layout at 900 dpi settles it:
they are SLOTS CUT INTO A SINGLE CONTIGUOUS THERMAL LAND, visible as a comb on
both flanks of one connected copper area, with the 5 by 3 grid of 15 vias
inside it. They are not separate pads. Ultra Librarian was therefore not
needed - TI's own package drawing, which the brief names as the primary source,
was sufficient once read at adequate resolution.

Geometry from TI 4210895-2/E LAND PATTERN DATA and 4208549-3/G THERMAL PAD
MECHANICAL DATA: signal lands 0.24 by 0.60 with R0.12, which at half the 0.24
width makes them fully rounded ovals; 0.5 mm pitch; seven per row; rows 2.8 mm
apart so y is plus or minus 1.4; x at 0, plus or minus 0.5, 1.0 and 1.5;
non-solder-mask-defined with 0.07 mm expansion all round; thermal pad 2.85 by
1.58 with plus or minus 0.10. Pin 1 is bottom-left in top view per the circled
callout on TI's Example Board Layout, numbering 1 to 7 left to right along the
bottom row then 8 to 14 back along the top.

Two deliberate implementation choices are documented in the footprint
description rather than left implicit. The comb is not reproduced; the plain
TI-dimensioned 2.85 by 1.58 envelope is used instead, which is conservative -
more thermal copper within the same outline. And paste uses
solder_paste_margin_ratio -0.05, which KiCad applies per side, giving 0.9
linear and therefore 0.81 area, matching TI's stated 81 percent solder coverage
by printed area on the centre thermal pad. TI's 15 thermal vias of 0.2 mm are
noted as a layout task, not p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
Parts:
- U12: footprint (none) -> AQROOT_Beta:TI_TPS63020_DSJ; Package 14-pin VSON (DSJ), 3 mm x 4 mm, with exposed thermal pad - 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 -> DSJ (R-PVSON-N14) 14-pin VSON with exposed thermal pad. Foo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
Changed lines of the file:
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@@
 			)
 		)
-		(property "Footprint" ""
+		(property "Footprint" "AQROOT_Beta:TI_TPS63020_DSJ"
 			(at 248.92 67.31 0)
 			(hide yes)
@@
 			)
 		)
-		(property "Package" "14-pin VSON (DSJ), 3 mm x 4 mm, with exposed thermal pad - exact DSJ land pattern still requires package-drawing verification"
+		(property "Package" "DSJ (R-PVSON-N14) 14-pin VSON with exposed thermal pad. Footprint built from TI drawings 4210895-2/E (LAND PATTERN DATA) and 4208549-3/G (THERMAL PAD MECHANICAL DATA): signal lands 0.24 x 0.60 oval R0.12, 0.5 pitch, 7 per row, rows 2.8 apart at y +/-1.4; NSMD with 0.07 mask expansion; thermal pad 2.85 +/-0.10 x 1.58 +/-0.10; paste ratio -0.05 giving TI's stated 81 percent coverage. Pin 1 bottom-left per TI's circled Example Board Layout callout, 1-7 along the bottom row then 8-14 back along the top. The 4X 0.20 flank features at 0.46 spacing were confirmed by 900 dpi rasterisation to be SLOTS IN A SINGLE CONTIGUOUS THERMAL PAD, not separate pads; the plain dimensioned 2.85 x 1.58 envelope is implemented instead of the comb, which is conservative. TI recommends 15 thermal vias of 0.2 mm (5x3) inside the pad - a layout task, not part of the footprint. See TI SLUA271."
 			(at 248.92 67.31 0)
 			(hide yes)

Commit message: AQROOT Beta: assign verified MAX17048 footprint
U14 (MAX17048G+T10) now carries AQROOT_Beta:MAX17048_T822, verified against
Maxim land pattern 90-0065 Rev E. Assigned in all three places per repo
convention: the MAX17048 library symbol, the 01_power_tree sheet cache and the
U14 instance. Three lines changed, nothing else.

Symbol-to-pad mapping verified 1:1 across exactly nine electrical pads:
1 CTG, 2 CELL, 3 VDD, 4 GND, 5 ~ALRT, 6 QSTRT, 7 SCL, 8 SDA, 9 EP. No phantom,
missing or duplicated pad numbers.

Netlist unchanged: U14 pin-to-net is byte-identical to the pre-change export
(1 GND, 2/3 BAT_PROTECTED_P, 4 GND, 5 MAX17048_ALRT_N, 6 unconnected,
7 I2C_SCL_INT, 8 I2C_SDA_INT, 9 GND). Across the whole design, zero components
changed any pin's net and the net count holds at 175.

Canonical ERC unchanged at 58 raw / 5 errors / 53 warnings, with 58 live
exclusions, 0 stale and 0 post-processed real defects, as expected for a
footprint-only assignment.

Footprint coverage 172 -> 173 of 186. Remaining without footprints: C12, C18,
C19, LS1, R24, SW1-SW8.

Co-Authored-By: Claude Opus 5 <noreply@anthropic.com>
Parts:
- U14: footprint (none) -> AQROOT_Beta:MAX17048_T822
Changed lines of the file:
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@@
 			)
 		)
-		(property "Footprint" ""
+		(property "Footprint" "AQROOT_Beta:MAX17048_T822"
 			(at 115.57 82.55 0)
 			(hide yes)

Commit message: AQROOT Beta: normalize the TPS63020 model to the physical TI package
Root-cause fix. Supersedes the temporary coincident pad-16 compatibility
shim added in 788fff0. No component moved, no routing, no geometry change.

TI SLVS916I (rev I, Oct 2019) section 5, "DSJ Package, 14-Pin VSON with
Exposed Thermal Pad", was re-verified: the Pin Functions table lists 14
numbered pins (1-14); PGND and the Exposed Thermal Pad both carry pin
number "-", and TI states "The exposed thermal pad is connected to PGND".
The physical device therefore has 14 numbered pins plus ONE unnumbered
exposed thermal pad which IS PGND. There is no pin 15 signal pin and no
pin 16 terminal of any kind.

AQROOT convention, now documented in the symbol, the footprint and the
decision log: pin/pad 15 named PGND_EP is the AQROOT/KiCad logical
identifier for TI's unnumbered exposed PGND thermal pad; it is NOT a
manufacturer package pin number. This matches the convention already used
for BQ25185 (EP 11), MAX17048 (EP 9) and ST25R3916 (EP 33) - the exposed
pad takes the next number after the last manufacturer pin.

Changes:
 - symbol AQROOT_Beta:TPS63020 - pin 16 (EP) removed; pin 15 renamed
   PGND -> PGND_EP, electrical type power_in (project EP convention);
   misleading Note property replaced with the TI-verified statement
 - 01_power_tree.kicad_sch - lib_symbols cache updated identically;
   (pin "16") removed from the U12 instance; the now-orphaned wire stub
   (256.54,88.9)-(256.54,87.63) and the GND power symbol at (256.54,88.9)
   removed so no dangling endpoint is created
 - footprint AQROOT_Beta:TI_TPS63020_DSJ - temporary coincident pad 16
   removed; back to 14 signal lands + one thermal land numbered 15.
   TI-verified geometry, pitch, row spacing, thermal copper, mask, paste,
   courtyard and via guidance all untouched
 - PCB - U12 pad-16 instance removed
 - 05 - Design Decisions Log.md - permanent record so the wrong model is
   not reintroduced

Verification:
 - symbol: 15 pins, contiguou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
Connections:
- net GND: no longer U12.16 (EP)
Changed lines of the file:
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@@
 	(wire
 		(pts
-			(xy 256.54 88.9) (xy 256.54 87.63)
-		)
-		(stroke
-			(width 0)
-			(type default)
-		)
-	)
-	(wire
-		(pts
 			(xy 63.5 149.86) (xy 63.5 151.13)
 		)
@@
 	)
 	(symbol
-		(lib_id "power:GND")
-		(at 256.54 88.9 0)
-		(unit 1)
-		(body_style 1)
-		(exclude_from_sim no)
-		(in_bom yes)
-		(on_board yes)
-		(in_pos_files yes)
-		(dnp no)
-		(fields_autoplaced yes)
-		(property "Reference" "#PWR0131"
-			(at 256.54 95.25 0)
-			(hide yes)
-			(show_name no)
-			(do_not_autoplace no)
-			(effects
-				(font
-					(size 1.27 1.27)
-				)
-			)
-		)
-		(property "Value" "GND"
-			(at 256.54 93.98 0)
-			(show_name no)
-			(do_not_autoplace no)
-			(effects
-				(font
-					(size 1.27 1.27)
-				)
-			)
-		)
-		(property "Footprint" ""
-			(at 256.54 88.9 0)
-			(hide yes)
-			(show_name no)
-			(do_not_autoplace no)
-			(effects
-				(font
-					(size 1.27 1.27)
-				)
-			)
-		)
-		(property "Datasheet" ""
-			(at 256.54 88.9 0)
-			(hide yes)
-			(show_name no)
-			(do_not_autoplace no)
-			(effects
-				(font
-					(size 1.27 1.27)
-				)
-			)
-		)
-		(property "Description" "Power symbol creates a global label with name \"GND\" , ground"
-			(at 256.54 88.9 0)
-			(hide yes)
-			(show_name no)
-			(do_not_autoplace no)
-			(effects
-				(font
-					(size 1.27 1.27)
-				)
-			)
-		)
-		(pin "1"
-		)
-		(instances
-			(project "aqroot-Beta"
-				(path "/8a0ad1ee-a49e-4cff-9a78-44823e373405/83b1880a-0a3b-496a-bce6-0dc4c72d8ece"
-					(reference "#PWR0131")
-					(unit 1)
-				)
-			)
-		)
-	)
-	(symbol
 		(lib_id "Device:C")
 		(at 54.61 62.23 0)
@@
 		(pin "15"
 		)
-		(pin "16"
-		)
 		(pin "14"

Commit message: AQROOT Beta: close final routing blockers
Closes the two BLOCKS_ROUTING items left by the pre-routing rule pass.
No traces drawn, no component moved, aqroot-Beta.kicad_dru untouched.

1. BQ25185 charge current locked at 300 mA.

R37 2k 1% -> 1k 1% on the ISET pin. ICHG = KISET/RISET = 300/1000 =
300 mA typ, 285/300/315 mA from the KISET spread and 270-330 mA at
TI's +/-10% ICHG_ACC spec. 0.15 C on the 2000 mAh Beta pack. IPRECHG
rises to 60 mA and ITERM to 30 mA. 1 kohm is TI's own figure in
SLUSF65A section 8.2.2.2, is far above RISET_SHORT (264 ohm), and
300 mA is far below the 1 A device maximum, so nothing is clipped.

R36 = 18 kohm is untouched: the input current limit stays ILIM500
(450/475/498 mA) and VBATREG stays 4.2 V. Both the schematic symbol and
the PCB footprint Value field were updated together, so parity picks up
no new field mismatch.

No power netclass width target changes. VBUS_CHG is set by ILIM, which
did not move; BAT_MAIN is sized by 1.5 A discharge and 3.125 A OCP;
SYS_MAIN is sized by the ~750 mA system load. IPC-2221B needs 0.057 mm
for 300 mA on 1 oz outer copper at dT=10 K, an order of magnitude below
every existing floor, so nothing was widened.

The real consequence is thermal and lands on U11. As a linear charger
with a power path, worst-case dissipation rises from ~0.46 W to ~0.69 W
(0.238 W on IN->SYS at 475 mA plus 0.450 W on the BATFET at 300 mA into
a depleted 3.0 V pack) in a 2.2 x 2.0 mm WSON-10. TREG folds charge
current back rather than failing, so this is a charge-time risk, but
U11's exposed-pad thermal vias are now required rather than optional
and the plan is revised from 1 to 2 THERMAL-class vias. Implementation
stays deferred to the routing/thermal pass.

Added BOM VERIFY: the cell/pack must permit >=300 mA charge, including
the pack protection circuit's own rating. Blocks BOM lock, not routing.

2. USB differential net names normalised to a _P/_N suffix.

  USB_D_P_CONN -> USB_D_CONN_P    USB_D_N_CONN -> USB_D_CONN_N
  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
Parts:
- R37: value 2k 1% -> 1k 1%
Connections:
- net USB_D_N_CONN renamed USB_D_CONN_N
- net USB_D_N_ESD renamed USB_D_ESD_N
- net USB_D_N_MCU renamed USB_D_MCU_N
- net USB_D_P_CONN renamed USB_D_CONN_P
- net USB_D_P_ESD renamed USB_D_ESD_P
- net USB_D_P_MCU renamed USB_D_MCU_P
Changed lines of the file:
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@@
 		)
 	)
-	(label "USB_D_N_CONN"
+	(label "USB_D_CONN_N"
 		(at 49.53 45.72 0)
 		(effects
@@
 		)
 	)
-	(label "USB_D_P_ESD"
+	(label "USB_D_ESD_P"
 		(at 153.67 46.99 0)
 		(effects
@@
 		)
 	)
-	(label "USB_D_N_MCU"
+	(label "USB_D_MCU_N"
 		(at 54.61 57.15 0)
 		(effects
@@
 		)
 	)
-	(label "USB_D_P_MCU"
+	(label "USB_D_MCU_P"
 		(at 76.2 57.15 0)
 		(effects
@@
 		)
 	)
-	(label "USB_D_P_CONN"
+	(label "USB_D_CONN_P"
 		(at 49.53 50.8 0)
 		(effects
@@
 		)
 	)
-	(label "USB_D_N_ESD"
+	(label "USB_D_ESD_N"
 		(at 165.1 25.4 180)
 		(effects
@@
 		)
 	)
-	(label "USB_D_P_ESD"
+	(label "USB_D_ESD_P"
 		(at 166.37 34.29 180)
 		(effects
@@
 		)
 	)
-	(label "USB_D_P_CONN"
+	(label "USB_D_CONN_P"
 		(at 139.7 46.99 180)
 		(effects
@@
 		)
 	)
-	(label "USB_D_N_ESD"
+	(label "USB_D_ESD_N"
 		(at 153.67 44.45 0)
 		(effects
@@
 		)
 	)
-	(label "USB_D_N_CONN"
+	(label "USB_D_CONN_N"
 		(at 139.7 44.45 180)
 		(effects
@@
 		)
 	)
-	(hierarchical_label "USB_D_N_MCU"
+	(hierarchical_label "USB_D_MCU_N"
 		(shape output)
 		(at 177.8 25.4 0)
@@
 		)
 	)
-	(hierarchical_label "USB_D_P_MCU"
+	(hierarchical_label "USB_D_MCU_P"
 		(shape output)
 		(at 177.8 34.29 0)
@@
 			)
 		)
-		(property "Value" "2k 1%"
+		(property "Value" "1k 1%"
 			(at 31.75 167.6399 0)
 			(show_name no)
