File: hardware/beta/kicad/aqroot-beta/02_mcu_core.kicad_sch (KiCad schematic)
At the start: 9 parts, among them SW1 BOOT, U1 ESP32-S3-WROOM-1

Commit message: AQROOT Beta: assign remaining test-point footprints
TP1-TP5 carried an empty Footprint property while TP6-TP12 all used
TestPoint:TestPoint_Pad_D1.0mm. They now match the project convention, so
every test point in the design has a footprint.

  TP1  02_mcu_core   /02_MCU_CORE/TEST_GPIO45
  TP2  02_mcu_core   /02_MCU_CORE/TEST_GPIO46
  TP3  05_i2c        /BMI270_INT1_STRAP
  TP4  05_i2c        /I2C_SDA_INT
  TP5  05_i2c        /I2C_SCL_INT

Property-value edit only - five lines. No symbol was moved, no pin
reconnected, no wire or label touched.

Verified with kicad-cli: netlist pin-to-net mapping byte-identical before
and after, each TP still on its original net. ERC unchanged: raw 48,
unique 24, excluded 24, real 0.

Co-Authored-By: Claude Opus 5 <noreply@anthropic.com>
Parts:
- TP1, TP2: footprint (none) -> TestPoint:TestPoint_Pad_D1.0mm
Changed lines of the file:
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@@
 			)
 		)
-		(property "Footprint" ""
+		(property "Footprint" "TestPoint:TestPoint_Pad_D1.0mm"
 			(at 193.04 111.76 0)
 			(hide yes)
@@
 			)
 		)
-		(property "Footprint" ""
+		(property "Footprint" "TestPoint:TestPoint_Pad_D1.0mm"
 			(at 172.72 111.76 0)
 			(hide yes)

Commit message: AQROOT Beta: assign standard passive footprints
Assigns footprints to 40 passives whose package is unambiguous from
existing project precedent. Property-value edits only - no symbol, wire,
label or net touched.

  28 resistors -> Resistor_SMD:R_0603_1608Metric
     R1 R2 R3-R17 R18 R19 R20 R21 R22 R23 R25 R26 R27 R28 R29
     Basis: all 39 already-assigned resistors in the project are 0603, and
     every one of these is signal-level (pull-ups, dividers, series
     termination, MOSFET gate network).

  12 capacitors -> Capacitor_SMD:C_0603_1608Metric
     C1 C2 C4 C5 C6 C7 C8 C9 C13 C14 C16 C17
     Basis: 100nF is 5/5 and 1uF is 4/4 for 0603 among already-assigned
     capacitors - unanimous.

DELIBERATELY NOT ASSIGNED - split precedent, needs a decision:
  C3, C15, C10  10uF   -> project uses BOTH C_1206 (x2) and C_0805 (x1)
  C11           4.7uF  -> single 0805 precedent, different subsystem
Bulk capacitors must not be blindly converted to 0603, and the existing
precedent does not settle 0805 vs 1206.

Also untouched per instruction: C12/R24/Q1 (TBD), C18/C19 (placeholder),
L1/L2, mechanical switches and connectors, and the four RF/module
placeholders.

Separately noted, NOT changed here: C24 is 22uF 25V X7R with
C_0603_1608Metric already assigned. A 22uF 25V X7R does not exist in 0603
and the project's other 22uF parts use 1206/0805 - this looks like a
pre-existing error and is flagged for the BOM pass, not silently altered.

Verified with kicad-cli: netlist pin-to-net mapping byte-identical before
and after. ERC unchanged: raw 48, unique 24, excluded 24, real 0.
Footprint coverage 97 -> 137 of 166 components.

Co-Authored-By: Claude Opus 5 <noreply@anthropic.com>
Parts:
- C1, C2: footprint (none) -> Capacitor_SMD:C_0603_1608Metric
- R1, R2: footprint (none) -> Resistor_SMD:R_0603_1608Metric
Changed lines of the file:
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@@
 			)
 		)
-		(property "Footprint" ""
+		(property "Footprint" "Resistor_SMD:R_0603_1608Metric"
 			(at 93.218 67.31 90)
 			(hide yes)
@@
 			)
 		)
-		(property "Footprint" ""
+		(property "Footprint" "Capacitor_SMD:C_0603_1608Metric"
 			(at 90.4748 74.93 0)
 			(hide yes)
@@
 			)
 		)
-		(property "Footprint" ""
+		(property "Footprint" "Capacitor_SMD:C_0603_1608Metric"
 			(at 173.6852 91.44 0)
 			(hide yes)
@@
 			)
 		)
-		(property "Footprint" ""
+		(property "Footprint" "Resistor_SMD:R_0603_1608Metric"
 			(at 78.232 86.36 90)
 			(hide yes)

Commit message: AQROOT Beta: assign remaining generic bulk-cap footprints
Assigns Capacitor_SMD:C_0805_2012Metric to the four bulk capacitors left
open by the standard-passive pass.

  C3   10uF   +3V3                  02_mcu_core     generic bulk decoupling
  C15  10uF   +3V3                  03_spi_a        generic bulk decoupling
  C10  10uF   +3V3                  06_audio        generic bulk decoupling
  C11  4.7uF  /07_IR/IR_RX_VS_LOCAL 07_ir           TSOP382 supply RC

Basis: these are NOT regulator input/output capacitors. The project's 1206
precedent (C26/C27 CIN, C29-C32 COUT) is a TPS63020-specific requirement -
the kicad README states '1206 preferred ... Close to VIN/PGND' for those
parts only, so it does not generalise. For generic 10uF/10V and 4.7uF/10V
bulk on a 3.3V rail, 0805 is adequate and is the project's generic
precedent (C33, C20). C11's role is documented at libraries/README.md:1264
as Vishay's TSOP382 application R1/C1 supply filter, paired with R21 100R.

Property-value edits only - four lines. No value, symbol, wire, label or
net touched.

Verified with kicad-cli: netlist pin-to-net mapping byte-identical before
and after. ERC unchanged: raw 48, unique 24, excluded 24, real 0.

Still open and deliberately untouched: exact MPNs and DC-bias derating for
these parts. A 10uF/10V 0805 X7R typically retains only ~60-70% of its
nominal capacitance at 3.3V, so effective capacitance must be confirmed at
the BOM pass - the package is locked here, the part is not.

Co-Authored-By: Claude Opus 5 <noreply@anthropic.com>
Parts:
- C3: footprint (none) -> Capacitor_SMD:C_0805_2012Metric
Changed lines of the file:
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@@
 			)
 		)
-		(property "Footprint" ""
+		(property "Footprint" "Capacitor_SMD:C_0805_2012Metric"
 			(at 190.1952 91.44 0)
 			(hide yes)

Commit message: AQROOT Beta: lock final user-button footprints
SW1-SW8 assigned Button_Switch_SMD:SW_SPST_PTS645Sx43SMTR92.

Classification: VERIFIED_VENDOR_EXACT. Checked against the C&K / Littelfuse
PTS645 series datasheet (Revised VL 01/29/26), RECOMMENDED PCB LAYOUT panels,
rasterised to confirm which feature each dimension attaches to. The drawing
gives 9.5 outer-edge to outer-edge and 6.4 inner-edge to inner-edge in X, and
5.8 outer to 3.2 inner in Y, which yields pads 1.55 (X) x 1.30 (Y) on centres of
+/-3.975 (X) and +/-2.25 (Y). The KiCad footprint implements 1.55 x 1.30 at
(+/-3.98, +/-2.25): exact on pad size and on the Y centre, with a 0.005 mm
rounding on the X centre that is far inside any fabrication tolerance.

The ratified premise that straight-SMT PTS645 variants share one published land
pattern is confirmed rather than assumed: the identical 9.5 / 6.4 / 5.8 / 3.2
set is published for both the 4.3 mm SMT G Type and the 7.3 mm straight SMT
variants. That is why the footprint can be locked while the actuator-height
suffix is not.

Pad mapping verified: four physical pads; C&K numbers 1 and 2 on the top row and
3 and 4 on the bottom row with 1-2 tied and 3-4 tied, so the footprint's pad 1
covers the top pair and pad 2 the bottom pair, matching the 2-pin
Switch:SW_Push symbol. No phantom or missing pads.

BOM status is FOOTPRINT LOCKED / BOM SUFFIX VERIFY. MPN is recorded as the
approved family notation PTS645Sx SMTR92 LFS with 160gf TARGET, ~5mm ACTUATOR
TARGET, ~0.25 mm travel and 100,000 operation class marked as selection targets.
No actuator height, force suffix, package code, travel or lifecycle figure was
invented.

SCOPE NOTE - the eight footprintless switches are SW1 plus SW2-SW8. SW1 is the
ESP32 BOOT strap button on 02_mcu_core, not a user-facing game button; it takes
the same part and land pattern but receives no plastic cap. The seven
user-facing buttons are SW2-SW8. SW9, the power slide switch, already had its
own footprint and was not touched.

Enclosur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
Parts:
- SW1: footprint (none) -> Button_Switch_SMD:SW_SPST_PTS645Sx43SMTR92; BOM_Status (none) -> C&K / Littelfuse PTS645 family, 6 mm SMD, top-actuated. FIN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; Footprint_Provenance (none) -> Land pattern VERIFIED_VENDOR_EXACT against the C&K / Littel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; MPN (none) -> PTS645Sx SMTR92 LFS; Manufacturer (none) -> C&K / Littelfuse; Mounting (none) -> BOARD_MOUNTED; Note (none) -> ESP32 BOOT strap button - electrically identical part, but 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; Package (none) -> 6.0 x 6.0 mm tactile switch, straight SMT gull-wing, 4 term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
Changed lines of the file:
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@@
 			)
 		)
-		(property "Footprint" ""
+		(property "Footprint" "Button_Switch_SMD:SW_SPST_PTS645Sx43SMTR92"
 			(at 87.63 90.17 0)
 			(hide yes)
@@
 			(at 87.63 95.25 0)
 			(hide yes)
+			(show_name no)
+			(do_not_autoplace no)
+			(effects
+				(font
+					(size 1.27 1.27)
+				)
+			)
+		)
+		(property "Manufacturer" "C&K / Littelfuse"
+			(at 87.63 95.25 0)
+			(hide yes)
+			(show_name no)
+			(do_not_autoplace no)
+			(effects
+				(font
+					(size 1.27 1.27)
+				)
+			)
+		)
+		(property "MPN" "PTS645Sx SMTR92 LFS"
+			(at 87.63 95.25 0)
+			(hide yes)
+			(show_name no)
+			(do_not_autoplace no)
+			(effects
+				(font
+					(size 1.27 1.27)
+				)
+			)
+		)
+		(property "Package" "6.0 x 6.0 mm tactile switch, straight SMT gull-wing, 4 terminals"
+			(at 87.63 95.25 0)
+			(hide yes)
+			(show_name no)
+			(do_not_autoplace no)
+			(effects
+				(font
+					(size 1.27 1.27)
+				)
+			)
+		)
+		(property "Mounting" "BOARD_MOUNTED"
+			(at 87.63 95.25 0)
+			(hide yes)
+			(show_name no)
+			(do_not_autoplace no)
+			(effects
+				(font
+					(size 1.27 1.27)
+				)
+			)
+		)
+		(property "BOM_Status" "C&K / Littelfuse PTS645 family, 6 mm SMD, top-actuated. FINAL SUFFIX VERIFY AT BOM LOCK - 160gf TARGET, ~5mm ACTUATOR TARGET, ~0.25 mm travel and 100,000 operation class are the selection targets, not a quoted commercial suffix. FOOTPRINT LOCKED / BOM SUFFIX VERIFY."
+			(at 87.63 95.25 0)
+			(hide yes)
+			(show_name no)
+			(do_not_autoplace no)
+			(effects
+				(font
+					(size 1.27 1.27)
+				)
+			)
+		)
+		(property "Footprint_Provenance" "Land pattern VERIFIED_VENDOR_EXACT against the C&K / Littelfuse PTS645 series datasheet (Revised VL 01/29/26), RECOMMENDED PCB LAYOUT / PCB LAYOUT panels. The drawing gives 9.5 outer-edge to outer-edge and 6.4 inner-edge to inner-edge in X, and 5.8 outer to 3.2 inner in Y, which yields pads 1.55 (X) x 1.30 (Y) on centres of +/-3.975 (X) and +/-2.25 (Y). KiCad Button_Switch_SMD:SW_SPST_PTS645Sx43SMTR92 implements 1.55 x 1.30 at (+/-3.98, +/-2.25) - exact on pad size and on the Y centre, with a 0.005 mm rounding on the X centre that is far inside any fabrication tolerance. The same land pattern is published for both the 4.3 mm SMT G Type and the 7.3 mm straight SMT variants, which is why the footprint can be locked before the actuator-height suffix is. Four physical pads; C&K numbers them 1 and 2 on the top row and 3 and 4 on the bottom row with 1-2 tied and 3-4 tied, so the KiCad footprint maps its pad 1 to the top pair and pad 2 to the bottom pair, matching the 2-pin Switch:SW_Push symbol."
+			(at 87.63 95.25 0)
+			(hide yes)
+			(show_name no)
+			(do_not_autoplace no)
+			(effects
+				(font
+					(size 1.27 1.27)
+				)
+			)
+		)
+		(property "Note" "ESP32 BOOT strap button - electrically identical part, but it is not a user-facing game button and does not receive a plastic cap. ENCLOSURE DESIGN TARGETS - these are AQROOT enclosure targets, NOT C&K switch specifications: individual plastic button caps, no membrane for Beta; 0.1-0.3 mm rest gap above the actuator with no preload; enclosure hard stop sized for ~0.3-0.4 mm total cap travel so the user cannot drive the tactile switch past its own travel."
+			(at 87.63 95.25 0)
+			(hide yes)

Commit message: AQROOT Beta: close final routing blockers
Closes the two BLOCKS_ROUTING items left by the pre-routing rule pass.
No traces drawn, no component moved, aqroot-Beta.kicad_dru untouched.

1. BQ25185 charge current locked at 300 mA.

R37 2k 1% -> 1k 1% on the ISET pin. ICHG = KISET/RISET = 300/1000 =
300 mA typ, 285/300/315 mA from the KISET spread and 270-330 mA at
TI's +/-10% ICHG_ACC spec. 0.15 C on the 2000 mAh Beta pack. IPRECHG
rises to 60 mA and ITERM to 30 mA. 1 kohm is TI's own figure in
SLUSF65A section 8.2.2.2, is far above RISET_SHORT (264 ohm), and
300 mA is far below the 1 A device maximum, so nothing is clipped.

R36 = 18 kohm is untouched: the input current limit stays ILIM500
(450/475/498 mA) and VBATREG stays 4.2 V. Both the schematic symbol and
the PCB footprint Value field were updated together, so parity picks up
no new field mismatch.

No power netclass width target changes. VBUS_CHG is set by ILIM, which
did not move; BAT_MAIN is sized by 1.5 A discharge and 3.125 A OCP;
SYS_MAIN is sized by the ~750 mA system load. IPC-2221B needs 0.057 mm
for 300 mA on 1 oz outer copper at dT=10 K, an order of magnitude below
every existing floor, so nothing was widened.

The real consequence is thermal and lands on U11. As a linear charger
with a power path, worst-case dissipation rises from ~0.46 W to ~0.69 W
(0.238 W on IN->SYS at 475 mA plus 0.450 W on the BATFET at 300 mA into
a depleted 3.0 V pack) in a 2.2 x 2.0 mm WSON-10. TREG folds charge
current back rather than failing, so this is a charge-time risk, but
U11's exposed-pad thermal vias are now required rather than optional
and the plan is revised from 1 to 2 THERMAL-class vias. Implementation
stays deferred to the routing/thermal pass.

Added BOM VERIFY: the cell/pack must permit >=300 mA charge, including
the pack protection circuit's own rating. Blocks BOM lock, not routing.

2. USB differential net names normalised to a _P/_N suffix.

  USB_D_P_CONN -> USB_D_CONN_P    USB_D_N_CONN -> USB_D_CONN_N
  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
Connections:
- net USB_D_N_MCU renamed USB_D_MCU_N
- net USB_D_P_MCU renamed USB_D_MCU_P
Changed lines of the file:
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@@
 		)
 	)
-	(hierarchical_label "USB_D_P_MCU"
+	(hierarchical_label "USB_D_MCU_P"
 		(shape bidirectional)
 		(at 149.86 86.36 0)
@@
 		)
 	)
-	(hierarchical_label "USB_D_N_MCU"
+	(hierarchical_label "USB_D_MCU_N"
 		(shape bidirectional)
 		(at 149.86 83.82 0)

Commit message: move SX1262_DIO1 to IO38, NFC_IRQ to IO18
SX1262_DIO1 could not escape U1.11 under any placement-preserving
routing: the U1 belly corridor holds exactly two 0.20 mm tracks and
both are consumed by SX1262_CS_N and SX1262_BUSY, while the USB F.Cu
pair forbids any through-via north of them. Deleting the entire
BMI270_INT1_STRAP net still left zero reachable via sites, and the
four-depth stack destroyed the last transition pocket. The trap is a
property of the pad, not the net, so swapping DIO1 with CS_N or BUSY
would only strand a more critical signal.

U1.31 / IO38 was chosen from a flood test of candidate host pads:
31,369 legal via sites at 1.100 mm best margin, on the south row and
on the correct side for the x63 E5 lane. IO45 and IO46 were rejected
as strapping pins reserved as test pads, and IO46's pad is trapped as
well.

Changes are two hierarchical labels in 02_mcu_core.kicad_sch and the
two matching pad net assignments. No copper moved: 493 tracks and 129
vias before and after, 0 added, 0 removed, 188 footprints unmoved.
SX1262_CS_N keeps E5 x62, U8.19 and its R27 pull-up; SX1262_BUSY keeps
E5 x64 and U8.14; SX1262_DIO1 keeps E5 x63 and U8.13 with only its MCU
endpoint moved.

NFC_IRQ now sits on U1.11 and is INTENTIONALLY NOT CONNECTED for Beta.
The hardware IRQ is deferred to the NFC-enablement respin; Beta NFC
scope is polling-based digital bring-up only, and ST25R3916
interrupt-status polling must be verified during bring-up.

DRC 0 electrical errors, ratsnest 419, schematic parity 261 delta 0
with no parity entry on either swapped net. ERC 116 total / 58 live,
unchanged. SX1262_DIO1 is not routed in this commit.

Co-Authored-By: Claude Opus 5 <noreply@anthropic.com>
Claude-Session: https://claude.ai/code/session_01N3T9f8EXqAwVAJudcbiTW4
Connections:
- net NFC_IRQ: now also U1.11 (IO18); no longer U1.31 (IO38)
- net SX1262_DIO1: now also U1.31 (IO38); no longer U1.11 (IO18)
Changed lines of the file:
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@@
 		)
 	)
-	(hierarchical_label "SX1262_DIO1"
+	(hierarchical_label "NFC_IRQ"
 		(shape input)
 		(at 149.86 81.28 0)
@@
 		)
 	)
-	(hierarchical_label "NFC_IRQ"
+	(hierarchical_label "SX1262_DIO1"
 		(shape input)
 		(at 149.86 99.06 0)
