File: hardware/beta/kicad/aqroot-beta/aqroot-Beta.kicad_pcb (KiCad board)
At the start: 4 copper layers, 74 x 155 mm, 188 parts, among them J1 CH280QV10-CT_50P, J2 Molex_5025700893, J3 USB_C_Receptacle_USB2.0_16P, J4 JST-PH-2 BATTERY, J5 COMMUNITY_HEADER_2x13, J6 JST-PH-2 SPEAKER, Q1 AO3400A, SW1 BOOT, SW2 UP, SW3 DOWN, SW4 LEFT, SW5 RIGHT, SW6 A_SELECT, SW7 B_BACK, SW8 HOME, SW9 SW_SPDT, U1 ESP32-S3-WROOM-1, U10 USBLC6-2SC6, U11 BQ25185, U12 TPS63020, U13 TPS61023, U14 MAX17048, U15 TPS22918, U16 TCA9517ADGK, U17 TPS61169DCKR, U2 TCA9535PWR, U3 TCA9535PWR, U4 BMI270, U5 MAX98357A, U6 TSOP38238, U7 E07-400M10S, U8 E22-900M22S, U9 ST25R3916-AQET

Commit message: route SX1262 CS_N and BUSY
Closes the two U1-origin SX1262 control nets. Each is a single copper
island: SX1262_CS_N over U1.10, U8.19 and R27.2 (R27 is a pull-up tee,
confirmed from the netlist, not a series element); SX1262_BUSY over
U1.12 and U8.14. Board ratsnest 424 -> 419, DRC 0 electrical errors.

The U1 belly corridor between the north pad row and the
BMI270_INT1_STRAP track is 1.200 mm and holds exactly two 0.20 mm
tracks, at y 18.300 and y 18.700, at exactly 0.2000 mm throughout.
Escape depth must increase eastward, and BUSY is capped by the strap,
so only two of the three controls can leave U1. SX1262_DIO1 is left
unrouted deliberately; its solution space is intact and it needs a
placement ruling.

The two nets take different corridors east because the I2C fan-out
barrier has a single 0.200 mm opening: BUSY runs the far-north lane
with a jog to y 8.750 around the I2C_SCL_INT via, CS_N runs a southern
In2 lane at y 82.250 / 80.700 that threads the SPI_A_MISO via row and
passes north of the J4 pads.

E5 crossings x 62.000 and x 64.000 consumed in place. 0 new vias in
either RF band, 0 new B.Cu band transit, no keepout incursions.
Tracks 459 -> 493, vias 123 -> 129, 0 objects removed, 188 footprints
unmoved. ERC 116 / 58 live and schematic parity 261 both unchanged.

Co-Authored-By: Claude Opus 5 <noreply@anthropic.com>
Claude-Session: https://claude.ai/code/session_01N3T9f8EXqAwVAJudcbiTW4
Routing:
- net /SX1262_BUSY: track 32.0 -> 195.1 mm, vias 0 -> 4
- net /SX1262_CS_N: track 32.0 -> 175.9 mm, vias 0 -> 2

Commit message: move SX1262_DIO1 to IO38, NFC_IRQ to IO18
SX1262_DIO1 could not escape U1.11 under any placement-preserving
routing: the U1 belly corridor holds exactly two 0.20 mm tracks and
both are consumed by SX1262_CS_N and SX1262_BUSY, while the USB F.Cu
pair forbids any through-via north of them. Deleting the entire
BMI270_INT1_STRAP net still left zero reachable via sites, and the
four-depth stack destroyed the last transition pocket. The trap is a
property of the pad, not the net, so swapping DIO1 with CS_N or BUSY
would only strand a more critical signal.

U1.31 / IO38 was chosen from a flood test of candidate host pads:
31,369 legal via sites at 1.100 mm best margin, on the south row and
on the correct side for the x63 E5 lane. IO45 and IO46 were rejected
as strapping pins reserved as test pads, and IO46's pad is trapped as
well.

Changes are two hierarchical labels in 02_mcu_core.kicad_sch and the
two matching pad net assignments. No copper moved: 493 tracks and 129
vias before and after, 0 added, 0 removed, 188 footprints unmoved.
SX1262_CS_N keeps E5 x62, U8.19 and its R27 pull-up; SX1262_BUSY keeps
E5 x64 and U8.14; SX1262_DIO1 keeps E5 x63 and U8.13 with only its MCU
endpoint moved.

NFC_IRQ now sits on U1.11 and is INTENTIONALLY NOT CONNECTED for Beta.
The hardware IRQ is deferred to the NFC-enablement respin; Beta NFC
scope is polling-based digital bring-up only, and ST25R3916
interrupt-status polling must be verified during bring-up.

DRC 0 electrical errors, ratsnest 419, schematic parity 261 delta 0
with no parity entry on either swapped net. ERC 116 total / 58 live,
unchanged. SX1262_DIO1 is not routed in this commit.

Co-Authored-By: Claude Opus 5 <noreply@anthropic.com>
Claude-Session: https://claude.ai/code/session_01N3T9f8EXqAwVAJudcbiTW4
Connections:
- U1 pad 11: /SX1262_DIO1 -> /NFC_IRQ
- U1 pad 31: /NFC_IRQ -> /SX1262_DIO1
Changed lines of the file:
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@@
 			(size 1.5 0.9)
 			(layers "B.Cu" "B.Mask" "B.Paste")
-			(net "/SX1262_DIO1")
+			(net "/NFC_IRQ")
 		)
 		(pad "12" smd rect
@@
 			(size 1.5 0.9)
 			(layers "B.Cu" "B.Mask" "B.Paste")
-			(net "/NFC_IRQ")
+			(net "/SX1262_DIO1")
 		)
 		(pad "32" smd rect

Commit message: route SX1262_DIO1 from IO38
Closes the last U1-origin SX1262 control. One copper island over U1.31
and U8.13, 148.407 mm, 14 tracks and 5 vias across B.Cu 7 / In2 5 /
F.Cu 2, minimum clearance 0.30000 mm copper across the whole net.
Board ratsnest 419 -> 417, DRC 0 electrical errors.

From U1.11 this net had zero reachable via sites under any
placement-preserving change. From U1.31 it routed on the first attempt
with half again the clearance the CS_N and BUSY escapes had to accept,
and with no zero-margin geometry anywhere.

Three walls, three answers. The SD_CS_N / SPI_A palisade plus
DISP_CS_N's In2 vertical block both B.Cu and In2 across x 23.7-27.4,
so a 4.6 mm F.Cu hop between two vias clears all five at once. NFC
RESERVED ends at y 35, so the long eastward run crosses x 28-54 freely
on B.Cu at y 39. The I2C In2 walls at y 76 and y 77 span the whole
descent corridor, so the descent stays on B.Cu at x 59.500, which is
clear from y 14.5 to 81.3.

The eastern transition drops to In2 at x 63.400 rather than 63.000:
that 0.400 mm offset lifts the via clear of BAT_PROTECTED_P from
0.200 mm to 0.400 mm, and a short In2 jog returns the net to the
x 63.000 lane before y 84. At U8 the net passes beneath BUSY's
approach on B.Cu rather than crossing it.

The x63 E5 crossing is consumed and no longer appears in the
free-endpoint audit; CS_N keeps x62 and BUSY keeps x64, none moved,
resized, duplicated or swapped. 0 new vias in either RF band, 0 new
B.Cu band transit, no keepout incursions.

NFC_IRQ remains 0 tracks / 0 vias / 0 zones. Its single ratsnest item
is the documented intentional-unrouted ledger entry, so 417 is the
correct end state.

Tracks 493 -> 506, vias 129 -> 134, 0 removed, all 18 additions on
/SX1262_DIO1. 188 footprints unmoved, 0 pad net assignments changed.
ERC 116 / 58 live and schematic parity 261 delta 0, both unchanged.

Co-Authored-By: Claude Opus 5 <noreply@anthropic.com>
Claude-Session: https://claude.ai/code/session_01N3T9f8EXqAwVAJudcbiTW4
Routing:
- net /SX1262_DIO1: track 32.0 -> 148.4 mm, vias 0 -> 5
Changed lines of the file:
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@@
 	(footprint "C_0603_1608Metric"
 		(layer "F.Cu")
-		(at 22 26.9)
+		(at 22.225 29.4 -90)
 		(descr "Capacitor SMD 0603 (1608 Metric), square (rectangular) end terminal, IPC-7351 nominal, (Body size source: IPC-SM-782 page 76, https://www.pcb-3d.com/wordpress/wp-content/uploads/ipc-sm-782a_amendment_1_and_2.pdf)")
 		(tags "capacitor")
-		(property "Reference" "C50"
-			(at 0 -1.43 0)
+		(property "Reference" "C55"
+			(at 0 -1.43 270)
 			(layer "F.SilkS")
 			(effects
@@
 			)
 		)
-		(property "Value" "10nF"
-			(at 0 1.43 0)
+		(property "Value" "2.2uF"
+			(at 0 1.43 270)
 			(layer "F.Fab")
 			(effects
@@
 		)
 		(property "Datasheet" ""
-			(at 0 0 0)
+			(at 0 0 270)
 			(layer "F.Fab")
 			(hide yes)
@@
 		)
 		(property "Description" ""
-			(at 0 0 0)
+			(at 0 0 270)
 			(layer "F.Fab")
 			(hide yes)
@@
 		)
 		(property "KiLib_Generator" "SMD_2terminal_chip_molded"
-			(at 0 0 0)
+			(at 0 0 270)
 			(layer "F.SilkS")
 			(hide yes)
@@
 		(duplicate_pad_numbers_are_jumpers no)
 		(fp_line
-			(start -0.14058 -0.51)
-			(end 0.14058 -0.51)
+			(start -0.14058 0.51)
+			(end 0.14058 0.51)
 			(stroke
 				(width 0.12)
@@
 		)
 		(fp_line
-			(start -0.14058 0.51)
-			(end 0.14058 0.51)
+			(start -0.14058 -0.51)
+			(end 0.14058 -0.51)
 			(stroke
 				(width 0.12)
@@
 		)
 		(fp_text user "${REFERENCE}"
-			(at 0 0 0)
+			(at 0 0 270)
 			(layer "F.Fab")
 			(effects
@@
 		)
 		(pad "1" smd roundrect
-			(at -0.775 0)
+			(at -0.775 0 270)
 			(size 0.9 0.95)
 			(layers "F.Cu" "F.Mask" "F.Paste")
 			(roundrect_rratio 0.25)
-			(net "/04_SPI_B_RADIOS_NFC/NFC_VDD_RF")
+			(net "/NFC_5V_PA_PENDING")
 		)
 		(pad "2" smd roundrect
-			(at 0.775 0)
+			(at 0.775 0 270)
 			(size 0.9 0.95)
 			(layers "F.Cu" "F.Mask" "F.Paste")
@@
 	(footprint "C_0603_1608Metric"
 		(layer "F.Cu")
-		(at 22.225 29.4 -90)
+		(at 22 26.9)
 		(descr "Capacitor SMD 0603 (1608 Metric), square (rectangular) end terminal, IPC-7351 nominal, (Body size source: IPC-SM-782 page 76, https://www.pcb-3d.com/wordpress/wp-content/uploads/ipc-sm-782a_amendment_1_and_2.pdf)")
 		(tags "capacitor")
-		(property "Reference" "C55"
-			(at 0 -1.43 270)
+		(property "Reference" "C50"
+			(at 0 -1.43 0)
 			(layer "F.SilkS")
 			(effects
@@
 			)
 		)
-		(property "Value" "2.2uF"
-			(at 0 1.43 270)
+		(property "Value" "10nF"
+			(at 0 1.43 0)
 			(layer "F.Fab")
 			(effects
@@
 		)
 		(property "Datasheet" ""
-			(at 0 0 270)
+			(at 0 0 0)
 			(layer "F.Fab")
 			(hide yes)
@@
 		)
 		(property "Description" ""
-			(at 0 0 270)
+			(at 0 0 0)
 			(layer "F.Fab")
 			(hide yes)
@@
 		)
 		(property "KiLib_Generator" "SMD_2terminal_chip_molded"
-			(at 0 0 270)
+			(at 0 0 0)
 			(layer "F.SilkS")
 			(hide yes)
@@
 		(duplicate_pad_numbers_are_jumpers no)
 		(fp_line
-			(start -0.14058 0.51)
-			(end 0.14058 0.51)
+			(start -0.14058 -0.51)
+			(end 0.14058 -0.51)
 			(stroke
 				(width 0.12)
@@
 		)
 		(fp_line
-			(start -0.14058 -0.51)
-			(end 0.14058 -0.51)
+			(start -0.14058 0.51)
+			(end 0.14058 0.51)
 			(stroke
 				(width 0.12)
@@
 		)
 		(fp_text user "${REFERENCE}"
-			(at 0 0 270)
+			(at 0 0 0)
 			(layer "F.Fab")
 			(effects
@@
 		)
 		(pad "1" smd roundrect
-			(at -0.775 0 270)
+			(at -0.775 0)
 			(size 0.9 0.95)
 			(layers "F.Cu" "F.Mask" "F.Paste")
 			(roundrect_rratio 0.25)
-			(net "/NFC_5V_PA_PENDING")
+			(net "/04_SPI_B_RADIOS_NFC/NFC_VDD_RF")
 		)
 		(pad "2" smd roundrect
-			(at 0.775 0 270)
+			(at 0.775 0)
 			(size 0.9 0.95)
 			(layers "F.Cu" "F.Mask" "F.Paste")
@@
 	)
 	(segment
+		(start 23.4 39)
+		(end 28 39)
+		(width 0.2)
+		(layer "F.Cu")
+		(net "/SX1262_DIO1")
+	)
+	(segment
+		(start 59.5 78)
+		(end 63.4 78)
+		(width 0.2)
+		(layer "F.Cu")
+		(net "/SX1262_DIO1")
+	)
+	(via
+		(at 23.4 39)
+		(size 0.6)
+		(drill 0.3)
+		(layers "F.Cu" "B.Cu")
+		(net "/SX1262_DIO1")
+	)
+	(via
+		(at 28 39)
+		(size 0.6)
+		(drill 0.3)
+		(layers "F.Cu" "B.Cu")
+		(net "/SX1262_DIO1")
+	)
+	(via
+		(at 59.5 78)
+		(size 0.6)
+		(drill 0.3)
+		(layers "F.Cu" "B.Cu")
+		(net "/SX1262_DIO1")
+	)
+	(via
+		(at 63.4 78)
+		(size 0.6)
+		(drill 0.3)
+		(layers "F.Cu" "B.Cu")
+		(net "/SX1262_DIO1")
+	)
+	(via
+		(at 63 132.5)
+		(size 0.6)
+		(drill 0.3)
+		(layers "F.Cu" "B.Cu")
+		(net "/SX1262_DIO1")
+	)
+	(segment
+		(start 19.2 35)
+		(end 19.2 38.6)
+		(width 0.2)
+		(layer "B.Cu")
+		(net "/SX1262_DIO1")
+	)
+	(segment
+		(start 19.2 38.6)
+		(end 23.4 38.6)
+		(width 0.2)
+		(layer "B.Cu")
+		(net "/SX1262_DIO1")
+	)
+	(segment
+		(start 23.4 38.6)
+		(end 23.4 39)
+		(width 0.2)
+		(layer "B.Cu")
+		(net "/SX1262_DIO1")
+	)
+	(segment
+		(start 28 39)
+		(end 59.5 39)
+		(width 0.2)
+		(layer "B.Cu")
+		(net "/SX1262_DIO1")
+	)
+	(segment
+		(start 59.5 39)
+		(end 59.5 78)
+		(width 0.2)
+		(layer "B.Cu")
+		(net "/SX1262_DIO1")
+	)
+	(segment
+		(start 63 132.5)
+		(end 63 134.73)
+		(width 0.2)
+		(layer "B.Cu")
+		(net "/SX1262_DIO1")
+	)
+	(segment
+		(start 63 134.73)
+		(end 58.6 134.73)
+		(width 0.2)
+		(layer "B.Cu")
+		(net "/SX1262_DIO1")
+	)
+	(segment
 		(start 63 85)
 		(end 63 117)
 		(width 0.2)
 		(layer "In2.Cu")
+		(net "/SX1262_DIO1")
+	)
+	(segment
+		(start 63.4 78)
+		(end 63.4 82)
+		(width 0.2)
+		(layer "In2.Cu")
+		(net "/SX1262_DIO1")
+	)
+	(segment
+		(start 63.4 82)
+		(end 63 83)
+		(width 0.2)
+		(layer "In2.Cu")
+		(net "/SX1262_DIO1")
+	)
+	(segment
+		(start 63 83)
+		(end 63 85)
+		(width 0.2)
+		(layer "In2.Cu")
+		(net "/SX1262_DIO1")
+	)
+	(segment
+		(start 63 117)
+		(end 63 132.5)
+		(width 0.2)
+		(layer "In2.Cu")

Commit message: route SX1262_RXEN from U3.19
Closes SX1262_RXEN: one island over U3.19, R74.1 and U8.6, 197.227 mm,
18 tracks and 4 vias across B.Cu 12 / In2 5 / F.Cu 1. Board ratsnest
417 -> 414, DRC 0 electrical errors. E5 x66 consumed.

Topology was verified from the netlist rather than assumed: R74.2 and
R13.2 are both GND, so both resistors are pull-down tees, not series
elements. Neither net originates at U1.

RXEN was routed first because it is by far the more constrained: its
source U3.19 sits at y 9.4 behind the I2C fan-out barrier whose only
0.200 mm opening SX1262_BUSY consumed in pass 3A-1, and it must cross
the whole board. U3 is a TSSOP-24 with 0.25 mm inter-pad gaps and
HEADER RESERVED 0.2 mm above its north edge, so U3.19 escapes south
into the package body gap, west above the I2C_SCL_INT B.Cu wall, and
crosses WAKE_INT_N's In2 on B.Cu. One B.Cu hop clears SX1262_BUSY's
In2 descent at x 61.

A mounting hole at (69.0, 13.0) radius 1.2 mm sat on the natural
eastward path; DRC caught it on the first write as copper_edge_clearance
0.0000 mm. The run now jogs to y 10.800, giving 2.200 mm against the
1.800 mm requirement. All four board cutouts are now checked explicitly
and that check is recorded as a standing route gate.

SX1262_RST_N is NOT routed in this commit. Its eastern half audits
legal end to end, but the western section fouls the TOUCH_RST_N via,
R4.1, R7.1, WAKE_INT_N B.Cu, the BQ25185_SYS F.Cu rail and comes within
0.100 mm of SX1262_DIO1's B.Cu descent. It is deferred rather than
compromised, and its x65 crossing is untouched.

Tracks 506 -> 523, vias 134 -> 138, 0 removed, all 21 additions on
/SX1262_RXEN. 188 footprints unmoved, 0 pad net assignments changed.
NFC_IRQ still 0 tracks / 0 vias / 0 zones. ERC 116 / 58 live and
schematic parity 261 delta 0, both unchanged.

Co-Authored-By: Claude Opus 5 <noreply@anthropic.com>
Claude-Session: https://claude.ai/code/session_01N3T9f8EXqAwVAJudcbiTW4
Routing:
- net /SX1262_RXEN: track 32.0 -> 197.2 mm, vias 0 -> 4
Changed lines of the file:
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@@
 	(footprint "C_0603_1608Metric"
 		(layer "B.Cu")
-		(at 28.5 79 180)
+		(at 46.1 82.5)
 		(descr "Capacitor SMD 0603 (1608 Metric), square (rectangular) end terminal, IPC-7351 nominal, (Body size source: IPC-SM-782 page 76, https://www.pcb-3d.com/wordpress/wp-content/uploads/ipc-sm-782a_amendment_1_and_2.pdf)")
 		(tags "capacitor")
-		(property "Reference" "C13"
-			(at 0 1.43 0)
+		(property "Reference" "C56"
+			(at 0 1.43 180)
 			(layer "B.SilkS")
 			(effects
@@
 			)
 		)
-		(property "Value" "100nF"
-			(at 0 -1.43 0)
+		(property "Value" "1uF"
+			(at 0 -1.43 180)
 			(layer "B.Fab")
 			(effects
@@
 		)
 		(property "Datasheet" ""
-			(at 0 0 0)
+			(at 0 0 180)
 			(layer "B.Fab")
 			(hide yes)
@@
 		)
 		(property "Description" ""
-			(at 0 0 0)
+			(at 0 0 180)
 			(layer "B.Fab")
 			(hide yes)
@@
 		)
 		(property "KiLib_Generator" "SMD_2terminal_chip_molded"
-			(at 0 0 0)
+			(at 0 0 180)
 			(layer "B.SilkS")
 			(hide yes)
@@
 		(duplicate_pad_numbers_are_jumpers no)
 		(fp_line
-			(start -0.14058 0.51)
-			(end 0.14058 0.51)
+			(start -0.14058 -0.51)
+			(end 0.14058 -0.51)
 			(stroke
 				(width 0.12)
@@
 		)
 		(fp_line
-			(start -0.14058 -0.51)
-			(end 0.14058 -0.51)
+			(start -0.14058 0.51)
+			(end 0.14058 0.51)
 			(stroke
 				(width 0.12)
@@
 		)
 		(fp_text user "${REFERENCE}"
-			(at 0 0 0)
+			(at 0 0 180)
 			(layer "B.Fab")
 			(effects
@@
 		)
 		(pad "1" smd roundrect
-			(at -0.775 0 180)
+			(at -0.775 0)
 			(size 0.9 0.95)
 			(layers "B.Cu" "B.Mask" "B.Paste")
@@
 		)
 		(pad "2" smd roundrect
-			(at 0.775 0 180)
+			(at 0.775 0)
 			(size 0.9 0.95)
 			(layers "B.Cu" "B.Mask" "B.Paste")
@@
 	(footprint "C_0603_1608Metric"
 		(layer "B.Cu")
-		(at 46.1 82.5)
+		(at 28.5 79 180)
 		(descr "Capacitor SMD 0603 (1608 Metric), square (rectangular) end terminal, IPC-7351 nominal, (Body size source: IPC-SM-782 page 76, https://www.pcb-3d.com/wordpress/wp-content/uploads/ipc-sm-782a_amendment_1_and_2.pdf)")
 		(tags "capacitor")
-		(property "Reference" "C56"
-			(at 0 1.43 180)
+		(property "Reference" "C13"
+			(at 0 1.43 0)
 			(layer "B.SilkS")
 			(effects
@@
 			)
 		)
-		(property "Value" "1uF"
-			(at 0 -1.43 180)
+		(property "Value" "100nF"
+			(at 0 -1.43 0)
 			(layer "B.Fab")
 			(effects
@@
 		)
 		(property "Datasheet" ""
-			(at 0 0 180)
+			(at 0 0 0)
 			(layer "B.Fab")
 			(hide yes)
@@
 		)
 		(property "Description" ""
-			(at 0 0 180)
+			(at 0 0 0)
 			(layer "B.Fab")
 			(hide yes)
@@
 		)
 		(property "KiLib_Generator" "SMD_2terminal_chip_molded"
-			(at 0 0 180)
+			(at 0 0 0)
 			(layer "B.SilkS")
 			(hide yes)
@@
 		(duplicate_pad_numbers_are_jumpers no)
 		(fp_line
-			(start -0.14058 -0.51)
-			(end 0.14058 -0.51)
+			(start -0.14058 0.51)
+			(end 0.14058 0.51)
 			(stroke
 				(width 0.12)
@@
 		)
 		(fp_line
-			(start -0.14058 0.51)
-			(end 0.14058 0.51)
+			(start -0.14058 -0.51)
+			(end 0.14058 -0.51)
 			(stroke
 				(width 0.12)
@@
 		)
 		(fp_text user "${REFERENCE}"
-			(at 0 0 180)
+			(at 0 0 0)
 			(layer "B.Fab")
 			(effects
@@
 		)
 		(pad "1" smd roundrect
-			(at -0.775 0)
+			(at -0.775 0 180)
 			(size 0.9 0.95)
 			(layers "B.Cu" "B.Mask" "B.Paste")
@@
 		)
 		(pad "2" smd roundrect
-			(at 0.775 0)
+			(at 0.775 0 180)
 			(size 0.9 0.95)
 			(layers "B.Cu" "B.Mask" "B.Paste")
@@
 	)
 	(segment
+		(start 70.6 129.65)
+		(end 70 129.65)
+		(width 0.2)
+		(layer "F.Cu")
+		(net "/SX1262_RXEN")
+	)
+	(via
+		(at 27 12.25)
+		(size 0.6)
+		(drill 0.3)
+		(layers "F.Cu" "B.Cu")
+		(net "/SX1262_RXEN")
+	)
+	(via
+		(at 60 12.6)
+		(size 0.6)
+		(drill 0.3)
+		(layers "F.Cu" "B.Cu")
+		(net "/SX1262_RXEN")
+	)
+	(via
+		(at 66 83.5)
+		(size 0.6)
+		(drill 0.3)
+		(layers "F.Cu" "B.Cu")
+		(net "/SX1262_RXEN")
+	)
+	(via
+		(at 70.6 129.65)
+		(size 0.6)
+		(drill 0.3)
+		(layers "F.Cu" "B.Cu")
+		(net "/SX1262_RXEN")
+	)
+	(segment
+		(start 22.325 9.6)
+		(end 22.325 10.6)
+		(width 0.2)
+		(layer "B.Cu")
+		(net "/SX1262_RXEN")
+	)
+	(segment
+		(start 22.325 10.6)
+		(end 17.5 10.6)
+		(width 0.2)
+		(layer "B.Cu")
+		(net "/SX1262_RXEN")
+	)
+	(segment
+		(start 17.5 10.6)
+		(end 17.5 13.5)
+		(width 0.2)
+		(layer "B.Cu")
+		(net "/SX1262_RXEN")
+	)
+	(segment
+		(start 17.5 13.5)
+		(end 25.5 13.5)
+		(width 0.2)
+		(layer "B.Cu")
+		(net "/SX1262_RXEN")
+	)
+	(segment
+		(start 25.5 13.5)
+		(end 25.5 12.25)
+		(width 0.2)
+		(layer "B.Cu")
+		(net "/SX1262_RXEN")
+	)
+	(segment
+		(start 25.5 12.25)
+		(end 27 12.25)
+		(width 0.2)
+		(layer "B.Cu")
+		(net "/SX1262_RXEN")
+	)
+	(segment
+		(start 60 12.6)
+		(end 66 12.6)
+		(width 0.2)
+		(layer "B.Cu")
+		(net "/SX1262_RXEN")
+	)
+	(segment
+		(start 66 12.6)
+		(end 66 10.8)
+		(width 0.2)
+		(layer "B.Cu")
+		(net "/SX1262_RXEN")
+	)
+	(segment
+		(start 66 10.8)
+		(end 72 10.8)
+		(width 0.2)
+		(layer "B.Cu")
+		(net "/SX1262_RXEN")
+	)
+	(segment
+		(start 72 10.8)
+		(end 72 83.5)
+		(width 0.2)
+		(layer "B.Cu")
+		(net "/SX1262_RXEN")
+	)
+	(segment
+		(start 72 83.5)
+		(end 66 83.5)
+		(width 0.2)
+		(layer "B.Cu")
+		(net "/SX1262_RXEN")
+	)
+	(segment
+		(start 70.6 129.65)
+		(end 71.5 129.65)
+		(width 0.2)
+		(layer "B.Cu")
+		(net "/SX1262_RXEN")
+	)
+	(segment
 		(start 66 85)
 		(end 66 117)
 		(width 0.2)
 		(layer "In2.Cu")
+		(net "/SX1262_RXEN")
+	)
+	(segment
+		(start 27 12.25)
+		(end 60 12.6)
+		(width 0.2)
+		(layer "In2.Cu")
+		(net "/SX1262_RXEN")
+	)
+	(segment
+		(start 66 83.5)
+		(end 66 85)
+		(width 0.2)
+		(layer "In2.Cu")
+		(net "/SX1262_RXEN")
+	)
+	(segment
+		(start 66 117)
+		(end 66 129.65)
+		(width 0.2)
+		(layer "In2.Cu")
+		(net "/SX1262_RXEN")
+	)
+	(segment
+		(start 66 129.65)
+		(end 70.6 129.65)
+		(width 0.2)
+		(layer "In2.Cu")
