File: hardware/beta-dm/kicad/aqroot-beta-dm/aqroot-Beta-DM.kicad_pcb (KiCad board)
At the start: 4 copper layers, 74 x 155 mm, 188 parts, among them J1 CH280QV10-CT_50P, J2 Molex_5025700893, J3 USB_C_Receptacle_USB2.0_16P, J4 JST-PH-2 BATTERY, J5 COMMUNITY_HEADER_2x13, J6 JST-PH-2 SPEAKER, Q1 AO3400A, SW1 BOOT, SW2 UP, SW3 DOWN, SW4 LEFT, SW5 RIGHT, SW6 A_SELECT, SW7 B_BACK, SW8 HOME, SW9 SW_SPDT, U1 ESP32-S3-WROOM-1, U10 USBLC6-2SC6, U11 BQ25185, U12 TPS63020, U13 TPS61023, U14 MAX17048, U15 TPS22918, U16 TCA9517ADGK, U17 TPS61169DCKR, U2 TCA9535PWR, U3 TCA9535PWR, U4 BMI270, U5 MAX98357A, U6 TSOP38238, U7 E07-400M10S, U8 E22-900M22S, U9 ST25R3916-AQET

Commit message: Beta-DM: add the outer-layer GND pours on F.Cu and B.Cu — B1 reaches 0
The board had no outer copper zones at all; In1.Cu carried the only plane.
Two supplementary GND zones now follow the In1 outline exactly (the 0.6 mm
inset octagon). In1 is untouched and remains the continuous board-wide
reference; no split-ground domain is created.

This closes the 15 fitted GND islands that the GND pass proved were
pour-resolvable rather than via-resolvable. Fitted GND pads off the main
island: 15 -> 0, measured with KiCad's connectivity engine, not by polygon
proximity. GND ratsnest 52 -> 18, all 18 DNP-only.

Post-pour ledger: 103 = A64 + B1(0) + B2(18) + C0 + D21.

Pad connection is SOLID, not thermal relief. Thermal relief was built and
measured first and is rejected on evidence: it left 15 starved_thermal DRC
errors because the fine-pitch pockets around U2, U3 and U4 cannot fit the
required two spokes, and it still left B1 at 4. Solid gives 0 errors and
B1 = 0, matches the convention the In1 plane already uses, and is the
preferred connection for the categories that matter here anyway - USB shell,
connector tabs, power and RF-module ground. Assembly note recorded in the
closeout doc: solid outer copper on small passives is a reflow heat-sink
consideration, and the DNP paste control already governs this stencil.

RF containment verified geometrically rather than trusting the flag: the
deepest penetration of any copperpour:not_allowed area by any filled pour
vertex is 0.000000 mm - every flagged vertex sits exactly on a keepout
boundary. NFC RESERVED, WROOM ANTENNA KEEPOUT, HEADER RESERVED, 915 KEEPOUT,
433 KEEPOUT and the west off-board area are all clean.

DRC 0 errors, 240 warnings, zero new warning types, 0 parity issues. Pour to
board edge 0.600 mm, to mounting-hole edge 0.501 mm. All hard-lock nets hold
with 0 must-work non-GND rats. XGPIO5's critical 0.50/0.25 via at
(20.400, 14.050) is unchanged, and all 55 GND stitch vias are preserved.

Objects added: 2 zones. Segm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
Routing:
- added copper zone on B.Cu, net GND
- added copper zone on F.Cu, net GND
Changed lines of the file:
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@@
+	)
+	(zone
+		(net "GND")
+		(layer "F.Cu")
+		(name "F.Cu GND POUR")
+		(hatch edge 0.5)
+		(connect_pads yes
+			(clearance 0.25)
+		)
+		(min_thickness 0.25)
+		(fill yes
+			(thermal_gap 0.5)
+			(thermal_bridge_width 0.5)
+			(island_removal_mode 0)
+		)
+		(polygon
+			(pts
+				(xy 0.6 3.4) (xy 3.4 0.6) (xy 70.6 0.6) (xy 73.4 3.4) (xy 73.4 151.6) (xy 70.6 154.4) (xy 3.4 154.4)
+				(xy 0.6 151.6)
+			)
+		)
 	)
 	(zone
@@
 			)
 		)
+	)
+	(zone
+		(net "GND")
+		(layer "B.Cu")
+		(name "B.Cu GND POUR")
+		(hatch edge 0.5)
+		(connect_pads yes
+			(clearance 0.25)
+		)
+		(min_thickness 0.25)
+		(fill yes
+			(thermal_gap 0.5)
+			(thermal_bridge_width 0.5)
+			(island_removal_mode 0)
+		)
+		(polygon
+			(pts
+				(xy 0.6 3.4) (xy 3.4 0.6) (xy 70.6 0.6) (xy 73.4 3.4) (xy 73.4 151.6) (xy 70.6 154.4) (xy 3.4 154.4)
+				(xy 0.6 151.6)
+			)
+		)
