File: hardware/beta-dm/kicad/aqroot-beta-dm/01_power_tree.kicad_sch (KiCad schematic)
At the start: 53 parts, among them J3 USB_C_Receptacle_USB2.0_16P, J4 JST-PH-2 BATTERY, SW9 SW_SPDT, U10 USBLC6-2SC6, U11 BQ25185, U12 TPS63020, U13 TPS61023, U14 MAX17048

Commit message: hardware(beta-dm): DNP becomes manufacturing data, not a markdown list
Marks the CTO-approved Beta-DM DNP set in KiCad's native convention and
generates the factory-facing package from it. No copper changes.

29 references gain (dnp yes) in the schematic and the matching `dnp` footprint
attribute on the PCB - the same convention the design already used for its five
pre-existing DNP parts C21, C22, R68, R49, R50, which is why nothing new was
invented here:

  NFC front end   U9 C45 C46 C47 C48 C49 C50 C51 C52 C53 C54
  NFC 5 V boost   U13 L2 R44 R45 C34 C35 C19 C55
  speaker         U5 J6
  IR transmitter  D1 Q1 R22 R23 R24
  IR receiver     U6 R21 C11

in_bom is deliberately left ON. A DNP part must still appear in the BOM flagged
DNP so the factory sees it and sees not to fit it; hiding it invites someone to
"helpfully" add it back. in_pos_files is left alone too - the position file is
generated with --exclude-dnp instead, which matches how the five pre-existing
DNP parts are already handled.

Generated into hardware/beta-dm/fab/:

  aqroot-Beta-DM-BOM-fitted.csv        parts to buy and place, DNP excluded
  aqroot-Beta-DM-BOM-full.csv          every part with a DNP column
  aqroot-Beta-DM-DO-NOT-POPULATE.csv   34 refs, each with its reason
  aqroot-Beta-DM-pos-fitted.csv        pick-and-place, DNP excluded
  aqroot-Beta-DM-pos-all.csv           reference only, do not feed the machine
  aqroot-Beta-DM-assembly-{top,bottom}.pdf   DNP parts crossed out
  ASSEMBLY-DNP-CONTROL.md              the control document

Verified: the fitted position file contains 139 of 173 footprints and none of
the 34 DNP refs; U9, U13, U5, J6, D1, Q1 and U6 are all absent from it. The
assembly PDFs cross out DNP automatically because the project already carries
crossoutdnponfab and sketchdnponfab.

Electrical audit of the ASSEMBLED circuit, not the artwork. No fitted IC pin is
left on a net with neither a driver nor a passive. SPI-B loses only U9's three
pins and keeps U1, U7 and U8, whic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
Parts:
- C34, C35, L2, R44, R45, U13: now not fitted
Changed lines of the file:
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@@
 		(on_board yes)
 		(in_pos_files yes)
-		(dnp no)
+		(dnp yes)
 		(fields_autoplaced yes)
 		(property "Reference" "L2"
@@
 		(on_board yes)
 		(in_pos_files yes)
-		(dnp no)
+		(dnp yes)
 		(fields_autoplaced yes)
 		(property "Reference" "C35"
@@
 		(on_board yes)
 		(in_pos_files yes)
-		(dnp no)
+		(dnp yes)
 		(fields_autoplaced yes)
 		(property "Reference" "U13"
@@
 		(on_board yes)
 		(in_pos_files yes)
-		(dnp no)
+		(dnp yes)
 		(fields_autoplaced yes)
 		(property "Reference" "C34"
@@
 		(on_board yes)
 		(in_pos_files yes)
-		(dnp no)
+		(dnp yes)
 		(property "Reference" "R44"
 			(at 152.654 176.53 90)
@@
 		(on_board yes)
 		(in_pos_files yes)
-		(dnp no)
+		(dnp yes)
 		(property "Reference" "R45"
 			(at 151.384 186.944 90)

Commit message: Beta-DM: close C24/J5 and freeze design-side PCBA release
The last design-side blocker is closed. C24's DC-bias gate is settled against
official Murata data, not a distributor description.

Murata's reference sheet carries no DC-bias curve and www.murata.com is serving
a maintenance page, so the numbers come from Murata's own SimSurfing
characteristic service, ds.murata.com/simserve/characsvdownload - the data the
SimSurfing viewer plots. Two curves at the stated condition 25 degC / AC 1 Vrms,
0-25 V in 0.125 V steps, archived verbatim in fab/datasheets/ along with the
AC-drive curve.

At the 4.5 V VSYS_REG operating point: 4.6773 uF, a change of -52.275 % from the
9.8005 uF measured at 0 V. TI BQ25185 SLUSF65A requires >1 uF effective, so the
typical part clears the floor by 4.68x. Stacking derations multiplicatively -
-10 % tolerance gives 4.210 uF, X5R -15 % temperature 3.578 uF, small-signal AC
drive 2.490 uF, an aging allowance 2.241 uF - it still holds at 2.24x. That last
stack deliberately over-derates: the AC term is measured at 0 V bias, where a
Class-II dielectric is most drive-sensitive, and flattens under bias.

C24 is LOCKED to Murata GRM188R61E106KA73D, 10 uF 25 V X5R 0603, FITTED. The
schematic value is landed and the symbol now carries Manufacturer and MPN.

No PCB change. kicad_pcb aaa04bfb and kicad_dru 050c83fc are unchanged, and all
17 Gerber/drill artifacts re-verify against their pre-edit SHA-256 manifest. The
PCB hash covers copper, every footprint and Edge.Cuts in one figure - the file
was never opened for writing. DRC 0 errors, schematic parity 0 errors, 103
unconnected matching the ledger exactly (A64 + B1(0) + B2(18) + C0 + D21), ERC
58 and byte-identical to the pre-edit report.

Both CPL files were re-exported from the unchanged board and came back
byte-identical, then C24's Val field alone was overridden to 10uF 25V X5R. Ref,
Package, PosX, PosY, Rot and Side are untouched and no other row moves; each
file is a one-line diff. Nothing ass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
Parts:
- C24: value 22uF 25V X7R -> 10uF 25V X5R; MPN (none) -> GRM188R61E106KA73D; Manufacturer (none) -> Murata
- J4: MPN (none) -> B2B-PH-K-S(LF)(SN); Manufacturer (none) -> JST
- U10: MPN (none) -> USBLC6-2SC6; Manufacturer (none) -> STMicroelectronics
Changed lines of the file:
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@@
 			)
 		)
+		(property "Manufacturer" "JST"
+			(at 252.73 132.08 0)
+			(hide yes)
+			(show_name no)
+			(do_not_autoplace no)
+			(effects
+				(font
+					(size 1.27 1.27)
+				)
+			)
+		)
+		(property "MPN" "B2B-PH-K-S(LF)(SN)"
+			(at 252.73 132.08 0)
+			(hide yes)
+			(show_name no)
+			(do_not_autoplace no)
+			(effects
+				(font
+					(size 1.27 1.27)
+				)
+			)
+		)
 		(pin "1"
 		)
@@
 			)
 		)
+		(property "Manufacturer" "STMicroelectronics"
+			(at 147.32 50.8 0)
+			(hide yes)
+			(show_name no)
+			(do_not_autoplace no)
+			(effects
+				(font
+					(size 1.27 1.27)
+				)
+			)
+		)
+		(property "MPN" "USBLC6-2SC6"
+			(at 147.32 50.8 0)
+			(hide yes)
+			(show_name no)
+			(do_not_autoplace no)
+			(effects
+				(font
+					(size 1.27 1.27)
+				)
+			)
+		)
 		(pin "2"
 		)
@@
 			)
 		)
-		(property "Value" "22uF 25V X7R"
+		(property "Value" "10uF 25V X5R"
 			(at 160.02 69.8499 0)
 			(show_name no)
@@
 			(at 156.21 68.58 0)
 			(hide yes)
+			(show_name no)
+			(do_not_autoplace no)
+			(effects
+				(font
+					(size 1.27 1.27)
+				)
+			)
+		)
+		(property "Manufacturer" "Murata"
+			(at 156.21 68.58 0)
+			(hide yes)
+			(show_name no)
+			(do_not_autoplace no)
+			(effects
+				(font
+					(size 1.27 1.27)
+				)
+			)
+		)
+		(property "MPN" "GRM188R61E106KA73D"
+			(at 156.21 68.58 0)
+			(hide yes)
