File: hardware/beta-dm/kicad/aqroot-beta-dm/09_community_header.kicad_sch (KiCad schematic)
At the start: 36 parts, among them J5 COMMUNITY_HEADER_2x13, U15 TPS22918, U16 TCA9517ADGK

Commit message: hardware(beta-dm): D2-D7 J5 ESD arrays DNP, U10 excluded by name
The J5 community-header ESD arrays become real manufacturing data on the
Demo Model. Each was audited pin by pin on the board first: every signal pin
touches exactly one net with GND on pin 2, so all six are shunt-only and
unfitting them removes protection without breaking a connection. The J5 ESD
network is entirely unrouted (see BETA-DM-RESIDUAL-BLOCKERS.md 2), so fitted
they would be unconnected parts on a demo board.

  D2 TPD2E009DBZR   I2C_SCL/SDA_EXT_HDR
  D3 TPD4E1B06DRLR  XGPIO0..3_HDR
  D4 TPD4E1B06DRLR  XGPIO4..7_HDR
  D5 TPD4E1B06DRLR  XGPIO8..11_HDR
  D6 TPD4E1B06DRLR  XGPIO12..13_HDR
  D7 TPD2E009DBZR   WAKE_ATTN_N_HDR / FAST_IO_GPIO43_HDR

FINAL RESTORE REQUIRED - the Final product ships header ESD fitted and routed.

U10 (USBLC6-2SC6) is the counter-example and is now stated by name in both the
assembly control document and the DNP list: USB data passes THROUGH it in
series (pins 3/1 in, 4/6 out, then R34/R33 to U1.14/U1.13), so unfitting it
open-circuits USB. "U10 MUST FIT - SERIES USB DATA PATH." Verified present in
the fitted BOM and the fitted placement file. D8 (NSR0240, backlight boost
catch diode) is likewise not an ESD part and stays fitted.

Encoding is KiCad-native: (dnp yes) on the six symbols, (attr smd dnp) on the
six footprints - 6 changed lines in each file, nothing else. All fab outputs
regenerated from the project.

DNP total 34 -> 40 (35 DM decisions + 5 pre-existing full-Beta).
BOM full 189 refs / fitted 149. Placement all 173 / fitted 133; the excluded
set is identical to the BOM's, so the two are self-consistent.
DRC 0 errors / 240 warnings / 230 unconnected - unchanged.
ERC 58 (5 errors / 53 warnings) - the recorded baseline, no regression.
hardware/beta/ untouched: 0 tracked changes, all four reference hashes match.

Co-Authored-By: Claude Opus 5 <noreply@anthropic.com>
Claude-Session: https://claude.ai/code/session_01NHhLoxp9EX3Khm68Metpp6
Parts:
- D2, D3, D4, D5, D6, D7: now not fitted
Changed lines of the file:
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@@
 		(on_board yes)
 		(in_pos_files yes)
-		(dnp no)
+		(dnp yes)
 		(property "Reference" "D6"
 			(at 138.684 135.382 0)
@@
 		(on_board yes)
 		(in_pos_files yes)
-		(dnp no)
+		(dnp yes)
 		(property "Reference" "D4"
 			(at 162.814 56.642 0)
@@
 		(on_board yes)
 		(in_pos_files yes)
-		(dnp no)
+		(dnp yes)
 		(property "Reference" "D3"
 			(at 195.834 85.852 0)
@@
 		(on_board yes)
 		(in_pos_files yes)
-		(dnp no)
+		(dnp yes)
 		(property "Reference" "D5"
 			(at 139.954 97.282 0)
@@
 		(on_board yes)
 		(in_pos_files yes)
-		(dnp no)
+		(dnp yes)
 		(property "Reference" "D7"
 			(at 254 142.24 0)
@@
 		(on_board yes)
 		(in_pos_files yes)
-		(dnp no)
+		(dnp yes)
 		(fields_autoplaced yes)
 		(property "Reference" "D2"

Commit message: hardware(beta-dm): LEAN-CORE scope - U15 and U16 DNP, ledger rebuilt to C6
Population and documentation only. NO ROUTING CHANGE: the object-level PCB diff
is exactly two footprint attributes -- pads 0, segments 0, vias 0, zones 0,
Edge.Cuts unchanged, placement unchanged. hardware/beta/ untouched.

Scope: buffered external J5 I2C and the switched accessory rail are Lean-DM
deferred, so U15 (TPS22918) and U16 (TCA9517A) have no Demo-Model function.
Internal I2C is a different net pair and remains MUST-WORK and hard-locked.

Dependency audit, run against KiCad's own connectivity by DELETING each
footprint on a scratch copy rather than merely marking it DNP:

  net             real board   U16 removed   U15 removed
  +3V3            1 island     1 island      1 island
  /I2C_SCL_INT    1 island     1 island      -
  /I2C_SDA_INT    1 island     1 island      -

Neither part is load-bearing for any live net; both DNPs are unconditional. An
earlier intermediate result from the project's approximate island code claimed
U15.1 was load-bearing for +3V3; that approximation is unreliable on a 430-item
net and KiCad's engine overrides it.

Support passives classified individually, not swept: R17 stays FITTED as the
only passive defining U3.20's node; C38, C39, C42, R46, R47, R48 are
DNP-ELIGIBLE and deliberately kept, following the C9/C10/R15/C18 precedent.

New fab requirement recorded: DNP footprints must receive no solder paste.
U15 and U16 are the first DNP parts with pads adjacent to live must-work nets
-- U16.1 (+3V3) sits 0.400 mm from U16.2 (internal I2C SCL).

Ledger rebuilt from the real board: 216 = A62 + B130 + C6 + D18.
C6 is re-derived, not assumed: XGPIO4/5/6/7 and BQ25185_STAT1/STAT2.
DRC unchanged at 0 errors, 240 warnings, 216 unconnected, parity 0.

Co-Authored-By: Claude Opus 5 <noreply@anthropic.com>
Claude-Session: https://claude.ai/code/session_017WGr8WtfBDVJyEdKckEXJh
Parts:
- U15, U16: now not fitted
Changed lines of the file:
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@@
 		(in_bom yes)
 		(on_board yes)
-		(in_pos_files yes)
-		(dnp no)
+		(in_pos_files no)
+		(dnp yes)
 		(property "Reference" "U16"
 			(at 232.156 87.376 0)
@@
 		(in_bom yes)
 		(on_board yes)
-		(in_pos_files yes)
-		(dnp no)
+		(in_pos_files no)
+		(dnp yes)
 		(fields_autoplaced yes)
 		(property "Reference" "U15"

Commit message: Beta-DM: clear both procurement blockers — C24 and J5
Both former STOPs are resolved, neither needed a PCB change.

C24. Correcting my own earlier statement: the SYS bulk requirement IS
specified. TI BQ25185 SLUSF65A (rev January 2026) section 8.2.2.3 gives
CSYS = 1 / 10 / 100 uF min/nom/max, requires greater than 1 uF AFTER derating,
recommends 25 V ceramics on IN and SYS specifically because of DC-bias
derating, and asks for placement as close as possible to the pins. VSYS_REG is
4.5 V. So the schematic's 25 V was not arbitrary - it follows TI. Only the
22 uF value and the 0603 package were wrong.

A second earlier error is corrected too. The previous pass counted C26+C27+C33
as 30 uF of SYS bulk available without C24. Measured from U11.1: C24 is
3.86 mm away with a 2.37 mm ground return, C33 is 8.43 mm, and C26/C27 are
20.4 and 20.8 mm from the charger but 3.63 and 4.70 mm from the TPS63020 -
they are the buck-boost CIN pair the decisions log already assigns, not
BQ25185 decoupling. C24 is the charger's local bulk capacitor.

So the DNP branch fails - the next bulk part is 2.2x further with a 2.9x
longer return - and the 0603 land instead takes a real part: Murata
GRM188R61E106KA73D, 10 uF 25 V X5R 0603, LCSC C344022. That hits TI's NOM
exactly, matches TI's 25 V recommendation, uses a dielectric TI explicitly
allows, fits the frozen land, and leaves total SYS nominal at 40.1 uF inside
the 1-100 uF window. C24 is at (64.0, 70.0) on F.Cu, clear of the display and
battery height shadows.

One check is outstanding and is not claimed as done: Murata's DC-bias curve
could not be retrieved, so the effective capacitance at 4.5 V is unproven. The
margin is large - 4.5 V is 18% of a 25 V rating and the part would have to lose
over 90% to fail - but per section 5 the value change is NOT landed. C24 stays
FITTED, the schematic still reads 22uF 25V X7R, and the substitution waits on
that curve.

J5 is locked to Samtec TSW-113-08-G-D-RA, right angle. Verified against Samtec
c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
Parts:
- J5: footprint Connector_PinHeader_2.54mm:PinHeader_2x13_P2.54mm_Vertical -> AQROOT_Beta:Samtec_TSW-113-08-G-D-RA
Changed lines of the file:
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@@
 			)
 		)
-		(property "Footprint" "Connector_PinHeader_2.54mm:PinHeader_2x13_P2.54mm_Vertical"
+		(property "Footprint" "AQROOT_Beta:Samtec_TSW-113-08-G-D-RA"
 			(at 257.81 124.46 0)
 			(hide yes)

Commit message: Beta-DM: close C24/J5 and freeze design-side PCBA release
The last design-side blocker is closed. C24's DC-bias gate is settled against
official Murata data, not a distributor description.

Murata's reference sheet carries no DC-bias curve and www.murata.com is serving
a maintenance page, so the numbers come from Murata's own SimSurfing
characteristic service, ds.murata.com/simserve/characsvdownload - the data the
SimSurfing viewer plots. Two curves at the stated condition 25 degC / AC 1 Vrms,
0-25 V in 0.125 V steps, archived verbatim in fab/datasheets/ along with the
AC-drive curve.

At the 4.5 V VSYS_REG operating point: 4.6773 uF, a change of -52.275 % from the
9.8005 uF measured at 0 V. TI BQ25185 SLUSF65A requires >1 uF effective, so the
typical part clears the floor by 4.68x. Stacking derations multiplicatively -
-10 % tolerance gives 4.210 uF, X5R -15 % temperature 3.578 uF, small-signal AC
drive 2.490 uF, an aging allowance 2.241 uF - it still holds at 2.24x. That last
stack deliberately over-derates: the AC term is measured at 0 V bias, where a
Class-II dielectric is most drive-sensitive, and flattens under bias.

C24 is LOCKED to Murata GRM188R61E106KA73D, 10 uF 25 V X5R 0603, FITTED. The
schematic value is landed and the symbol now carries Manufacturer and MPN.

No PCB change. kicad_pcb aaa04bfb and kicad_dru 050c83fc are unchanged, and all
17 Gerber/drill artifacts re-verify against their pre-edit SHA-256 manifest. The
PCB hash covers copper, every footprint and Edge.Cuts in one figure - the file
was never opened for writing. DRC 0 errors, schematic parity 0 errors, 103
unconnected matching the ledger exactly (A64 + B1(0) + B2(18) + C0 + D21), ERC
58 and byte-identical to the pre-edit report.

Both CPL files were re-exported from the unchanged board and came back
byte-identical, then C24's Val field alone was overridden to 10uF 25V X5R. Ref,
Package, PosX, PosY, Rot and Side are untouched and no other row moves; each
file is a one-line diff. Nothing ass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
Parts:
- J5: MPN (none) -> TSW-113-08-G-D-RA; Manufacturer (none) -> Samtec
Changed lines of the file:
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@@
+			)
+		)
+		(property "Manufacturer" "Samtec"
+			(at 257.81 124.46 0)
+			(hide yes)
+			(show_name no)
+			(do_not_autoplace no)
+			(effects
+				(font
+					(size 1.27 1.27)
+				)
+			)
+		)
+		(property "MPN" "TSW-113-08-G-D-RA"
+			(at 257.81 124.46 0)
+			(hide yes)
+			(show_name no)
+			(do_not_autoplace no)
+			(effects
+				(font
+					(size 1.27 1.27)
+				)
 			)
 		)
