File: hardware/beta-dm/kicad/aqroot-beta-dm/08_buttons_expanders.kicad_sch (KiCad schematic)
At the start: 26 parts, among them SW2 UP, SW3 DOWN, SW4 LEFT, SW5 RIGHT, SW6 A_SELECT, SW7 B_BACK, SW8 HOME, U2 TCA9535PWR, U3 TCA9535PWR

Commit message: Beta-DM: close C24/J5 and freeze design-side PCBA release
The last design-side blocker is closed. C24's DC-bias gate is settled against
official Murata data, not a distributor description.

Murata's reference sheet carries no DC-bias curve and www.murata.com is serving
a maintenance page, so the numbers come from Murata's own SimSurfing
characteristic service, ds.murata.com/simserve/characsvdownload - the data the
SimSurfing viewer plots. Two curves at the stated condition 25 degC / AC 1 Vrms,
0-25 V in 0.125 V steps, archived verbatim in fab/datasheets/ along with the
AC-drive curve.

At the 4.5 V VSYS_REG operating point: 4.6773 uF, a change of -52.275 % from the
9.8005 uF measured at 0 V. TI BQ25185 SLUSF65A requires >1 uF effective, so the
typical part clears the floor by 4.68x. Stacking derations multiplicatively -
-10 % tolerance gives 4.210 uF, X5R -15 % temperature 3.578 uF, small-signal AC
drive 2.490 uF, an aging allowance 2.241 uF - it still holds at 2.24x. That last
stack deliberately over-derates: the AC term is measured at 0 V bias, where a
Class-II dielectric is most drive-sensitive, and flattens under bias.

C24 is LOCKED to Murata GRM188R61E106KA73D, 10 uF 25 V X5R 0603, FITTED. The
schematic value is landed and the symbol now carries Manufacturer and MPN.

No PCB change. kicad_pcb aaa04bfb and kicad_dru 050c83fc are unchanged, and all
17 Gerber/drill artifacts re-verify against their pre-edit SHA-256 manifest. The
PCB hash covers copper, every footprint and Edge.Cuts in one figure - the file
was never opened for writing. DRC 0 errors, schematic parity 0 errors, 103
unconnected matching the ledger exactly (A64 + B1(0) + B2(18) + C0 + D21), ERC
58 and byte-identical to the pre-edit report.

Both CPL files were re-exported from the unchanged board and came back
byte-identical, then C24's Val field alone was overridden to 10uF 25V X5R. Ref,
Package, PosX, PosY, Rot and Side are untouched and no other row moves; each
file is a one-line diff. Nothing ass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
Parts:
- U2, U3: MPN (none) -> TCA9535PWR; Manufacturer (none) -> Texas Instruments
Changed lines of the file:
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@@
+			)
+		)
+		(property "Manufacturer" "Texas Instruments"
+			(at 194.31 100.33 0)
+			(hide yes)
+			(show_name no)
+			(do_not_autoplace no)
+			(effects
+				(font
+					(size 1.27 1.27)
+				)
+			)
+		)
+		(property "MPN" "TCA9535PWR"
+			(at 194.31 100.33 0)
+			(hide yes)
+			(show_name no)
+			(do_not_autoplace no)
+			(effects
+				(font
+					(size 1.27 1.27)
+				)
 			)
 		)
@@
 			(hide yes)
 			(show_name no)
+			(do_not_autoplace no)
+			(effects
+				(font
+					(size 1.27 1.27)
+				)
+			)
+		)
+		(property "Manufacturer" "Texas Instruments"
+			(at 109.22 100.33 0)
+			(hide yes)
+			(show_name no)
+			(do_not_autoplace no)
+			(effects
+				(font
+					(size 1.27 1.27)
+				)
+			)
+		)
+		(property "MPN" "TCA9535PWR"
+			(at 109.22 100.33 0)
+			(hide yes)
+			(show_name no)

Commit message: Beta-DM: finalize JLC component matching and manual-source plan
Both CTO rulings applied, the two remaining engineering gates closed with real
manufacturer data, and the E list is empty.

D8. The old lock NSR0240V2T5G is a SOD-523 part and the land is SOD-323, so it
never fitted - a defect in our own ledger that only surfaced because JLC's
matcher suggested the package-correct sibling. Now locked to onsemi
NSR0240HT1G, SOD-323, 40 V, 250 mA Schottky. It is NOT pinned to a JLC code:
C152519 shows 13 in stock against a 116-piece minimum purchase and a negative
presale balance, so it cannot be bought today. Pinning an unbuyable code only
fails at checkout. Manual source; two pieces of a 2-pin SOD-323 are trivial.

SW1-SW8. All eight locked to one part, C&K PTS645SM43SMTR92LFS / C221880,
1.6 N, SMD-4P 6x6 mm gull wing, 4.3 mm actuator, stock 8462. The 'x' in
PTS645Sx43SMTR92 was always the actuation-force letter and the design had never
fixed it; M = 1.6 N is the Beta-DM feel baseline, revisitable after hands-on
testing. JLC's lone hanxia match for SW5 is rejected - it would have made one
button differ from the other seven.

C26/C27 hard gate: PASS. Murata GRM31CR71E106KA12L, 10 uF 25 V X7R 1206,
C77093, stock 226763. TI SLUSF65A 8.2.2.3 also asks for 25 V parts on IN/SYS.
Official Murata SimSurfing data at 25 degC / AC 1 Vrms: 10.923 uF at 0 V and
9.000 uF at 4.5 V, a change of -17.60 %. Per capacitor that is 9.00 uF against
the >=5 uF floor and 18.0 uF combined against the >=10 uF floor, 1.80x both.
With -10 % tolerance, 8.10 uF each and 16.2 uF combined, 1.62x both; with X7R
-15 % temperature on top, 6.885 uF and 13.77 uF, 1.38x both. The obsolete
GRM21BR71A106KE51L was never a candidate.

R32/R35/R42 closed with numbers rather than judgement. The netlist shows R35 is
the only power-node jumper of the three - it bridges USB_VBUS_RAW to
USB_VBUS_CHG, while R32 is a shield tie and R42 a PS/SYNC strap. The rule text
names R42 as the power node; the netlist says R35, and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
Parts:
- SW2, SW3, SW4, SW5, SW6, SW7, SW8: MPN PTS645Sx SMTR92 LFS -> PTS645SM43SMTR92LFS
Changed lines of the file:
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@@
 			)
 		)
-		(property "MPN" "PTS645Sx SMTR92 LFS"
+		(property "MPN" "PTS645SM43SMTR92LFS"
 			(at 168.91 153.67 0)
 			(hide yes)
@@
 			)
 		)
-		(property "MPN" "PTS645Sx SMTR92 LFS"
+		(property "MPN" "PTS645SM43SMTR92LFS"
 			(at 125.73 153.67 0)
 			(hide yes)
@@
 			)
 		)
-		(property "MPN" "PTS645Sx SMTR92 LFS"
+		(property "MPN" "PTS645SM43SMTR92LFS"
 			(at 102.87 153.67 0)
 			(hide yes)
@@
 			)
 		)
-		(property "MPN" "PTS645Sx SMTR92 LFS"
+		(property "MPN" "PTS645SM43SMTR92LFS"
 			(at 148.59 153.67 0)
 			(hide yes)
@@
 			)
 		)
-		(property "MPN" "PTS645Sx SMTR92 LFS"
+		(property "MPN" "PTS645SM43SMTR92LFS"
 			(at 82.55 153.67 0)
 			(hide yes)
@@
 			)
 		)
-		(property "MPN" "PTS645Sx SMTR92 LFS"
+		(property "MPN" "PTS645SM43SMTR92LFS"
 			(at 38.1 153.67 0)
 			(hide yes)
@@
 			)
 		)
-		(property "MPN" "PTS645Sx SMTR92 LFS"
+		(property "MPN" "PTS645SM43SMTR92LFS"
 			(at 59.69 153.67 0)
 			(hide yes)
