File: hardware/beta-v2/kicad/aqroot-beta-v2/aqroot-Beta-v2.kicad_sch (KiCad schematic)
At the start: 0 parts

Commit message: hardware: migrate Full Beta v2 community expansion
Sheet 09 migrated (FBV2-S1-009). All nine schematic sheets now carry the Full
Beta v2 architecture and fork_equivalence.py's "still Beta-DM" list is empty.

Three CTO rulings implemented. O-6 ratified: U23, the third PCAL9535APW,118 at
0x22, and the front RGB are locked architecture; B-37 retired with 11 spare
expander pins. O-4 approved: U16 TCA9517A -> TI TCA4307DGKR (LCSC C880333),
FITTED where the old part was DNP. P-18 closed with no I2C mux.

Sheet 09 was rebuilt, not patched, and was hiding two serious defects: J5
contact 1 carried permanent raw +3V3 against D-057, and the community port had
no power at all - 01:ACC_3V3_SW and 09:ACC_3V3_SW were different nets, the
latter fed by a second, DNP TPS22918. Also removed: the 26-pin 2x13 male
header, XGPIO10-13, FAST_IO_GPIO43_HDR, RESERVED_NC. Sixth consecutive sheet
with a load-bearing inherited DNP.

Connector footprint built from the Samtec RECOMMENDED PCB LAYOUT REV B FIG 3:
2.54 mm in row, 7.87 +/-0.05 mm row-to-row, 0.71 mm PTH, 27.94 mm pin field.
All 24 contacts verified pin by pin against D-084.

External I2C pull-ups re-derived: the inherited 4.7k gives 796 ns against a
300 ns fast-mode budget at 200 pF and could never have worked; now 1.5k =
254 ns. Both current limits re-derived rather than copied - 3.3 V stays 1.5k
but the accessory-short case moved 86% -> 89% of the TPS63020's 2 A.

5 V enables split per the CTO refinement: ACC_5V_BOOST_EN on U3 P13 and
ACC_5V_SW_EN on U23 P04, each with its own 100k pull-down. B-08 closed in
copper with Q10, source facing the connector. All six TVS arrays were DNP and
are now fitted; one TPD4E1B06DRLR MPN covers all sixteen exposed contacts.

#FLG0105, deleted by the rebuild, turned out to be the only power-output driver
on the entire GND net and was re-created with a note explaining its role.

ERC 42/1/41 -> 27/0/27 - zero errors for the first time. 321 components, 0
duplicate references, 0 without a footprint, 224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
Other:
- sheet 01_POWER_TREE ports: added ACC_3V3_SW, ACC_5V_BOOST_EN, ACC_5V_SW, ACC_5V_SW_EN; removed ACC_5V_EN
- sheet 08_BUTTONS_EXPANDERS ports: added ACC_5V_BOOST_EN, ACC_5V_SW_EN, ACC_DETECT_N; removed ACC_5V_EN
- sheet 09_COMMUNITY_HEADER ports: added ACC_3V3_SW, ACC_5V_SW, ACC_DETECT_N, NATIVE_A, NATIVE_B; removed FAST_IO_U0TXD_ROOTPROBE_CS, XGPIO10, XGPIO11, XGPIO12, XGPIO13
Changed lines of the file:
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@@
 	(wire
 		(pts
-			(xy 133.35 250.19) (xy 135.89 250.19)
-		)
-		(stroke
-			(width 0)
-			(type default)
-		)
-	)
-	(wire
-		(pts
 			(xy 144.78 105.41) (xy 144.78 107.95)
 		)
@@
 	(wire
 		(pts
-			(xy 133.35 261.62) (xy 135.89 261.62)
-		)
-		(stroke
-			(width 0)
-			(type default)
-		)
-	)
-	(wire
-		(pts
 			(xy 334.01 115.57) (xy 334.01 113.03)
 		)
@@
 	(wire
 		(pts
-			(xy 133.35 257.81) (xy 135.89 257.81)
-		)
-		(stroke
-			(width 0)
-			(type default)
-		)
-	)
-	(wire
-		(pts
 			(xy 223.52 38.1) (xy 226.06 38.1)
 		)
@@
 	(wire
 		(pts
-			(xy 52.07 257.81) (xy 54.61 257.81)
-		)
-		(stroke
-			(width 0)
-			(type default)
-		)
-	)
-	(wire
-		(pts
 			(xy 290.83 67.31) (xy 293.37 67.31)
 		)
@@
 	(wire
 		(pts
-			(xy 133.35 254) (xy 135.89 254)
-		)
-		(stroke
-			(width 0)
-			(type default)
-		)
-	)
-	(wire
-		(pts
 			(xy 223.52 78.74) (xy 226.06 78.74)
 		)
@@
 		)
 	)
-	(label "XGPIO10"
-		(at 135.89 250.19 0)
-		(effects
-			(font
-				(size 1.27 1.27)
-			)
-			(justify left bottom)
-		)
-	)
 	(label "XGPIO9"
 		(at 391.16 157.48 0)
@@
 		)
 	)
-	(label "XGPIO13"
-		(at 135.89 261.62 0)
-		(effects
-			(font
-				(size 1.27 1.27)
-			)
-			(justify left bottom)
-		)
-	)
 	(label "I2S_BCLK"
 		(at 144.78 107.95 0)
@@
 		)
 	)
-	(label "FAST_IO_U0TXD_ROOTPROBE_CS"
-		(at 52.07 257.81 180)
-		(effects
-			(font
-				(size 1.27 1.27)
-			)
-			(justify right bottom)
-		)
-	)
 	(label "ACC_PWR_EN"
 		(at 52.07 218.44 180)
@@
 		)
 	)
-	(label "XGPIO11"
-		(at 135.89 254 0)
-		(effects
-			(font
-				(size 1.27 1.27)
-			)
-			(justify left bottom)
-		)
-	)
 	(label "DISP_RST_N"
 		(at 358.14 110.49 0)
@@
 		)
 	)
-	(label "XGPIO12"
-		(at 135.89 257.81 0)
-		(effects
-			(font
-				(size 1.27 1.27)
-			)
-			(justify left bottom)
-		)
-	)
 	(label "XGPIO8"
 		(at 391.16 154.94 0)
@@
 			)
 		)
-		(pin "ACC_5V_EN" input
+		(pin "ACC_5V_BOOST_EN" input
 			(at 105.41 74.93 0)
 			(effects
@@
 			)
 		)
+		(pin "ACC_5V_SW_EN" input
+			(at 105.41 82.55 0)
+			(effects
+				(font
+					(size 1.27 1.27)
+				)
+				(justify right)
+			)
+		)
+		(pin "ACC_3V3_SW" output
+			(at 105.41 86.36 0)
+			(effects
+				(font
+					(size 1.27 1.27)
+				)
+				(justify right)
+			)
+		)
+		(pin "ACC_5V_SW" output
+			(at 105.41 90.17 0)
+			(effects
+				(font
+					(size 1.27 1.27)
+				)
+				(justify right)
+			)
+		)
 		(instances
 			(project "aqroot-Beta-v2"
@@
 			)
 		)
-		(pin "ACC_5V_EN" output
+		(pin "ACC_5V_BOOST_EN" output
 			(at 388.62 185.42 0)
 			(effects
@@
 			)
 		)
+		(pin "ACC_5V_SW_EN" output
+			(at 388.62 172.72 0)
+			(effects
+				(font
+					(size 1.27 1.27)
+				)
+				(justify right)
+			)
+		)
+		(pin "ACC_DETECT_N" input
+			(at 388.62 187.96 0)
+			(effects
+				(font
+					(size 1.27 1.27)
+				)
+				(justify right)
+			)
+		)
 		(instances
 			(project "aqroot-Beta-v2"
@@
 			)
 		)
-		(pin "FAST_IO_U0TXD_ROOTPROBE_CS" input
-			(at 54.61 257.81 180)
-			(effects
-				(font
-					(size 1.27 1.27)
-				)
-				(justify left)
-			)
-		)
 		(pin "I2C_SCL_INT" input
 			(at 54.61 243.84 180)
@@
 			)
 		)
-		(pin "XGPIO10" bidirectional
+		(pin "NATIVE_A" bidirectional
 			(at 133.35 250.19 0)
 			(effects
@@
 			)
 		)
-		(pin "XGPIO11" bidirectional
+		(pin "NATIVE_B" bidirectional
 			(at 133.35 254 0)
 			(effects
@@
 			)
 		)
-		(pin "XGPIO12" bidirectional
+		(pin "ACC_3V3_SW" input
 			(at 133.35 257.81 0)
 			(effects
@@
 			)
 		)
-		(pin "XGPIO13" bidirectional
+		(pin "ACC_5V_SW" input
 			(at 133.35 261.62 0)
 			(effects
@@
 			)
 		)
+		(pin "ACC_DETECT_N" output
+			(at 133.35 265.43 0)
+			(effects
+				(font
+					(size 1.27 1.27)
+				)
+				(justify right)
+			)
+		)
 		(instances
 			(project "aqroot-Beta-v2"
@@
 		)
 	)
-	(label "ACC_5V_EN"
+	(label "ACC_5V_BOOST_EN"
 		(at 391.16 185.42 0)
 		(effects
@@
 		)
 	)
-	(label "ACC_5V_EN"
+	(label "ACC_5V_BOOST_EN"
 		(at 107.95 74.93 0)
 		(effects
@@
 		(effects
 			(font
+				(size 1.27 1.27)
+			)
+			(justify left bottom)
+		)
+	)
+	(wire
+		(pts
+			(xy 133.35 250.19) (xy 135.89 250.19)
+		)
+		(stroke
+			(width 0)
+			(type default)
+		)
+	)
+	(label "NATIVE_A"
+		(at 135.89 250.19 0)
+		(effects
+			(font
+				(size 1.27 1.27)
+			)
+			(justify left bottom)
+		)
+	)
+	(wire
+		(pts
+			(xy 133.35 254) (xy 135.89 254)
+		)
+		(stroke
+			(width 0)
+			(type default)
+		)
+	)
+	(label "NATIVE_B"
+		(at 135.89 254 0)
+		(effects
+			(font
+				(size 1.27 1.27)
+			)
+			(justify left bottom)
+		)
+	)
+	(wire
+		(pts
+			(xy 133.35 257.81) (xy 135.89 257.81)
+		)
+		(stroke
+			(width 0)
+			(type default)
+		)
+	)
+	(label "ACC_3V3_SW"
+		(at 135.89 257.81 0)
+		(effects
+			(font
+				(size 1.27 1.27)
+			)
+			(justify left bottom)
+		)
+	)
+	(wire
+		(pts
+			(xy 133.35 261.62) (xy 135.89 261.62)
+		)
+		(stroke
+			(width 0)
+			(type default)
+		)
+	)
+	(label "ACC_5V_SW"
+		(at 135.89 261.62 0)
+		(effects
+			(font
+				(size 1.27 1.27)
+			)
+			(justify left bottom)
+		)
+	)
+	(wire
+		(pts
+			(xy 133.35 265.43) (xy 135.89 265.43)
+		)
+		(stroke
+			(width 0)
+			(type default)
+		)
+	)
+	(label "ACC_DETECT_N"
+		(at 135.89 265.43 0)
+		(effects
+			(font
+				(size 1.27 1.27)
+			)
+			(justify left bottom)
+		)
+	)
+	(wire
+		(pts
+			(xy 388.62 172.72) (xy 391.16 172.72)
+		)
+		(stroke
+			(width 0)
+			(type default)
+		)
+	)
+	(label "ACC_5V_SW_EN"
+		(at 391.16 172.72 0)
+		(effects
+			(font
+				(size 1.27 1.27)
+			)
+			(justify left bottom)
+		)
+	)
+	(wire
+		(pts
+			(xy 388.62 187.96) (xy 391.16 187.96)
+		)
+		(stroke
+			(width 0)
+			(type default)
+		)
+	)
+	(label "ACC_DETECT_N"
+		(at 391.16 187.96 0)
+		(effects
+			(font
+				(size 1.27 1.27)
+			)
+			(justify left bottom)
+		)
+	)
+	(wire
+		(pts
+			(xy 105.41 82.55) (xy 107.95 82.55)
+		)
+		(stroke
+			(width 0)
+			(type default)
+		)
+	)
+	(label "ACC_5V_SW_EN"
+		(at 107.95 82.55 0)
+		(effects
+			(font
+				(size 1.27 1.27)
+			)
+			(justify left bottom)
+		)
+	)
+	(wire
+		(pts
+			(xy 105.41 86.36) (xy 107.95 86.36)
+		)
+		(stroke
+			(width 0)
+			(type default)
+		)
+	)
+	(label "ACC_3V3_SW"
+		(at 107.95 86.36 0)
+		(effects
+			(font
+				(size 1.27 1.27)
+			)
+			(justify left bottom)
+		)
+	)
+	(wire
+		(pts
+			(xy 105.41 90.17) (xy 107.95 90.17)
+		)
+		(stroke
+			(width 0)
+			(type default)
+		)
+	)
+	(label "ACC_5V_SW"
+		(at 107.95 90.17 0)
+		(effects
+			(font
