File: hardware/beta-v2/kicad/aqroot-beta-v2/02_mcu_core.kicad_sch (KiCad schematic)
At the start: 9 parts, among them SW1 BOOT, U1 ESP32-S3-WROOM-1

Commit message: hardware: migrate Full Beta v2 MCU core (FBV2-S1-002)
Closes the two power-tree values the CTO ruled on and migrates 02_MCU_CORE.
Task gate FBV2-S1-MCU-CORE = PASS. FBV2-S1 itself is 2 of 9 sheets.

P-20 - R95 680R -> 560R. Recovery recomputed from the captured circuit:
8.36 mA nominal at VBUS 5.0 V into a 0 V pack, 7.93-8.80 mA across 4.75-5.25 V,
back inside the accepted 5-10 mA band that B-26 is measured against.

The recomputation also showed that 680R was NOT arbitrary:
(5.00 - 0.32 + 4.2) / 680 = 13.06 mA is exactly B-27's recorded ~13 mA
single-fault ceiling. With 560R that ceiling becomes ~15.9 mA nominal and
~16.6 mA worst case - 0.0066 C on a 2500 mAh pack, still bounded by R95, still
unidirectional through D12, still self-annunciating. B-27 is amended in place
rather than left reading a number that is no longer true. The trade is explicit:
~21% more recovery current for ~22% more single-fault current.

P-21 - the OV trip is derived, not typed. The datasheet threshold was fetched
first (LTC4368, Farnell mirror 2243878): V_OV 492.5 / 500 / 507.5 mV rising,
hysteresis 20 / 25 / 32 mV, UV/OV leakage 10 nA max, "Adjustable +/-1.5%".
R77 4.02M -> 3.65M 1%, R78 unchanged at 442k:
0.500 x (3.65M + 442k) / 442k = 4.629 V.
Nominal 4.63 V; 4.48-4.78 V over comparator and 1% resistor tolerance;
4.44-4.82 V including worst-case OV pin leakage; release 4.40 V nominal.
Above a 4.35 V-class pack with 129 mV of worst-case margin, 420 mV below the
5.05 V first capture, and no lockout hazard because release sits above float.
3.65M is already R91's value, so this REMOVES a BOM line.

02_MCU_CORE migrated:

- GPIO38 = NATIVE_A and GPIO47 = NATIVE_B, both hierarchical and bidirectional.
  SX1262_DIO1 no longer reaches the MCU at all; under D-089 it terminates on the
  internal expander U2, which is sheet 08.
- GPIO46 = DISP_BL_CTL. GPIO46 is a strapping pin that MUST read LOW at reset -
  GPIO0 = 0 alone does not select Joint Download Boot, GPIO46 = 0 is also
  required. Three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
Parts:
- added R108, R110: 10k, Resistor_SMD:R_0603_1608Metric, symbol Device:R
- added R109: 0R FIT, Resistor_SMD:R_0603_1608Metric, symbol Device:R
- added R111: 10k DNP, Resistor_SMD:R_0603_1608Metric, symbol Device:R
- added TP35: UART0_TXD_TEST, TestPoint:TestPoint_Pad_D1.0mm, symbol Connector:TestPoint
- TP1: value GPIO45_TEST -> GPIO45_STRAP_TEST
- TP2: value GPIO46_TEST -> GPIO46_STRAP_TEST
Connections:
- net BMI270_INT1_STRAP: now also R110.1
- net DISP_BL_CTL: now also R109.2; no longer U1.24 (IO47)
- net GND: now also R108.2, R110.2, R111.2
- net FAST_IO_U0TXD_ROOTPROBE_CS renamed UART0_TXD_DBG
- net UART0_TXD_DBG: now also TP35.1
- net SX1262_DIO1 renamed NATIVE_A
- net TEST_GPIO45 renamed GPIO45_VDDSPI_STRAP
- net GPIO45_VDDSPI_STRAP: now also R111.1
- net TEST_GPIO46 renamed DISP_BL_CTL_STRAP
- net DISP_BL_CTL_STRAP: now also R108.1, R109.1
- new net NATIVE_B: U1.24 (IO47)
Other:
- note added: "=== FBV2-S1 MCU CORE (FBV2-S1-002) - GPIO38/47 RELEASED TO THE COMMUNITY PORT, GPIO46 TAKES THE BACKLIGHT ==="
- note added: "GPIO38 = NATIVE_A and GPIO47 = NATIVE_B leave this sheet as the two native community fast-IO signals (D-084). SX1262_DIO1 no longer reaches the MCU: it terminates on the internal PCAL9535A U2 (D-089), which is sheet 08 and is NOT migrated yet."
- note added: "GPIO43 (U0TXD) is withdrawn from the community port (D-106) and is internal debug only - TP35 carries the ROM boot log, which is the only view of a first board whose USB does not enumerate. GPIO44 (U0RXD) is IR RX, so UART0 is TX-only; ROM download recovery is via the native USB Serial/JTAG on GPIO19/20, not UART0."
- note added: "STRAPS. GPIO0: R2 10k pull-up + SW1 direct to GND, no capacitor (Espressif forbids bulk C here). GPIO46: R108 10k pull-down at the pin, and R109 0R FIT isolates the TPS61169 CTRL so the strap survives even if CTRL sources current - GPIO46 MUST be LOW at reset or Joint Download Boot is unreachable. GPIO3: R110 10k pull-down, LOW selects the USB Serial/JTAG source; external JTAG would land on GPIO3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"

Commit message: hardware: migrate Full Beta v2 display and microSD (FBV2-S1-003)
Fits R111 per CTO ruling and migrates 03_SPI_A_DISPLAY_SD. Task gate
FBV2-S1-DISPLAY-SD = PASS. FBV2-S1 itself is 3 of 9 sheets.

THE INHERITED J1 WOULD HAVE PRODUCED A DEAD DISPLAY, TWICE OVER.

J1 still used the 2.8-inch CH280QV10_CT_50P pin table while its Value and
Footprint fields already read FH69-50S-0.5SH. Pin count matched, connector
matched, ERC was silent. The pin FUNCTIONS did not match ER-TFT035IPS-6:

  panel pin 1/2/3   old: LEDK / LED-A1 / LED-A2   new: LEDA / LEDK / LEDK
                    -> backlight reverse-biased, no light
  panel pin 36/37   old: WR_RS->DISP_DC / RS_SCL->SPI_A_SCK
                    new: WRX(SCL) / D-CX
                    -> clock and D/C swapped, no valid command ever reaches
                       the panel
  panel pin 4,5,6   old: LED-A3, LED-A4, IM0(grounded)   new: NC
  panel pin 7,8,9   old: IM1,IM2,IM3   new: IM0,IM1,IM2  (all three were
                    already +3V3, so 1 1 1 was correct by luck)
  panel pin 46      CTP IRQ, not represented at all

Neither fault is visible from a pin count, a connector MPN or an ERC run. A new
project-library symbol ER-TFT035IPS-6_50P was authored with the vendor table
verbatim (datasheet Rev 2.0 sec 4.1), deliberately keeping the old pin geometry
so the migration is a pin-function change and not a redraw. CH280QV10_CT_50P
stays in the library - Beta-DM still uses it - and is dropped from sheet 03's
symbol cache.

R111 FITTED (D-111). 10k, GPIO45_VDDSPI_STRAP -> GND. VDD_SPI is held LOW
deterministically instead of relying on the chip's internal pull-down alone.
TP1 retained, no capacitance on the net, no peripheral on GPIO45.

B-43 CLOSED WITH A PRIMARY SOURCE (D-116). TPS61169 datasheet SNVSA40B:
R_PD, CTRL pin internal pull-down resistor, 300 kohm, with V_H/V_L = 1.2/0.4 V
and t_SD = 2.5 ms. CTRL's only internal element pulls DOWN, so there is no
mechanism by which the backlight driver can raise the GPIO46 strap. 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
Parts:
- R111: value 10k DNP -> 10k; now fitted
Changed lines of the file:
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@@
 		(on_board yes)
 		(in_pos_files yes)
-		(dnp yes)
+		(dnp no)
 		(fields_autoplaced yes)
 		(property "Reference" "R111"
@@
 			)
 		)
-		(property "Value" "10k DNP"
+		(property "Value" "10k"
 			(at 102.87 116.83999999999999 0)
 			(show_name no)
@@
 		)
 	)
-	(text "STRAPS. GPIO0: R2 10k pull-up + SW1 direct to GND, no capacitor (Espressif forbids bulk C here). GPIO46: R108 10k pull-down at the pin, and R109 0R FIT isolates the TPS61169 CTRL so the strap survives even if CTRL sources current - GPIO46 MUST be LOW at reset or Joint Download Boot is unreachable. GPIO3: R110 10k pull-down, LOW selects the USB Serial/JTAG source; external JTAG would land on GPIO39-42, which are I2S. GPIO45: R111 10k DNP, VDD_SPI stays 3.3 V; fit it if the internal pull-down is ever in doubt."
+	(text "STRAPS. GPIO0: R2 10k pull-up + SW1 direct to GND, no capacitor (Espressif forbids bulk C here). GPIO46: R108 10k pull-down at the pin, and R109 0R FIT isolates the TPS61169 CTRL so the strap survives even if CTRL sources current - GPIO46 MUST be LOW at reset or Joint Download Boot is unreachable. GPIO3: R110 10k pull-down, LOW selects the USB Serial/JTAG source; external JTAG would land on GPIO39-42, which are I2S. GPIO45: R111 10k FITTED (CTO ruling, FBV2-S1-003) so VDD_SPI is deterministic, not reliant on the internal pull-down alone. VDD_SPI stays 3.3 V. GPIO45 carries no peripheral and no capacitance - TP1 only."
 		(exclude_from_sim no)
 		(at 20.0 42.0 0)

Commit message: hardware: close Full Beta v2 S2 release blockers
Closes B-03, B-63, B-70 and B-71's schematic-side work. Property-only
changes to the nine sheets plus the microphone footprint; ERC unchanged
at 27 / 0 errors / 27 with an identical violation histogram, and the PCB
is untouched and still bit-identical to Beta-DM.

B-03 - all eight remaining Tier-2 footprints compared dimension by
dimension against retrieved manufacturer drawings. Y1 moves from
candidate to lock (Yajingxin TXM27.12M0004322DBBDO00T, C362365, 3421 in
stock) with a land that matches the vendor's Suggested Layout exactly.
The MAX98357A looked like a genuine defect - outline 21-0136 gives
T1633-5 an EP of 1.50/1.60/1.70 while the land is 1.23 - and is not:
land pattern 90-0032 Rev E is issued for T1633-5, -5C and -7C together
and specifies one land for all three, so no project-local footprint was
created.

B-63 - the microphone acoustic port is now drawn rather than described.
1.05 mm NPTH taken from the drawing's own pad-4 ring inner diameter,
paste pulled back 0.10 mm as a declared stencil choice, keepout marked,
bottom-port orientation recorded.

B-70 - L5/L6 lock to Murata LQW18AN39NG80D. The DCR is a first-order
term here: 0.20 ohm max against R_q = 1.1 ohm drops network Q from 25.3
to about 21.4, so the antenna must be tuned with this exact part fitted
and the first lever is R_q, not 39 nH.

B-71 - 65 LCSC fields written in, three MPN strings corrected. J6 and J7
carried bare order codes that resolve to zero-stock listings while the
plating-suffixed strings are abundantly stocked. Six substitution traps
recorded in the symbols themselves, including BAT54W offered for
BAT54WS - a single diode for a series pair - and a clone for the battery
reverse-polarity pass FETs.

Eight DNP parts still carried no recorded reason and now do. The design
has zero unexplained DNP.

Co-Authored-By: Claude Opus 5 <noreply@anthropic.com>
Claude-Session: https://claude.ai/code/session_0133CdFHfKcCH8oPWqJZWe7o
Parts:
- SW1: LCSC (none) -> C221880; Note2 (none) -> SOURCING 2026-08-23 (FBV2-S2-002) (B-71). Genuine C&K PTS64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
- U1: LCSC (none) -> C2913202
Changed lines of the file:
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@@
+			)
+		)
+		(property "LCSC" "C2913202"
+			(at 133.35 96.52 0)
+			(hide yes)
+			(show_name no)
+			(do_not_autoplace no)
+			(effects
+				(font
+					(size 1.27 1.27)
+				)
 			)
 		)
@@
 			(at 87.63 95.25 0)
 			(hide yes)
+			(show_name no)
+			(do_not_autoplace no)
+			(effects
+				(font
+					(size 1.27 1.27)
+				)
+			)
+		)
+		(property "Note2" "SOURCING 2026-08-23 (FBV2-S2-002) (B-71). Genuine C&K PTS645SM43SMTR92LFS is LCSC C221880, stock 8432. A loose keyword search returns G-Switch GT-TC089A-H043-L1 (C843623) instead - a DIFFERENT MANUFACTURER whose land pattern has not been checked against the C&K G-Type layout this footprint was built from. Seven buttons per board is 35 placements for the first five; do not let a search shortcut swap them. LCSC/JLC library state verified live on 2026-08-23 through the JLCPCB parts API (D-096). Stock is a snapshot, not a guarantee."
+			(at 87.63 95.25 0)
+			(hide yes)
+			(show_name no)
+			(do_not_autoplace no)
+			(effects
+				(font
+					(size 1.27 1.27)
+				)
+			)
+		)
+		(property "LCSC" "C221880"
+			(at 87.63 95.25 0)
+			(hide yes)
