File: hardware/beta-v2/kicad/aqroot-beta-v2/03_spi_a_display_sd.kicad_sch (KiCad schematic)
At the start: 18 parts, among them J1 FH69-50S-0.5SH, J2 Molex_5025700893, U17 TPS61169DCKR

Commit message: hardware: migrate Full Beta v2 display and microSD (FBV2-S1-003)
Fits R111 per CTO ruling and migrates 03_SPI_A_DISPLAY_SD. Task gate
FBV2-S1-DISPLAY-SD = PASS. FBV2-S1 itself is 3 of 9 sheets.

THE INHERITED J1 WOULD HAVE PRODUCED A DEAD DISPLAY, TWICE OVER.

J1 still used the 2.8-inch CH280QV10_CT_50P pin table while its Value and
Footprint fields already read FH69-50S-0.5SH. Pin count matched, connector
matched, ERC was silent. The pin FUNCTIONS did not match ER-TFT035IPS-6:

  panel pin 1/2/3   old: LEDK / LED-A1 / LED-A2   new: LEDA / LEDK / LEDK
                    -> backlight reverse-biased, no light
  panel pin 36/37   old: WR_RS->DISP_DC / RS_SCL->SPI_A_SCK
                    new: WRX(SCL) / D-CX
                    -> clock and D/C swapped, no valid command ever reaches
                       the panel
  panel pin 4,5,6   old: LED-A3, LED-A4, IM0(grounded)   new: NC
  panel pin 7,8,9   old: IM1,IM2,IM3   new: IM0,IM1,IM2  (all three were
                    already +3V3, so 1 1 1 was correct by luck)
  panel pin 46      CTP IRQ, not represented at all

Neither fault is visible from a pin count, a connector MPN or an ERC run. A new
project-library symbol ER-TFT035IPS-6_50P was authored with the vendor table
verbatim (datasheet Rev 2.0 sec 4.1), deliberately keeping the old pin geometry
so the migration is a pin-function change and not a redraw. CH280QV10_CT_50P
stays in the library - Beta-DM still uses it - and is dropped from sheet 03's
symbol cache.

R111 FITTED (D-111). 10k, GPIO45_VDDSPI_STRAP -> GND. VDD_SPI is held LOW
deterministically instead of relying on the chip's internal pull-down alone.
TP1 retained, no capacitance on the net, no peripheral on GPIO45.

B-43 CLOSED WITH A PRIMARY SOURCE (D-116). TPS61169 datasheet SNVSA40B:
R_PD, CTRL pin internal pull-down resistor, 300 kohm, with V_H/V_L = 1.2/0.4 V
and t_SD = 2.5 ms. CTRL's only internal element pulls DOWN, so there is no
mechanism by which the backlight driver can raise the GPIO46 strap. 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
Parts:
- added R112: 0R DNP, Resistor_SMD:R_0603_1608Metric, symbol Device:R
- added R113: 100k, Resistor_SMD:R_0603_1608Metric, symbol Device:R
- added TP36: DISP_SDO_TEST, TestPoint:TestPoint_Pad_D1.0mm, symbol Connector:TestPoint
- C43: value 4.7uF -> 4.7uF 10V X5R
- J1: symbol AQROOT_Beta:CH280QV10_CT_50P -> AQROOT_Beta:ER-TFT035IPS-6_50P
- R69: value 2.55R -> 1.87R 1%
- R70, R71, R72, R73: value 39R -> 33R 1%
Connections:
- net +3V3: now also R113.1
- net DISP_DC: now also J1.37 (DCX); no longer J1.36 (~{WR_RS})
- net GND: no longer J1.6 (IM0)
- net LED_K: now also J1.2 (LEDK), J1.3 (LEDK); no longer J1.1 (LEDK)
- net SPI_A_MISO: now also R112.2; no longer J1.33 (SDO)
- net SPI_A_SCK: now also J1.36 (WRX_SCL); no longer J1.37 (RS_SCL)
- net TOUCH_INT_N: now reaches J1.46 (CTP_IRQ)
- net LED_A1 renamed LED_A
- net LED_A: now also J1.1 (LEDA), R71.2, R72.2, R73.2; no longer J1.2 (LED-A1)
- removed net LED_A2: J1.3 (LED-A2), R71.2
- net LED_A3: no longer names the net of J1.4 (NC)
- net LED_A3: no longer R72.2
- net LED_A4: no longer names the net of J1.5 (NC)
- net LED_A4: no longer R73.2
- net SD_CARD_DETECT_TBD renamed SD_CARD_DETECT_N
- net SD_CARD_DETECT_N: now also R113.2
- new net DISP_SDO: J1.33 (SDO), R112.1, TP36.1
- no-connect marks 4 -> 6
Other:
- note added: "=== FBV2-S1 DISPLAY / TOUCH / microSD (FBV2-S1-003) - PANEL LOCKED: EastRising ER-TFT035IPS-6 + ER-TPC035-6 ==="
- note added: "BACKLIGHT: 6 LEDs in parallel, one anode. R69 = 1.87R 1% -> I_LED = VREF/R69 = 100.5 / 109.1 / 117.6 mA over the 188/204/220 mV VREF band, under the panel 120 mA maximum. R70-R73 4 x 33R in parallel = 8.25R ballast on the single LED_A node. Peak switch current 263 mA against the TPS61169 1.2 A minimum limit = 4.6x."
- note added: "DISPLAY SDO: R112 is 0R DNP BY DEFAULT. The ILI9488 datasheet says to leave SDO open when unused and does not specify its high-Z behaviour while CSX is high; SPI-A is shared with the microSD. AQROOT never reads the display, so fitting R112 risks a core feature to gain an unused one. TP36 still observes SDO. Fit R112 only if register readback is ever required."
- note added: "GPIO46 STRAP: TPS61169 CTRL has a 300 kOhm INTERNAL PULL-DOWN (SNVSA40B) and a 1.2 V logic high, so CTRL can only pull GPIO46 DOWN - it can never corrupt the strap, and the backlight is off through reset. With R108 10k on sheet 02 the node sits at 9.68k to GND. R109 0R is retained as a general isolation and rework escape, no longer as the strap defence."
- note added: "J1 pin numbering is taken VERBATIM from ER-TFT035IPS-6_Datasheet Rev 2.0 sec 4.1. It is NOT the CH280QV10-CT numbering. Two pin groups moved and would have been dead on arrival: pins 36/37 are WRX(SCL)/D-CX on this panel and were SCL/D-C reversed on the old part, and pin 1 is LEDA with LEDK on 2+3, where the old part had LEDK on 1 and four anodes on 2-5."
- note added: "SD CARD DETECT: J2.11 DETECT_LEVER is grounded and J2.10 DET-SW is pulled up by R113 100k, so the net is a real two-state signal. SD_CARD_DETECT_N assumes the usual push-push convention - switch closes on insertion, LOW = card present. Polarity is a firmware constant on a PCAL9535A input, never a board change (B-46)."

Commit message: hardware: migrate Full Beta v2 buttons expanders and RGB status
Sheet 08 migrated (FBV2-S1-008), resumed after a session-limit interruption.
All prior work was uncommitted working-tree change; it was inspected, kept and
finished rather than restarted.

Both expanders are NXP PCAL9535APW,118, verified against PCAL9535A Rev. 2
(23-Jan-2015) and NOT treated as a behavioural drop-in: it powers up with every
interrupt masked, the opposite of the TCA9535. U2 = 0x20, U3 = 0x21 preserved.

The two-expander allocation genuinely fails: 35 committed signals against 32
pins, with zero free native GPIO (so the WS2812 escape is impossible),
RESERVED_SPARE mandated by D-094 and ten XGPIO locked by D-082. Closed by U23,
a third PCAL9535APW,118 at 0x22 carrying only the front RGB and the reserved
spare - no new MPN, no new footprint, no new driver, no new rail, and B-37
retired with 12 spare I/O. Core, community and safety functions are placed
before the RGB by construction.

Landed: BQ25185_STAT1/STAT2 (10k pull-ups), SD_CARD_DETECT_N, TOUCH_INT_N,
SX1262_DIO1 on U2; ACC_3V3_EN, ACC_5V_EN, ACC_DETECT_N, ACC_POWER_FAULT_N on
U3. RESERVED_SPARE created on U23 P03 with R130 and TP41 - it had never existed.

Front RGB: D13 MEIHUA MHPA3528RGBCT (LCSC C409779), common anode, R124 1k /
R125 680R / R126 390R = 1.50 / 1.03 / 1.67 mA, white 4.20 mA. Dark by
construction with no external pull-ups.

IR receiver reverted to TSOP38238 (AGC2), TSOP38438 retained as a documented
drop-in fallback. Closes O-5.

Sheets 01 and 03 touched only to promote six local labels to hierarchical so
the required nets could reach the expanders; no component, value, topology or
DNP state changed.

ERC 42 messages / 1 error / 41 warnings - identical violation set to the
recovered tree and better than the 45/2/43 pre-sheet-08 baseline. Zero new
errors. fork_equivalence.py PASS, netclass_probe.py PASS, PCB still
bit-identical to Beta-DM. Sheet 09 untouched.

Co-Authored-By: Claude Opus 5 <noreply@anthropic.com>
Claud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
Changed lines of the file:
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@@
 		)
 	)
-	(label "SD_CARD_DETECT_N"
+	(hierarchical_label "SD_CARD_DETECT_N"
+		(shape output)
 		(at 165.1 81.28 0)
 		(effects
@@
 				(size 1.27 1.27)
 			)
-			(justify left bottom)
+			(justify left)
 		)
 	)

Commit message: hardware: close Full Beta v2 S2 release blockers
Closes B-03, B-63, B-70 and B-71's schematic-side work. Property-only
changes to the nine sheets plus the microphone footprint; ERC unchanged
at 27 / 0 errors / 27 with an identical violation histogram, and the PCB
is untouched and still bit-identical to Beta-DM.

B-03 - all eight remaining Tier-2 footprints compared dimension by
dimension against retrieved manufacturer drawings. Y1 moves from
candidate to lock (Yajingxin TXM27.12M0004322DBBDO00T, C362365, 3421 in
stock) with a land that matches the vendor's Suggested Layout exactly.
The MAX98357A looked like a genuine defect - outline 21-0136 gives
T1633-5 an EP of 1.50/1.60/1.70 while the land is 1.23 - and is not:
land pattern 90-0032 Rev E is issued for T1633-5, -5C and -7C together
and specifies one land for all three, so no project-local footprint was
created.

B-63 - the microphone acoustic port is now drawn rather than described.
1.05 mm NPTH taken from the drawing's own pad-4 ring inner diameter,
paste pulled back 0.10 mm as a declared stencil choice, keepout marked,
bottom-port orientation recorded.

B-70 - L5/L6 lock to Murata LQW18AN39NG80D. The DCR is a first-order
term here: 0.20 ohm max against R_q = 1.1 ohm drops network Q from 25.3
to about 21.4, so the antenna must be tuned with this exact part fitted
and the first lever is R_q, not 39 nH.

B-71 - 65 LCSC fields written in, three MPN strings corrected. J6 and J7
carried bare order codes that resolve to zero-stock listings while the
plating-suffixed strings are abundantly stocked. Six substitution traps
recorded in the symbols themselves, including BAT54W offered for
BAT54WS - a single diode for a series pair - and a clone for the battery
reverse-polarity pass FETs.

Eight DNP parts still carried no recorded reason and now do. The design
has zero unexplained DNP.

Co-Authored-By: Claude Opus 5 <noreply@anthropic.com>
Claude-Session: https://claude.ai/code/session_0133CdFHfKcCH8oPWqJZWe7o
Parts:
- D8: LCSC (none) -> C152519; Note2 (none) -> SOURCING 2026-08-23 (FBV2-S2-002) (B-71). Genuine onsemi NS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
- L3: LCSC (none) -> C5156236
- R112: Note2 (none) -> DNP BY DESIGN - documented 2026-08-23 (FBV2-S2-002). R112 i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
- U17: LCSC (none) -> C71045
Changed lines of the file:
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@@
+			)
+		)
+		(property "LCSC" "C71045"
+			(at 215.9 146.05 0)
+			(hide yes)
+			(show_name no)
+			(do_not_autoplace no)
+			(effects
+				(font
+					(size 1.27 1.27)
+				)
 			)
 		)
@@
 			)
 		)
+		(property "LCSC" "C5156236"
+			(at 196.85 128.27 0)
+			(hide yes)
+			(show_name no)
+			(do_not_autoplace no)
+			(effects
+				(font
+					(size 1.27 1.27)
+				)
+			)
+		)
 		(property "Manufacturer" "Coilcraft"
 			(at 196.85 128.27 0)
@@
 			(at 247.65 135.89 0)
 			(hide yes)
+			(effects
+				(font
+					(size 1.27 1.27)
+				)
+			)
+		)
+		(property "Note2" "SOURCING 2026-08-23 (FBV2-S2-002) (B-71). Genuine onsemi NSR0240HT1G is LCSC C152519 but STOCK IS 7 against a need of 5 for the first five. A loose keyword search returns FUXINSEMI SD103AWS (C915626) instead - THAT IS A DIFFERENT PART AND MUST NOT BE ORDERED IN ITS PLACE. Buy from a broadline distributor and consign if LCSC stock has moved. LCSC/JLC library state verified live on 2026-08-23 through the JLCPCB parts API (D-096). Stock is a snapshot, not a guarantee."
+			(at 247.65 135.89 0)
+			(hide yes)
+			(show_name no)
+			(do_not_autoplace no)
+			(effects
+				(font
+					(size 1.27 1.27)
+				)
+			)
+		)
+		(property "LCSC" "C152519"
+			(at 247.65 135.89 0)
+			(hide yes)
+			(show_name no)
+			(do_not_autoplace no)
 			(effects
 				(font
@@
 			(at 151.13 135.89 0)
 			(hide yes)
+			(show_name no)
+			(do_not_autoplace no)
+			(effects
+				(font
+					(size 1.27 1.27)
+				)
+			)
+		)
+		(property "Note2" "DNP BY DESIGN - documented 2026-08-23 (FBV2-S2-002). R112 is a 0 R link between the display module SDO (/03_SPI_A_DISPLAY_SD/DISP_SDO) and the shared /SPI_A_MISO bus. It is DNP so the display CANNOT drive the bus the microSD card also reads on; the display is written to, never read from, on the first build. Fitting it is a no-respin provision under D-049 for panel register read-back during bring-up, and it MUST NOT be fitted while MX-8 (microSD and display never transact simultaneously on SPI-A) is relied on for bus integrity. It had no note at all before FBV2-S2-002."
+			(at 151.13 135.89 0)
+			(hide yes)
