File: hardware/beta-v2/kicad/aqroot-beta-v2/04_spi_b_radios_nfc.kicad_sch (KiCad schematic)
At the start: 22 parts, among them U7 E07-400M10S, U8 E22-900M22S, U9 ST25R3916-AQET

Commit message: hardware: migrate Full Beta v2 radios and NFC (FBV2-S1-004)
Sheet 04. Task gate FBV2-S1-RADIOS-NFC = PASS. FBV2-S1 itself is 4 of 9 sheets.

ERC: 4 errors -> 2. Total 86 -> 68. Zero added, eighteen removed. This is the
first migration task to REDUCE the project's error count, and it did so by
deleting placeholder architecture rather than by suppressing anything.

ZERO *_TBD NETS REMAIN ANYWHERE IN THE PROJECT. Sheet 04 alone retired fourteen.

RF ARCHITECTURE LOCKED (D-118).
433 MHz: INTERNAL flex. U7 IPEX -> 100 mm coax -> Taoglas FXP450.07.0100C against
a plastic wall. 915 MHz: EXTERNAL. U8 IPEX -> short pigtail -> top-panel SMA
female bulkhead, user-changeable. Neither band has a motherboard 50 ohm RF trace,
a matching network, an RF switch or a diplexer - both modules present their own
matched 50 ohm port, so the board's RF involvement at 433/915 is zero copper.
This supersedes the internal-FXP890 plan for 915 in "12 - RF and Antenna Plan".
The U7 IPEX socket must remain SERVICE-ACCESSIBLE with the shell open: if
internal 433 performance disappoints on the first units the flex unplugs and an
external pigtail replaces it with no PCB respin. That is an FBV2-P1 placement
constraint and the reason an internal antenna is an acceptable first-build risk.

433 ANTENNA VERIFIED, MATING PROVEN RATHER THAN ASSUMED (D-119). Taoglas
datasheet SPE-23-8-180-A, verbatim: "410-470MHz Flexible PCB Antenna with 100mm
1.37 IPEX MHFI". 47 x 17 x 0.28 mm, adhesive mount, gain -0.36 / -1.57 /
-0.05 dBi, Active, 54 in stock, $5.52 @ 1, MOQ 1. The antenna terminates in IPEX
MHF I and Ebyte's manual lists the E07-400M10S interface as IPEX-1 / stamp hole;
MHF I, IPEX-1 and U.FL are one mating interface, so no cable variant is needed.
Mechanical reservation recorded for FBV2-P1: plastic wall, LEFT/LOWER-SIDE, NOT
on the PCB, clear of the LiPo, the NFC loop and ferrite, the speaker magnet,
large ground pours, metal bosses, the USB shell, the 915 bulkhead/pigtail and the
IR structures.

915 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
Parts:
- added C69, C70, C76, C78: 220pF 50V C0G TUNE, Capacitor_SMD:C_0603_1608Metric, symbol Device:C
- added C71, C72, C73, C74: 100pF 50V C0G TUNE, Capacitor_SMD:C_0603_1608Metric, symbol Device:C
- added C75, C77: 47pF 50V C0G TUNE, Capacitor_SMD:C_0603_1608Metric, symbol Device:C
- added C79, C80: 10pF 50V C0G TUNE, Capacitor_SMD:C_0603_1608Metric, symbol Device:C
- added L5, L6: 220nH TUNE, Inductor_SMD:L_0603_1608Metric, symbol Device:L
- added R114, R115: 0R TUNE, Resistor_SMD:R_0603_1608Metric, symbol Device:R
- added R116, R117: 1k TUNE, Resistor_SMD:R_0603_1608Metric, symbol Device:R
- added TP37: NFC_ANT_A_TEST, TestPoint:TestPoint_Pad_D1.0mm, symbol Connector:TestPoint
- added TP38: NFC_ANT_B_TEST, TestPoint:TestPoint_Pad_D1.0mm, symbol Connector:TestPoint
- added Y1: 27.12MHz 10pF 3225-4P, Crystal:Crystal_SMD_3225-4Pin_3.2x2.5mm, symbol Device:Crystal_GND24
Connections:
- net GND: now also C69.2, C70.2, C73.2, C74.2, C76.2, C78.2, C79.2, C80.2, Y1.2 (G), Y1.4 (G)
- net CC1101_ANT_TBD: no longer names the net of U7.21 (ANT)
- net NFC_5V_PA_PENDING renamed NFC_SUPPLY
- net NFC_AAT_A_TBD: no longer names the net of U9.18 (AAT_A)
- net NFC_AAT_B_TBD: no longer names the net of U9.19 (AAT_B)
- net NFC_CSI_TBD: no longer names the net of U9.25 (CSI)
- net NFC_CSO_TBD: no longer names the net of U9.2 (CSO)
- net NFC_EXT_LM_TBD: no longer names the net of U9.17 (EXT_LM)
- net NFC_MCU_CLK_TBD: no longer names the net of U9.28 (MCU_CLK)
- net NFC_RFI1_TBD renamed NFC_RFI1
- net NFC_RFI1: now also R116.2
- net NFC_RFI2_TBD renamed NFC_RFI2
- net NFC_RFI2: now also R117.2
- net NFC_RFO1_TBD renamed NFC_RFO1
- net NFC_RFO1: now also L5.1
- net NFC_RFO2_TBD renamed NFC_RFO2
- net NFC_RFO2: now also L6.1
- net NFC_XIN_TBD renamed NFC_XIN
- net NFC_XIN: now also C80.1, Y1.3
- net NFC_XOUT_TBD renamed NFC_XOUT
- net NFC_XOUT: now also C79.1, Y1.1
- net RF_ANT_TBD: no longer names the net of U8.21 (ANT)
- new net NFC_ANT_A: C75.1, R114.2, TP37.1
- new net NFC_ANT_B: C77.1, R115.2, TP38.1
- new net NFC_EMCA: C69.1, C71.1, C73.1, L5.2
- new net NFC_EMCB: C70.1, C72.1, C74.1, L6.2
- new net NFC_MATCH_A: C71.2, R114.1
- new net NFC_MATCH_B: C72.2, R115.1
- new net NFC_RXA: C75.2, C76.1, R116.1
- new net NFC_RXB: C77.2, C78.1, R117.1
- no-connect marks 1 -> 9
Other:
- note added: "433 MHz: INTERNAL Taoglas FXP450.07.0100C flex (410-470 MHz, 47 x 17 x 0.28 mm, 100 mm 1.37 mm coax, IPEX MHF-I) onto the U7 module socket. 915 MHz: EXTERNAL - U8 IPEX -> short pigtail -> top-panel SMA bulkhead. NEITHER band has a board RF trace, a matching network or an RF switch. Module pin 21 (stamp hole) is the alternative feed and stays NC on both modules."
- note added: "=== FBV2-S1 RADIOS + NFC (FBV2-S1-004) - RF ARCHITECTURE LOCKED ==="
- note added: "=== NFC FRONT END - TOPOLOGY IS REAL, VALUES ARE NOT FINAL ==="
- note added: "Every part marked TUNE is an INITIAL VALUE. The matching and RX-divider values cannot be finalised until the 45 x 45 mm antenna impedance is measured and the ST antenna matching tool (STSW-ST25R004) is run against it. TP37/TP38 are the measurement points - probe NFC_ANT_A / NFC_ANT_B with a VNA before fitting a final set. All tuning parts are 0603 so they can be reworked by hand."
- note added: "NOT FITTED on the first build, and the pins are explicitly NC: AAT_A / AAT_B (automatic antenna tuning needs external varactors, and DS12484 warns against combining AAT with hardware wake-up), CSI / CSO (capacitive sensing), EXT_LM (external load-modulation MOSFET - the internal load modulator is used), MCU_CLK (the ESP32-S3 has its own clocks)."
- note added: "ONE HIGH-POWER TRANSMITTER AT A TIME (MX-1). CC1101 TX, SX1262 +22 dBm TX and the NFC field are mutually exclusive until measurement proves concurrency safe."
- note added: "RX chain per side: antenna -> C_rx_series -> [C_rx_shunt to GND] -> R_rx -> RFIx. The divider must keep RFIx inside its input range at full field; it is sized with the same tool run."
- note added: "SUPPLY: VDD (pin 8) and VDD_TX (pin 10) now sit on NFC_SUPPLY, not on the Beta-DM boost output - this closes B-41. NFC_SUPPLY is +3V3 on the first build through the R106 FIT link on sheet 01; the R107 DNP link is the no-respin 5 V fallback. VDD_IO (pin 1) stays on +3V3. FIRMWARE MUST SET sup3V."
- note added: "TX chain per side: RFOx -> L_EMC -> [C_EMC + C_p to GND] -> C_s -> R_q -> antenna. C_EMC and C_p are two separate shunt footprints on the same node ON PURPOSE: it gives two trim positions instead of one. R_q is fitted 0 R and is raised to widen bandwidth / lower Q if the read range needs it."
- note added: "The U7 IPEX socket must stay SERVICE-ACCESSIBLE with the enclosure open: if internal 433 performance disappoints on the first units, the flex unplugs and an external pigtail goes in its place with NO PCB respin (D-049)."

Commit message: hardware: finalize Full Beta v2 NFC antenna interface (FBV2-S1-004B)
Sheet 04 closeout. Task gate FBV2-S1-NFC-ANTENNA-LOCK = PASS.
ERC 68 -> 68: zero added, zero removed, the violation lists are identical.
301 components, 0 duplicate references, 0 without a footprint.

B-06 IS CLOSED. "NFC is undesigned, not merely unrouted" has been on the blocker
list since the pre-design audit and is not true any more: crystal, matching
topology, antenna, connector and supply all exist. What remains is tuning, which
is a bench activity, not a design gap.

NFC IC LOCKED - P-17 CLOSED (D-126). ST25R3916-AQET. The B variant is not
adopted: non-B is active production, it preserves capacitive low-power sensing,
AQROOT is not an EMVCo payment terminal, AWS is not worth trading sourcing
simplicity and feature breadth for, and the first build already has 3.3 V plus a
no-respin 5 V fallback. This agrees with the FBV2-S1-004 recommendation on
independent grounds - the non-B is the only one of the two with an LCSC part
number (C5267441) and therefore a JLCPCB assembly path, at roughly half the unit
cost. MPN metadata verified present in the schematic, not merely in prose: Value,
MPN, Manufacturer and LCSC all carry it. U9's Package description was rewritten -
it still named NFC_5V_PA_PENDING as the supply and told the reader the RF and
oscillator pins were "on explicit named TBD nets - DO NOT ROUTE", and both
statements stopped being true in FBV2-S1-004.

NFC ANTENNA LOCKED, OFF-BOARD - B-53 CLOSED (D-127). Taoglas
FXC.46.52.0075X.A.dg, verified verbatim from Taoglas SPE-22-8-131-C: "Circular
Form Factor Flexible Near Field Communications Antenna", 13.56 MHz, "Diameter:
46 mm", "Thickness: 0.27 mm - FXC.46.52.0075X.A.dg - NFC with ferrite and 75mm
Twisted Pair 28AWG cable with ACH(F) connector", "Peel and stick 3M adhesive",
typical interrogation distance 40 mm. This replaces the abstract 45x45 mm
custom-antenna assumption and keeps the antenna off the main PCB - which is what
avoids puttin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
Parts:
- added J7: BM02B-ACHSS-GAN-ETF, Connector_JST:JST_ACH_BM02B-ACHSS-GAN-ETF_1x02-1MP_P1.20mm_Vertical, symbol Connector_Generic:Conn_01x02
- C71, C72: value 100pF 50V C0G TUNE -> 300pF 50V C0G TUNE
- C73, C74: value 100pF 50V C0G TUNE -> 1.8nF 50V C0G TUNE
- R114, R115: value 0R TUNE -> 1R0 TUNE
- U9: Package UFQFPN32 5x5x0.55, 0.5 mm pitch, 32 lands + exposed pad 33. Normal internal RF-regulator mode: VDD_IO on +3V3; VDD and VDD_TX both on NFC_5V_PA_PENDING; I2C_EN grounded to select SPI; VDD_DR sourced from the VDD_RF regulated node - NOT tied to VDD_TX, which would be the regulator-bypass configuration and is not used for Beta. Regulator outputs VDD_D, VDD_A, VDD_RF and VDD_AM plus reference AGDC each carry ST-specified local decoupling. Exposed pad grounded per ST. RF, oscillator and AAT/EXT_LM/CSI pins are on explicit named TBD nets - DO NOT ROUTE until NFC antenna and matching design. -> UFQFPN32 5x5x0.55, 0.5 mm pitch, 32 lands + exposed pad 33. LOCKED 2026-08-23 (FBV2-S1-004B): ST25R3916-AQET, NOT the B variant. Normal internal RF-regulator mode: VDD_IO on +3V3; VDD and VDD_TX both on NFC_SUPPLY, which is +3V3 on the first build through the R106 FIT link with the R107 DNP link as the no-respin 5 V fallback; I2C_EN grounded to select SPI; VDD_DR sourced from the VDD_RF regulated node - NOT tied to VDD_TX, which would be the regulator-bypass configuration and is not used. Regulator outputs VDD_D, VDD_A, VDD_RF and VDD_AM plus reference AGDC each carry ST-specified local decoupling. Exposed pad grounded per ST. FIRMWARE MUST SET sup3V. AAT_A/AAT_B, CSI/CSO, EXT_LM and MCU_CLK are explicit no-connects. RF front end and 27.12 MHz crystal are captured; every matching value is TUNE until STSW-ST25R004 is run.
- Y1: LCSC (none) -> C362365; MPN (none) -> TXM27.12M0004322DBBDO00T; Manufacturer (none) -> Yajingxin; Note (none) -> CANDIDATE against a live LCSC listing, not a lock (D-096). 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
Connections:
- net NFC_ANT_A: now also J7.1 (Pin_1)
- net NFC_ANT_B: now also J7.2 (Pin_2)
Other:
- note added: "=== NFC ANTENNA INTERFACE - LOCKED OFF-BOARD (FBV2-S1-004B) ==="
- note added: "Antenna: Taoglas FXC.46.52.0075X.A.dg - 13.56 MHz circular flex, 46 mm diameter, 0.27 mm thick WITH FERRITE, peel-and-stick 3M adhesive, 75 mm twisted pair 28 AWG, ACH(F) connector, typical interrogation distance 40 mm. IT DOES NOT GO ON THE PCB."
- note added: "J7 BM02B-ACHSS-GAN-ETF, JST ACH, 2 circuits, 1.2 mm, SMT, gold, 2.0 A. It mates the ACHR-02V-S housing, which is the ACH(F) connector already fitted to the antenna cable - so the antenna is REPLACEABLE WITHOUT SOLDERING. JST classes ACH as TOP ENTRY: the socket drops on vertically and the wires leave horizontally. Leave vertical clearance above J7 for mating."
- note added: "MATCHING BASIS: L = 1.09 uH, Rs = 1.6 R, Q0 = 58 at 13.56 MHz. R_q 1R0 per leg brings Q to about 26 for ISO14443 bandwidth - that value is derived from the antenna alone and is the most solid number here. C_s 300pF and C_p 1.8nF come from an L-match to an ASSUMED 20 R per side driver target; the EMC pair L5/L6 + C69/C70 has NOT been re-derived against the new shunt and is NOT yet a working filter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"

Commit message: hardware: correct Full Beta v2 NFC antenna and matching (FBV2-S1-004C)
Sheet 04. Task gate FBV2-S1-NFC-MATCHING = PASS.
ERC 68 -> 68: zero added, zero removed. Errors remain 2, both inherited.

TWO DEFECTS TURNED UP THAT WERE NOT ON THE BRIEF.

1. The RX divider would have over-driven the receiver. At full field the antenna
sits at 49.5 V pk-pk differential, 24.8 V pk-pk per side. The placeholder
47pF / 220pF divider has a ratio of 0.176 and would therefore have put about
4.4 V pk-pk on RFI1/RFI2 - against a 3.0 V regulated analog rail. That is a
part-stress condition, not a tuning imperfection, and it had been carried since
the topology was first drawn without ever being checked against a real antenna
voltage. New divider 27pF / 620pF, ratio 0.0417, gives about 1.03 V pk-pk per
side - over 3x headroom. Purely capacitive, no DC path, and it adds only ~26 pF
of shunt at the antenna node.

2. The E24 grid is brutally steep at the series matching capacitor. C_s sits
close to series resonance where dZ/dC is enormous, so the two E24 neighbours of
the ideal 284 pF are not close in effect:
    270 pF/leg -> ~16 ohm differential -> 0.55 W -> ~257 mA, OVER BUDGET
    284 pF ideal -> 36 ohm -> 0.247 W -> ~115 mA
    300 pF/leg -> ~68 ohm differential -> 0.13 W -> ~60 mA   <- SELECTED
300 pF is chosen on purpose, on the low-current side: on a first board an
under-driven antenna is a one-component swap, while an over-driven one risks the
driver and the +3V3 budget on first power-up. 187 mA of coil current in a 46 mm
loop is still a serviceable field, about 72% of what the 36 ohm design would
give, and the shortfall is recoverable by rework.

ANTENNA VARIANT CORRECTED A -> B (D-131). FXC.46.52.0075X.A.dg is superseded;
FXC.46.52.0075X.B.dg is locked. Verified verbatim from Taoglas SPE-24-8-104-B:
"NFC Flex Antenna (46*0.3mm) with a Reverse Ferrite Layer and adhesive backing",
"13.56 MHz Antenna", "Diameter: 46mm", "FXC.46.52.0075X.B.dg - NFC with ferrite
and 75mm Twisted Pair 28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
Parts:
- C69, C70: value 220pF 50V C0G TUNE -> 100pF 50V C0G TUNE
- C73, C74: value 1.8nF 50V C0G TUNE -> 1.5nF 50V C0G TUNE
- C75, C77: value 47pF 50V C0G TUNE -> 27pF 50V C0G TUNE
- C76, C78: value 220pF 50V C0G TUNE -> 620pF 50V C0G TUNE
- J7: Note Board-side NFC antenna interface. Off-board antenna: Taoglas FXC.46.52.0075X.A.dg -> Board-side NFC antenna interface. Off-board antenna: Taoglas FXC.46.52.0075X.B.dg (REVERSE ferrite, adhesive to the inner rear shell)
- L5, L6: value 220nH TUNE -> 39nH TUNE
- R114, R115: value 1R0 TUNE -> 1R1 1% TUNE
Other:
- note added: "Antenna: Taoglas FXC.46.52.0075X.B.dg - the B VERSION, REVERSE FERRITE LAYER (SPE-24-8-104-B). 13.56 MHz, 46 mm diameter, 0.3 mm, peel-and-stick 3M adhesive, 75 mm twisted pair 28 AWG, ACH(F). Stack order is ADHESIVE / FLEX ANTENNA / FERRITE, so it bonds ADHESIVE-SIDE to the INNER REAR SHELL and reads OUTWARD through the plastic with the ferrite facing INWARD at the PCB and battery (Taoglas APN-2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"
- note added: "MATCHING BASIS (FBV2-S1-004C, AN5276 Rev 6 workflow): FXC.46.B published La 1.10 uH, Rs 1.50 R, Q 60.37, SRF 395 MHz. wL = 93.72 R at 13.56 MHz. CALCULATED FIRST-BUILD SET, not final tuning: R_q 1R1 per leg -> R_total 3.70 R -> Q 25.3. C_s 300pF per leg (ideal 284pF; 300pF is the E24 neighbour on the SAFE, lower-current side) -> about 68 R differential, 0.13 W, coil current about 187 mA, driver a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"
- note removed: "Antenna: Taoglas FXC.46.52.0075X.A.dg - 13.56 MHz circular flex, 46 mm diameter, 0.27 mm thick WITH FERRITE, peel-and-stick 3M adhesive, 75 mm twisted pair 28 AWG, ACH(F) connector, typical interrogation distance 40 mm. IT DOES NOT GO ON THE PCB."
- note removed: "MATCHING BASIS: L = 1.09 uH, Rs = 1.6 R, Q0 = 58 at 13.56 MHz. R_q 1R0 per leg brings Q to about 26 for ISO14443 bandwidth - that value is derived from the antenna alone and is the most solid number here. C_s 300pF and C_p 1.8nF come from an L-match to an ASSUMED 20 R per side driver target; the EMC pair L5/L6 + C69/C70 has NOT been re-derived against the new shunt and is NOT yet a working filter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"
Changed lines of the file:
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@@
 			)
 		)
-		(property "Value" "220nH TUNE"
+		(property "Value" "39nH TUNE"
 			(at 311.15000000000003 130.81 0)
 			(show_name no)
@@
 			)
 		)
-		(property "Value" "220pF 50V C0G TUNE"
+		(property "Value" "100pF 50V C0G TUNE"
 			(at 323.85 138.43 0)
 			(show_name no)
@@
 			)
 		)
-		(property "Value" "1.8nF 50V C0G TUNE"
+		(property "Value" "1.5nF 50V C0G TUNE"
 			(at 335.28000000000003 138.43 0)
 			(show_name no)
@@
 			)
 		)
-		(property "Value" "1R0 TUNE"
+		(property "Value" "1R1 1% TUNE"
 			(at 361.95000000000005 130.81 0)
 			(show_name no)
@@
 			)
 		)
-		(property "Value" "220nH TUNE"
+		(property "Value" "39nH TUNE"
 			(at 311.15000000000003 176.53 0)
 			(show_name no)
@@
 			)
 		)
-		(property "Value" "220pF 50V C0G TUNE"
+		(property "Value" "100pF 50V C0G TUNE"
 			(at 323.85 184.15 0)
 			(show_name no)
@@
 			)
 		)
-		(property "Value" "1.8nF 50V C0G TUNE"
+		(property "Value" "1.5nF 50V C0G TUNE"
 			(at 335.28000000000003 184.15 0)
 			(show_name no)
@@
 			)
 		)
-		(property "Value" "1R0 TUNE"
+		(property "Value" "1R1 1% TUNE"
 			(at 361.95000000000005 176.53 0)
 			(show_name no)
@@
 			)
 		)
-		(property "Value" "47pF 50V C0G TUNE"
+		(property "Value" "27pF 50V C0G TUNE"
 			(at 311.15000000000003 222.25 0)
 			(show_name no)
@@
 			)
 		)
-		(property "Value" "220pF 50V C0G TUNE"
+		(property "Value" "620pF 50V C0G TUNE"
 			(at 323.85 229.87 0)
 			(show_name no)
@@
 			)
 		)
-		(property "Value" "47pF 50V C0G TUNE"
+		(property "Value" "27pF 50V C0G TUNE"
 			(at 311.15000000000003 255.27 0)
 			(show_name no)
@@
 			)
 		)
-		(property "Value" "220pF 50V C0G TUNE"
+		(property "Value" "620pF 50V C0G TUNE"
 			(at 323.85 262.89 0)
 			(show_name no)
@@
 			)
 		)
-		(property "Note" "Board-side NFC antenna interface. Off-board antenna: Taoglas FXC.46.52.0075X.A.dg"
+		(property "Note" "Board-side NFC antenna interface. Off-board antenna: Taoglas FXC.46.52.0075X.B.dg (REVERSE ferrite, adhesive to the inner rear shell)"
 			(at 0 0 0)
 			(hide yes)
@@
 		)
 	)
-	(text "Antenna: Taoglas FXC.46.52.0075X.A.dg - 13.56 MHz circular flex, 46 mm diameter, 0.27 mm thick WITH FERRITE, peel-and-stick 3M adhesive, 75 mm twisted pair 28 AWG, ACH(F) connector, typical interrogation distance 40 mm. IT DOES NOT GO ON THE PCB."
+	(text "Antenna: Taoglas FXC.46.52.0075X.B.dg - the B VERSION, REVERSE FERRITE LAYER (SPE-24-8-104-B). 13.56 MHz, 46 mm diameter, 0.3 mm, peel-and-stick 3M adhesive, 75 mm twisted pair 28 AWG, ACH(F). Stack order is ADHESIVE / FLEX ANTENNA / FERRITE, so it bonds ADHESIVE-SIDE to the INNER REAR SHELL and reads OUTWARD through the plastic with the ferrite facing INWARD at the PCB and battery (Taoglas APN-24-8-001). The A version is for bonding onto a PCB or component surface and is NOT the right part here. IT DOES NOT GO ON THE PCB."
 		(exclude_from_sim no)
 		(at 380.0 112.0 0)
@@
 		)
 	)
-	(text "MATCHING BASIS: L = 1.09 uH, Rs = 1.6 R, Q0 = 58 at 13.56 MHz. R_q 1R0 per leg brings Q to about 26 for ISO14443 bandwidth - that value is derived from the antenna alone and is the most solid number here. C_s 300pF and C_p 1.8nF come from an L-match to an ASSUMED 20 R per side driver target; the EMC pair L5/L6 + C69/C70 has NOT been re-derived against the new shunt and is NOT yet a working filter. EVERYTHING STAYS TUNE UNTIL STSW-ST25R004 IS RUN. Do not build to these values."
+	(text "MATCHING BASIS (FBV2-S1-004C, AN5276 Rev 6 workflow): FXC.46.B published La 1.10 uH, Rs 1.50 R, Q 60.37, SRF 395 MHz. wL = 93.72 R at 13.56 MHz. CALCULATED FIRST-BUILD SET, not final tuning: R_q 1R1 per leg -> R_total 3.70 R -> Q 25.3. C_s 300pF per leg (ideal 284pF; 300pF is the E24 neighbour on the SAFE, lower-current side) -> about 68 R differential, 0.13 W, coil current about 187 mA, driver about 60 mA. C_p 1.5nF completes the L-match. EMC: L 39nH with the 1.6nF total shunt gives f_c 20.1 MHz - AN5276 forbids a cut-off between 13 and 14 MHz, and the old 220nH pair sat at 7.6 MHz, BELOW the carrier. RX divider 27pF / 620pF holds RFI at about 1.0 Vpp per side against a 3.0 V regulated rail; the previous 47pF / 220pF would have driven it to about 4.4 Vpp, ABOVE the rail. FINAL VALUES COME FROM A VNA WITH THE REAR SHELL, PCB AND BATTERY IN PLACE."
 		(exclude_from_sim no)
 		(at 380.0 118.0 0)
