File: hardware/beta-v2/kicad/aqroot-beta-v2/06_audio.kicad_sch (KiCad schematic)
At the start: 7 parts, among them J6 JST-PH-2 SPEAKER, U5 MAX98357A

Commit message: hardware: migrate Full Beta v2 audio (FBV2-S1-006)
Sheet 06. Task gate FBV2-S1-AUDIO = PASS.
ERC 45 -> 45: zero added, zero removed. Errors remain 2, both inherited.

THE BIGGEST FINDING WAS NOT ON THE BRIEF.

U5 (the MAX98357A) and J6 (the speaker connector) arrived from Beta-DM marked
DNP. Nobody wrote that down - it is in the inherited file. It means the entire
speaker output path has never been populated on any AQROOT board, while C9 and
C10 WERE fitted, decoupling an amplifier that was not there.

The brief says voice output remains required and Full Beta v2 is the
feature-complete design, so both are now fitted. Everything below - the power
budget, the speaker choice, the EMI provision - describes a path being built for
the first time, and bring-up should read it that way.

This is the third load-bearing inherited DNP in two tasks (U16, R49/R50, U15,
D2/D3 on sheet 09 at FBV2-S1-005). A DNP on a Beta-DM sheet is a statement about
the reduced build, not about the architecture, and every migrated sheet has to
re-decide it rather than inherit it.

THE MICROPHONE IS NOT A DROP-IN, FOR A STRONGER REASON THAN SIZE.

  ICS-43434              DMM-4026-B-I2S-R
  6 pads                 7 pads
  3.5 x 2.65 x 0.98 mm   4.00 x 3.00 x 1.00 mm
  -                      CONFIG pin, no ICS equivalent

The pin count differs, so both a new symbol and a new footprint were built from
the PUI drawing (Rev A, 5/26/2021). Every pin was re-derived: LR->GND selects the
left I2S slot; CONFIG->GND is MANDATORY ("Pull to ground. The state of this pin
is used at power-up."); VDD 1.62-3.63 V with C8 100 nF; WS/SCK/SD unchanged.

R120 100 kOhm on I2S_MIC_DIN is a DATA-SHEET REQUIREMENT, not a preference:
"The SD trace should have a 100 kOhm pull down resistor to discharge the line
during the time that all microphones on the bus have tri-stated their outputs."
With one microphone the line still tri-states for the entire unused half of every
frame, and the inherited sheet had no pull-down at al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
Parts:
- removed MK1: ICS-43434, Sensor_Audio:InvenSense_ICS-43434-6_3.5x2.65mm, symbol Sensor_Audio:ICS-43434
- added C81, C82: 1nF DNP, Capacitor_SMD:C_0603_1608Metric, symbol Device:C
- added MK1: DMM-4026-B-I2S, AQROOT_Beta:PUI_DMM-4026-B-I2S_4.0x3.0mm, symbol AQROOT_Beta:DMM-4026-B-I2S
- added R120: 100k, Resistor_SMD:R_0603_1608Metric, symbol Device:R
- added R121, R122: 0R, Resistor_SMD:R_0603_1608Metric, symbol Device:R
- J6: Note Board-side speaker connector. OFF-BOARD SPEAKER / 8R >=0.5W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 -> Board-side speaker connector, RETAINED in FBV2-S1-006. J6 p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; now fitted
- LS1: value 8R_SPEAKER_OFFBOARD -> AS02008MR-LW152-R; MPN SKU FINALIZES WITH ENCLOSURE -> AS02008MR-LW152-R; Manufacturer TBD - selected with the enclosure -> PUI Audio; Note OFF_BOARD / WIRED SPEAKER / 8R >=0.5W / SKU FINALIZES WITH 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 -> OFF-BOARD, ENCLOSURE-MOUNTED, WIRED THROUGH J6. LS1 is draw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; Package OFF_BOARD WIRED SPEAKER, 8 ohm, >=0.5 W, ~15 mm class. No P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 -> OFF_BOARD wired speaker, 20 mm diameter x 3 mm, 152 mm flyi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
- U5: MPN (none) -> MAX98357AETE+T; Manufacturer (none) -> Analog Devices (Maxim); Note (none) -> RETAINED after a lifecycle check in FBV2-S1-006: analog.com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; Package (none) -> TQFN-16, 3 x 3 mm, 0.5 mm pitch, exposed pad; now fitted
Connections:
- net +3V3: now also U5.2 (GAIN_SLOT), MK1.3 (VDD)
- net GND: now also C81.2, C82.2, MK1.1 (LR), MK1.2 (CONFIG), MK1.4 (GND), R120.2; no longer U5.2 (GAIN_SLOT)
- net I2S_BCLK: now also MK1.6 (SCK)
- net I2S_LRCLK: now also MK1.5 (WS)
- net I2S_MIC_DIN: now also MK1.7 (SD), R120.1
- net SPK_N: now also R122.1; no longer J6.2 (Pin_2), LS1.2
- net SPK_P: now also R121.1; no longer J6.1 (Pin_1), LS1.1
- new net SPK_N_CONN: C82.1, J6.2 (Pin_2), LS1.2, R122.2
- new net SPK_P_CONN: C81.1, J6.1 (Pin_1), LS1.1, R121.2
Other:
- note added: "AUDIO ARCHITECTURE - MIGRATED FBV2-S1-006 MK1 PUI DMM-4026-B-I2S-R (REPLACES ICS-43434) LR -> GND = LEFT I2S SLOT CONFIG-> GND = MANDATORY, READ AT POWER-UP VDD 1.62-3.63 V, C8 100nF LOCAL SD TRI-STATES OFF-SLOT -> R120 100k PULL-DOWN (DATA-SHEET REQUIREMENT, NOT A CHOICE) 7 PADS, NOT 6. NEW SYMBOL AND NEW FOOTPRINT. U5 MAX98357AETE+T 3.3 V, PRODUCTION GAIN_SLOT -> VDD = 6 dB (WAS GND = 12 dB) AT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"
- note added: "SPEAKER - LOCKED FBV2-S1-006 LS1 = PUI AUDIO AS02008MR-LW152-R 20 mm DIA x 3 mm, 8R +/-15%, 0.5 W RATED / 0.8 W MAX, 86 +/-3 dBA @ 0.1 W / 0.1 m, 500-4000 Hz = VOICE BAND, NOT MUSIC, 152 mm UL1571 AWG#32 LEADS, RED +, BLACK -. OFF-BOARD, ENCLOSURE-MOUNTED, WIRED VIA J6. LS1 IS EXCLUDED FROM THE BOARD (on_board no). J6 pin 1 = SPK_P J6 pin 2 = SPK_N MATING: JST PHR-2 + SPH-002T-P0.5S. AWG#32 IS IN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"
- note removed: "AUDIO ARCHITECTURE LOCKED ICS-43434: LEFT I2S SLOT - LR PIN TIED TO GND MAX98357A: 3.3V SUPPLY GAIN_SLOT TIED TO GND - 12 dB GAIN DIFFERENTIAL FILTERLESS SPEAKER OUTPUT SPEAKER IS OFF-BOARD - WIRED VIA J6 (JST PH 2.0 mm) VERIFY OUTPUT LEVEL AND THERMALS ON BETA SPEAKER SKU FINALISES WITH THE ENCLOSURE"
- note removed: "SPEAKER IS OFF-BOARD OFF-BOARD SPEAKER 8R >=0.5W JST PH 2.0 mm ENCLOSURE-MOUNTED LS1 represents the wired speaker beyond J6 and is EXCLUDED FROM THE BOARD. J6 pin 1 = SPK_P = MAX98357A OUTP J6 pin 2 = SPK_N = MAX98357A OUTN OBSERVE POLARITY WHEN CRIMPING Speaker SKU finalises with the enclosure."

Commit message: hardware: close Full Beta v2 S2 release blockers
Closes B-03, B-63, B-70 and B-71's schematic-side work. Property-only
changes to the nine sheets plus the microphone footprint; ERC unchanged
at 27 / 0 errors / 27 with an identical violation histogram, and the PCB
is untouched and still bit-identical to Beta-DM.

B-03 - all eight remaining Tier-2 footprints compared dimension by
dimension against retrieved manufacturer drawings. Y1 moves from
candidate to lock (Yajingxin TXM27.12M0004322DBBDO00T, C362365, 3421 in
stock) with a land that matches the vendor's Suggested Layout exactly.
The MAX98357A looked like a genuine defect - outline 21-0136 gives
T1633-5 an EP of 1.50/1.60/1.70 while the land is 1.23 - and is not:
land pattern 90-0032 Rev E is issued for T1633-5, -5C and -7C together
and specifies one land for all three, so no project-local footprint was
created.

B-63 - the microphone acoustic port is now drawn rather than described.
1.05 mm NPTH taken from the drawing's own pad-4 ring inner diameter,
paste pulled back 0.10 mm as a declared stencil choice, keepout marked,
bottom-port orientation recorded.

B-70 - L5/L6 lock to Murata LQW18AN39NG80D. The DCR is a first-order
term here: 0.20 ohm max against R_q = 1.1 ohm drops network Q from 25.3
to about 21.4, so the antenna must be tuned with this exact part fitted
and the first lever is R_q, not 39 nH.

B-71 - 65 LCSC fields written in, three MPN strings corrected. J6 and J7
carried bare order codes that resolve to zero-stock listings while the
plating-suffixed strings are abundantly stocked. Six substitution traps
recorded in the symbols themselves, including BAT54W offered for
BAT54WS - a single diode for a series pair - and a clone for the battery
reverse-polarity pass FETs.

Eight DNP parts still carried no recorded reason and now do. The design
has zero unexplained DNP.

Co-Authored-By: Claude Opus 5 <noreply@anthropic.com>
Claude-Session: https://claude.ai/code/session_0133CdFHfKcCH8oPWqJZWe7o
Parts:
- J6: LCSC (none) -> C131337; MPN B2B-PH-K-S -> B2B-PH-K-S(LF)(SN); Note2 (none) -> SOURCING 2026-08-23 (FBV2-S2-002) (B-71). J4 and J6 are the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
- LS1: LCSC (none) -> C3311653
- MK1: LCSC (none) -> C3171792; Note2 (none) -> SOURCING 2026-08-23 (FBV2-S2-002) (B-71). PUI Audio DMM-402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
- U5: LCSC (none) -> C910544; Note2 (none) -> B-03 FOOTPRINT VERIFIED TIER 1 2026-08-23 (FBV2-S2-002). Bo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
Changed lines of the file:
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@@
+			)
+		)
+		(property "Note2" "B-03 FOOTPRINT VERIFIED TIER 1 2026-08-23 (FBV2-S2-002). Both cited Maxim documents were retrieved and read. Package outline 21-0136 gives 16L TQFN 3x3, e = 0.50 BSC, b = 0.20/0.25/0.30, L = 0.30/0.40/0.50, and lists EXPOSED PAD VARIATIONS in which T1633-5 is 1.50/1.60/1.70 while T1633-2/-4/-7C are 0.95/1.10/1.25. THAT LOOKED LIKE A CONTRADICTION with a 1.23 mm land and it is not: Maxim land pattern 90-0032 Rev E, titled \"PACKAGE LAND PATTERN, [T1633] 16L TQFN, 3X3 MM\", is issued for PKG CODES [T1633-5], [T1633-5C] AND [T1633-7C] together and specifies ONE land for all three - EP 1.23 x 1.23, perimeter pads 0.80 x 0.30, pitch 0.50, pad centreline span 2.85, IPC-7351A, tolerance +/-0.02. So the land question does not depend on which EP variant the MAX98357AETE+T carries. Numerical comparison with Package_DFN_QFN:TQFN-16-1EP_3x3mm_P0.5mm_EP1.23x1.23mm: EP 1.23 x 1.23 EXACT; pitch 0.50 EXACT; pad INNER edge 1.025 EXACT (so EP-to-signal clearance is Maxim s own 0.410 mm); pad centre 1.4375 vs 1.425 (+0.0125, inside the drawing tolerance); pad length 0.825 vs 0.80 (+0.025 toe); pad WIDTH 0.25 vs 0.30 (-0.05, zero side fillet, but a 0.25 mm pad gap and a safer mask dam at 0.5 mm pitch). NO PROJECT-LOCAL FOOTPRINT IS NEEDED - the two deviations are <= 0.05 mm, IPC-7351B compliant, and both are on the safe side for a first build. EP paste is four 0.5 x 0.5 apertures = 66% coverage, which is correct QFN practice."
+			(at 219.71 80.01 0)
+			(hide yes)
+			(show_name no)
+			(do_not_autoplace no)
+			(effects
+				(font
+					(size 1.27 1.27)
+				)
+			)
+		)
+		(property "LCSC" "C910544"
+			(at 219.71 80.01 0)
+			(hide yes)
+			(show_name no)
+			(do_not_autoplace no)
+			(effects
+				(font
+					(size 1.27 1.27)
+				)
 			)
 		)
@@
 			)
 		)
+		(property "Note2" "SOURCING 2026-08-23 (FBV2-S2-002) (B-71). J4 and J6 are the same JST PH 2-pin header but carried two different MPN strings - J4 the (LF)(SN) plating suffix, J6 the bare code. That was not cosmetic: the bare code is LCSC C20504437 with STOCK 0 while B2B-PH-K-S(LF)(SN) is C131337 with 378913 in stock. Both are now the stocked string. LCSC/JLC library state verified live on 2026-08-23 through the JLCPCB parts API (D-096). Stock is a snapshot, not a guarantee."
+			(at 241.3 110.49 0)
+			(hide yes)
+			(show_name no)
+			(do_not_autoplace no)
+			(effects
+				(font
+					(size 1.27 1.27)
+				)
+			)
+		)
+		(property "LCSC" "C131337"
+			(at 241.3 110.49 0)
+			(hide yes)
+			(show_name no)
+			(do_not_autoplace no)
+			(effects
+				(font
+					(size 1.27 1.27)
+				)
+			)
+		)
 		(property "Manufacturer" "JST"
 			(at 241.3 110.49 0)
@@
 			)
 		)
-		(property "MPN" "B2B-PH-K-S"
+		(property "MPN" "B2B-PH-K-S(LF)(SN)"
 			(at 241.3 110.49 0)
 			(hide yes)
@@
 		)
 		(property "Description" "PUI Audio bottom-port MEMS I2S microphone, 7-pad, 4.0 x 3.0 x 1.0 mm"
+			(at 116.84 81.28 0)
+			(hide yes)
+			(show_name no)
+			(do_not_autoplace no)
+			(effects
+				(font
+					(size 1.27 1.27)
+				)
+			)
+		)
+		(property "Note2" "SOURCING 2026-08-23 (FBV2-S2-002) (B-71). PUI Audio DMM-4026-B-I2S-R is in the LCSC catalogue as C3171792 but STOCK IS 0. Buy from Digi-Key/Mouser and consign - a 7-pad bottom-port MEMS microphone is not a hand-placement candidate. B-63 CLOSED at the same time: see the footprint file, which now carries the acoustic port, the paste pullback and the keepout. LCSC/JLC library state verified live on 2026-08-23 through the JLCPCB parts API (D-096). Stock is a snapshot, not a guarantee."
+			(at 116.84 81.28 0)
+			(hide yes)
+			(show_name no)
+			(do_not_autoplace no)
+			(effects
+				(font
+					(size 1.27 1.27)
+				)
+			)
+		)
+		(property "LCSC" "C3171792"
 			(at 116.84 81.28 0)
 			(hide yes)
@@
 			(at 247.65 140.97 0)
 			(hide yes)
+			(show_name no)
+			(do_not_autoplace no)
+			(effects
+				(font
+					(size 1.27 1.27)
+				)
+			)
+		)
+		(property "LCSC" "C3311653"
+			(at 247.65 140.97 0)
+			(hide yes)
