File: hardware/beta-v2/kicad/aqroot-beta-v2/08_buttons_expanders.kicad_sch (KiCad schematic)
At the start: 26 parts, among them SW2 UP, SW3 DOWN, SW4 LEFT, SW5 RIGHT, SW6 A_SELECT, SW7 B_BACK, SW8 HOME, U2 TCA9535PWR, U3 TCA9535PWR

Commit message: hardware: migrate Full Beta v2 buttons expanders and RGB status
Sheet 08 migrated (FBV2-S1-008), resumed after a session-limit interruption.
All prior work was uncommitted working-tree change; it was inspected, kept and
finished rather than restarted.

Both expanders are NXP PCAL9535APW,118, verified against PCAL9535A Rev. 2
(23-Jan-2015) and NOT treated as a behavioural drop-in: it powers up with every
interrupt masked, the opposite of the TCA9535. U2 = 0x20, U3 = 0x21 preserved.

The two-expander allocation genuinely fails: 35 committed signals against 32
pins, with zero free native GPIO (so the WS2812 escape is impossible),
RESERVED_SPARE mandated by D-094 and ten XGPIO locked by D-082. Closed by U23,
a third PCAL9535APW,118 at 0x22 carrying only the front RGB and the reserved
spare - no new MPN, no new footprint, no new driver, no new rail, and B-37
retired with 12 spare I/O. Core, community and safety functions are placed
before the RGB by construction.

Landed: BQ25185_STAT1/STAT2 (10k pull-ups), SD_CARD_DETECT_N, TOUCH_INT_N,
SX1262_DIO1 on U2; ACC_3V3_EN, ACC_5V_EN, ACC_DETECT_N, ACC_POWER_FAULT_N on
U3. RESERVED_SPARE created on U23 P03 with R130 and TP41 - it had never existed.

Front RGB: D13 MEIHUA MHPA3528RGBCT (LCSC C409779), common anode, R124 1k /
R125 680R / R126 390R = 1.50 / 1.03 / 1.67 mA, white 4.20 mA. Dark by
construction with no external pull-ups.

IR receiver reverted to TSOP38238 (AGC2), TSOP38438 retained as a documented
drop-in fallback. Closes O-5.

Sheets 01 and 03 touched only to promote six local labels to hierarchical so
the required nets could reach the expanders; no component, value, topology or
DNP state changed.

ERC 42 messages / 1 error / 41 warnings - identical violation set to the
recovered tree and better than the 45/2/43 pre-sheet-08 baseline. Zero new
errors. fork_equivalence.py PASS, netclass_probe.py PASS, PCB still
bit-identical to Beta-DM. Sheet 09 untouched.

Co-Authored-By: Claude Opus 5 <noreply@anthropic.com>
Claud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
Parts:
- removed R10: 10k, Resistor_SMD:R_0603_1608Metric, symbol Device:R
- removed R11: 10K, Resistor_SMD:R_0603_1608Metric, symbol Device:R
- removed SW8: HOME, Button_Switch_SMD:SW_SPST_PTS645Sx43SMTR92, symbol Switch:SW_Push
- added C83: 100nF, Capacitor_SMD:C_0603_1608Metric, symbol Device:C
- added D13: MHPA3528RGBCT, AQROOT_Beta:MEIHUA_MHPA3528RGBCT_PLCC4_3.5x2.8mm, symbol AQROOT_Beta:MHPA3528RGBCT
- added R124: 1k, Resistor_SMD:R_0603_1608Metric, symbol Device:R
- added R125: 680R, Resistor_SMD:R_0603_1608Metric, symbol Device:R
- added R126: 390R, Resistor_SMD:R_0603_1608Metric, symbol Device:R
- added R127, R128: 10k, Resistor_SMD:R_0603_1608Metric, symbol Device:R
- added R129, R130: 100k, Resistor_SMD:R_0603_1608Metric, symbol Device:R
- added TP41: TestPoint, TestPoint:TestPoint_Pad_D1.0mm, symbol Connector:TestPoint
- added U23: PCAL9535APW, Package_SO:TSSOP-24_4.4x7.8mm_P0.65mm, symbol AQROOT_Beta:PCAL9535APW
- U2: value TCA9535PWR -> PCAL9535APW; symbol Interface_Expansion:TCA9535PWR -> AQROOT_Beta:PCAL9535APW; I2C_Address (none) -> 0x20; MPN TCA9535PWR -> PCAL9535APW,118; Manufacturer Texas Instruments -> NXP Semiconductors; Note (none) -> FBV2-S1-008: TCA9535PWR -> NXP PCAL9535APW,118. PIN-TO-PIN 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
- U3: value TCA9535PWR -> PCAL9535APW; symbol Interface_Expansion:TCA9535PWR -> AQROOT_Beta:PCAL9535APW; I2C_Address (none) -> 0x21; MPN TCA9535PWR -> PCAL9535APW,118; Manufacturer Texas Instruments -> NXP Semiconductors; Note (none) -> FBV2-S1-008: TCA9535PWR -> NXP PCAL9535APW,118. PIN-TO-PIN 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
Connections:
- net +3V3: now also C83.1, D13.1 (A), R127.1, R128.1, R129.1, R130.1, U23.2 (A1), U23.24 (VCC)
- net GND: now also C83.2, U23.12 (GND), U23.21 (A0), U23.3 (A2)
- net I2C_SCL_INT: now also U23.22 (SCL)
- net I2C_SDA_INT: now also U23.23 (SDA)
- net WAKE_INT_N: now also U23.1 (~{INT})
- net BTN_HOME_N renamed TOUCH_INT_N
- net RGB_B_CTL renamed SD_CARD_DETECT_N
- net RGB_G_CTL renamed BQ25185_STAT2
- net BQ25185_STAT2: now also R128.2
- net RGB_R_CTL renamed BQ25185_STAT1
- net BQ25185_STAT1: now also R127.2
- net ROOTPROBE_IRQ_READY_N renamed SX1262_DIO1
- net XGPIO10 renamed ACC_3V3_EN
- net XGPIO11 renamed ACC_5V_EN
- net XGPIO12 renamed ACC_DETECT_N
- net ACC_DETECT_N: now also R129.2
- net XGPIO13 renamed ACC_POWER_FAULT_N
- new net: D13.2 (BK), R126.2
- new net: D13.3 (GK), R125.2
- new net: D13.4 (RK), R124.2
- new net FRONT_RGB_B_N: R126.1, U23.6 (P02)
- new net FRONT_RGB_G_N: R125.1, U23.5 (P01)
- new net FRONT_RGB_R_N: R124.1, U23.4 (P00)
- new net RESERVED_SPARE: R130.2, TP41.1, U23.7 (P03)
- no-connect marks 0 -> 12
Other:
- note added: "BUTTONS - MIGRATED FBV2-S1-008 SIX BUTTONS: UP, DOWN, LEFT, RIGHT, A/SELECT, B/BACK. HOME (SW8) AND ITS PULL-UP R10 ARE REMOVED - THE SIX-BUTTON SET IS THE LOCKED ONE. VOLUME BUTTONS NEVER EXISTED ELECTRICALLY AND ARE NOT INVENTED HERE. ACTIVE LOW: 10 k EXTERNAL PULL-UP TO +3V3, SWITCH TO GND. THE PULL-UPS STAY EXTERNAL EVEN THOUGH THE PCAL9535A HAS INTERNAL 100 k ONES - 100 k WITH THE PCAL 1 uA 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"
- note added: "EXPANDER INTERRUPTS - FBV2-S1-008 ALL THREE /INT PINS ARE OPEN-DRAIN AND WIRE-OR ONTO WAKE_INT_N, WHICH R3 10 k PULLS TO +3V3 AND WHICH REACHES GPIO21. THE PULL-UP IS MANDATORY - THE DATA SHEET SAYS SO - AND IT IS WHAT MAKES THE LINE DETERMINISTIC (INACTIVE HIGH) BEFORE ANY REGISTER IS WRITTEN. GPIO21 IS NOT A STRAPPING PIN, SO A HELD INTERRUPT CANNOT BLOCK ROM DOWNLOAD. PCAL9535A POWERS UP WITH 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"
- note added: "FRONT RGB STATUS LIGHT - IMPLEMENTED FBV2-S1-008 D13 = MEIHUA MHPA3528RGBCT (LCSC C409779) COMMON ANODE, SMD3528-4P 3.5 x 2.8 x 1.85 mm, 120 deg, WATER CLEAR, 69k IN STOCK, $0.084/2k. PIN 1 = A, 2 = BLUE K, 3 = GREEN K, 4 = RED K. NOTE THIS IS **NOT** Device:LED_ARGB ORDER (THAT SYMBOL HAS 2 = RED, 4 = BLUE). THREE RESISTORS, CALCULATED SEPARATELY FROM THE LOW-CURRENT Fig.4 CURVES - THE TABULATED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"
- note added: "PIN BUDGET - READ THIS BEFORE ADDING ANYTHING TWO PCAL9535A ARE 32 PINS. COMMITTED DEMAND IS 35: 5 SAFE-STATE CONTROL OUTPUTS U2 P00-P04 6 USER BUTTONS U2 P10-P15 5 TRANSITIONAL / TELEMETRY INPUTS TOUCH_INT_N, SX1262_DIO1, SD_CARD_DETECT_N, BQ25185_STAT1, BQ25185_STAT2 10 XGPIO U3, D-082 4 ACCESSORY CONTROL / STATUS U3 P12-P15 1 SX1262_RXEN + 1 ACC_PWR_EN U3 P16/P17 1 RESERVED_SPARE D-094 3 FRONT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"
- note added: "U2 INTERNAL EXPANDER - MIGRATED FBV2-S1-008 NXP PCAL9535APW,118 I2C ADDRESS 0x20 A0 = A1 = A2 = GND PORT 0 = P00-P04 OUT, P05-P07 IN (06h = E0h) PORT 1 = 8 INPUTS (07h = FFh) 16 / 16 USED - ZERO SPARE P00 TOUCH_RST_N OUT ACTIVE LOW P01 SX1262_RST_N OUT ACTIVE LOW P02 NFC_5V_EN OUT ACTIVE HIGH P03 AMP_SD_MODE OUT ACTIVE HIGH P04 DISP_RST_N OUT ACTIVE LOW P05 BQ25185_STAT1 IN R127 10k UP P06 BQ2518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"
- note added: "U23 THIRD EXPANDER - ADDED FBV2-S1-008 NXP PCAL9535APW,118 I2C ADDRESS 0x22 A1 = +3V3, A0 = A2 = GND (0100 010) 0x22 IS FREE: THE INTERNAL BUS HOLDS 0x20 U2, 0x21 U3, 0x36 MAX17048, 0x38 FT6236, 0x68 BMI270. P00 FRONT_RGB_R_N OUT, SINKS 1.50 mA VIA R124 1k P01 FRONT_RGB_G_N OUT, SINKS 1.03 mA VIA R125 680R P02 FRONT_RGB_B_N OUT, SINKS 1.67 mA VIA R126 390R P03 RESERVED_SPARE R130 100k UP + TP41 (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"
- note added: "U3 COMMUNITY EXPANDER - MIGRATED FBV2-S1-008 NXP PCAL9535APW,118 I2C ADDRESS 0x21 A0 = +3V3, A1 = A2 = GND P00-P07 XGPIO0-7 COMMUNITY, BIDIRECTIONAL P10 XGPIO8 P11 XGPIO9 P12 ACC_3V3_EN OUT R98 100k DOWN, SHEET 01 P13 ACC_5V_EN OUT R102 100k DOWN, SHEET 01 P14 ACC_DETECT_N IN R129 100k UP, HERE P15 ACC_POWER_FAULT_N IN R103 100k UP, SHEET 01 P16 SX1262_RXEN OUT R74 PULL-DOWN, SHEET 04 P17 ACC_PWR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"
- note removed: "RGB OUTPUT IMPLEMENTATION PENDING RGB_R_CTL / RGB_G_CTL / RGB_B_CTL LED TYPE, POLARITY, CURRENT RESISTORS AND SAFE-STATE PULL DIRECTION NOT SELECTED DO NOT ROUTE"
- note removed: "U60 INTERNAL EXPANDER I2C ADDRESS 0x20 ARCHITECTURE LOCKED"
- note removed: "U61 COMMUNITY EXPANDER I2C ADDRESS 0x21 ARCHITECTURE LOCKED"

Commit message: hardware: migrate Full Beta v2 community expansion
Sheet 09 migrated (FBV2-S1-009). All nine schematic sheets now carry the Full
Beta v2 architecture and fork_equivalence.py's "still Beta-DM" list is empty.

Three CTO rulings implemented. O-6 ratified: U23, the third PCAL9535APW,118 at
0x22, and the front RGB are locked architecture; B-37 retired with 11 spare
expander pins. O-4 approved: U16 TCA9517A -> TI TCA4307DGKR (LCSC C880333),
FITTED where the old part was DNP. P-18 closed with no I2C mux.

Sheet 09 was rebuilt, not patched, and was hiding two serious defects: J5
contact 1 carried permanent raw +3V3 against D-057, and the community port had
no power at all - 01:ACC_3V3_SW and 09:ACC_3V3_SW were different nets, the
latter fed by a second, DNP TPS22918. Also removed: the 26-pin 2x13 male
header, XGPIO10-13, FAST_IO_GPIO43_HDR, RESERVED_NC. Sixth consecutive sheet
with a load-bearing inherited DNP.

Connector footprint built from the Samtec RECOMMENDED PCB LAYOUT REV B FIG 3:
2.54 mm in row, 7.87 +/-0.05 mm row-to-row, 0.71 mm PTH, 27.94 mm pin field.
All 24 contacts verified pin by pin against D-084.

External I2C pull-ups re-derived: the inherited 4.7k gives 796 ns against a
300 ns fast-mode budget at 200 pF and could never have worked; now 1.5k =
254 ns. Both current limits re-derived rather than copied - 3.3 V stays 1.5k
but the accessory-short case moved 86% -> 89% of the TPS63020's 2 A.

5 V enables split per the CTO refinement: ACC_5V_BOOST_EN on U3 P13 and
ACC_5V_SW_EN on U23 P04, each with its own 100k pull-down. B-08 closed in
copper with Q10, source facing the connector. All six TVS arrays were DNP and
are now fitted; one TPD4E1B06DRLR MPN covers all sixteen exposed contacts.

#FLG0105, deleted by the rebuild, turned out to be the only power-output driver
on the entire GND net and was re-created with a note explaining its role.

ERC 42/1/41 -> 27/0/27 - zero errors for the first time. 321 components, 0
duplicate references, 0 without a footprint, 224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
Connections:
- net ACC_5V_SW_EN: now reaches U23.8 (P04)
- net ACC_5V_EN renamed ACC_5V_BOOST_EN
- no-connect marks 12 -> 11
Other:
- note added: "U3 COMMUNITY EXPANDER - MIGRATED FBV2-S1-008 NXP PCAL9535APW,118 I2C ADDRESS 0x21 A0 = +3V3, A1 = A2 = GND P00-P07 XGPIO0-7 COMMUNITY, BIDIRECTIONAL P10 XGPIO8 P11 XGPIO9 P12 ACC_3V3_EN OUT R98 100k DOWN, SHEET 01 P13 ACC_5V_BOOST_EN OUT R102 100k DOWN, SHEET 01 P14 ACC_DETECT_N IN R129 100k UP, HERE P15 ACC_POWER_FAULT_N IN R103 100k UP, SHEET 01 P16 SX1262_RXEN OUT R74 PULL-DOWN, SHEET 04 P17 A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"
- note removed: "U3 COMMUNITY EXPANDER - MIGRATED FBV2-S1-008 NXP PCAL9535APW,118 I2C ADDRESS 0x21 A0 = +3V3, A1 = A2 = GND P00-P07 XGPIO0-7 COMMUNITY, BIDIRECTIONAL P10 XGPIO8 P11 XGPIO9 P12 ACC_3V3_EN OUT R98 100k DOWN, SHEET 01 P13 ACC_5V_EN OUT R102 100k DOWN, SHEET 01 P14 ACC_DETECT_N IN R129 100k UP, HERE P15 ACC_POWER_FAULT_N IN R103 100k UP, SHEET 01 P16 SX1262_RXEN OUT R74 PULL-DOWN, SHEET 04 P17 ACC_PWR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"

Commit message: hardware: close Full Beta v2 S2 release blockers
Closes B-03, B-63, B-70 and B-71's schematic-side work. Property-only
changes to the nine sheets plus the microphone footprint; ERC unchanged
at 27 / 0 errors / 27 with an identical violation histogram, and the PCB
is untouched and still bit-identical to Beta-DM.

B-03 - all eight remaining Tier-2 footprints compared dimension by
dimension against retrieved manufacturer drawings. Y1 moves from
candidate to lock (Yajingxin TXM27.12M0004322DBBDO00T, C362365, 3421 in
stock) with a land that matches the vendor's Suggested Layout exactly.
The MAX98357A looked like a genuine defect - outline 21-0136 gives
T1633-5 an EP of 1.50/1.60/1.70 while the land is 1.23 - and is not:
land pattern 90-0032 Rev E is issued for T1633-5, -5C and -7C together
and specifies one land for all three, so no project-local footprint was
created.

B-63 - the microphone acoustic port is now drawn rather than described.
1.05 mm NPTH taken from the drawing's own pad-4 ring inner diameter,
paste pulled back 0.10 mm as a declared stencil choice, keepout marked,
bottom-port orientation recorded.

B-70 - L5/L6 lock to Murata LQW18AN39NG80D. The DCR is a first-order
term here: 0.20 ohm max against R_q = 1.1 ohm drops network Q from 25.3
to about 21.4, so the antenna must be tuned with this exact part fitted
and the first lever is R_q, not 39 nH.

B-71 - 65 LCSC fields written in, three MPN strings corrected. J6 and J7
carried bare order codes that resolve to zero-stock listings while the
plating-suffixed strings are abundantly stocked. Six substitution traps
recorded in the symbols themselves, including BAT54W offered for
BAT54WS - a single diode for a series pair - and a clone for the battery
reverse-polarity pass FETs.

Eight DNP parts still carried no recorded reason and now do. The design
has zero unexplained DNP.

Co-Authored-By: Claude Opus 5 <noreply@anthropic.com>
Claude-Session: https://claude.ai/code/session_0133CdFHfKcCH8oPWqJZWe7o
Parts:
- SW2, SW3, SW4, SW5, SW6, SW7: LCSC (none) -> C221880; Note2 (none) -> SOURCING 2026-08-23 (FBV2-S2-002) (B-71). Genuine C&K PTS64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
- U2, U23, U3: LCSC (none) -> C2669683; Note2 (none) -> SOURCING 2026-08-23 (FBV2-S2-002) (B-71) - FIRST-BUILD BLOC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
Changed lines of the file:
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@@
 			)
 		)
+		(property "Note2" "SOURCING 2026-08-23 (FBV2-S2-002) (B-71). Genuine C&K PTS645SM43SMTR92LFS is LCSC C221880, stock 8432. A loose keyword search returns G-Switch GT-TC089A-H043-L1 (C843623) instead - a DIFFERENT MANUFACTURER whose land pattern has not been checked against the C&K G-Type layout this footprint was built from. Seven buttons per board is 35 placements for the first five; do not let a search shortcut swap them. LCSC/JLC library state verified live on 2026-08-23 through the JLCPCB parts API (D-096). Stock is a snapshot, not a guarantee."
+			(at 125.73 153.67 0)
+			(hide yes)
+			(show_name no)
+			(do_not_autoplace no)
+			(effects
+				(font
+					(size 1.27 1.27)
+				)
+			)
+		)
+		(property "LCSC" "C221880"
+			(at 125.73 153.67 0)
+			(hide yes)
+			(show_name no)
+			(do_not_autoplace no)
+			(effects
+				(font
+					(size 1.27 1.27)
+				)
+			)
+		)
 		(property "Manufacturer" "C&K / Littelfuse"
 			(at 125.73 153.67 0)
@@
 			)
 		)
+		(property "Note2" "SOURCING 2026-08-23 (FBV2-S2-002) (B-71). Genuine C&K PTS645SM43SMTR92LFS is LCSC C221880, stock 8432. A loose keyword search returns G-Switch GT-TC089A-H043-L1 (C843623) instead - a DIFFERENT MANUFACTURER whose land pattern has not been checked against the C&K G-Type layout this footprint was built from. Seven buttons per board is 35 placements for the first five; do not let a search shortcut swap them. LCSC/JLC library state verified live on 2026-08-23 through the JLCPCB parts API (D-096). Stock is a snapshot, not a guarantee."
+			(at 102.87 153.67 0)
+			(hide yes)
+			(show_name no)
+			(do_not_autoplace no)
+			(effects
+				(font
+					(size 1.27 1.27)
+				)
+			)
+		)
+		(property "LCSC" "C221880"
+			(at 102.87 153.67 0)
+			(hide yes)
+			(show_name no)
+			(do_not_autoplace no)
+			(effects
+				(font
+					(size 1.27 1.27)
+				)
+			)
+		)
 		(property "Manufacturer" "C&K / Littelfuse"
 			(at 102.87 153.67 0)
@@
 			)
 		)
+		(property "Note2" "SOURCING 2026-08-23 (FBV2-S2-002) (B-71) - FIRST-BUILD BLOCKER. NXP PCAL9535APW,118 is LCSC C2669683 with STOCK 1 against a need of FIFTEEN (three per board, five boards). This part cannot be JLC-turnkey-sourced today. Buy fifteen plus spares from a broadline distributor and CONSIGN them to JLC so they stay MACHINE-PLACED - a TSSOP-24 at 0.65 mm pitch, fifteen times, is not a hand-assembly job. LCSC/JLC library state verified live on 2026-08-23 through the JLCPCB parts API (D-096). Stock is a snapshot, not a guarantee."
+			(at 167.64 74.93 0)
+			(hide yes)
+			(show_name no)
+			(do_not_autoplace no)
+			(effects
+				(font
+					(size 1.27 1.27)
+				)
+			)
+		)
+		(property "LCSC" "C2669683"
+			(at 167.64 74.93 0)
+			(hide yes)
+			(show_name no)
+			(do_not_autoplace no)
+			(effects
+				(font
+					(size 1.27 1.27)
+				)
+			)
+		)
 		(property "Manufacturer" "NXP Semiconductors"
 			(at 194.31 100.33 0)
@@
 			)
 		)
+		(property "Note2" "SOURCING 2026-08-23 (FBV2-S2-002) (B-71) - FIRST-BUILD BLOCKER. NXP PCAL9535APW,118 is LCSC C2669683 with STOCK 1 against a need of FIFTEEN (three per board, five boards). This part cannot be JLC-turnkey-sourced today. Buy fifteen plus spares from a broadline distributor and CONSIGN them to JLC so they stay MACHINE-PLACED - a TSSOP-24 at 0.65 mm pitch, fifteen times, is not a hand-assembly job. LCSC/JLC library state verified live on 2026-08-23 through the JLCPCB parts API (D-096). Stock is a snapshot, not a guarantee."
+			(at 82.55 74.93 0)
+			(hide yes)
+			(show_name no)
+			(do_not_autoplace no)
+			(effects
+				(font
+					(size 1.27 1.27)
+				)
+			)
+		)
+		(property "LCSC" "C2669683"
+			(at 82.55 74.93 0)
+			(hide yes)
+			(show_name no)
+			(do_not_autoplace no)
+			(effects
+				(font
+					(size 1.27 1.27)
+				)
+			)
+		)
 		(property "Manufacturer" "NXP Semiconductors"
 			(at 109.22 100.33 0)
@@
 			)
 		)
+		(property "Note2" "SOURCING 2026-08-23 (FBV2-S2-002) (B-71). Genuine C&K PTS645SM43SMTR92LFS is LCSC C221880, stock 8432. A loose keyword search returns G-Switch GT-TC089A-H043-L1 (C843623) instead - a DIFFERENT MANUFACTURER whose land pattern has not been checked against the C&K G-Type layout this footprint was built from. Seven buttons per board is 35 placements for the first five; do not let a search shortcut swap them. LCSC/JLC library state verified live on 2026-08-23 through the JLCPCB parts API (D-096). Stock is a snapshot, not a guarantee."
+			(at 148.59 153.67 0)
+			(hide yes)
+			(show_name no)
+			(do_not_autoplace no)
+			(effects
+				(font
+					(size 1.27 1.27)
+				)
+			)
+		)
+		(property "LCSC" "C221880"
+			(at 148.59 153.67 0)
+			(hide yes)
+			(show_name no)
+			(do_not_autoplace no)
+			(effects
+				(font
+					(size 1.27 1.27)
+				)
+			)
+		)
 		(property "Manufacturer" "C&K / Littelfuse"
 			(at 148.59 153.67 0)
@@
 			)
 		)
+		(property "Note2" "SOURCING 2026-08-23 (FBV2-S2-002) (B-71). Genuine C&K PTS645SM43SMTR92LFS is LCSC C221880, stock 8432. A loose keyword search returns G-Switch GT-TC089A-H043-L1 (C843623) instead - a DIFFERENT MANUFACTURER whose land pattern has not been checked against the C&K G-Type layout this footprint was built from. Seven buttons per board is 35 placements for the first five; do not let a search shortcut swap them. LCSC/JLC library state verified live on 2026-08-23 through the JLCPCB parts API (D-096). Stock is a snapshot, not a guarantee."
+			(at 82.55 153.67 0)
+			(hide yes)
+			(show_name no)
+			(do_not_autoplace no)
+			(effects
+				(font
+					(size 1.27 1.27)
+				)
+			)
+		)
+		(property "LCSC" "C221880"
+			(at 82.55 153.67 0)
+			(hide yes)
+			(show_name no)
+			(do_not_autoplace no)
+			(effects
+				(font
+					(size 1.27 1.27)
+				)
+			)
+		)
 		(property "Manufacturer" "C&K / Littelfuse"
 			(at 82.55 153.67 0)
@@
 			)
 		)
+		(property "Note2" "SOURCING 2026-08-23 (FBV2-S2-002) (B-71). Genuine C&K PTS645SM43SMTR92LFS is LCSC C221880, stock 8432. A loose keyword search returns G-Switch GT-TC089A-H043-L1 (C843623) instead - a DIFFERENT MANUFACTURER whose land pattern has not been checked against the C&K G-Type layout this footprint was built from. Seven buttons per board is 35 placements for the first five; do not let a search shortcut swap them. LCSC/JLC library state verified live on 2026-08-23 through the JLCPCB parts API (D-096). Stock is a snapshot, not a guarantee."
+			(at 38.1 153.67 0)
+			(hide yes)
+			(show_name no)
+			(do_not_autoplace no)
+			(effects
+				(font
+					(size 1.27 1.27)
+				)
+			)
+		)
+		(property "LCSC" "C221880"
+			(at 38.1 153.67 0)
+			(hide yes)
+			(show_name no)
+			(do_not_autoplace no)
+			(effects
+				(font
+					(size 1.27 1.27)
+				)
+			)
+		)
 		(property "Manufacturer" "C&K / Littelfuse"
 			(at 38.1 153.67 0)
@@
 			)
 		)
+		(property "Note2" "SOURCING 2026-08-23 (FBV2-S2-002) (B-71). Genuine C&K PTS645SM43SMTR92LFS is LCSC C221880, stock 8432. A loose keyword search returns G-Switch GT-TC089A-H043-L1 (C843623) instead - a DIFFERENT MANUFACTURER whose land pattern has not been checked against the C&K G-Type layout this footprint was built from. Seven buttons per board is 35 placements for the first five; do not let a search shortcut swap them. LCSC/JLC library state verified live on 2026-08-23 through the JLCPCB parts API (D-096). Stock is a snapshot, not a guarantee."
+			(at 59.69 153.67 0)
+			(hide yes)
+			(show_name no)
+			(do_not_autoplace no)
+			(effects
+				(font
+					(size 1.27 1.27)
+				)
+			)
+		)
+		(property "LCSC" "C221880"
+			(at 59.69 153.67 0)
+			(hide yes)
+			(show_name no)
+			(do_not_autoplace no)
+			(effects
+				(font
+					(size 1.27 1.27)
+				)
+			)
+		)
 		(property "Manufacturer" "C&K / Littelfuse"
 			(at 59.69 153.67 0)
@@
 			(at 200.66 250.19 0)
 			(hide yes)
+			(show_name no)
+			(do_not_autoplace no)
+			(effects
+				(font
+					(size 1.27 1.27)
+				)
+			)
+		)
+		(property "Note2" "SOURCING 2026-08-23 (FBV2-S2-002) (B-71) - FIRST-BUILD BLOCKER. NXP PCAL9535APW,118 is LCSC C2669683 with STOCK 1 against a need of FIFTEEN (three per board, five boards). This part cannot be JLC-turnkey-sourced today. Buy fifteen plus spares from a broadline distributor and CONSIGN them to JLC so they stay MACHINE-PLACED - a TSSOP-24 at 0.65 mm pitch, fifteen times, is not a hand-assembly job. LCSC/JLC library state verified live on 2026-08-23 through the JLCPCB parts API (D-096). Stock is a snapshot, not a guarantee."
+			(at 200.66 250.19 0)
+			(hide yes)
+			(show_name no)
+			(do_not_autoplace no)
+			(effects
+				(font
+					(size 1.27 1.27)
+				)
+			)
+		)
+		(property "LCSC" "C2669683"
+			(at 200.66 250.19 0)
+			(hide yes)
