File: hardware/beta-v2/kicad/aqroot-beta-v2/01_power_tree.kicad_sch (KiCad schematic)
At the start: 136 parts, among them J3 USB_C_Receptacle_USB2.0_16P, J4 JST-PH-2 BATTERY, Q2 NTMD4820N, Q3 NTMD4820N, Q4 BSS138, Q5 AO3401A, Q6 BSS138, Q7 BSS138, Q8 BSS138, Q9 BSS138, SW9 SW_SPDT, U10 USBLC6-2SC6, U11 BQ25185, U12 TPS63020, U13 TPS61023, U14 MAX17048, U18 LTC4368-1, U19 TLV7032, U20 TPS22950C, U21 TPS61023, U22 TPS22950C

Commit message: hardware: migrate Full Beta v2 MCU core (FBV2-S1-002)
Closes the two power-tree values the CTO ruled on and migrates 02_MCU_CORE.
Task gate FBV2-S1-MCU-CORE = PASS. FBV2-S1 itself is 2 of 9 sheets.

P-20 - R95 680R -> 560R. Recovery recomputed from the captured circuit:
8.36 mA nominal at VBUS 5.0 V into a 0 V pack, 7.93-8.80 mA across 4.75-5.25 V,
back inside the accepted 5-10 mA band that B-26 is measured against.

The recomputation also showed that 680R was NOT arbitrary:
(5.00 - 0.32 + 4.2) / 680 = 13.06 mA is exactly B-27's recorded ~13 mA
single-fault ceiling. With 560R that ceiling becomes ~15.9 mA nominal and
~16.6 mA worst case - 0.0066 C on a 2500 mAh pack, still bounded by R95, still
unidirectional through D12, still self-annunciating. B-27 is amended in place
rather than left reading a number that is no longer true. The trade is explicit:
~21% more recovery current for ~22% more single-fault current.

P-21 - the OV trip is derived, not typed. The datasheet threshold was fetched
first (LTC4368, Farnell mirror 2243878): V_OV 492.5 / 500 / 507.5 mV rising,
hysteresis 20 / 25 / 32 mV, UV/OV leakage 10 nA max, "Adjustable +/-1.5%".
R77 4.02M -> 3.65M 1%, R78 unchanged at 442k:
0.500 x (3.65M + 442k) / 442k = 4.629 V.
Nominal 4.63 V; 4.48-4.78 V over comparator and 1% resistor tolerance;
4.44-4.82 V including worst-case OV pin leakage; release 4.40 V nominal.
Above a 4.35 V-class pack with 129 mV of worst-case margin, 420 mV below the
5.05 V first capture, and no lockout hazard because release sits above float.
3.65M is already R91's value, so this REMOVES a BOM line.

02_MCU_CORE migrated:

- GPIO38 = NATIVE_A and GPIO47 = NATIVE_B, both hierarchical and bidirectional.
  SX1262_DIO1 no longer reaches the MCU at all; under D-089 it terminates on the
  internal expander U2, which is sheet 08.
- GPIO46 = DISP_BL_CTL. GPIO46 is a strapping pin that MUST read LOW at reset -
  GPIO0 = 0 alone does not select Joint Download Boot, GPIO46 = 0 is also
  required. Three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
Parts:
- R77: value 4.02M 1% -> 3.65M 1%
- R95: value 680R 1% 1206 -> 560R 1% 1206
Other:
- note added: "LTC4368-1 ONLY (the -2 trips at -3 mV and blocks charging). RETRY grounded = latch-off; SHDN toggled low-then-high clears it. UV unused: 510k to VIN per datasheet (V_UV/V_OV = 492.5 / 500 / 507.5 mV, hysteresis 20 / 25 / 32 mV). OV TRIP (P-21, D-104): R77 3.65M / R78 442k -> 4.63 V nominal, 4.48-4.78 V over comparator + 1% resistor tolerance. Release 4.40 V nominal. Above a 4.35 V-class pack, wel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"
- note added: "Q6/Q7/Q8 in series form the AND. Q9 inverts FAULT (active-low) so FAULT-ASSERTED becomes a positive enable. Recovery current = (VBUS - Vf) / R95; single-fault ceiling into a reversed cell = (VBUS - Vf + 4.2) / R95. R95 = 560R LOCKED (P-20, D-105): 8.4 mA nominal at VBUS 5.0 V into a 0 V pack (7.9-8.9 mA over 4.75-5.25 V), inside the accepted 5-10 mA band. Single-fault ceiling rises to 15.9 mA nom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"
- note removed: "LTC4368-1 ONLY (the -2 trips at -3 mV and blocks charging). RETRY grounded = latch-off; SHDN toggled low-then-high clears it. UV unused: 510k to VIN per datasheet. VALUE TO VERIFY items are marked in the audit."
- note removed: "Q6/Q7/Q8 in series form the AND. Q9 inverts FAULT (active-low) so FAULT-ASSERTED becomes a positive enable. Recovery current = (VBUS - Vf) / R95; single-fault ceiling into a reversed cell = (VBUS - Vf + 4.2) / R95."
Changed lines of the file:
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@@
 		)
 	)
-	(text "LTC4368-1 ONLY (the -2 trips at -3 mV and blocks charging). RETRY grounded = latch-off; SHDN toggled low-then-high clears it. UV unused: 510k to VIN per datasheet. VALUE TO VERIFY items are marked in the audit."
+	(text "LTC4368-1 ONLY (the -2 trips at -3 mV and blocks charging). RETRY grounded = latch-off; SHDN toggled low-then-high clears it. UV unused: 510k to VIN per datasheet (V_UV/V_OV = 492.5 / 500 / 507.5 mV, hysteresis 20 / 25 / 32 mV).\nOV TRIP (P-21, D-104): R77 3.65M / R78 442k -> 4.63 V nominal, 4.48-4.78 V over comparator + 1% resistor tolerance. Release 4.40 V nominal. Above a 4.35 V-class pack, well below the 5.05 V first capture."
 		(exclude_from_sim no)
 		(at 20 239.5 0)
@@
 			)
 		)
-		(property "Value" "4.02M 1%"
+		(property "Value" "3.65M 1%"
 			(at 210.28 257.25 0)
 			(show_name no)
@@
 		)
 	)
-	(text "Q6/Q7/Q8 in series form the AND. Q9 inverts FAULT (active-low) so FAULT-ASSERTED becomes a positive enable. Recovery current = (VBUS - Vf) / R95; single-fault ceiling into a reversed cell = (VBUS - Vf + 4.2) / R95."
+	(text "Q6/Q7/Q8 in series form the AND. Q9 inverts FAULT (active-low) so FAULT-ASSERTED becomes a positive enable. Recovery current = (VBUS - Vf) / R95; single-fault ceiling into a reversed cell = (VBUS - Vf + 4.2) / R95.\nR95 = 560R LOCKED (P-20, D-105): 8.4 mA nominal at VBUS 5.0 V into a 0 V pack (7.9-8.9 mA over 4.75-5.25 V), inside the accepted 5-10 mA band. Single-fault ceiling rises to 15.9 mA nominal / 16.6 mA worst case - B-27 restated, still ~0.007 C."
 		(exclude_from_sim no)
 		(at 20 332.5 0)
@@
 			)
 		)
-		(property "Value" "680R 1% 1206"
+		(property "Value" "560R 1% 1206"
 			(at 175.99 381.71 0)
 			(show_name no)

Commit message: hardware: migrate Full Beta v2 radios and NFC (FBV2-S1-004)
Sheet 04. Task gate FBV2-S1-RADIOS-NFC = PASS. FBV2-S1 itself is 4 of 9 sheets.

ERC: 4 errors -> 2. Total 86 -> 68. Zero added, eighteen removed. This is the
first migration task to REDUCE the project's error count, and it did so by
deleting placeholder architecture rather than by suppressing anything.

ZERO *_TBD NETS REMAIN ANYWHERE IN THE PROJECT. Sheet 04 alone retired fourteen.

RF ARCHITECTURE LOCKED (D-118).
433 MHz: INTERNAL flex. U7 IPEX -> 100 mm coax -> Taoglas FXP450.07.0100C against
a plastic wall. 915 MHz: EXTERNAL. U8 IPEX -> short pigtail -> top-panel SMA
female bulkhead, user-changeable. Neither band has a motherboard 50 ohm RF trace,
a matching network, an RF switch or a diplexer - both modules present their own
matched 50 ohm port, so the board's RF involvement at 433/915 is zero copper.
This supersedes the internal-FXP890 plan for 915 in "12 - RF and Antenna Plan".
The U7 IPEX socket must remain SERVICE-ACCESSIBLE with the shell open: if
internal 433 performance disappoints on the first units the flex unplugs and an
external pigtail replaces it with no PCB respin. That is an FBV2-P1 placement
constraint and the reason an internal antenna is an acceptable first-build risk.

433 ANTENNA VERIFIED, MATING PROVEN RATHER THAN ASSUMED (D-119). Taoglas
datasheet SPE-23-8-180-A, verbatim: "410-470MHz Flexible PCB Antenna with 100mm
1.37 IPEX MHFI". 47 x 17 x 0.28 mm, adhesive mount, gain -0.36 / -1.57 /
-0.05 dBi, Active, 54 in stock, $5.52 @ 1, MOQ 1. The antenna terminates in IPEX
MHF I and Ebyte's manual lists the E07-400M10S interface as IPEX-1 / stamp hole;
MHF I, IPEX-1 and U.FL are one mating interface, so no cable variant is needed.
Mechanical reservation recorded for FBV2-P1: plastic wall, LEFT/LOWER-SIDE, NOT
on the PCB, clear of the LiPo, the NFC loop and ferrite, the speaker magnet,
large ground pours, metal bosses, the USB shell, the 915 bulkhead/pigtail and the
IR structures.

915 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
Changed lines of the file:
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@@
 		)
 	)
-	(hierarchical_label "NFC_5V_PA_PENDING"
-		(shape output)
+	(label "NFC_5V_PA_PENDING"
 		(at 147.32 168.91 0)
 		(effects
@@
 				(size 1.27 1.27)
 			)
-			(justify left)
+			(justify left bottom)
 		)
 	)
@@
 		)
 	)
-	(label "NFC_SUPPLY"
+	(hierarchical_label "NFC_SUPPLY"
+		(shape output)
 		(at 488.95 400.05 0)
 		(fields_autoplaced yes)
@@
 				(size 1.0 1.0)
 			)
-			(justify left bottom)
+			(justify left)
 		)
 	)
@@
 					(unit 1)
 				)
+			)
+		)
+	)
+	(wire
+		(pts
+			(xy 527.05 396.24) (xy 527.05 400.05)
+		)
+		(stroke
+			(width 0)
+			(type default)
+		)
+	)
+	(label "NFC_SUPPLY"
+		(at 527.05 400.05 0)
+		(effects
+			(font
+				(size 1.27 1.27)
+			)
+			(justify left bottom)
+		)
+	)
+	(symbol
+		(lib_id "power:PWR_FLAG")
+		(at 527.05 396.24 0)
+		(unit 1)
+		(body_style 1)
+		(exclude_from_sim no)
+		(in_bom yes)
+		(on_board yes)
+		(in_pos_files yes)
+		(dnp no)
+		(fields_autoplaced yes)
+		(property "Reference" "#FLG614"
+			(at 529.5899999999999 394.97 0)
+			(show_name no)
+			(do_not_autoplace no)
+			(effects
+				(font
+					(size 1.27 1.27)
+				)
+				(justify left)
+			)
+		)
+		(property "Value" "PWR_FLAG"
+			(at 529.5899999999999 397.51 0)
+			(show_name no)
+			(do_not_autoplace no)
+			(effects
+				(font
+					(size 1.27 1.27)
+				)
+				(justify left)
+			)
+		)
+		(property "Footprint" ""
+			(at 527.05 396.24 0)
+			(hide yes)
+			(show_name no)
+			(do_not_autoplace no)
+			(effects
+				(font
+					(size 1.27 1.27)
+				)
+			)
+		)
+		(property "Datasheet" ""
+			(at 527.05 396.24 0)
+			(hide yes)
+			(show_name no)
+			(do_not_autoplace no)
+			(effects
+				(font
+					(size 1.27 1.27)
+				)
+			)
+		)
+		(property "Description" ""
+			(at 527.05 396.24 0)
+			(hide yes)
+			(show_name no)
+			(do_not_autoplace no)
+			(effects
+				(font
+					(size 1.27 1.27)
+				)
+			)
+		)
+		(pin "1"
+		)
+		(instances
+			(project "aqroot-Beta-v2"
+				(path "/8a0ad1ee-a49e-4cff-9a78-44823e373405/83b1880a-0a3b-496a-bce6-0dc4c72d8ece"
+					(reference "#FLG614")
+					(unit 1)
+				)

Commit message: hardware: migrate Full Beta v2 buttons expanders and RGB status
Sheet 08 migrated (FBV2-S1-008), resumed after a session-limit interruption.
All prior work was uncommitted working-tree change; it was inspected, kept and
finished rather than restarted.

Both expanders are NXP PCAL9535APW,118, verified against PCAL9535A Rev. 2
(23-Jan-2015) and NOT treated as a behavioural drop-in: it powers up with every
interrupt masked, the opposite of the TCA9535. U2 = 0x20, U3 = 0x21 preserved.

The two-expander allocation genuinely fails: 35 committed signals against 32
pins, with zero free native GPIO (so the WS2812 escape is impossible),
RESERVED_SPARE mandated by D-094 and ten XGPIO locked by D-082. Closed by U23,
a third PCAL9535APW,118 at 0x22 carrying only the front RGB and the reserved
spare - no new MPN, no new footprint, no new driver, no new rail, and B-37
retired with 12 spare I/O. Core, community and safety functions are placed
before the RGB by construction.

Landed: BQ25185_STAT1/STAT2 (10k pull-ups), SD_CARD_DETECT_N, TOUCH_INT_N,
SX1262_DIO1 on U2; ACC_3V3_EN, ACC_5V_EN, ACC_DETECT_N, ACC_POWER_FAULT_N on
U3. RESERVED_SPARE created on U23 P03 with R130 and TP41 - it had never existed.

Front RGB: D13 MEIHUA MHPA3528RGBCT (LCSC C409779), common anode, R124 1k /
R125 680R / R126 390R = 1.50 / 1.03 / 1.67 mA, white 4.20 mA. Dark by
construction with no external pull-ups.

IR receiver reverted to TSOP38238 (AGC2), TSOP38438 retained as a documented
drop-in fallback. Closes O-5.

Sheets 01 and 03 touched only to promote six local labels to hierarchical so
the required nets could reach the expanders; no component, value, topology or
DNP state changed.

ERC 42 messages / 1 error / 41 warnings - identical violation set to the
recovered tree and better than the 45/2/43 pre-sheet-08 baseline. Zero new
errors. fork_equivalence.py PASS, netclass_probe.py PASS, PCB still
bit-identical to Beta-DM. Sheet 09 untouched.

Co-Authored-By: Claude Opus 5 <noreply@anthropic.com>
Claud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
Changed lines of the file:
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@@
 		)
 	)
-	(label "BQ25185_STAT1"
+	(hierarchical_label "BQ25185_STAT1"
+		(shape output)
 		(at 73.66 107.95 0)
 		(effects
@@
 				(size 1.27 1.27)
 			)
-			(justify left bottom)
+			(justify left)
 		)
 	)
@@
 		)
 	)
-	(label "BQ25185_STAT2"
+	(hierarchical_label "BQ25185_STAT2"
+		(shape output)
 		(at 73.66 110.49 0)
 		(effects
@@
 				(size 1.27 1.27)
 			)
-			(justify left bottom)
+			(justify left)
 		)
 	)
@@
 		)
 	)
-	(label "ACC_3V3_EN"
+	(hierarchical_label "ACC_3V3_EN"
+		(shape input)
 		(at 441.96 254.0 0)
-		(fields_autoplaced yes)
 		(effects
 			(font
 				(size 1.0 1.0)
 			)
-			(justify left bottom)
+			(justify left)
 		)
 	)
@@
 		)
 	)
-	(label "ACC_POWER_FAULT_N"
+	(hierarchical_label "ACC_POWER_FAULT_N"
+		(shape output)
 		(at 378.46 284.48 0)
-		(fields_autoplaced yes)
 		(effects
 			(font
 				(size 1.0 1.0)
 			)
-			(justify left bottom)
+			(justify left)
 		)
 	)
@@
 		)
 	)
-	(label "ACC_5V_EN"
+	(hierarchical_label "ACC_5V_EN"
+		(shape input)
 		(at 532.13 340.36 0)
-		(fields_autoplaced yes)
 		(effects
 			(font
 				(size 1.0 1.0)
 			)
-			(justify left bottom)
+			(justify left)
 		)
 	)

Commit message: hardware: migrate Full Beta v2 community expansion
Sheet 09 migrated (FBV2-S1-009). All nine schematic sheets now carry the Full
Beta v2 architecture and fork_equivalence.py's "still Beta-DM" list is empty.

Three CTO rulings implemented. O-6 ratified: U23, the third PCAL9535APW,118 at
0x22, and the front RGB are locked architecture; B-37 retired with 11 spare
expander pins. O-4 approved: U16 TCA9517A -> TI TCA4307DGKR (LCSC C880333),
FITTED where the old part was DNP. P-18 closed with no I2C mux.

Sheet 09 was rebuilt, not patched, and was hiding two serious defects: J5
contact 1 carried permanent raw +3V3 against D-057, and the community port had
no power at all - 01:ACC_3V3_SW and 09:ACC_3V3_SW were different nets, the
latter fed by a second, DNP TPS22918. Also removed: the 26-pin 2x13 male
header, XGPIO10-13, FAST_IO_GPIO43_HDR, RESERVED_NC. Sixth consecutive sheet
with a load-bearing inherited DNP.

Connector footprint built from the Samtec RECOMMENDED PCB LAYOUT REV B FIG 3:
2.54 mm in row, 7.87 +/-0.05 mm row-to-row, 0.71 mm PTH, 27.94 mm pin field.
All 24 contacts verified pin by pin against D-084.

External I2C pull-ups re-derived: the inherited 4.7k gives 796 ns against a
300 ns fast-mode budget at 200 pF and could never have worked; now 1.5k =
254 ns. Both current limits re-derived rather than copied - 3.3 V stays 1.5k
but the accessory-short case moved 86% -> 89% of the TPS63020's 2 A.

5 V enables split per the CTO refinement: ACC_5V_BOOST_EN on U3 P13 and
ACC_5V_SW_EN on U23 P04, each with its own 100k pull-down. B-08 closed in
copper with Q10, source facing the connector. All six TVS arrays were DNP and
are now fitted; one TPD4E1B06DRLR MPN covers all sixteen exposed contacts.

#FLG0105, deleted by the rebuild, turned out to be the only power-output driver
on the entire GND net and was re-created with a note explaining its role.

ERC 42/1/41 -> 27/0/27 - zero errors for the first time. 321 components, 0
duplicate references, 0 without a footprint, 224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
Parts:
- added R131: 100k, Resistor_SMD:R_0603_1608Metric, symbol Device:R
- added TP47: TestPoint, TestPoint:TestPoint_Pad_D1.0mm, symbol Connector:TestPoint
Connections:
- net GND: now also R131.2
- net ACC_5V_EN renamed ACC_5V_BOOST_EN
- net ACC_5V_BOOST_EN: no longer U22.1 (ON)
- new net ACC_5V_SW_EN: R131.1, TP47.1, U22.1 (ON)

Commit message: hardware: close Full Beta v2 pre-placement schematic issues
FBV2-S2-001 pre-placement release audit. The audit found a fabrication-blocking
defect on the first thing it looked at.

U9 ST25R3916-AQET and its twelve mandatory supply-decoupling capacitors (C19,
C45-C55) were still marked DNP, inherited from Beta-DM, against D-035 ("NFC is
mandatory in the FIRST Full Beta v2 fabrication. No DNP showcase shortcut") and
D-055 ("NFC must be FITTED and functional on the first fabrication"). Everything
around the chip was already fitted - the 27.12 MHz crystal, the complete
differential matching network, the antenna connector, the SPI wiring. The first
five boards would have carried a finished 13.56 MHz front end with no NFC chip
on it. All thirteen parts are now FIT. Seventh consecutive sheet with a
load-bearing inherited DNP.

Six missing MPNs added: D9 -> PMEG2010AEH,115 and Q4/Q6-Q9 -> BSS138LT1G. Every
active and every connector now carries an exact MPN.

Two undocumented placeholders resolved. R68 is a 0R DNP bypass across SW9, the
hard power switch - fitting it wires the unit permanently ON and defeats the
only way to power down a hung or unflashed board; it is now marked DNP AND IT
MUST STAY DNP. C21/C22 are dead pads with one terminal no-connect flagged.

Two stale "FOOTPRINT STILL BLOCKED" notes on L1 and L2 withdrawn - both land
patterns had already been built from the manufacturer drawings. L1 and L4
headroom recorded: 1.4x and 2.8x on Isat, which closes B-68.

16 DNP parts remain and every one is documented. Zero unexplained DNP.

ERC 27 / 0 errors / 27, unchanged. 0 duplicate references, 0 unresolved
footprint references, 0 orphan nets, 0 *_TBD. fork_equivalence.py PASS,
netclass_probe.py PASS. PCB untouched and still bit-identical to Beta-DM. No
PCB placement or routing was started.

Co-Authored-By: Claude Opus 5 <noreply@anthropic.com>
Claude-Session: https://claude.ai/code/session_0133CdFHfKcCH8oPWqJZWe7o
Parts:
- C21, C22: Note (none) -> FBV2-S2-001: **DEAD PAD - DNP, AND ONE TERMINAL IS DELIBERA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
- D9: MPN (none) -> PMEG2010AEH,115; Manufacturer (none) -> Nexperia; Note SECONDARY clamp only - P2 isolation is the primary defence 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 -> FBV2-S2-001: exact order code added - the schematic previou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
- L1: Note Coilcraft doc 745-1 rev 03/10/26: 1.5 uH +/-20%; DCR 14.40 mOhm typ / 15.80 max; SRF 59 MHz typ; Isat 4.1 A (10% drop) / 4.4 A (20%) / 4.6 A (30%); Irms 6.7 A (20K rise) / 9.1 A (40K). Body 4.0 x 4.0 mm +/-0.3, height 2.10 mm max, terminals 0.82 x 1.57 mm. LCSC C3033018. Coilcraft marks the start (short) lead - connect high dv/dt there for lowest EMI; the footprint must carry that orientation marker. FOOTPRINT STILL BLOCKED: the recommended land pattern prints 0.98 / 2.37 / 3.4 mm but text extraction does not reveal which dimension is the span, so pad centres cannot be fixed without reading the drawing. -> Coilcraft doc 745-1 rev 03/10/26: 1.5 uH +/-20%; DCR 14.40 mOhm typ / 15.80 max; SRF 59 MHz typ; Isat 4.1 A (10% drop) / 4.4 A (20%) / 4.6 A (30%); Irms 6.7 A (20K rise) / 9.1 A (40K). Body 4.0 x 4.0 mm +/-0.3, height 2.10 mm max, terminals 0.82 x 1.57 mm. LCSC C3033018. Coilcraft marks the start (short) lead - connect high dv/dt there for lowest EMI, and the footprint carries that orientation marker. **FBV2-S2-001: THE 'FOOTPRINT STILL BLOCKED' NOTE THAT USED TO SIT HERE IS STALE AND IS WITHDRAWN.** The land pattern was subsequently built from Coilcraft document 745-3 rev 03/10/26 'Recommended Land Pattern' with the dimensions read off the drawing leader lines rather than inferred from text order: pad 0.98 mm wide x 3.4 mm long at 2.37 mm centre-to-centre. **HEADROOM CHECK, FBV2-S2-001:** at the TPS63020 worst case - 2 A out of 3.3 V from a 3.0 V cell - the average inductor current is about 2.44 A and the peak about 2.9 A, against Isat 4.1 A at the 10 % inductance-drop point. That is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
- L2: Note Wurth datasheet for 74438357010 (WE-MAPI 4030): 1 uH +/-20%; RDC 11.6 mOhm typ / 13.5 max; Isat 6.2 A (10% drop) / 12.5 A (30%); IRP,40K 10.25 A max; fres 59 MHz. Body 4.1 x 4.1 mm +/-0.2, height 3.1 mm max. Marked with start-of-winding. These ratings supersede the earlier 'take from datasheet' placeholder and satisfy the outstanding check that L2 be rated for the TI TPS61023 5V boost. FOOTPRINT STILL BLOCKED: recommended land pattern prints 1.39 / 3.35 / 3.7 mm but which is the span is not recoverable from text; prefer Wurth's own EDA/KiCad asset. -> Wurth datasheet for 74438357010 (WE-MAPI 4030): 1 uH +/-20%; RDC 11.6 mOhm typ / 13.5 max; Isat 6.2 A (10% drop) / 12.5 A (30%); IRP,40K 10.25 A max; fres 59 MHz. Body 4.1 x 4.1 mm +/-0.2, height 3.1 mm max. Marked with start-of-winding. **FBV2-S2-001: THE 'FOOTPRINT STILL BLOCKED' NOTE THAT USED TO SIT HERE IS STALE AND IS WITHDRAWN** - the land pattern was built from the same datasheet's 'Recommended Land Pattern' (rev 003.001, 2024-02-27) with the dimensions read off the drawing leader lines. **THIS PART IS DNP HERE** - it is the NFC 5 V fallback inductor (D-055/D-056) - **but the SAME MPN IS FITTED AS `L4` on the accessory 5 V boost, and its Isat of 6.2 A closes B-68**: the accessory boost peak inductor current is 2.19 A at the 0.86 A worst-high current limit with V_SYS at 3.0 V, so the margin is 2.8x on Isat and 4.7x on IRP.
- Q4: MPN (none) -> BSS138LT1G; Manufacturer (none) -> onsemi; Note open-drain SHDN pull-down; NEVER sources from +3V3 -> FBV2-S2-001: exact order code added - the schematic previou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
- Q6: MPN (none) -> BSS138LT1G; Manufacturer (none) -> onsemi; Note AND input 1 - pack polarity correct -> FBV2-S2-001: exact order code added - the schematic previou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
- Q7: MPN (none) -> BSS138LT1G; Manufacturer (none) -> onsemi; Note AND input 2 - pack below handoff threshold -> FBV2-S2-001: exact order code added - the schematic previou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
- Q8: MPN (none) -> BSS138LT1G; Manufacturer (none) -> onsemi; Note AND input 3 - LTC4368 FAULT asserted -> FBV2-S2-001: exact order code added - the schematic previou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
- Q9: MPN (none) -> BSS138LT1G; Manufacturer (none) -> onsemi; Note inverts active-low FAULT for the AND chain -> FBV2-S2-001: exact order code added - the schematic previou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
- R68: Note (none) -> FBV2-S2-001: **DNP AND IT MUST STAY DNP. THIS IS NOT A TUNI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
