File: hardware/beta-v2/kicad/aqroot-beta-v2/01_power_tree.kicad_sch (KiCad schematic)
At the start: 138 parts, among them J3 USB_C_Receptacle_USB2.0_16P, J4 JST-PH-2 BATTERY, Q2 NTMD4820N, Q3 NTMD4820N, Q4 BSS138, Q5 AO3401A, Q6 BSS138, Q7 BSS138, Q8 BSS138, Q9 BSS138, SW9 SW_SPDT, U10 USBLC6-2SC6, U11 BQ25185, U12 TPS63020, U13 TPS61023, U14 MAX17048, U18 LTC4368-1, U19 TLV7032, U20 TPS22950C, U21 TPS61023, U22 TPS22950C

Commit message: hardware: close Full Beta v2 S2 release blockers
Closes B-03, B-63, B-70 and B-71's schematic-side work. Property-only
changes to the nine sheets plus the microphone footprint; ERC unchanged
at 27 / 0 errors / 27 with an identical violation histogram, and the PCB
is untouched and still bit-identical to Beta-DM.

B-03 - all eight remaining Tier-2 footprints compared dimension by
dimension against retrieved manufacturer drawings. Y1 moves from
candidate to lock (Yajingxin TXM27.12M0004322DBBDO00T, C362365, 3421 in
stock) with a land that matches the vendor's Suggested Layout exactly.
The MAX98357A looked like a genuine defect - outline 21-0136 gives
T1633-5 an EP of 1.50/1.60/1.70 while the land is 1.23 - and is not:
land pattern 90-0032 Rev E is issued for T1633-5, -5C and -7C together
and specifies one land for all three, so no project-local footprint was
created.

B-63 - the microphone acoustic port is now drawn rather than described.
1.05 mm NPTH taken from the drawing's own pad-4 ring inner diameter,
paste pulled back 0.10 mm as a declared stencil choice, keepout marked,
bottom-port orientation recorded.

B-70 - L5/L6 lock to Murata LQW18AN39NG80D. The DCR is a first-order
term here: 0.20 ohm max against R_q = 1.1 ohm drops network Q from 25.3
to about 21.4, so the antenna must be tuned with this exact part fitted
and the first lever is R_q, not 39 nH.

B-71 - 65 LCSC fields written in, three MPN strings corrected. J6 and J7
carried bare order codes that resolve to zero-stock listings while the
plating-suffixed strings are abundantly stocked. Six substitution traps
recorded in the symbols themselves, including BAT54W offered for
BAT54WS - a single diode for a series pair - and a clone for the battery
reverse-polarity pass FETs.

Eight DNP parts still carried no recorded reason and now do. The design
has zero unexplained DNP.

Co-Authored-By: Claude Opus 5 <noreply@anthropic.com>
Claude-Session: https://claude.ai/code/session_0133CdFHfKcCH8oPWqJZWe7o
Parts:
- C24, C26: LCSC (none) -> C344022
- C34, C35, R44, R45: Note2 (none) -> DNP BY DESIGN AND CORRECTLY SO - documented 2026-08-23 (FBV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
- D10, D11, D12: Note2 (none) -> SOURCING 2026-08-23 (FBV2-S2-002) (B-71). NEXPERIA BAT54WS,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
- D9: LCSC (none) -> C110921
- F1: LCSC (none) -> C187597; Note2 (none) -> SOURCING 2026-08-23 (FBV2-S2-002) (B-71). Littelfuse 046600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
- J3: LCSC (none) -> C5184243
- J4: LCSC (none) -> C131337; Note2 (none) -> SOURCING 2026-08-23 (FBV2-S2-002) (B-71). B2B-PH-K-S(LF)(SN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
- L1: LCSC (none) -> C3033018
- L2: LCSC (none) -> C5542269; Note2 (none) -> DNP BY DESIGN AND CORRECTLY SO - documented 2026-08-23 (FBV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
- L4: LCSC (none) -> C5542269; Manufacturer Wurth -> Wurth Elektronik; Note2 (none) -> SOURCING 2026-08-23 (FBV2-S2-002) (B-71). Wurth 74438357010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
- Q2, Q3: LCSC (none) -> C905372; Note2 (none) -> SOURCING 2026-08-23 (FBV2-S2-002) (B-71) - FIRST-BUILD BLOC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
- Q4, Q6, Q7, Q8, Q9: LCSC (none) -> C82045; Note2 (none) -> SOURCING 2026-08-23 (FBV2-S2-002) (B-71). Genuine onsemi BS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
- Q5: LCSC (none) -> C15127
- SW9: LCSC (none) -> C221660
- U10: LCSC (none) -> C7519
- U11: LCSC (none) -> C19725033
- U12: LCSC (none) -> C15483
- U13: LCSC (none) -> C919459; Note2 (none) -> DNP BY DESIGN AND CORRECTLY SO - documented 2026-08-23 (FBV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
- U14: LCSC (none) -> C2682616
- U18: LCSC (none) -> C688397; Note2 (none) -> SOURCING 2026-08-23 (FBV2-S2-002) (B-71) - FIRST-BUILD BLOC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
- U19: LCSC (none) -> C2871498; Note2 (none) -> SOURCING 2026-08-23 (FBV2-S2-002) (B-71). TLV7032DDFR is LC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
- U20, U22: LCSC (none) -> C7587833
- U21: LCSC (none) -> C919459

Commit message: hardware: lock final first-five procurement alternatives
Two CTO-approved substitutions, both verified live under D-096 against the
JLCPCB parts API on 2026-08-23, both adopted.

F1: Littelfuse 0466005.NR -> 0466005.NRHF, LCSC C187597 -> C57525.
The halogen-free ordering option of the same 466 / Nano2 family: 5 A,
32 VAC / 32 VDC, 50 A interrupting, fast acting, 1206. The two LCSC records
carry a character-for-character identical parametric string. Stock 0 -> 29,328.
Same footprint, same electrical function, connectivity untouched. (D-210)

D10/D11/D12: Nexperia BAT54WS,115 -> Diodes Incorporated BAT54WS-7-F,
LCSC C124205, 46,819 in stock. One independent Schottky, 30 V, 100 mA
continuous, 600 mA surge, SOD-323. (D-211)

BAT54WS IS NOT A SERIES PAIR. The prior sourcing note said it was, in six
documents including the symbols themselves. SOD-323 is a two-terminal package,
every BAT54WS in the LCSC library from eight manufacturers is catalogued
"1 Independent", and D10/D11/D12 are each one two-pin Device:D_Schottky on a
two-pad Diode_SMD:D_SOD-323 - D10 and D11 form the ratiometric bridge as two
separate matched components. The design was never wrong; the note was.
BAT54W,115 stays rejected because it is SOT-323 (SC-70), a footprint mismatch.

Electrically verified, no material mismatch. The bridge comparison
(BAT_RAW + V_F11 - V_F10)/2 cancels the absolute drop and runs at ~1.1 uA
through 4.4 M. D12 sees ~16.6 mA worst case against 100 mA continuous - 6x -
and D-105's 5-10 mA recovery band needs no revision.

Assembly: F1 class C -> B, D10-D12 class D -> B. Both machine-placed.
Consignment 11 -> 9 part numbers; class D is now empty. Still exactly two
hand-soldered parts per board (J5, D1).

ERC 27 -> 27, zero errors, histogram identical. Netlist 224 nets / 991 nodes,
identical. The diff is property-only: no wire, label, junction, no-connect,
symbol or pin line changed. fork_equivalence PASS, netclass_probe PASS.
PCB byte-identical and still bit-identical to Beta-DM.
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
Parts:
- D10, D11, D12: LCSC (none) -> C124205; MPN BAT54WS,115 -> BAT54WS-7-F; Manufacturer Nexperia -> Diodes Incorporated; Note2 SOURCING 2026-08-23 (FBV2-S2-002) (B-71). NEXPERIA BAT54WS,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 -> PROCUREMENT LOCKED 2026-08-23 (FBV2-MECH-002, D-211). Diode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
- F1: LCSC C187597 -> C57525; MPN 0466005.NR -> 0466005.NRHF; Note2 SOURCING 2026-08-23 (FBV2-S2-002) (B-71). Littelfuse 046600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 -> PROCUREMENT LOCKED 2026-08-23 (FBV2-MECH-002, D-210). Litte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
Changed lines of the file:
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@@
 			)
 		)
-		(property "Note2" "SOURCING 2026-08-23 (FBV2-S2-002) (B-71). Littelfuse 0466005.NR is LCSC C187597 with STOCK 0. The halogen-free 0466005.NRHF (C57525) has 29338 in stock and is the same 0466 5 A 1206 Nano2 fuse family, but it is a DIFFERENT ORDER CODE and is recorded as a CANDIDATE, not a substitution. Consign the .NR from a broadline distributor unless the .NRHF is signed off. LCSC/JLC library state verified live on 2026-08-23 through the JLCPCB parts API (D-096). Stock is a snapshot, not a guarantee."
+		(property "Note2" "PROCUREMENT LOCKED 2026-08-23 (FBV2-MECH-002, D-210). Littelfuse 0466005.NRHF, LCSC C57525 - the HALOGEN-FREE ORDERING OPTION of the same Littelfuse 466 / Nano2 family: 5 A, 32 VAC / 32 VDC, 50 A interrupting, fast acting, 1206. SAME FOOTPRINT AND SAME ELECTRICAL FUNCTION as the 0466005.NR it replaces - the HF suffix is a manufacturer ordering option, not an electrical redesign. F1 connectivity and footprint are UNCHANGED. The .NR order code (C187597) is STOCK 0; .NRHF verified live 2026-08-23 through the JLCPCB parts API at 29328 in stock, JLC EXTENDED - machine-placed, NO CONSIGNMENT. Stock is a snapshot, not a guarantee (D-096)."
 			(at 36.29 252.75 0)
 			(hide yes)
@@
 			)
 		)
-		(property "LCSC" "C187597"
+		(property "LCSC" "C57525"
 			(at 36.29 252.75 0)
 			(hide yes)
@@
 			)
 		)
-		(property "MPN" "0466005.NR"
+		(property "MPN" "0466005.NRHF"
 			(at 36.29 249.75 0)
 			(hide yes)
@@
 			)
 		)
-		(property "Note2" "SOURCING 2026-08-23 (FBV2-S2-002) (B-71). NEXPERIA BAT54WS,115 IS NOT IN THE LCSC/JLC LIBRARY AT ALL. A loose search for \"BAT54WS,115\" returns Nexperia BAT54W,115 (C8657) - that is the SINGLE diode, not the SERIES PAIR, and it must not be substituted. Two correct routes: buy the Nexperia part from a broadline distributor and consign it, or use the documented equivalent Diodes Incorporated BAT54WS-7-F, LCSC C124205, stock 46819 - same SOD-323 series-pair Schottky. THE EQUIVALENT IS DOCUMENTED, NOT ADOPTED: it needs a one-line sign-off before the order. LCSC/JLC library state verified live on 2026-08-23 through the JLCPCB parts API (D-096). Stock is a snapshot, not a guarantee."
+		(property "Note2" "PROCUREMENT LOCKED 2026-08-23 (FBV2-MECH-002, D-211). Diodes Incorporated BAT54WS-7-F, LCSC C124205, verified live 2026-08-23 through the JLCPCB parts API: ONE INDEPENDENT Schottky diode, 30 V, 100 mA continuous, 600 mA surge, VF 1 V max at 100 mA, IR 2 uA at 25 V, SOD-323, 46819 in stock, JLC EXTENDED - machine-placed, NO CONSIGNMENT. CORRECTION TO THE EARLIER SOURCING NOTE: BAT54WS IS NOT A SERIES PAIR. SOD-323 is a TWO-TERMINAL package, every BAT54WS in the LCSC library from every manufacturer is listed as 1 Independent, and D10, D11 and D12 are each ONE diode on the two-pin Device:D_Schottky symbol. D10 and D11 form the ratiometric polarity bridge as TWO SEPARATE MATCHED COMPONENTS, so BAT54WS-7-F matches the actual architecture exactly. THE REAL REJECTION CRITERION FOR ANY ALTERNATE IS: single independent diode, SOD-323 land pattern, adequate VF / leakage / current, matched type for D10 and D11, and live sourcing. Nexperia BAT54W,115 (C8657) is rejected because it is a SOT-323 (SC-70) part - a FOOTPRINT MISMATCH against Diode_SMD:D_SOD-323 - NOT because of diode count. Stock is a snapshot, not a guarantee (D-096)."
 			(at 41.37 337.84 0)
 			(hide yes)
@@
 			)
 		)
-		(property "Manufacturer" "Nexperia"
+		(property "LCSC" "C124205"
+			(at 41.37 337.84 0)
+			(hide yes)
+			(show_name no)
+			(do_not_autoplace no)
+			(effects
+				(font
+					(size 1.0 1.0)
+				)
+				(justify left)
+			)
+		)
+		(property "Manufacturer" "Diodes Incorporated"
 			(at 41.37 336.34 0)
 			(hide yes)
@@
 			)
 		)
-		(property "MPN" "BAT54WS,115"
+		(property "MPN" "BAT54WS-7-F"
 			(at 41.37 334.84 0)
 			(hide yes)
@@
 			)
 		)
-		(property "Note2" "SOURCING 2026-08-23 (FBV2-S2-002) (B-71). NEXPERIA BAT54WS,115 IS NOT IN THE LCSC/JLC LIBRARY AT ALL. A loose search for \"BAT54WS,115\" returns Nexperia BAT54W,115 (C8657) - that is the SINGLE diode, not the SERIES PAIR, and it must not be substituted. Two correct routes: buy the Nexperia part from a broadline distributor and consign it, or use the documented equivalent Diodes Incorporated BAT54WS-7-F, LCSC C124205, stock 46819 - same SOD-323 series-pair Schottky. THE EQUIVALENT IS DOCUMENTED, NOT ADOPTED: it needs a one-line sign-off before the order. LCSC/JLC library state verified live on 2026-08-23 through the JLCPCB parts API (D-096). Stock is a snapshot, not a guarantee."
+		(property "Note2" "PROCUREMENT LOCKED 2026-08-23 (FBV2-MECH-002, D-211). Diodes Incorporated BAT54WS-7-F, LCSC C124205, verified live 2026-08-23 through the JLCPCB parts API: ONE INDEPENDENT Schottky diode, 30 V, 100 mA continuous, 600 mA surge, VF 1 V max at 100 mA, IR 2 uA at 25 V, SOD-323, 46819 in stock, JLC EXTENDED - machine-placed, NO CONSIGNMENT. CORRECTION TO THE EARLIER SOURCING NOTE: BAT54WS IS NOT A SERIES PAIR. SOD-323 is a TWO-TERMINAL package, every BAT54WS in the LCSC library from every manufacturer is listed as 1 Independent, and D10, D11 and D12 are each ONE diode on the two-pin Device:D_Schottky symbol. D10 and D11 form the ratiometric polarity bridge as TWO SEPARATE MATCHED COMPONENTS, so BAT54WS-7-F matches the actual architecture exactly. THE REAL REJECTION CRITERION FOR ANY ALTERNATE IS: single independent diode, SOD-323 land pattern, adequate VF / leakage / current, matched type for D10 and D11, and live sourcing. Nexperia BAT54W,115 (C8657) is rejected because it is a SOT-323 (SC-70) part - a FOOTPRINT MISMATCH against Diode_SMD:D_SOD-323 - NOT because of diode count. Stock is a snapshot, not a guarantee (D-096)."
 			(at 41.37 351.81 0)
 			(hide yes)
@@
 			)
 		)
-		(property "Manufacturer" "Nexperia"
+		(property "LCSC" "C124205"
+			(at 41.37 351.81 0)
+			(hide yes)
+			(show_name no)
+			(do_not_autoplace no)
+			(effects
+				(font
+					(size 1.0 1.0)
+				)
+				(justify left)
+			)
+		)
+		(property "Manufacturer" "Diodes Incorporated"
 			(at 41.37 350.31 0)
 			(hide yes)
@@
 			)
 		)
-		(property "MPN" "BAT54WS,115"
+		(property "MPN" "BAT54WS-7-F"
 			(at 41.37 348.81 0)
 			(hide yes)
@@
 			)
 		)
-		(property "Note2" "SOURCING 2026-08-23 (FBV2-S2-002) (B-71). NEXPERIA BAT54WS,115 IS NOT IN THE LCSC/JLC LIBRARY AT ALL. A loose search for \"BAT54WS,115\" returns Nexperia BAT54W,115 (C8657) - that is the SINGLE diode, not the SERIES PAIR, and it must not be substituted. Two correct routes: buy the Nexperia part from a broadline distributor and consign it, or use the documented equivalent Diodes Incorporated BAT54WS-7-F, LCSC C124205, stock 46819 - same SOD-323 series-pair Schottky. THE EQUIVALENT IS DOCUMENTED, NOT ADOPTED: it needs a one-line sign-off before the order. LCSC/JLC library state verified live on 2026-08-23 through the JLCPCB parts API (D-096). Stock is a snapshot, not a guarantee."
+		(property "Note2" "PROCUREMENT LOCKED 2026-08-23 (FBV2-MECH-002, D-211). Diodes Incorporated BAT54WS-7-F, LCSC C124205, verified live 2026-08-23 through the JLCPCB parts API: ONE INDEPENDENT Schottky diode, 30 V, 100 mA continuous, 600 mA surge, VF 1 V max at 100 mA, IR 2 uA at 25 V, SOD-323, 46819 in stock, JLC EXTENDED - machine-placed, NO CONSIGNMENT. CORRECTION TO THE EARLIER SOURCING NOTE: BAT54WS IS NOT A SERIES PAIR. SOD-323 is a TWO-TERMINAL package, every BAT54WS in the LCSC library from every manufacturer is listed as 1 Independent, and D10, D11 and D12 are each ONE diode on the two-pin Device:D_Schottky symbol. D10 and D11 form the ratiometric polarity bridge as TWO SEPARATE MATCHED COMPONENTS, so BAT54WS-7-F matches the actual architecture exactly. THE REAL REJECTION CRITERION FOR ANY ALTERNATE IS: single independent diode, SOD-323 land pattern, adequate VF / leakage / current, matched type for D10 and D11, and live sourcing. Nexperia BAT54W,115 (C8657) is rejected because it is a SOT-323 (SC-70) part - a FOOTPRINT MISMATCH against Diode_SMD:D_SOD-323 - NOT because of diode count. Stock is a snapshot, not a guarantee (D-096)."
 			(at 41.37 384.83 0)
 			(hide yes)
@@
 			)
 		)
-		(property "Manufacturer" "Nexperia"
+		(property "LCSC" "C124205"
+			(at 41.37 384.83 0)
+			(hide yes)
+			(show_name no)
+			(do_not_autoplace no)
+			(effects
+				(font
+					(size 1.0 1.0)
+				)
+				(justify left)
+			)
+		)
+		(property "Manufacturer" "Diodes Incorporated"
 			(at 41.37 383.33 0)
 			(hide yes)
@@
 			)
 		)
-		(property "MPN" "BAT54WS,115"
+		(property "MPN" "BAT54WS-7-F"
 			(at 41.37 381.83 0)
 			(hide yes)
