File: hardware/beta-v2/kicad/aqroot-beta-v2/09_community_header.kicad_sch (KiCad schematic)
At the start: 36 parts, among them J5 COMMUNITY_PORT_2x12, Q10 2N7002, U16 TCA4307DGKR

Commit message: hardware: adopt standard AQROOT expansion interface
Replace the community port's presentation, not its electronics.

J5 becomes a Samtec SSQ-124-02-G-S-RA: 1 x 24, 2.54 mm, female, right-angle,
one pin per line -- the same manufacturer as the BCS-112-S-D-HE it supersedes,
so the account and the small-quantity behaviour are already known. Body
61.47 mm, pin span 58.42 mm, mates a .025 in (0.635 mm) square post, which is
the ordinary male-header and Dupont standard. New project footprint, drawn from
the Samtec SSW/SSQ datasheet and the Sullins 1-row right-angle recommended
layout (drawing 10493), which is also where the 6.53 mm tail-row-to-mating-face
depth comes from -- the dimension the whole right-wall fit turns on.

J8 adds Qwiic / STEMMA QT: JST SM04B-SRSS-TB, SH 1.0 mm, 4 circuit, side entry,
SMT and machine-placed, so the manual-assembly list stays at two parts. Pin
order 1 GND / 2 3V3 / 3 SDA / 4 SCL is the ecosystem standard, identical for
SparkFun Qwiic and Adafruit STEMMA QT. It taps EXT_SDA / EXT_SCL downstream of
U16 and the 22 ohm pair, at D2's clamp, and so costs ZERO components: no second
buffer, no mux, no repeater, no extra pull-ups, no second TVS. Power is
ACC_3V3_SW because U16's own VCC already is; an unswitched feed would create a
powered-device / unpowered-bus state. ACC_5V_SW is not on it and cannot be.

Pin order is ORDER-B, superseding EXP-001's ORDER-A. ORDER-A was safe against a
one-position slip, which the closed-end recess already makes impossible; it was
not safe against someone turning the accessory around. ORDER-B is symmetric by
construction, so a full 24-pin accessory inserted 180 degrees maps 5V to 5V,
GND to GND, 3V3 to 3V3 and 3.3 V logic to 3.3 V logic on every remaining
contact. Power-to-signal maps under reversal: zero, proved pin by pin from the
exported netlist.

All 24 electrical functions retained. Not one protection component removed:
twelve 100 ohm GPIO resistors, the 22 ohm I2C pair, the 330 ohm WAKE resistor,
four TPD4E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
Parts:
- added J8: QWIIC_STEMMA_QT, Connector_JST:JST_SH_SM04B-SRSS-TB_1x04-1MP_P1.00mm_Horizontal, symbol Connector_Generic:Conn_01x04
- J5: value COMMUNITY_PORT_2x12 -> COMMUNITY_PORT_1x24; footprint AQROOT_Beta:Samtec_BCS-112-S-D-HE -> AQROOT_Beta:Samtec_SSQ-124-02-G-S-RA
Connections:
- net ACC_3V3_SW: now also J5.22 (Pin_22), J8.2 (Pin_2); no longer J5.15 (Pin_15)
- net ACC_5V_SW: now also J5.1 (Pin_1), J5.24 (Pin_24); no longer J5.10 (Pin_10), J5.22 (Pin_22)
- net ACC_DETECT_N_HDR: now also J5.21 (Pin_21); no longer J5.23 (Pin_23)
- net EXT_SCL: now also J5.5 (Pin_5), J8.4 (Pin_4); no longer J5.2 (Pin_2)
- net EXT_SDA: now also J5.4 (Pin_4), J8.3 (Pin_3); no longer J5.6 (Pin_6)
- net GND: now also J5.19 (Pin_19), J5.2 (Pin_2), J5.23 (Pin_23), J5.6 (Pin_6), J8.1 (Pin_1); no longer J5.16 (Pin_16), J5.21 (Pin_21), J5.4 (Pin_4), J5.9 (Pin_9)
- net NATIVE_B_HDR: now also J5.8 (Pin_8); no longer J5.11 (Pin_11)
- net WAKE_ATTN_N_HDR: now also J5.20 (Pin_20); no longer J5.14 (Pin_14)
- net XGPIO0_HDR: now also J5.9 (Pin_9); no longer J5.1 (Pin_1)
- net XGPIO1_HDR: now also J5.10 (Pin_10); no longer J5.5 (Pin_5)
- net XGPIO2_HDR: now also J5.11 (Pin_11); no longer J5.8 (Pin_8)
- net XGPIO5_HDR: now also J5.14 (Pin_14); no longer J5.17 (Pin_17)
- net XGPIO6_HDR: now also J5.15 (Pin_15); no longer J5.18 (Pin_18)
- net XGPIO7_HDR: now also J5.16 (Pin_16); no longer J5.19 (Pin_19)
- net XGPIO8_HDR: now also J5.17 (Pin_17); no longer J5.20 (Pin_20)
- net XGPIO9_HDR: now also J5.18 (Pin_18); no longer J5.24 (Pin_24)
Other:
- note added: "QWIIC / STEMMA QT - FBV2-EXP-002 (D-238) J8 = JST SM04B-SRSS-TB(LF)(SN), SH 1.0 mm, 4 circuit, SIDE ENTRY SMT. 1 GND / 2 3V3 / 3 SDA / 4 SCL is the ECOSYSTEM STANDARD ORDER - Qwiic and STEMMA QT are identical here, so every cable in either ecosystem mates. IT ADDS NO COMPONENT. It taps the PROTECTED EXTERNAL segment at EXT_SDA / EXT_SCL - downstream of U16 and of the R47/R48 22 R pair, at D2's cl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"
