File: hardware/demo/kicad/aqroot-demo/01_power_tree.kicad_sch (KiCad schematic)
At the start: 138 parts, among them J3 USB_C_Receptacle_USB2.0_16P, J4 JST-PH-2 BATTERY, Q2 NTMD4820N, Q3 NTMD4820N, Q4 BSS138, Q5 AO3401A, Q6 BSS138, Q7 BSS138, Q8 BSS138, Q9 BSS138, SW9 SW_SPDT, U10 USBLC6-2SC6, U11 BQ25185, U12 TPS63020, U13 TPS61023, U14 MAX17048, U18 LTC4368-1, U19 TLV7032, U20 TPS22950C, U21 TPS61023, U22 TPS22950C

Commit message: demo: apply schematic simplification ECO
Parts:
- R131: Note ACC_5V_SW_EN safe-state pull-down, ADDED FBV2-S1-009. The CTO split the single ACC_5V_EN into ACC_5V_BOOST_EN (U3 P13 -> U21 EN) and ACC_5V_SW_EN (U23 P04 -> U22 ON), so the new net needs its own 100 k to ground. THE PULL-DOWN IS MANDATORY, NOT A CONVENIENCE: SLVSFJ2B specifies a 500 kOhm smart pull-down inside the TPS22950C and STILL REQUIRES AN EXTERNAL ONE, and the PCAL9535A powers up with every pin high-impedance - so without this resistor the 5 V accessory contact would be defined only by leakage between power-on and the first firmware write. 100 k matches R98 and R102 and costs 33 uA when the pin is driven high. -> ACC_5V_SW_EN safe-state pull-down, ADDED FBV2-S1-009. The CTO split the single ACC_5V_EN into ACC_5V_BOOST_EN (U3 P13 -> U21 EN) and ACC_5V_SW_EN (U3 P03 -> U22 ON), so the new net needs its own 100 k to ground. THE PULL-DOWN IS MANDATORY, NOT A CONVENIENCE: SLVSFJ2B specifies a 500 kOhm smart pull-down inside the TPS22950C and STILL REQUIRES AN EXTERNAL ONE, and the PCAL9535A powers up with every pin high-impedance - so without this resistor the 5 V accessory contact would be defined only by leakage between power-on and the first firmware write. 100 k matches R98 and R102 and costs 33 uA when the pin is driven high.
Changed lines of the file:
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@@
 			)
 		)
-		(property "Note" "ACC_5V_SW_EN safe-state pull-down, ADDED FBV2-S1-009. The CTO split the single ACC_5V_EN into ACC_5V_BOOST_EN (U3 P13 -> U21 EN) and ACC_5V_SW_EN (U23 P04 -> U22 ON), so the new net needs its own 100 k to ground. THE PULL-DOWN IS MANDATORY, NOT A CONVENIENCE: SLVSFJ2B specifies a 500 kOhm smart pull-down inside the TPS22950C and STILL REQUIRES AN EXTERNAL ONE, and the PCAL9535A powers up with every pin high-impedance - so without this resistor the 5 V accessory contact would be defined only by leakage between power-on and the first firmware write. 100 k matches R98 and R102 and costs 33 uA when the pin is driven high."
+		(property "Note" "ACC_5V_SW_EN safe-state pull-down, ADDED FBV2-S1-009. The CTO split the single ACC_5V_EN into ACC_5V_BOOST_EN (U3 P13 -> U21 EN) and ACC_5V_SW_EN (U3 P03 -> U22 ON), so the new net needs its own 100 k to ground. THE PULL-DOWN IS MANDATORY, NOT A CONVENIENCE: SLVSFJ2B specifies a 500 kOhm smart pull-down inside the TPS22950C and STILL REQUIRES AN EXTERNAL ONE, and the PCAL9535A powers up with every pin high-impedance - so without this resistor the 5 V accessory contact would be defined only by leakage between power-on and the first firmware write. 100 k matches R98 and R102 and costs 33 uA when the pin is driven high."
 			(at 0 0 0)
 			(hide yes)
