File: hardware/demo/kicad/aqroot-demo/01_power_tree.kicad_sch (KiCad schematic)
At the start: 136 parts, among them J3 USB_C_Receptacle_USB2.0_16P, J4 JST-PH-2 BATTERY, Q2 NTMD4820N, Q3 NTMD4820N, Q4 BSS138, Q5 AO3401A, Q6 BSS138, Q7 BSS138, Q8 BSS138, Q9 BSS138, SW9 SW_SPDT, U10 USBLC6-2SC6, U11 BQ25185, U12 TPS63020, U13 TPS61023, U14 MAX17048, U18 LTC4368-1, U19 TLV7032, U20 TPS22950C, U21 TPS61023, U22 TPS22950C

Commit message: demo: D-743 -- the charger could not complete a charge. TI halved tMAXCHG in August and this board's ICHG was chosen against the old number.
R37 was 1 kOhm, so SLUSF65B 6.1.1.4's ICHG = KISET/RISET programmed 300 mA (TI's own worked example).  R36 was 18 kOhm = ILIM500.  And SLUSF65B revision B (August 2026) changed tMAXCHG from 720 min to 360 min -- the only line in its revision history.  300 mA x 360 min = 1800 mAh against a 2500-3000 mAh cell, so the charger stopped at 60-72 % state of charge and section 6.3.7.7 disabled charging with a non-recoverable fault, clearable only by toggling CE or VIN -- and U11.4 /CE is hard-tied to GND, so the user must unplug the cable.  The design was CORRECT against SLUSF65A (720 min x 300 mA = 3600 mAh); a vendor documentation change invalidated it and nothing here re-read the datasheet for four weeks.

FIX: R37 1 k -> 390 R (ICHG 769 mA typ) and R36 18 k -> 13 k (ILIM1100).  R36 is a LOOKUP row, not a trim: 13 kOhm keeps VBATREG at 4.2 V and VLOWV at 3.0 V and moves only the input limit, so D-269/D-186 are untouched.  It had to move because the part is linear -- input current IS charge current, and ILIM500 caps ICHG plus system load at 500 mA.  390 R beat the arithmetically nearer 374 R on the live distributor record: 0603WAF3740T5E is EXTENDED with stock 1, while 0603WAF3900T5E (C23151) and 0603WAF1302T5E (C22797) are both JLC BASIC with six-figure stock, same UNI-ROYAL family so D-614's reasoning carries.  Margin 286 min at 3000 mAh and 238 at 2500, against 360; TREG 100 C governs the low-VBAT corner rather than a fixed current ceiling, and first-article thermal measurement is recorded as required.

Doubling the input limit doubled what USB_VBUS_CHG carries, and no instrument here could say whether it could -- every ampacity tool on this board is a DIFF.  audit_rail_ampacity.py is absolute: it walks the CARRYING path (this net has eleven pads and nine are microamp telemetry over 200 mm, so judging the net by its narrowest trac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
Parts:
- R36: value 18k 1% -> 13k 1%; LCSC C25810 -> C22797; MPN 0603WAF1802T5E -> 0603WAF1302T5E; Note (none) -> D-743 CHANGED THIS VALUE FROM 18 kOhm TO 13 kOhm, AND IT IS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; Note_Sourcing SOURCING D-614. EXACT_PRIOR from the beta-dm audit line '18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 -> SOURCING D-743, live JLCPCB record refreshed 2026-09-18 and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
- R37: value 1k 1% -> 390R 1%; LCSC C21190 -> C23151; MPN 0603WAF1001T5E -> 0603WAF3900T5E; Note (none) -> D-743 CHANGED THIS VALUE FROM 1 kOhm TO 390 Ohm. IT PROGRAM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; Note_Sourcing SOURCING D-614. EXACT_PRIOR from the beta-dm audit line '1k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 -> SOURCING D-743, live JLCPCB record refreshed 2026-09-18 and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
Changed lines of the file:
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@@
 			)
 		)
-		(property "Value" "18k 1%"
+		(property "Value" "13k 1%"
 			(at 48.26 171.4499 0)
 			(show_name no)
@@
 			)
 		)
-		(property "MPN" "0603WAF1802T5E"
+		(property "MPN" "0603WAF1302T5E"
 			(at 45.72 170.18 0)
 			(hide yes)
@@
 			)
 		)
-		(property "LCSC" "C25810"
+		(property "LCSC" "C22797"
 			(at 45.72 170.18 0)
 			(hide yes)
@@
 			)
 		)
-		(property "Note_Sourcing" "SOURCING D-614. EXACT_PRIOR from the beta-dm audit line '18k 1%' (REJECTED - JLC match wrong); manufacturer derived from the UNI-ROYAL(Uniroyal Elec) part-number family and corroborated by the audit text; tolerance 1.0% meets 1.0%."
+		(property "Note_Sourcing" "SOURCING D-743, live JLCPCB record refreshed 2026-09-18 and archived in hardware/demo/manufacturing/evidence/jlc-live/. C22797, UNI-ROYAL 0603WAF1302T5E, 13 kOhm +-1% 100 mW 0603, JLCPCB BASIC library, stock 500493, RoHS. Replaces C25810 / 0603WAF1802T5E (18 kOhm), which is retained in git history only. The part FAMILY is unchanged, so the D-614 manufacturer and land-pattern reasoning carries over unaltered; only the resistance moved."
 			(at 45.72 170.18 0)
 			(hide yes)
@@
 		(property "Description" "Resistor"
 			(at 45.72 170.18 0)
+			(hide yes)
+			(show_name no)
+			(do_not_autoplace no)
+			(effects
+				(font
+					(size 1.27 1.27)
+				)
+			)
+		)
+		(property "Note" "D-743 CHANGED THIS VALUE FROM 18 kOhm TO 13 kOhm, AND IT IS NOT A TRIM - IT SELECTS A DIFFERENT ROW OF THE BQ25185's ILIM/VSET RESISTOR MAP. SLUSF65B Table 6-1 is a lookup, not a formula: 18 kOhm = ILIM500 + VBATREG 4.2 V + VLOWV 3.0 V; 13 kOhm = ILIM1100 + VBATREG 4.2 V + VLOWV 3.0 V. *** THE BATTERY REGULATION VOLTAGE AND THE PRECHARGE THRESHOLD ARE THEREFORE UNCHANGED AT 4.2 V AND 3.0 V. Only the INPUT CURRENT LIMIT moves, 500 mA to 1100 mA. D-269 and D-186 battery-safety requirements are untouched by this change. *** WHY IT HAD TO MOVE: the BQ25185 is a linear charger, so input current and charge current are the same current. ILIM500 caps ICHG + system load at 500 mA, and SLUSF65B revision B (August 2026) halved the fast-charge safety timer tMAXCHG from 720 min to 360 min. At any charge current ILIM500 permits, a 2500-3000 mAh cell cannot reach termination before the timer expires, and section 6.3.7.7 then DISABLES CHARGING with a non-recoverable fault that only a CE or VIN toggle clears - and CE is hard-tied to GND on this board, so only unplugging the USB cable clears it. See R37's note for the charge-current half of the same decision and for the arithmetic. CONSEQUENCE ON THE SOURCE: this board's USB-C is a plain 5.1 kOhm Rd sink (R30/R31) and does not read the source's Rp advertisement, so at ILIM1100 it may draw more than a legacy 500 mA USB 2.0 port offers. The BQ25185's battery-tracking VINDPM (target VBAT + 330 mV, SLUSF65B section 5.5) is the designed mitigation and folds the input current back as VIN sags. A 500 mA-class source therefore charges more slowly and will not complete a cycle inside tMAXCHG; charge from a 1 A or better source. Reading the Type-C Rp advertisement is a Rev-B item."
+			(at 0 0 0)
 			(hide yes)
 			(show_name no)
@@
 			)
 		)
-		(property "Value" "1k 1%"
+		(property "Value" "390R 1%"
 			(at 31.75 167.6399 0)
 			(show_name no)
@@
 			)
 		)
-		(property "MPN" "0603WAF1001T5E"
+		(property "MPN" "0603WAF3900T5E"
 			(at 29.21 166.37 0)
 			(hide yes)
@@
 			)
 		)
-		(property "LCSC" "C21190"
+		(property "LCSC" "C23151"
 			(at 29.21 166.37 0)
 			(hide yes)
@@
 			)
 		)
-		(property "Note_Sourcing" "SOURCING D-614. EXACT_PRIOR from the beta-dm audit line '1k 1%' (REJECTED - JLC match wrong); manufacturer derived from the UNI-ROYAL(Uniroyal Elec) part-number family and corroborated by the audit text; tolerance 1.0% meets 1.0%."
+		(property "Note_Sourcing" "SOURCING D-743, live JLCPCB record refreshed 2026-09-18 and archived in hardware/demo/manufacturing/evidence/jlc-live/. C23151, UNI-ROYAL 0603WAF3900T5E, 390 Ohm +-1% 100 mW 0603, JLCPCB BASIC library, stock 353079, RoHS. Replaces C21190 / 0603WAF1001T5E (1 kOhm). The nearer arithmetic value 374 Ohm (0603WAF3740T5E, C23149) was REJECTED on the live record: EXTENDED library and stock 1. The part FAMILY is unchanged, so D-614's manufacturer and land-pattern reasoning carries over; only the resistance moved."
 			(at 29.21 166.37 0)
 			(hide yes)
@@
 			(hide yes)
 			(show_name no)
+			(do_not_autoplace no)
+			(effects
+				(font
+					(size 1.27 1.27)
+				)
+			)
+		)
+		(property "Note" "D-743 CHANGED THIS VALUE FROM 1 kOhm TO 390 Ohm. IT PROGRAMS THE BQ25185 FAST-CHARGE CURRENT AND THE OLD VALUE COULD NOT FINISH A CHARGE. SLUSF65B section 6.1.1.4: ICHG = KISET / RISET with KISET = 300 AOhm typical (285 to 315 over the range 10 mA < ICHG < 1000 mA, Table 5-1). 1 kOhm gave ICHG = 300 mA; 390 Ohm gives ICHG = 769 mA typical, 714 to 808 mA over the KISET range. *** THE DEFECT: SLUSF65B revision B (August 2026) changed tMAXCHG from 720 min to 360 min - the only line in its revision history. At 300 mA the charger delivers 300 mA x 360 min = 1800 mAh before the fast-charge safety timer expires, against a fitted cell of 2500 to 3000 mAh, so it stops at roughly 60 to 72 percent state of charge and section 6.3.7.7 DISABLES CHARGING with a non-recoverable fault. The design was correct against SLUSF65A, where tMAXCHG was 720 min and 300 mA x 12 h = 3600 mAh covered the whole envelope. A vendor documentation change invalidated it. *** THE NEW MARGIN: a 1S CC/CV cycle to 4.2 V terminating at ITERM = 10 percent of ICHG takes about 1.22 x C / ICHG. At 769 mA that is 286 min for 3000 mAh and 238 min for 2500 mAh, against 360 min - 21 and 34 percent margin. At the KISET minimum of 714 mA it is 308 min for 3000 mAh, still inside. THERMAL: the BQ25185 is linear and dissipates PSYS + PBAT = (VIN - VSYS) x IIN + (VSYS - VBAT) x IBAT with VSYS regulated to 4.5 V. At 769 mA, VBAT 3.7 V, VIN 5.0 V and a 50 mA system load that is about 1.03 W, and at RthetaJA 68.3 K/W (SLUSF65B section 5.3) about 70 K of rise. TREG is 100 C, so the part THERMALLY REGULATES - it reduces charge current itself rather than overheating - below roughly VBAT 3.9 V in a 40 C enclosure, which is where the cell holds least charge. TSHUT is 150 C and is not approached. This is deliberate: ICHG is set at the value the package can sustain for most of the cycle and TREG governs the rest. RISET_SHORT is 264 Ohm maximum, so 390 Ohm is well clear of the short-detect threshold that would latch a fault at startup. FIRST-ARTICLE MEASUREMENT REQUIRED: measure charge current, total charge time and U11 case temperature on the first assembled unit, in the enclosure, at the fitted cell capacity. Prefer the 2500 mAh end of the DEVICE_SPEC envelope; the 3000 mAh end at 40 C ambient has the least margin."
+			(at 0 0 0)
+			(hide yes)
+			(show_name no)

Commit message: demo: D-750 and D-751 -- the external first-spin review found four real defects, and finishing its repairs found two more.
An external first-spin review (Fable 5.1 + Astra) reopened DEMO_READY_FOR_FAB at
b593b97 and named thirteen items.  Four were real defects on the frozen package:
J5's BOM identity still named the 2x12 BCS-112-S-D-HE that D-237 superseded eight
months ago, U14.6 QSTRT was physically floating behind a deliberate no_connect,
audit_rail_ampacity.py computed at 0.0174 mm inner copper against a board that
declares 0.0152 mm, and neither boost converter had a local input capacitor --
the nearest was 36.6 mm and the *named* input part 93.5 mm away.  A fifth,
item 7, is a design-condition failure: TI guarantees the TPS61169 OFF only when
the LED array's minimum Vf exceeds the maximum VIN, this panel is 2.9-3.2 V on a
3.3 V rail, and the shutdown DC path converges at about 25 mA -- a fifth of full
brightness, with no firmware mitigation because +3V3 is switched by SW9.

D-750 closed all of them and dispositioned the other nine, item by item, with
FIRST-ARTICLE and PROCUREMENT work explicitly separated from pre-order blockers.
The charger input was re-laid 250.8 -> 189.8 mm and 440 -> 216 mOhm, which is
what buys the 360 min tMAXCHG its margin; C83 and C84 were fitted on the existing
C33/C64 BOM line; Q11, the backlight true-off disconnect, was fitted on Q1's line.

D-751 FINISHED THE TRANSACTION, AND EACH THING IT TOUCHED HELD ANOTHER DEFECT.

* Q11 was on the board as a symbol and a BOM line and NOT as a circuit: three
  unapproved open edges, all three of them its own pins.  Routed with three
  --tap-first taps, 16.26 mm and four barrels.  The first run was REFUSED for a
  0.44 mm dangling In2 stub the tap left past its T; trimmed, re-run clean.
* placement_contract.py HAD NO WORD FOR AN ADDED PART, so the whole standing
  suite read "placement FAIL" for a legitimate act.  --add exists; PL7 now holds
  an ADDED pad to the same foreign-copper clearance a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
Parts:
- added C83, C84: 10uF 10V X7R, Capacitor_SMD:C_0805_2012Metric, symbol Device:C
Connections:
- net BQ25185_SYS: now also C83.1, C84.1
- net GND: now also U14.6 (QSTRT), C83.2, C84.2
- no-connect marks 6 -> 5
