File: hardware/demo/kicad/aqroot-demo/01_power_tree.kicad_sch (KiCad schematic)
At the start: 138 parts, among them J3 USB_C_Receptacle_USB2.0_16P, J4 JST-PH-2 BATTERY, Q2 NTMD4820N, Q3 NTMD4820N, Q4 BSS138, Q5 AO3401A, Q6 BSS138, Q7 BSS138, Q8 BSS138, Q9 BSS138, SW9 SW_SPDT, U10 USBLC6-2SC6, U11 BQ25185, U12 TPS63020, U13 TPS61023, U14 MAX17048, U18 LTC4368-1, U19 TLV7032, U20 TPS22950C, U21 TPS61023, U22 TPS22950C

Commit message: demo: D-753 -- a policy is not an enforcement mechanism, so the accessory envelope is silicon now.
D-750 closed the external first-spin review's combined-load item as a PUBLISHED
LIMIT: "firmware must not raise both accessory rails to their per-rail maxima
together".  The independent re-review answered that this is not an enforcement
mechanism, and it is not -- THIS BOARD HAS NO ACCESSORY CURRENT MEASUREMENT.
Firmware can choose whether a rail is ON; it cannot know what an arbitrary
external accessory then draws.  The only thing that bounds an accessory is the
TPS22950C's own current limit, and at the values D-750 shipped those limits sat
far above what the policy permitted.

AND THE BOARD WAS WORSE THAN THE REVIEW SAID.  At the 3.0 V cell corner with the
full 1.0 A internal +3V3 load, U12 at 90 % and U21 at 88 % into 4.95 V, against
a BQ25185 IBAT_OCP MINIMUM of 2.5625 A (3.125 A typ +/-18 %), two states a user
could reach with CONFORMING accessories already tripped the pack protection: the
5 V rail alone at its limiter drew 2.930 A, and both rails merely at the current
each one GUARANTEES drew 2.737 A.  Not a thermal or copper failure -- a reset --
but nothing on the board prevented it.

R97 1.5 k -> 2.7 k and R101 1.65 k -> 2.7 k.  TI SLVSFJ2B equation 1 gives
ILIM = 1.18 x R[kOhm]^-1.072 = 0.407 A typ, and the widest tolerance ratio the
part's own EC table publishes (0.68x / 1.32x of typ over -40..+125 C) brackets
each rail at 0.277 A guaranteed and 0.537 A worst case.  The same four states
become 1.879 / 2.229 / 2.079 / 2.886 A: nothing a user can reach exceeds the
minimum trip (worst 13 % under it), and only a SIMULTANEOUS DOUBLE LIMITER FAULT
reaches 2.886 A, which trips the charger's own OCP and auto-retries -- below the
LTC4368's 3.33 A (50 mV across R75 15 mOhm) and far below F1's 5 A one-shot.

THE RAILS GOT MORE USABLE, NOT LESS: 0.277 A guaranteed each against the 0.15 A
at 5 V / 0.23 A at 3.3 V the superseded policy permitted at this corner.  No
copper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
Parts:
- R101: value 1.65k 1% -> 2.7k 1%; LCSC C4088673 -> C13167; MPN ERJ-PA3F1651V -> 0603WAF2701T5E; Manufacturer PANASONIC -> UNI-ROYAL(Uniroyal Elec); Note ILIM = 0.69 A typ (0.52-0.86 A) -> D-753 THE ACCESSORY CONCURRENCY LIMIT BECOMES HARDWARE. WAS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; Note_Sourcing SOURCING D-615 LIVE_RECORD. JLCPCB record read 2026-09-05T0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 -> SOURCING D-753 2026-09-18, verified live per D-096 through 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
- R97: value 1.5k 1% -> 2.7k 1%; LCSC C22843 -> C13167; MPN 0603WAF1501T5E -> 0603WAF2701T5E; Note ILIM = 1.18 x R[kOhm]^-1.072 = 0.76 A typ (0.57-0.96 A) -> D-753 THE ACCESSORY CONCURRENCY LIMIT BECOMES HARDWARE. WAS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; Note_Sourcing SOURCING D-615 LIVE_RECORD. JLCPCB record read 2026-09-05T0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 -> SOURCING D-753 2026-09-18, verified live per D-096 through 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
Changed lines of the file:
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@@
 			)
 		)
-		(property "Value" "1.5k 1%"
+		(property "Value" "2.7k 1%"
 			(at 422.37 258.52 0)
 			(show_name no)
@@
 			)
 		)
-		(property "MPN" "0603WAF1501T5E"
+		(property "MPN" "0603WAF2701T5E"
 			(at 422.37 255.52 0)
 			(hide yes)
@@
 			)
 		)
-		(property "LCSC" "C22843"
+		(property "LCSC" "C13167"
 			(at 422.37 255.52 0)
 			(hide yes)
@@
 			)
 		)
-		(property "Note_Sourcing" "SOURCING D-615 LIVE_RECORD. JLCPCB record read 2026-09-05T00:59:59Z: base library, stock 3722075, land 0603, Operating Temperature -55℃~+155℃; Power(Watts) 100mW; Resistance 1.5kΩ; Temperature Coefficient ±100ppm/℃; Tolerance ±1%; Type Thick Film Resistor; Voltage-Supply(Max) 75V. Gates: land working voltage vs the highest node; 2x the strict over-bound."
+		(property "Note_Sourcing" "SOURCING D-753 2026-09-18, verified live per D-096 through the JLCPCB parts API: LCSC C13167, UNI-ROYAL(Uniroyal Elec) 0603WAF2701T5E, 2.7 kOhm +/-1 %, 0603, 100 mW, +/-100 ppm/C, -55..+155 C, componentLibraryType = BASE (no extended-part fee), stock 1406950.  Same 0603WAF series as most of this board's 1 %% resistors.  R101's superseded ERJ-PA3F1651V was an EXTENDED part with 2763 in stock, so this also removes a sourcing risk."
 			(at 422.37 255.52 0)
 			(hide yes)
@@
 			)
 		)
-		(property "Note" "ILIM = 1.18 x R[kOhm]^-1.072 = 0.76 A typ (0.57-0.96 A)"
+		(property "Note" "D-753 THE ACCESSORY CONCURRENCY LIMIT BECOMES HARDWARE.  WAS 1.5 kOhm = 0.76 A typ, up to 1.01 A at the same tolerance.  TI SLVSFJ2B equation 1: ILIM = 1.18 x R[kOhm]^-1.072, so 2.7 kOhm sets 0.407 A typ; applying the WIDEST published tolerance ratio in the part's own EC table (min 0.68x / max 1.32x of typ over -40..+125 C, read off the 19.2 kOhm row) gives a guaranteed 0.277 A and a worst-case 0.537 A.  WHY IT MOVED: DEVICE_SPEC 6.3a answered the external first-spin review's combined-load item with a POLICY -- 'firmware must not raise both accessory rails to their per-rail maxima together' -- and a policy is not an enforcement mechanism.  THIS BOARD HAS NO ACCESSORY CURRENT MEASUREMENT: firmware can choose whether a rail is ON, and cannot know what an arbitrary external accessory then draws.  At the old values the hardware permitted far more than the policy did.  Modelled at the 3.0 V cell corner with the full 1.0 A internal +3V3 load, U12 at 90 % and U21 at 88 % into 4.95 V: the 5 V rail ALONE at its limiter drew 2.93 A and both rails at their GUARANTEED currents drew 2.74 A, against a BQ25185 IBAT_OCP MINIMUM of 2.5625 A (3.125 A typ, +/-18 %) -- so loads the Community Port invites could trip the pack protection and reset the device.  At 2.7 kOhm on both rails: 3V3 alone 1.88 A (+27 % margin), 5V alone 2.23 A (+13 %), BOTH at their guaranteed currents 2.08 A (+19 %).  Only a SIMULTANEOUS DOUBLE LIMITER FAULT reaches 2.89 A, which trips the BQ25185 OCP and auto-retries -- below the LTC4368's 3.33 A (50 mV / R75 15 mOhm) and far below F1's 5 A. THE ENVELOPE IS NOW BOUNDED BY SILICON AND NOT BY A DOCUMENT.  The rail still guarantees 0.277 A, which is MORE than the superseded policy permitted at this corner (0.15 A at 5 V / 0.23 A at 3.3 V).  Pinned by checks/demo_feature_contract.py F6."
 			(at 422.37 252.52 0)
 			(hide yes)
@@
 			)
 		)
-		(property "Value" "1.65k 1%"
+		(property "Value" "2.7k 1%"
 			(at 510.0 344.88 0)
 			(show_name no)
@@
 			)
 		)
-		(property "Manufacturer" "PANASONIC"
+		(property "Manufacturer" "UNI-ROYAL(Uniroyal Elec)"
 			(at 510.0 341.88 0)
 			(hide yes)
@@
 			)
 		)
-		(property "MPN" "ERJ-PA3F1651V"
+		(property "MPN" "0603WAF2701T5E"
 			(at 510.0 341.88 0)
 			(hide yes)
@@
 			)
 		)
-		(property "LCSC" "C4088673"
+		(property "LCSC" "C13167"
 			(at 510.0 341.88 0)
 			(hide yes)
@@
 			)
 		)
-		(property "Note_Sourcing" "SOURCING D-615 LIVE_RECORD. JLCPCB record read 2026-09-05T00:59:59Z: expand library, stock 2763, land 0603, Operating Temperature -55℃~+155℃; Power(Watts) 250mW; Resistance 1.65kΩ; Temperature Coefficient ±100ppm/℃; Tolerance ±1%; Type Thick Film Resistor. Gates: land working voltage vs the highest node; 2x the strict over-bound."
+		(property "Note_Sourcing" "SOURCING D-753 2026-09-18, verified live per D-096 through the JLCPCB parts API: LCSC C13167, UNI-ROYAL(Uniroyal Elec) 0603WAF2701T5E, 2.7 kOhm +/-1 %, 0603, 100 mW, +/-100 ppm/C, -55..+155 C, componentLibraryType = BASE (no extended-part fee), stock 1406950.  Same 0603WAF series as most of this board's 1 %% resistors.  R101's superseded ERJ-PA3F1651V was an EXTENDED part with 2763 in stock, so this also removes a sourcing risk."
 			(at 510.0 341.88 0)
 			(hide yes)
@@
 			)
 		)
-		(property "Note" "ILIM = 0.69 A typ (0.52-0.86 A)"
+		(property "Note" "D-753 THE ACCESSORY CONCURRENCY LIMIT BECOMES HARDWARE.  WAS 1.65 kOhm = 0.69 A typ, up to 0.91 A at the same tolerance.  TI SLVSFJ2B equation 1: ILIM = 1.18 x R[kOhm]^-1.072, so 2.7 kOhm sets 0.407 A typ; applying the WIDEST published tolerance ratio in the part's own EC table (min 0.68x / max 1.32x of typ over -40..+125 C, read off the 19.2 kOhm row) gives a guaranteed 0.277 A and a worst-case 0.537 A.  WHY IT MOVED: DEVICE_SPEC 6.3a answered the external first-spin review's combined-load item with a POLICY -- 'firmware must not raise both accessory rails to their per-rail maxima together' -- and a policy is not an enforcement mechanism.  THIS BOARD HAS NO ACCESSORY CURRENT MEASUREMENT: firmware can choose whether a rail is ON, and cannot know what an arbitrary external accessory then draws.  At the old values the hardware permitted far more than the policy did.  Modelled at the 3.0 V cell corner with the full 1.0 A internal +3V3 load, U12 at 90 % and U21 at 88 % into 4.95 V: the 5 V rail ALONE at its limiter drew 2.93 A and both rails at their GUARANTEED currents drew 2.74 A, against a BQ25185 IBAT_OCP MINIMUM of 2.5625 A (3.125 A typ, +/-18 %) -- so loads the Community Port invites could trip the pack protection and reset the device.  At 2.7 kOhm on both rails: 3V3 alone 1.88 A (+27 % margin), 5V alone 2.23 A (+13 %), BOTH at their guaranteed currents 2.08 A (+19 %).  Only a SIMULTANEOUS DOUBLE LIMITER FAULT reaches 2.89 A, which trips the BQ25185 OCP and auto-retries -- below the LTC4368's 3.33 A (50 mV / R75 15 mOhm) and far below F1's 5 A. THE ENVELOPE IS NOW BOUNDED BY SILICON AND NOT BY A DOCUMENT.  The rail still guarantees 0.277 A, which is MORE than the superseded policy permitted at this corner (0.15 A at 5 V / 0.23 A at 3.3 V).  Pinned by checks/demo_feature_contract.py F6."
 			(at 510.0 338.88 0)
 			(hide yes)

Commit message: demo: D-765 -- the accessory envelope was right and the silicon could not legally hold it
D-753's accessory-power envelope is retained to the digit; the PART could not
legally be set that low.  TI SLVSFJ2B section 5 -- the Device Comparison Table
of the datasheet D-753 itself cited -- gives the fitted TPS22950C an ILIM range
of 0.5-3.5 A, and this board programs 0.407 A.  The 0.05 A floor and the
"certified from 66 mA" UL note D-753 reasoned from belong to the base TPS22950,
which TI sells only in a WCSP package this board cannot use.  Three places in
this repository already held the right number -- POWER_FAULT_STATE_TABLE.md
says "treat 500 mA as the floor, not the target" -- and F6 had no clause that
could express the act at all, because it never read the limiter's part number.

U20/U22 are now the TPS22950-Q1 (SLVSGP6A, orderable TPS22950CQDDCRQ1, LCSC
C17349276, Active/Production, 4050 in stock), whose single specified ILIM range
is 0.05-3.5 A.  Same DDC0006A land pattern, same pinout, same ILIM equation and
EC rows, same auto-retry, same always-on true RCB, same FLT semantics, same
170 C TSD, plus AEC-Q100 grade 1, for about US$0.03 per device.  NO resistor, NO
copper and NO envelope number changed: F6 reproduces D-753's four modes exactly
(1.8786 / 2.2292 / 2.0791 / 2.8857 A, 13.01 % margin) and the .kicad_dru parsed
class table is proven byte-identical.

F6 keeps D-753's two clauses unweakened and adds three: the limiter must be a
part with a published range, the setting must be inside THAT part's range over
the resistor's whole tolerance band, and both rails must carry one MPN.  Eight
live controls, all refused; f6e is the board D-753 shipped and is refused by the
new range clause alone.

Also: kicad-cli sch export bom EXITS 0 while silently omitting an entire sheet
whose symbol is unparseable -- which made routing_ledger report 114 nets instead
of 174 -- so generate() now reconciles its population set against the board.
d750-critical-identity.json had pinne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
Parts:
- R103: Note single pull-up for the wired-OR of both TPS22950C FLT outpu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 -> single pull-up for the wired-OR of both TPS22950-Q1 FLT out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
- R131: Note ACC_5V_SW_EN safe-state pull-down, ADDED FBV2-S1-009. The CTO split the single ACC_5V_EN into ACC_5V_BOOST_EN (U3 P13 -> U21 EN) and ACC_5V_SW_EN (U3 P03 -> U22 ON), so the new net needs its own 100 k to ground. THE PULL-DOWN IS MANDATORY, NOT A CONVENIENCE: SLVSFJ2B specifies a 500 kOhm smart pull-down inside the TPS22950C and STILL REQUIRES AN EXTERNAL ONE, and the PCAL9535A powers up with every pin high-impedance - so without this resistor the 5 V accessory contact would be defined only by leakage between power-on and the first firmware write. 100 k matches R98 and R102 and costs 33 uA when the pin is driven high. -> ACC_5V_SW_EN safe-state pull-down, ADDED FBV2-S1-009. The CTO split the single ACC_5V_EN into ACC_5V_BOOST_EN (U3 P13 -> U21 EN) and ACC_5V_SW_EN (U3 P03 -> U22 ON), so the new net needs its own 100 k to ground. THE PULL-DOWN IS MANDATORY, NOT A CONVENIENCE: SLVSGP6A specifies a 500 kOhm smart pull-down inside the TPS22950-Q1 and it is not a substitute for an external one, and the PCAL9535A powers up with every pin high-impedance - so without this resistor the 5 V accessory contact would be defined only by leakage between power-on and the first firmware write. 100 k matches R98 and R102 and costs 33 uA when the pin is driven high.
- U20, U22: value TPS22950C -> TPS22950-Q1; symbol AQROOT_Beta:TPS22950C -> AQROOT_Beta:TPS22950-Q1; LCSC C7587833 -> C17349276; MPN TPS22950CDDCR -> TPS22950CQDDCRQ1
Other:
- note added: "=== C. COMMUNITY ACCESSORY POWER (D-086 / D-087 / D-088) - ONE TPS22950-Q1 MPN ON BOTH RAILS (D-765), FLT WIRE-OR (D-094) ==="
- note added: "ACC_3V3: +3V3 -> TPS22950-Q1 -> ACC_3V3_SW. R_ILIM 2.7k ~ 0.407 A typ, 0.277 A GUARANTEED / 0.537 A worst case (D-753). There is no accessory current measurement, so the LIMITER is the envelope and the GUARANTEE is the published figure."
- note added: "ACC_5V: BQ25185_SYS -> dedicated TPS61023 (5.0 V) -> dedicated TPS22950-Q1 -> ACC_5V_SW. R_ILIM 2.7k ~ 0.407 A typ, 0.277 A GUARANTEED / 0.537 A worst case (D-753). NOT USB VBUS. NOT the NFC fallback boost (O-3 REJECTED)."
- note removed: "=== C. COMMUNITY ACCESSORY POWER (D-086 / D-087 / D-088) - ONE TPS22950C FAMILY ON BOTH RAILS, FLT WIRE-OR (D-094) ==="
- note removed: "ACC_3V3: +3V3 -> TPS22950C -> ACC_3V3_SW. R_ILIM 1.5k ~ 0.76 A typ; PUBLISHED LIMIT 400 mA TOTAL across both connector contacts."
- note removed: "ACC_5V: BQ25185_SYS -> dedicated TPS61023 (5.0 V) -> dedicated TPS22950C -> ACC_5V_SW. R_ILIM 1.65k ~ 0.69 A typ; PUBLISHED LIMIT 300 mA TOTAL. NOT USB VBUS. NOT the NFC fallback boost (O-3 REJECTED)."
Changed lines of the file:
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@@
 		)
 	)
-	(text "=== C. COMMUNITY ACCESSORY POWER (D-086 / D-087 / D-088) - ONE TPS22950C FAMILY ON BOTH RAILS, FLT WIRE-OR (D-094) ==="
+	(text "=== C. COMMUNITY ACCESSORY POWER (D-086 / D-087 / D-088) - ONE TPS22950-Q1 MPN ON BOTH RAILS (D-765), FLT WIRE-OR (D-094) ==="
 		(exclude_from_sim no)
 		(at 330 232.0 0)
@@
 		)
 	)
-	(text "ACC_3V3: +3V3 -> TPS22950C -> ACC_3V3_SW. R_ILIM 1.5k ~ 0.76 A typ; PUBLISHED LIMIT 400 mA TOTAL across both connector contacts."
+	(text "ACC_3V3: +3V3 -> TPS22950-Q1 -> ACC_3V3_SW. R_ILIM 2.7k ~ 0.407 A typ, 0.277 A GUARANTEED / 0.537 A worst case (D-753). There is no accessory current measurement, so the LIMITER is the envelope and the GUARANTEE is the published figure."
 		(exclude_from_sim no)
 		(at 330 236.0 0)
@@
 		)
 	)
-	(text "ACC_5V: BQ25185_SYS -> dedicated TPS61023 (5.0 V) -> dedicated TPS22950C -> ACC_5V_SW. R_ILIM 1.65k ~ 0.69 A typ; PUBLISHED LIMIT 300 mA TOTAL. NOT USB VBUS. NOT the NFC fallback boost (O-3 REJECTED)."
+	(text "ACC_5V: BQ25185_SYS -> dedicated TPS61023 (5.0 V) -> dedicated TPS22950-Q1 -> ACC_5V_SW. R_ILIM 2.7k ~ 0.407 A typ, 0.277 A GUARANTEED / 0.537 A worst case (D-753). NOT USB VBUS. NOT the NFC fallback boost (O-3 REJECTED)."
 		(exclude_from_sim no)
 		(at 330 239.5 0)
@@
 	)
 	(symbol
-		(lib_id "AQROOT_Beta:TPS22950C")
+		(lib_id "AQROOT_Beta:TPS22950-Q1")
 		(at 359.41 261.62 0)
 		(unit 1)
@@
 			)
 		)
-		(property "Value" "TPS22950C"
+		(property "Value" "TPS22950-Q1"
 			(at 361.41 258.52 0)
 			(show_name no)
@@
 			)
 		)
-		(property "Datasheet" ""
+		(property "Datasheet" "https://www.ti.com/lit/ds/symlink/tps22950-q1.pdf"
 			(at 361.41 255.52 0)
 			(hide yes)
@@
 			)
 		)
-		(property "LCSC" "C7587833"
+		(property "LCSC" "C17349276"
 			(at 361.41 254.02 0)
 			(hide yes)
@@
 			)
 		)
-		(property "MPN" "TPS22950CDDCR"
+		(property "MPN" "TPS22950CQDDCRQ1"
 			(at 361.41 251.02 0)
 			(hide yes)
@@
 			)
 		)
-		(property "Note" "single pull-up for the wired-OR of both TPS22950C FLT outputs (D-094)"
+		(property "Note" "single pull-up for the wired-OR of both TPS22950-Q1 FLT outputs (D-094)"
 			(at 510.0 252.52 0)
 			(hide yes)
@@
 	)
 	(symbol
-		(lib_id "AQROOT_Beta:TPS22950C")
+		(lib_id "AQROOT_Beta:TPS22950-Q1")
 		(at 430.53 320.04 0)
 		(unit 1)
@@
 			)
 		)
-		(property "Value" "TPS22950C"
+		(property "Value" "TPS22950-Q1"
 			(at 432.53 316.94 0)
 			(show_name no)
@@
 			)
 		)
-		(property "Datasheet" ""
+		(property "Datasheet" "https://www.ti.com/lit/ds/symlink/tps22950-q1.pdf"
 			(at 432.53 313.94 0)
 			(hide yes)
@@
 			)
 		)
-		(property "LCSC" "C7587833"
+		(property "LCSC" "C17349276"
 			(at 432.53 312.44 0)
 			(hide yes)
@@
 			)
 		)
-		(property "MPN" "TPS22950CDDCR"
+		(property "MPN" "TPS22950CQDDCRQ1"
 			(at 432.53 309.44 0)
 			(hide yes)
@@
 			)
 		)
-		(property "Note" "ACC_5V_SW_EN safe-state pull-down, ADDED FBV2-S1-009. The CTO split the single ACC_5V_EN into ACC_5V_BOOST_EN (U3 P13 -> U21 EN) and ACC_5V_SW_EN (U3 P03 -> U22 ON), so the new net needs its own 100 k to ground. THE PULL-DOWN IS MANDATORY, NOT A CONVENIENCE: SLVSFJ2B specifies a 500 kOhm smart pull-down inside the TPS22950C and STILL REQUIRES AN EXTERNAL ONE, and the PCAL9535A powers up with every pin high-impedance - so without this resistor the 5 V accessory contact would be defined only by leakage between power-on and the first firmware write. 100 k matches R98 and R102 and costs 33 uA when the pin is driven high."
+		(property "Note" "ACC_5V_SW_EN safe-state pull-down, ADDED FBV2-S1-009. The CTO split the single ACC_5V_EN into ACC_5V_BOOST_EN (U3 P13 -> U21 EN) and ACC_5V_SW_EN (U3 P03 -> U22 ON), so the new net needs its own 100 k to ground. THE PULL-DOWN IS MANDATORY, NOT A CONVENIENCE: SLVSGP6A specifies a 500 kOhm smart pull-down inside the TPS22950-Q1 and it is not a substitute for an external one, and the PCAL9535A powers up with every pin high-impedance - so without this resistor the 5 V accessory contact would be defined only by leakage between power-on and the first firmware write. 100 k matches R98 and R102 and costs 33 uA when the pin is driven high."
 			(at 0 0 0)
 			(hide yes)
