File: hardware/demo/kicad/aqroot-demo/01_power_tree.kicad_sch (KiCad schematic)
At the start: 138 parts, among them J3 USB_C_Receptacle_USB2.0_16P, J4 JST-PH-2 BATTERY, Q2 NTMD4820N, Q3 NTMD4820N, Q4 BSS138, Q5 AO3401A, Q6 BSS138, Q7 BSS138, Q8 BSS138, Q9 BSS138, SW9 SW_SPDT, U10 USBLC6-2SC6, U11 BQ25185, U12 TPS63020, U13 TPS61023, U14 MAX17048, U18 LTC4368-1, U19 TLV7032, U20 TPS22950-Q1, U21 TPS61023, U22 TPS22950-Q1

Commit message: demo: D-771 -- the board published an accessory budget its own limiter could refuse to deliver, and ordered its battery protection chain against a typical
Closes the external-review hold on D-770.

(1) THE ENVELOPE HAD ONLY EVER BEEN CHECKED FROM ABOVE.  Every clause D-753
and D-765 wrote asks whether an accessory can pull TOO MUCH; none asks whether
the rail DELIVERS what the product promises.  D-098 locks the first five boards
at ACC_3V3_SW = 400 mA TOTAL and ACC_5V_SW = 300 mA TOTAL, and at 2.7 kOhm each
limiter GUARANTEED only 0.277 A.  R97 -> 1.78 kOhm (0.428 A guaranteed, +7.0 %)
and R101 -> 2.32 kOhm (0.322 A guaranteed, +7.4 %).

(2) THE PROTECTION CHAIN WAS ORDERED AGAINST A TYPICAL.  ADI guarantees the
LTC4368 forward threshold only as 40/50/60 mV; at R75 = 15 mOhm the LATCHING
breaker's band (2.640-4.040 A) OVERLAPPED the charger's RECOVERABLE IBAT_OCP
band (2.5625-3.6875 A), and RETRY is grounded here.  The board D-765 shipped
reached 2.886 A in double fault, above the breaker's own minimum: the clause
was FALSE on the board that passed it.  R75 -> 10 mOhm, same Bourns CRA2512-FZ
series and same 2512 land; the breaker is now 3.960-6.061 A, entirely above
IBAT_OCP's maximum.

F6 gains three clauses (published budget, chain ordered over tolerance,
converter capability) and six controls -- two of which are the boards D-753 and
D-765 actually shipped.  F7 gains the three passives, a BOM-row matcher that
parses GROUPED reference rows, and positive identity assertions.  The rail
ampacity audit gains the two accessory rails, declares +3V3 as pour-delivered,
and its method self-check now PARSES the .kicad_dru table it always claimed to
re-derive -- it had been reading a frozen copy that already carried a row D-753
retired.  .kicad_dru gains section 5f and its 5e residual is re-derived.

board 5849b658 -> c15672df; ZERO copper objects added or removed and every
copper Gerber byte-identical apart from its timestamp.  Connectivity 174/173/1
owner-approved/0 unappro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
Parts:
- R101: value 2.7k 1% -> 2.32k 1%; LCSC C13167 -> C22905; MPN 0603WAF2701T5E -> 0603WAF2321T5E; Note D-753 THE ACCESSORY CONCURRENCY LIMIT BECOMES HARDWARE. WAS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 -> D-771 THE PUBLISHED ACCESSORY BUDGET BECOMES A GUARANTEE. D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; Note_Sourcing SOURCING D-753 2026-09-18, verified live per D-096 through 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 -> SOURCING D-771 2026-09-18, verified live per D-096 through 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
- R75: value 15mR 1% 1W -> 10mR 1% 3W; LCSC C2073490 -> C840621; MPN CRA2512-FZ-R015ELF -> CRA2512-FZ-R010ELF; Note R_SENSE: I_OC,FWD = 50 mV / 15 mR = 3.33 A -> R_SENSE, LTC4368-1 FORWARD BREAKER. D-771 MOVED THIS FROM 1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; Note_Sourcing SOURCING D-615 LIVE_RECORD. JLCPCB record read 2026-09-05T0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 -> SOURCING D-771 2026-09-18, verified live per D-096 through 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
- R97: value 2.7k 1% -> 1.78k 1%; LCSC C13167 -> C22849; MPN 0603WAF2701T5E -> 0603WAF1781T5E; Note D-753 THE ACCESSORY CONCURRENCY LIMIT BECOMES HARDWARE. WAS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 -> D-771 THE PUBLISHED ACCESSORY BUDGET BECOMES A GUARANTEE. D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; Note_Sourcing SOURCING D-753 2026-09-18, verified live per D-096 through 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 -> SOURCING D-771 2026-09-18, verified live per D-096 through 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
Other:
- note added: "ACC_3V3: +3V3 -> TPS22950-Q1 -> ACC_3V3_SW. R_ILIM 1.78k ~ 0.636 A typ, 0.428 A GUARANTEED / 0.849 A worst case (D-771; was 2.7k at D-753). There is no accessory current measurement, so the LIMITER is the envelope and the GUARANTEE is the published figure -- and D-098 PUBLISHES 400 mA TOTAL for this rail across BOTH its J5 contacts, which 2.7k could not guarantee."
- note added: "ACC_5V: BQ25185_SYS -> dedicated TPS61023 (5.0 V) -> dedicated TPS22950-Q1 -> ACC_5V_SW. R_ILIM 2.32k ~ 0.479 A typ, 0.322 A GUARANTEED / 0.639 A worst case (D-771; was 2.7k at D-753), against the 300 mA TOTAL D-098 PUBLISHES for this rail across BOTH its J5 contacts. NOT USB VBUS. NOT the NFC fallback boost (O-3 REJECTED)."
- note added: "JST J4 -> F1 (5A backstop) -> BAT_RAW -> Q2 (stage 1, 2 FETs) -> BAT_MID -> Q3 (stage 2, 2 FETs) -> BAT_SENSE -> R75 10mR (D-771; was 15mR) -> BAT_PROTECTED_P -> BQ25185 BAT."
- note added: "LTC4368-1 ONLY (the -2 trips at -3 mV and blocks charging). RETRY grounded = latch-off; SHDN toggled low-then-high clears it. D-771 FORWARD BREAKER, OVER TOLERANCE: ADI Rev C guarantees dVSENSE,F as 40 / 50 / 60 mV over temperature -- 50 mV is a TYPICAL. R75 is 10 mOhm (was 15), so the breaker trips at 3.960 / 5.000 / 6.061 A, ENTIRELY ABOVE the BQ25185 IBAT_OCP band 2.5625 / 3.125 / 3.6875 A. TH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"
- note added: "REVERSE-POLARITY PROTECTION - IMPLEMENTED (FBV2-S1) D-050 / D-052 / D-064 / D-068. The placeholder is RETIRED. See block A, lower left, for the captured circuit: BAT_CONNECTOR_P -> F1 -> BAT_RAW -> Q2 -> BAT_MID -> Q3 -> BAT_SENSE -> R75 10mR -> BAT_PROTECTED_P -> U11 BAT Controller U18 LTC4368-1. Recovery branch in block B. BAT_CONNECTOR_P AND BAT_PROTECTED_P REMAIN INTENTIONALLY DISTINCT NETS. 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"
- note removed: "ACC_3V3: +3V3 -> TPS22950-Q1 -> ACC_3V3_SW. R_ILIM 2.7k ~ 0.407 A typ, 0.277 A GUARANTEED / 0.537 A worst case (D-753). There is no accessory current measurement, so the LIMITER is the envelope and the GUARANTEE is the published figure."
- note removed: "ACC_5V: BQ25185_SYS -> dedicated TPS61023 (5.0 V) -> dedicated TPS22950-Q1 -> ACC_5V_SW. R_ILIM 2.7k ~ 0.407 A typ, 0.277 A GUARANTEED / 0.537 A worst case (D-753). NOT USB VBUS. NOT the NFC fallback boost (O-3 REJECTED)."
- note removed: "JST J4 -> F1 (5A backstop) -> BAT_RAW -> Q2 (stage 1, 2 FETs) -> BAT_MID -> Q3 (stage 2, 2 FETs) -> BAT_SENSE -> R75 15mR -> BAT_PROTECTED_P -> BQ25185 BAT."
- note removed: "LTC4368-1 ONLY (the -2 trips at -3 mV and blocks charging). RETRY grounded = latch-off; SHDN toggled low-then-high clears it. UV unused: 510k to VIN per datasheet (V_UV/V_OV = 492.5 / 500 / 507.5 mV, hysteresis 20 / 25 / 32 mV). OV TRIP (P-21, D-104): R77 3.65M / R78 442k -> 4.63 V nominal, 4.48-4.78 V over comparator + 1% resistor tolerance. Release 4.40 V nominal. Above a 4.35 V-class pack, wel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"
- note removed: "REVERSE-POLARITY PROTECTION - IMPLEMENTED (FBV2-S1) D-050 / D-052 / D-064 / D-068. The placeholder is RETIRED. See block A, lower left, for the captured circuit: BAT_CONNECTOR_P -> F1 -> BAT_RAW -> Q2 -> BAT_MID -> Q3 -> BAT_SENSE -> R75 15mR -> BAT_PROTECTED_P -> U11 BAT Controller U18 LTC4368-1. Recovery branch in block B. BAT_CONNECTOR_P AND BAT_PROTECTED_P REMAIN INTENTIONALLY DISTINCT NETS. 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"

Commit message: demo: D-773 -- the 5 V setpoint was a number from a reference voltage TI does not publish, and it decides this board's thinnest margin
Third and last of the chain the CTO's withdrawal opened.  The pack cost of
ACC_5V_SW scales DIRECTLY with the boost's output voltage, and that voltage was
a constant in two places that disagreed:

    checks/demo_feature_contract.py   V_ACC5V = 4.95
    architecture/ARCHITECTURE.md      "VREF 0.6 V -> 4.99 V"

Both were derived from VREF = 0.6 V.  TI SLVSF14B gives the TPS61023's FB
reference as 580 / 595 / 610 mV in PWM mode -- typ 595, not 600 -- and R99's
own symbol note had carried the correct 0.595 V all along (the D-765 pattern:
this repository already held the number, in the one place nobody read).

Over R99 732k and R100 100k at their 1 % bands the real setpoint is
4.742 / 4.950 / 5.165 V.  Costed at 5.165 V, D-771's R101 = 2.32 kOhm left
0.52 % of margin between the 5 V rail at its limiter and IBAT_OCP's minimum --
the thinnest state this board has, and nobody knew the number.

R101 -> 2.37 kOhm (0603WAF2371T5E, LCSC C25964, same UNI-ROYAL 0603WAF series,
same 0603 land, verified live per D-096).  It is the E96 value nearest the
centre of its own COMPUTED legal window: below 2.298 kOhm the limiter's worst
case reaches the pack's minimum trip, above 2.478 kOhm the rail can no longer
guarantee the 300 mA D-098 publishes.  Delivery headroom 7.4 % -> 4.9 %, pack
margin 0.52 % -> 1.62 %.  D-771's 2.32 kOhm BROKE NO CLAUSE and this entry does
not pretend it did -- the control written to claim so was found not to refuse
and was replaced by one at 2.2 kOhm, past the computed bound.

F6 now DERIVES the setpoint from R99/R100/U21 read off the board, runs the
envelope on the worst case, reports the typical beside it, and gains a clause
nothing had ever checked: the divider's worst-case high must clear the
TPS61023's own VOVP minimum of 5.5 V (it does, by 6.1 %).  Three new controls,
all refused; F6 runs TWENTY-ONE.  F7's R101 entry ret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
Parts:
- R101: value 2.32k 1% -> 2.37k 1%; LCSC C22905 -> C25964; MPN 0603WAF2321T5E -> 0603WAF2371T5E; Note D-771 THE PUBLISHED ACCESSORY BUDGET BECOMES A GUARANTEE. D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 -> D-773 THE 5 V SETPOINT WAS A NUMBER FROM A WRONG REFERENCE,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; Note_Sourcing SOURCING D-771 2026-09-18, verified live per D-096 through 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 -> SOURCING D-773 2026-09-19, verified live per D-096 through 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
- R99: Note VOUT = 0.595 V x (1 + 732k/100k) = 4.95 V - identical divid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 -> ACC_5V_RAW SETPOINT. VOUT = VREF x (1 + R99/R100) = 4.95 V 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
Changed lines of the file:
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@@
 			)
 		)
-		(property "Note" "VOUT = 0.595 V x (1 + 732k/100k) = 4.95 V - identical divider to the NFC boost (BOM consolidation)"
+		(property "Note" "ACC_5V_RAW SETPOINT.  VOUT = VREF x (1 + R99/R100) = 4.95 V TYPICAL at 732k/100k - identical divider to the NFC boost (BOM consolidation).  D-773 PUT THE BAND BESIDE THE TYPICAL, because the pack cost of the accessory 5 V rail scales directly with this voltage and the envelope must be costed at the worst case.  TI SLVSF14B Electrical Characteristics gives VREF as 580 / 595 / 610 mV in PWM mode (585 / 601 in PFM); over R99 and R100 at their own 1 %% bands the setpoint is 4.742 / 4.950 / 5.165 V.  THIS NOTE WAS ALREADY RIGHT -- it has carried 0.595 V since it was written -- while architecture/ARCHITECTURE.md published 4.99 V from a VREF of 0.6 V and checks/demo_feature_contract.py carried 4.95 as a bare constant.  The contract now DERIVES the band from R99, R100 and U21 read off the board, runs the envelope on the 5.165 V worst case, and refuses a divider whose worst case reaches the TPS61023's own VOVP minimum of 5.5 V; this one clears it by 6.1 %%.  Pinned by checks/demo_feature_contract.py F6."
 			(at 461.74 338.88 0)
 			(hide yes)
@@
 			)
 		)
-		(property "Value" "2.32k 1%"
+		(property "Value" "2.37k 1%"
 			(at 510.0 344.88 0)
 			(show_name no)
@@
 			)
 		)
-		(property "MPN" "0603WAF2321T5E"
+		(property "MPN" "0603WAF2371T5E"
 			(at 510.0 341.88 0)
 			(hide yes)
@@
 			)
 		)
-		(property "LCSC" "C22905"
+		(property "LCSC" "C25964"
 			(at 510.0 341.88 0)
 			(hide yes)
@@
 			)
 		)
-		(property "Note_Sourcing" "SOURCING D-771 2026-09-18, verified live per D-096 through the JLCPCB parts API.  LCSC C22905, UNI-ROYAL(Uniroyal Elec) 0603WAF2321T5E, 2.32 kOhm +/-1 %, 0603, 100 mW, +/-100 ppm/C, -55..+155 C, componentLibraryType = expand, stock 6268.  SAME 0603WAF SERIES AND SAME MANUFACTURER as the 0603WAF2701T5E it replaces; same 0603 land, so no copper changes."
+		(property "Note_Sourcing" "SOURCING D-773 2026-09-19, verified live per D-096 through the JLCPCB parts API.  LCSC C25964, UNI-ROYAL(Uniroyal Elec) 0603WAF2371T5E, 2.37 kOhm +/-1 %%, 0603, 100 mW, +/-100 ppm/C, -55..+155 C, componentLibraryType = expand, stock 11268.  SAME 0603WAF SERIES, SAME MANUFACTURER and same 0603 land as the 0603WAF2321T5E it replaces, so no footprint, no copper and no assembly step changes -- only the resistance."
 			(at 510.0 341.88 0)
 			(hide yes)
@@
 			)
 		)
-		(property "Note" "D-771 THE PUBLISHED ACCESSORY BUDGET BECOMES A GUARANTEE.  D-753 made the accessory envelope hardware and D-765 corrected the silicon, but every clause either wrote asks only whether an accessory can pull TOO MUCH.  None asked whether the rail DELIVERS what the product promises.  D-098 (2026-08-23) locks the first five boards at ACC_3V3_SW = 400 mA TOTAL and ACC_5V_SW = 300 mA TOTAL and requires those numbers in accessory-facing documentation in those words -- and 2.7 kOhm GUARANTEES only 0.277 A on either rail.  The board published a budget its own limiter could refuse to deliver, on the two contacts the Community Port exists for.  TI SLVSGP6A equation 1: ILIM = 1.18 x R[kOhm]^-1.072, bracketed by the widest tolerance ratio in the part's own EC table (0.68x / 1.32x of typ over -40..+125 C, read off the 19.2 kOhm row) and by the programming resistor's own 1 % band, which D-771 also folded in -- the envelope modes had used the NOMINAL resistor alone.  R101 = 2.32 kOhm programs 0.479 A typ and brackets the 5 V rail at 0.322 A GUARANTEED / 0.639 A worst case, so the published 300 mA is guaranteed with 7.4 % headroom.  The 5 V rail is the expensive one: at the 3.0 V cell corner it costs 1.875 A of pack current per amp delivered, so its worst case alone draws 2.420 A against a 2.5625 A IBAT_OCP minimum -- 5.6 %, the thinnest margin on this board and the reason R101 cannot go lower.  U21 can source it: SLVSF14B equation 1 with ILIM_SW at its 2.7 A EC MINIMUM and L4 at its -20 %% corner gives 0.973 A at this operating point.  WAS 2.7 kOhm (D-753); 1.65 kOhm before that (D-750).  Pinned by checks/demo_feature_contract.py F6."
+		(property "Note" "D-773 THE 5 V SETPOINT WAS A NUMBER FROM A WRONG REFERENCE, AND IT DECIDES THIS RAIL'S MARGIN.  D-771 set R101 = 2.32 kOhm against a boost output modelled at 4.95 V, and ARCHITECTURE.md published 4.99 V; BOTH were derived from VREF = 0.6 V.  TI SLVSF14B's Electrical Characteristics gives the TPS61023's FB reference as 580 / 595 / 610 mV in PWM mode -- the TYPICAL is 595 mV, not 600 -- so over R99 732k and R100 100k at their own 1 %% bands the real setpoint is 4.742 / 4.950 / 5.165 V.  THE PACK COST OF THIS RAIL SCALES DIRECTLY WITH THAT VOLTAGE: at the worst-case 5.165 V the 5 V rail alone at its limiter drew 2.549 A against a BQ25185 IBAT_OCP MINIMUM of 2.5625 A -- 0.52 %% of margin, on the thinnest state this board has.  R101 = 2.37 kOhm programs 0.468 A typ and brackets the rail at 0.315 A GUARANTEED / 0.624 A worst case: the published 300 mA is still guaranteed with 4.9 %% headroom and the pack margin becomes 1.62 %%.  IT IS THE E96 VALUE NEAREST THE CENTRE OF ITS OWN LEGAL WINDOW, which is 2.298 .. 2.478 kOhm -- below 2.298 the limiter's worst case trips the pack, above 2.478 the rail cannot guarantee what D-098 publishes.  F6 now DERIVES the setpoint from R99/R100 and the part's own VREF band instead of carrying a constant, runs the envelope on the worst case, reports the typical beside it, and refuses a divider whose worst-case high reaches the TPS61023's own VOVP minimum of 5.5 V (margin 6.1 %%).  WAS 2.32 kOhm (D-771); 2.7 kOhm (D-753); 1.65 kOhm (D-750).  Pinned by checks/demo_feature_contract.py F6."
 			(at 510.0 338.88 0)
 			(hide yes)
