File: hardware/demo/kicad/aqroot-demo/01_power_tree.kicad_sch (KiCad schematic)
At the start: 138 parts, among them J3 USB_C_Receptacle_USB2.0_16P, J4 JST-PH-2 BATTERY, Q2 NTMD4820N, Q3 NTMD4820N, Q4 BSS138, Q5 AO3401A, Q6 BSS138, Q7 BSS138, Q8 BSS138, Q9 BSS138, SW9 SW_SPDT, U10 USBLC6-2SC6, U11 BQ25185, U12 TPS63020, U13 TPS61023, U14 MAX17048, U18 LTC4368-1, U19 TLV7032, U20 TPS22950-Q1, U21 TPS61023, U22 TPS22950-Q1

Commit message: demo: D-776 -- the as-built limits told firmware to read a signal this board does not have, and the list of signals it does not have is now computed off the copper
THE GENERATED FIRMWARE MAP'S OWN AS-BUILT LIMITS -- a block headed "facts
firmware cannot discover and must not get wrong" -- told firmware to infer
charging state "from VBUS presence plus the MAX17048 trend".  THERE IS NO
VBUS-PRESENCE SIGNAL ON THIS BOARD.  R104 150k and R105 220k divide
USB_VBUS_CHG to 2.973 V, C68 filters it, all three are FITTED, and
/01_POWER_TREE/VBUS_PRESENT reaches TP31 AND NOTHING ELSE -- no U1 pin, no
U2/U3 bit.  The same sentence stood in 01_power_tree.kicad_sch, in
08_buttons_expanders.kicad_sch and in Firmware/README.md, and the sheet-01
telemetry note added "raw VBUS never reaches the expander", which reads as
though the DIVIDED level does.

TWO MORE OF THE SAME SHAPE WERE UNDECLARED BESIDE IT, found by asking the
question of the whole board instead of one note:

  * /01_POWER_TREE/LTC4368_FAULT_N -- the LATCHING battery breaker's own FAULT
    output, reaching R81, R82, TP18 and Q9's GATE, whose drain is REC_FAULT_B
    and disappears into the autonomous dead-cell recovery chain.  FIRMWARE
    CANNOT OBSERVE THAT THE BATTERY BREAKER HAS TRIPPED.
  * Net-(U12-PG) -- the TPS63020's POWER GOOD, reaching R41 1M and TP8 only.

THE REAL DEFECT IS THAT THE LIST WAS REMEMBERED.  `limits` already carried
FUEL_GAUGE_ALRT_NOT_WIRED and ACC_BUS_READY_NOT_WIRED -- the PATTERN was right
and had been applied twice, BY HAND, so three nets of exactly that shape were
never added and one of them was named by another limit as though readable.

SO THE LIST IS DERIVED.  A net is FIRMWARE-REACHABLE iff it touches a pad of
U1, U2 or U3; BENCH-PROBED iff it touches a TP pad.  gen_firmware_hw_map.py
enumerates every net that is probed and not reachable OFF THE COPPER and
REFUSES TO EMIT if one is undeclared, or if a declaration names a net that has
since been wired -- both directions, which is the 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
Parts:
- U13: Note D-742 (2026-09-18) RECORDS TWO THINGS ABOUT THIS PART THAT FIRMWARE AND ANY REVIEWER MUST READ TOGETHER. (1) PIN 3 STAT2 IS INTENTIONALLY UNCONNECTED ON AQROOT DEMO - OWNER DECISION, 2026-09-17. The /BQ25185_STAT2 net is retained and fully routed on its other three contacts (R128 10k pull-up to +3V3, TP7 test point, and U2.19 = PCAL9535A U2 P16), but U11.3 itself has no escape. MEASURED REASON (D-734, re-measured D-741): U11.2's BAT_PROTECTED_P escape must leave on its own land centreline y=78.200 mm because 0.200 mm of pad clearance to U11.1's SYS land at y>=78.500 mm pins it there; D-269's 0.300 mm battery-conductor clearance then caps STAT2's escape at y<=77.800 mm, and U11.4's GND land at y<=77.500 mm floors it at y>=77.700 mm. The window is 0.100 mm against this board's published 0.200 mm minimum track width. It does not move with U11's position and it does not move with rotation, because BAT is pin 2 and STAT2 is pin 3 in every DLH0010A. A via-in-pad escape is impossible too: th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 -> D-742 (2026-09-18) RECORDS TWO THINGS ABOUT THIS PART THAT FIRMWARE AND ANY REVIEWER MUST READ TOGETHER. (1) PIN 3 STAT2 IS INTENTIONALLY UNCONNECTED ON AQROOT DEMO - OWNER DECISION, 2026-09-17. The /BQ25185_STAT2 net is retained and fully routed on its other three contacts (R128 10k pull-up to +3V3, TP7 test point, and U2.19 = PCAL9535A U2 P16), but U11.3 itself has no escape. MEASURED REASON (D-734, re-measured D-741): U11.2's BAT_PROTECTED_P escape must leave on its own land centreline y=78.200 mm because 0.200 mm of pad clearance to U11.1's SYS land at y>=78.500 mm pins it there; D-269's 0.300 mm battery-conductor clearance then caps STAT2's escape at y<=77.800 mm, and U11.4's GND land at y<=77.500 mm floors it at y>=77.700 mm. The window is 0.100 mm against this board's published 0.200 mm minimum track width. It does not move with U11's position and it does not move with rotation, because BAT is pin 2 and STAT2 is pin 3 in every DLH0010A. A via-in-pad escape is impossible too: th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
Other:
- note added: "VBUS_PRESENT: divided to 2.973 V at VBUS 5.0 V by R104 150k / R105 220k, filtered by C68. *** D-776 CORRECTED THE SECOND HALF OF THIS SENTENCE. It read 'raw VBUS NEVER reaches the expander', which reads as though the DIVIDED level does. IT DOES NOT: this node reaches TP31 and nothing else. The divider, the filter and the test point are all fitted and correct; the connection to a readable pin was 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"
- note removed: "VBUS_PRESENT: divided to 2.97 V at VBUS 5.0 V - raw VBUS NEVER reaches the expander. NFC: 3.3 V link FIT, 5 V link DNP, mutually exclusive, no trace cut needed to convert."
Changed lines of the file:
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@@
 			)
 		)
-		(property "Note" "D-742 (2026-09-18) RECORDS TWO THINGS ABOUT THIS PART THAT FIRMWARE AND ANY REVIEWER MUST READ TOGETHER. (1) PIN 3 STAT2 IS INTENTIONALLY UNCONNECTED ON AQROOT DEMO - OWNER DECISION, 2026-09-17. The /BQ25185_STAT2 net is retained and fully routed on its other three contacts (R128 10k pull-up to +3V3, TP7 test point, and U2.19 = PCAL9535A U2 P16), but U11.3 itself has no escape. MEASURED REASON (D-734, re-measured D-741): U11.2's BAT_PROTECTED_P escape must leave on its own land centreline y=78.200 mm because 0.200 mm of pad clearance to U11.1's SYS land at y>=78.500 mm pins it there; D-269's 0.300 mm battery-conductor clearance then caps STAT2's escape at y<=77.800 mm, and U11.4's GND land at y<=77.500 mm floors it at y>=77.700 mm. The window is 0.100 mm against this board's published 0.200 mm minimum track width. It does not move with U11's position and it does not move with rotation, because BAT is pin 2 and STAT2 is pin 3 in every DLH0010A. A via-in-pad escape is impossible too: the smallest barrel this board's own floors permit is 0.450 mm across and the land is 0.750 x 0.200 mm. SLUSF65B Table 4-1 states that STAT1 and STAT2 may be left floating if unused, so this is electrically inert. R128 and TP7 are RETAINED so the signal stays probeable and bodgeable for bench bring-up and a Rev-B respin; DO NOT DEPOPULATE THEM. (2) THE CHARGE-STATE DECODE THIS BOARD CARRIED WAS INVERTED ON STAT1, AND D-742 CORRECTED IT. The authority is SLUSF65B (August 2026) section 6.3.10 Table 6-2; the 'Table 7-2' the old notes cited is not a status table at all. THE CORRECT TABLE: STAT1 HIGH + STAT2 HIGH = charge completed, sleep, or charge disabled (including VBAT > VRCH); STAT1 HIGH + STAT2 LOW = NORMAL CHARGING IN PROGRESS; STAT1 LOW + STAT2 HIGH = RECOVERABLE FAULT (VIN_OVP, TS HOT, TS COLD, TSHUT, system short protection); STAT1 LOW + STAT2 LOW = NON-RECOVERABLE OR LATCH-OFF FAULT (ILIM/ISET pin short, BATOCP, safety timer expired). The retired text had STAT1 LOW meaning 'charging' and STAT1 HIGH with STAT2 LOW meaning 'fault' - both rows exactly backwards. COLLAPSED ONTO STAT1 ALONE, WHICH IS ALL THIS REVISION HAS: STAT1 LOW = FAULT, DIRECTLY OBSERVED (recoverable versus non-recoverable is not distinguishable); STAT1 HIGH = NOT FAULTED, and ambiguous between charging and charge-complete / sleep / disabled. THE DEMO KEEPS FAULT DETECTION AND LOSES THE CHARGING-VERSUS-COMPLETE DISTINCTION - the opposite way round from what D-734 and the owner decision assumed while working from the inverted table. Firmware must treat STAT1 LOW as a real charger fault, and must label any charging-versus-complete claim as an INFERENCE from VBUS_PRESENT and the MAX17048 voltage and state-of-charge trend. The no-battery limit cycle of section 6.3.10 toggles STAT2 while STAT1 stays HIGH, so it is not observable here either. REV-B: this needs a charger whose STAT2 pin is not adjacent to BAT, or a package with a land taller than 0.200 mm. A different U11 departure geometry alone removes only the second of the two walls and is not sufficient. PRIMARY SOURCE, IN THE REPOSITORY: hardware/demo/kicad/aqroot-demo/vendor/BQ25185/ti-bq25185-slusf65b-2026-08.pdf, sha256 c73ed7d63e6532bb05e26df30edd37c6ac2de310c1222a84a77625e15e133684."
+		(property "Note" "D-742 (2026-09-18) RECORDS TWO THINGS ABOUT THIS PART THAT FIRMWARE AND ANY REVIEWER MUST READ TOGETHER. (1) PIN 3 STAT2 IS INTENTIONALLY UNCONNECTED ON AQROOT DEMO - OWNER DECISION, 2026-09-17. The /BQ25185_STAT2 net is retained and fully routed on its other three contacts (R128 10k pull-up to +3V3, TP7 test point, and U2.19 = PCAL9535A U2 P16), but U11.3 itself has no escape. MEASURED REASON (D-734, re-measured D-741): U11.2's BAT_PROTECTED_P escape must leave on its own land centreline y=78.200 mm because 0.200 mm of pad clearance to U11.1's SYS land at y>=78.500 mm pins it there; D-269's 0.300 mm battery-conductor clearance then caps STAT2's escape at y<=77.800 mm, and U11.4's GND land at y<=77.500 mm floors it at y>=77.700 mm. The window is 0.100 mm against this board's published 0.200 mm minimum track width. It does not move with U11's position and it does not move with rotation, because BAT is pin 2 and STAT2 is pin 3 in every DLH0010A. A via-in-pad escape is impossible too: the smallest barrel this board's own floors permit is 0.450 mm across and the land is 0.750 x 0.200 mm. SLUSF65B Table 4-1 states that STAT1 and STAT2 may be left floating if unused, so this is electrically inert. R128 and TP7 are RETAINED so the signal stays probeable and bodgeable for bench bring-up and a Rev-B respin; DO NOT DEPOPULATE THEM. (2) THE CHARGE-STATE DECODE THIS BOARD CARRIED WAS INVERTED ON STAT1, AND D-742 CORRECTED IT. The authority is SLUSF65B (August 2026) section 6.3.10 Table 6-2; the 'Table 7-2' the old notes cited is not a status table at all. THE CORRECT TABLE: STAT1 HIGH + STAT2 HIGH = charge completed, sleep, or charge disabled (including VBAT > VRCH); STAT1 HIGH + STAT2 LOW = NORMAL CHARGING IN PROGRESS; STAT1 LOW + STAT2 HIGH = RECOVERABLE FAULT (VIN_OVP, TS HOT, TS COLD, TSHUT, system short protection); STAT1 LOW + STAT2 LOW = NON-RECOVERABLE OR LATCH-OFF FAULT (ILIM/ISET pin short, BATOCP, safety timer expired). The retired text had STAT1 LOW meaning 'charging' and STAT1 HIGH with STAT2 LOW meaning 'fault' - both rows exactly backwards. COLLAPSED ONTO STAT1 ALONE, WHICH IS ALL THIS REVISION HAS: STAT1 LOW = FAULT, DIRECTLY OBSERVED (recoverable versus non-recoverable is not distinguishable); STAT1 HIGH = NOT FAULTED, and ambiguous between charging and charge-complete / sleep / disabled. THE DEMO KEEPS FAULT DETECTION AND LOSES THE CHARGING-VERSUS-COMPLETE DISTINCTION - the opposite way round from what D-734 and the owner decision assumed while working from the inverted table. Firmware must treat STAT1 LOW as a real charger fault, and must NOT claim a charging-versus-complete state at all. *** D-776 CORRECTED THIS SENTENCE. It named VBUS_PRESENT as an input firmware could use, and VBUS_PRESENT REACHES TP31 AND NOTHING ELSE - no MCU pin and no expander bit - so THIS BOARD HAS NO USB-PRESENT SIGNAL AT ALL. The only remaining input is the MAX17048 voltage and state-of-charge TREND, which is weak and slow. Firmware must NOT display a charging state on this revision; display state-of-charge. The native USB CDC link detects a USB HOST, not a charger, and a dumb 5 V supply charges this board invisibly. See AQROOT_VBUS_PRESENT_UNREADABLE in the generated firmware map, whose list of probed-but-unreadable nets is COMPUTED off the copper. REV-B: move R104/R105/C68/TP31 beside U3 - USB_VBUS_CHG already runs within about 3 mm of U3's west column - and land VBUS_PRESENT on U3 P06; zero BOM change. Hauling it from where it sits now is NO_PATH at 0.200 mm on all three routable layers at both 0.10 and 0.05 mm lattices, with both ends launching (44 and 7 escapes). *** The no-battery limit cycle of section 6.3.10 toggles STAT2 while STAT1 stays HIGH, so it is not observable here either. REV-B: this needs a charger whose STAT2 pin is not adjacent to BAT, or a package with a land taller than 0.200 mm. A different U11 departure geometry alone removes only the second of the two walls and is not sufficient. PRIMARY SOURCE, IN THE REPOSITORY: hardware/demo/kicad/aqroot-demo/vendor/BQ25185/ti-bq25185-slusf65b-2026-08.pdf, sha256 c73ed7d63e6532bb05e26df30edd37c6ac2de310c1222a84a77625e15e133684."
 			(at 53.34 105.41 0)
 			(hide yes)
@@
 		)
 	)
-	(text "VBUS_PRESENT: divided to 2.97 V at VBUS 5.0 V - raw VBUS NEVER reaches the expander. NFC: 3.3 V link FIT, 5 V link DNP, mutually exclusive, no trace cut needed to convert."
+	(text "VBUS_PRESENT: divided to 2.973 V at VBUS 5.0 V by R104 150k / R105 220k, filtered by C68. *** D-776 CORRECTED THE SECOND HALF OF THIS SENTENCE. It read 'raw VBUS NEVER reaches the expander', which reads as though the DIVIDED level does. IT DOES NOT: this node reaches TP31 and nothing else. The divider, the filter and the test point are all fitted and correct; the connection to a readable pin was never made, so THIS REVISION HAS NO USB-PRESENT SIGNAL. 2.973 V would be a valid PCAL9535A logic HIGH on +3V3 (VIH = 2.31 V) at an 89.2 kOhm source impedance, so the intended connection is electrically sound and is a REV-B item: move R104/R105/C68/TP31 beside U3 and land on U3 P06. *** NFC: 3.3 V link FIT, 5 V link DNP, mutually exclusive, no trace cut needed to convert."
 		(exclude_from_sim no)
 		(at 460 366.0 0)

Commit message: demo: D-777 · D-778 · D-779 -- the battery connector had no rating in this repository, the derating rule was run against the specification instead of the part, and an extracted datasheet changed a unit that a proof was built on
Closes the round-3 external review hold on D-776.  All six reproduced items
are closed by measurement.  NO COPPER MOVED: every copper Gerber, both drill
files and Edge_Cuts are byte-identical to the D-776 package apart from
timestamps.  One BOM row changed -- C85 100nF -> 1uF, onto a line this board
already buys.  Board 8c548ece -> 880a2ece.

D-777  J4 is a JST B2B-PH-K-S(LF)(SN), published at 2 A AC/DC (AWG #24) --
       the LOWEST number in the battery path, below the BQ25185's 2.5625 A
       IBAT_OCP minimum, D-771's 3.960 A breaker and F1's 5 A fuse.  D-775's
       published simultaneous envelope sat at 2.2715 A, 13.6 % OVER, and
       D-776 passed in that state.  Holding it under 2 A by VCELL alone needs
       a 4.16 V pack, so the bounded term is the internal one: while BOTH
       accessory rails are enabled firmware RESERVES the sub-GHz TX path, the
       NFC field and the IR transmitter, enforced in SpiBusB::beginTransmit.
       The connection carries 1.8797 A, 6.0 % inside its rating; D-098's
       400/300 mA are both still guaranteed.  Rating, rated gauge, applicable
       wire range and the pack's lead gauge are all PARSED from archived
       vendor text.  The JST B2B-XH-A 3 A upgrade is confirmed live, costed
       and deferred to REV-B (needs an owner protected-copper exception on
       BAT_CONNECTOR_P); a first-article J4 temperature-rise measurement is
       added instead.

D-778  Twenty-four value strings UNDERSTATE the part the BOM buys, so three
       of D-774's five derating exceptions were against a rating this board
       does not have.  Ratings now come from the part, joined reference ->
       LCSC -> the committed live distributor record; all 76 fitted
       capacitors covered, a missing record is a re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
Parts:
- R75: Note R_SENSE, LTC4368-1 FORWARD BREAKER. D-771 MOVED THIS FROM 15 mOhm. ADI LTC4368 Rev C Electrical Characteristics guarantees dVSENSE,F -- the forward overcurrent fault threshold -- as 40 / 50 / 60 mV over the full operating temperature range. 50 mV is a TYPICAL, and every document in this repository had used it as a limit. At 15 mOhm +/-1 % the breaker's real band was 2.640 .. 4.040 A, which OVERLAPPED the BQ25185's IBAT_OCP band of 2.5625 .. 3.6875 A (3.125 A typ +/-18 %, SLUSF65B) by 1.05 A -- and RETRY is grounded, so this breaker LATCHES OFF and is cleared only by toggling SHDN while IBAT_OCP hiccups and auto-retries. On an unlucky unit the LATCHING protection fired first. At 10 mOhm +/-1 % the band is 3.960 .. 6.061 A, ENTIRELY ABOVE IBAT_OCP's 3.6875 A maximum, so the recoverable protection is guaranteed to act first on EVERY unit. The breaker still beats F1: its propagation delay is 3-18 us (tp(GATE)) against a 5 A fast-acting Nano2 that needs 5 s at 200 % of rating, so ordering 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 -> R_SENSE, LTC4368-1 FORWARD BREAKER. D-771 MOVED THIS FROM 15 mOhm. ADI LTC4368 Rev C Electrical Characteristics guarantees dVSENSE,F -- the forward overcurrent fault threshold -- as 40 / 50 / 60 mV over the full operating temperature range. 50 mV is a TYPICAL, and every document in this repository had used it as a limit. At 15 mOhm +/-1 % the breaker's real band was 2.640 .. 4.040 A, which OVERLAPPED the BQ25185's IBAT_OCP band of 2.5625 .. 3.6875 A (3.125 A typ +/-18 %, SLUSF65B) by 1.05 A -- and RETRY is grounded, so this breaker LATCHES OFF and is cleared only by toggling SHDN while IBAT_OCP hiccups and re-enables the BATFET after tREC_SC. D-779 COMPLETES THAT SENTENCE from SLUSF65B 6.3.7.3: the hiccup is not indefinite -- 4 to 7 consecutive trips inside a 2 s window leave the BATFET OFF until a valid VIN is connected, so a SUSTAINED battery overcurrent is a battery-only dead stop that needs USB to clear. The ordering D-771 set is unchanged and still right; what changes is the stat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
Changed lines of the file:
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@@
 			)
 		)
-		(property "Note" "R_SENSE, LTC4368-1 FORWARD BREAKER.  D-771 MOVED THIS FROM 15 mOhm.  ADI LTC4368 Rev C Electrical Characteristics guarantees dVSENSE,F -- the forward overcurrent fault threshold -- as 40 / 50 / 60 mV over the full operating temperature range.  50 mV is a TYPICAL, and every document in this repository had used it as a limit.  At 15 mOhm +/-1 % the breaker's real band was 2.640 .. 4.040 A, which OVERLAPPED the BQ25185's IBAT_OCP band of 2.5625 .. 3.6875 A (3.125 A typ +/-18 %, SLUSF65B) by 1.05 A -- and RETRY is grounded, so this breaker LATCHES OFF and is cleared only by toggling SHDN while IBAT_OCP hiccups and auto-retries.  On an unlucky unit the LATCHING protection fired first.  At 10 mOhm +/-1 % the band is 3.960 .. 6.061 A, ENTIRELY ABOVE IBAT_OCP's 3.6875 A maximum, so the recoverable protection is guaranteed to act first on EVERY unit.  The breaker still beats F1: its propagation delay is 3-18 us (tp(GATE)) against a 5 A fast-acting Nano2 that needs 5 s at 200 % of rating, so ordering against the one-shot fuse is a TIME-CURRENT result, not a threshold comparison.  Reverse threshold scales with it: -42/-50/-58 mV gives 4.16 .. 5.86 A, still far above any charge current this board programs (ICHG 769 mA).  Dissipation falls from 0.146 W to 0.098 W at 3.125 A, and D-193's fuel-gauge offset from 26 mV to 17 mV at the 1.75 A pack worst case.  Pinned by checks/demo_feature_contract.py F6."
+		(property "Note" "R_SENSE, LTC4368-1 FORWARD BREAKER.  D-771 MOVED THIS FROM 15 mOhm.  ADI LTC4368 Rev C Electrical Characteristics guarantees dVSENSE,F -- the forward overcurrent fault threshold -- as 40 / 50 / 60 mV over the full operating temperature range.  50 mV is a TYPICAL, and every document in this repository had used it as a limit.  At 15 mOhm +/-1 % the breaker's real band was 2.640 .. 4.040 A, which OVERLAPPED the BQ25185's IBAT_OCP band of 2.5625 .. 3.6875 A (3.125 A typ +/-18 %, SLUSF65B) by 1.05 A -- and RETRY is grounded, so this breaker LATCHES OFF and is cleared only by toggling SHDN while IBAT_OCP hiccups and re-enables the BATFET after tREC_SC.  D-779 COMPLETES THAT SENTENCE from SLUSF65B 6.3.7.3: the hiccup is not indefinite -- 4 to 7 consecutive trips inside a 2 s window leave the BATFET OFF until a valid VIN is connected, so a SUSTAINED battery overcurrent is a battery-only dead stop that needs USB to clear.  The ordering D-771 set is unchanged and still right; what changes is the stated consequence of reaching the recoverable limit.  On an unlucky unit the LATCHING protection fired first.  At 10 mOhm +/-1 % the band is 3.960 .. 6.061 A, ENTIRELY ABOVE IBAT_OCP's 3.6875 A maximum, so the recoverable protection is guaranteed to act first on EVERY unit.  The breaker still beats F1: its propagation delay is 3-18 us (tp(GATE)) against a 5 A fast-acting Nano2 that needs 5 s at 200 % of rating, so ordering against the one-shot fuse is a TIME-CURRENT result, not a threshold comparison.  Reverse threshold scales with it: -42/-50/-58 mV gives 4.16 .. 5.86 A, still far above any charge current this board programs (ICHG 769 mA).  Dissipation falls from 0.146 W to 0.098 W at 3.125 A, and D-193's fuel-gauge offset from 26 mV to 17 mV at the 1.75 A pack worst case.  Pinned by checks/demo_feature_contract.py F6."
 			(at 84.55 251.25 0)
 			(hide yes)
