File: hardware/demo/kicad/aqroot-demo/01_power_tree.kicad_sch (KiCad schematic)
At the start: 138 parts, among them J3 USB_C_Receptacle_USB2.0_16P, J4 JST-PH-2 BATTERY, Q2 NTMD4820N, Q3 NTMD4820N, Q4 BSS138, Q5 AO3401A, Q6 BSS138, Q7 BSS138, Q8 BSS138, Q9 BSS138, SW9 SW_SPDT, U10 USBLC6-2SC6, U11 BQ25185, U12 TPS63020, U13 TPS61023, U14 MAX17048, U18 LTC4368-1, U19 TLV7032, U20 TPS22950-Q1, U21 TPS61023, U22 TPS22950-Q1

Commit message: demo: D-780/D-781 close Round-3 Q11 and battery blockers
Parts:
- J4: value JST-PH-2 BATTERY -> BATTERY PIGTAIL 26AWG; LCSC C131337 -> (none); MPN B2B-PH-K-S(LF)(SN) -> D-781-BAT-PIGTAIL; Manufacturer JST -> AQROOT manual harness; Note2 SOURCING 2026-08-23 (FBV2-S2-002) (B-71). B2B-PH-K-S(LF)(SN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 -> D-781 2026-09-19. J4 is NOT a purchased PCB connector and i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; now left out of the parts list
Changed lines of the file:
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@@
 		(body_style 1)
 		(exclude_from_sim no)
-		(in_bom yes)
+		(in_bom no)
 		(on_board yes)
-		(in_pos_files yes)
+		(in_pos_files no)
 		(dnp no)
 		(fields_autoplaced yes)
@@
 			)
 		)
-		(property "Value" "JST-PH-2 BATTERY"
+		(property "Value" "BATTERY PIGTAIL 26AWG"
 			(at 255.27 134.6199 0)
 			(show_name no)
@@
 			)
 		)
-		(property "Datasheet" ""
+		(property "Datasheet" "docs/full-beta-v2/assembly/BATTERY_HARNESS.json"
 			(at 252.73 132.08 0)
 			(hide yes)
@@
 			)
 		)
-		(property "Description" "Generic connector, single row, 01x02, script generated (kicad-library-utils/schlib/autogen/connector/)"
+		(property "Description" "Manual battery pigtail land: two 0.75 mm PTH pads at 2.00 mm pitch; no JST header fitted. Board-side 26 AWG red/black wires terminate in frozen Molex Micro-Lock Plus 2.0 W/W harness per D-781."
 			(at 252.73 132.08 0)
 			(hide yes)
@@
 			)
 		)
-		(property "Note2" "SOURCING 2026-08-23 (FBV2-S2-002) (B-71). B2B-PH-K-S(LF)(SN) = LCSC C131337, stock 378913. J6 was normalised to this same string. LCSC/JLC library state verified live on 2026-08-23 through the JLCPCB parts API (D-096). Stock is a snapshot, not a guarantee."
+		(property "Note2" "D-781 2026-09-19. J4 is NOT a purchased PCB connector and is excluded from BOM/CPL. Reuse the existing two plated holes without moving protected battery copper. Use Molex 2175012101 red and 2175011101 black factory pre-crimped 26 AWG pigtails in 5055700201; solder red to J4.1 BAT_CONNECTOR_P and black to J4.2 GND after a stripped-conductor fit check in an actual finished 0.75 mm J4 PTH. Battery side is 2137192021 + 2137201000 after incoming lead-OD qualification; final detachable interface is Micro-Lock Plus 2.0 W/W. See assembly/BATTERY_HARNESS.json and THT_LEAD_TRIM.md."
 			(at 252.73 132.08 0)
 			(hide yes)
@@
 			)
 		)
-		(property "LCSC" "C131337"
+		(property "LCSC" ""
 			(at 252.73 132.08 0)
 			(hide yes)
@@
 			)
 		)
-		(property "Manufacturer" "JST"
+		(property "Manufacturer" "AQROOT manual harness"
 			(at 252.73 132.08 0)
 			(hide yes)
@@
 			)
 		)
-		(property "MPN" "B2B-PH-K-S(LF)(SN)"
+		(property "MPN" "D-781-BAT-PIGTAIL"
 			(at 252.73 132.08 0)
 			(hide yes)
