File: hardware/demo/kicad/aqroot-demo/09_community_header.kicad_sch (KiCad schematic)
At the start: 37 parts, among them J5 COMMUNITY_PORT_1x24, J8 QWIIC_STEMMA_QT, Q10 2N7002, U16 TCA4307DGKR

Commit message: demo: apply schematic simplification ECO
Parts:
- removed D3: TPD4E1B06DRLR, Package_TO_SOT_SMD:SOT-563, symbol AQROOT_Beta:TPD4E1B06DRLR
- removed R51, R52, R53, R54, R57, R58, R59, R60: 100R 1%, Resistor_SMD:R_0603_1608Metric, symbol Device:R
Connections:
- net XGPIO0_HDR: no longer names the net of J5.9 (Pin_9)
- net XGPIO1_HDR: no longer names the net of J5.10 (Pin_10)
- net XGPIO2_HDR: no longer names the net of J5.11 (Pin_11)
- net XGPIO3_HDR: no longer names the net of J5.12 (Pin_12)
- net XGPIO6_HDR: no longer names the net of J5.15 (Pin_15)
- net XGPIO6_HDR: no longer D4.4 (IO3)
- net XGPIO7_HDR: no longer names the net of J5.16 (Pin_16)
- net XGPIO7_HDR: no longer D4.6 (IO4)
- net XGPIO8_HDR: no longer names the net of J5.17 (Pin_17)
- net XGPIO8_HDR: no longer D5.1 (IO1)
- net XGPIO9_HDR: no longer names the net of J5.18 (Pin_18)
- net XGPIO9_HDR: no longer D5.3 (IO2)
- no-connect marks 4 -> 16
Other:
- note added: "ACCESSORY POWER SEQUENCING - CTO RULING, FBV2-S1-009 THE SINGLE ACC_5V_EN IS SPLIT INTO TWO INDEPENDENT ENABLES: U3 P13 ACC_5V_BOOST_EN -> TPS61023 EN (U21, SHEET 01) U3 P03 ACC_5V_SW_EN -> TPS22950C ON (U22, SHEET 01) BOTH CARRY THEIR OWN 100 k EXTERNAL PULL-DOWN, SO BOTH ARE OFF BEFORE FIRMWARE RUNS. THE TWO 5 V CONTROLS REMAIN INDEPENDENT. POWER-UP: 1 VERIFY ACC_DETECT_N ASSERTED 2 ACC_3V3_EN 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"
- note added: "COMMUNITY EXPANSION PORT - AQROOT DEMO SCHEMATIC ECO J5 = 24-CONTACT ORDER-B PHYSICAL INTERFACE 1 5V 2 GND 3 3V3 4 SDA 5 SCL 6 GND 7 NATIVE_A 8 NATIVE_B 9 NC 10 NC 11 NC 12 NC 13 XGPIO4 14 XGPIO5 15 NC 16 NC 17 NC 18 NC 19 GND 20 WAKE 21 DET 22 3V3 23 GND 24 5V AQROOT DEMO EXPOSES ONLY XGPIO4 AND XGPIO5. CONTACTS 9-12 AND 15-18 ARE EXPLICITLY NC. BOTH SWITCHED-RAIL CONTACT PAIRS SHARE THEIR EXIST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"
- note removed: "ACCESSORY POWER SEQUENCING - CTO RULING, FBV2-S1-009 THE SINGLE ACC_5V_EN IS SPLIT INTO TWO INDEPENDENT ENABLES: U3 P13 ACC_5V_BOOST_EN -> TPS61023 EN (U21, SHEET 01) U23 P04 ACC_5V_SW_EN -> TPS22950C ON (U22, SHEET 01) BOTH CARRY THEIR OWN 100 k EXTERNAL PULL-DOWN, SO BOTH ARE OFF BEFORE FIRMWARE RUNS. U23 P04 WAS A SPARE; ELEVEN ORDINARY SPARES PLUS RESERVED_SPARE REMAIN. POWER-UP: 1 VERIFY ACC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"
- note removed: "COMMUNITY EXPANSION PORT - MIGRATED FBV2-S1-009 J5 = SAMTEC BCS-112-S-D-HE 2 x 12, 24 ACTIVE CONTACTS 2.54 mm, FEMALE, HORIZONTAL ENTRY, THROUGH-HOLE, 30 uin GOLD FOOTPRINT FIG 3 REV B: 2.54 IN ROW, 7.87 BETWEEN ROWS, 0.71 PTH 1 XGPIO0 2 EXT_SCL 3 ACC_3V3_SW 4 GND 5 XGPIO1 6 EXT_SDA 7 NATIVE_A 8 XGPIO2 9 GND 10 ACC_5V_SW 11 NATIVE_B 12 XGPIO3 13 XGPIO4 14 WAKE_ATTN_N 15 ACC_3V3_SW 16 GND 17 XGPIO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"
