File: hardware/demo/kicad/aqroot-demo/09_community_header.kicad_sch (KiCad schematic)
At the start: 28 parts, among them J5 COMMUNITY_PORT_1x24, J8 QWIIC_STEMMA_QT, Q10 2N7002, U16 TCA4307DGKR

Commit message: demo: the BOM is THREE QUARTERS orderable -- 122 part identities grafted from prior CTO audits, every one re-read off the PART instead of the line, and four gates that had never been run (D-614)
NO COPPER CHANGED.  The authoritative board is byte-identical at
c8e421aa50144fe396aedb5e226aaabeb815bd69ffaf6e04f549ded43831d103 and 26 of the
package's 28 artifacts are normalised-sha-identical to D-613's; the two that
moved are the two BOM views.

FAB7 coverage 25.9% -> 75.3%, orderable references 64 -> 186 of 247.
36 BOM lines / 122 references gained Manufacturer / MPN / LCSC -- 487 properties
across nine schematic sheets, replayable to byte-identical sheets.

Four things the mechanical answer would have got wrong: a REJECTED audit row's
JLC Manufacturer column names the match that was THROWN OUT (16 of 31 grafts);
the rating belongs to the PART, not the line; the designator is not the
identity; and the beta-dm 0 ohm current gate had never been run on five of the
Demo's eight links.

Two defects in the instruments fixed: the value parser could not read 15mR, and
MANIFEST.json hashed only the ROOT schematic sheet while nine child sheets
changed.

Re-proved on this tree: verify_promotion.py 14/14, FAB1-FAB6 + FAB8 PASS,
POP1-POP4, P1-P4, protected copper 15 nets / 393 objects IDENTICAL.
FAB7 still FAILS and is partitioned: 8 lines / 16 parts TUNE, 26 lines /
45 parts genuinely open.

Co-Authored-By: Claude Opus 5 <noreply@anthropic.com>
Parts:
- C37, C38: LCSC (none) -> C106858; MPN (none) -> CC0603KRX7R8BB105; Manufacturer (none) -> YAGEO; Note_Sourcing (none) -> SOURCING D-614. EXACT_PRIOR from the beta-dm audit line '1u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
- C39: LCSC (none) -> C14663; MPN (none) -> CC0603KRX7R9BB104; Manufacturer (none) -> YAGEO; Note_Sourcing (none) -> SOURCING D-614. EXACT_PRIOR from the beta-dm audit line '10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
- J8: MPN (none) -> SM04B-SRSS-TB(LF)(SN); Manufacturer (none) -> JST; Note_Sourcing (none) -> SOURCING D-614. REFERENCE_RULING from the beta-dm audit lin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
- R46, R63: LCSC (none) -> C25804; MPN (none) -> 0603WAF1002T5E; Manufacturer (none) -> UNI-ROYAL(Uniroyal Elec); Note_Sourcing (none) -> SOURCING D-614. EXACT_PRIOR from the beta-dm audit line '10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
- R47, R48: LCSC (none) -> C23345; MPN (none) -> 0603WAF220JT5E; Manufacturer (none) -> UNI-ROYAL(Uniroyal Elec); Note_Sourcing (none) -> SOURCING D-614. EXACT_PRIOR from the beta-dm audit line '22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
- R55, R56, R61, R62, R64: LCSC (none) -> C22775; MPN (none) -> 0603WAF1000T5E; Manufacturer (none) -> UNI-ROYAL(Uniroyal Elec); Note_Sourcing (none) -> SOURCING D-614. EXACT_PRIOR from the beta-dm audit line '10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
- R66: LCSC (none) -> C23138; MPN (none) -> 0603WAF3300T5E; Manufacturer (none) -> UNI-ROYAL(Uniroyal Elec); Note_Sourcing (none) -> SOURCING D-614. EXACT_PRIOR from the beta-dm audit line '33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

Commit message: demo: the BOM is 100% ORDERABLE and the safety part was ordered in the WRONG PACKAGE -- 61 identities ruled against a live distributor record, and a screen that asks the C26 question of every line at once (D-615)
D-614 named this task and named what stopped it: D-096 binds -- a part number
configured from an ordering scheme is a hypothesis until a distributor record
confirms lifecycle and stock, and that session had none to read.  This one read
the JLCPCB catalogue 225 times and KEPT every answer, each stamped with the UTC
minute it was read.

NO COPPER CHANGED.  The authoritative board is byte-identical at
c8e421aa50144fe396aedb5e226aaabeb815bd69ffaf6e04f549ded43831d103.

FAB7 IS CLOSED.  Coverage 75.3% -> 100.0%, orderable 186 -> 247 of 247,
needs_a_sourcing_decision ZERO lines, and fab_package_contract.py reads
FAB1-FAB8 PASS for the first time.

THE FINDING.  screen_part_land_parity.py asks D-613's C26 question of every
sourced line at once against the catalogue's own package field: 119 lines carry
a code, 75 are comparable, 74 MATCH and U18 did not.  The land is MSOP-10; the
BOM ordered LTC4368IDD-1#PBF, and DD is DFN-10-EP(3x3) -- against D-099, which
locked LTC4368IMS-1#PBF under FBV2-PWR-002's "no bottom-terminated parts" on
the single most safety-critical component.  The cached library symbol AND the
project .kicad_sym both still carried it, with a Package field describing a DFN
beside a Footprint field already reading MSOP-10.  Corrected to
LTC4368IMS-1#TRPBF, LCSC C688401 -- the tape-and-reel order code of the
identical device, D-210's precedent, not an electrical change.

Three things the obvious answer would have got wrong: R69 is 1.87 ohm and its
part is 0603WAF187KT5E while 0603WAF1873T5E is 187 kOhm; R95's node over-bound
UNDERSTATES its dissipation because a reversed cell adds in series (154 mW vs
54 mW); and R24/C12's Value strings are looser than their own symbol notes.
NET_MAX_DC grew 17 -> 48 established nodes to give the new dissipation gate
nu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
Parts:
- J8: LCSC (none) -> C160404; Note_Sourcing SOURCING D-614. REFERENCE_RULING from the beta-dm audit lin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 -> SOURCING D-615 LIVE_RECORD, SUPERSEDING THE D-614 REFERENCE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
- R49, R50: LCSC (none) -> C22843; MPN (none) -> 0603WAF1501T5E; Manufacturer (none) -> UNI-ROYAL(Uniroyal Elec); Note_Sourcing (none) -> SOURCING D-615 LIVE_RECORD. JLCPCB record read 2026-09-05T0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
Changed lines of the file:
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@@
+			)
+		)
+		(property "Manufacturer" "UNI-ROYAL(Uniroyal Elec)"
+			(at 251.46 45.72 0)
+			(hide yes)
+			(show_name no)
+			(do_not_autoplace no)
+			(effects
+				(font
+					(size 1.27 1.27)
+				)
+			)
+		)
+		(property "MPN" "0603WAF1501T5E"
+			(at 251.46 45.72 0)
+			(hide yes)
+			(show_name no)
+			(do_not_autoplace no)
+			(effects
+				(font
+					(size 1.27 1.27)
+				)
+			)
+		)
+		(property "LCSC" "C22843"
+			(at 251.46 45.72 0)
+			(hide yes)
+			(show_name no)
+			(do_not_autoplace no)
+			(effects
+				(font
+					(size 1.27 1.27)
+				)
+			)
+		)
+		(property "Note_Sourcing" "SOURCING D-615 LIVE_RECORD. JLCPCB record read 2026-09-05T00:59:59Z: base library, stock 3722075, land 0603, Operating Temperature -55℃~+155℃; Power(Watts) 100mW; Resistance 1.5kΩ; Temperature Coefficient ±100ppm/℃; Tolerance ±1%; Type Thick Film Resistor; Voltage-Supply(Max) 75V. Gates: land working voltage vs the highest node; 2x the strict over-bound."
+			(at 251.46 45.72 0)
+			(hide yes)
+			(show_name no)
+			(do_not_autoplace no)
+			(effects
+				(font
+					(size 1.27 1.27)
+				)
 			)
 		)
@@
 			)
 		)
+		(property "Manufacturer" "UNI-ROYAL(Uniroyal Elec)"
+			(at 264.16 45.72 0)
+			(hide yes)
+			(show_name no)
+			(do_not_autoplace no)
+			(effects
+				(font
+					(size 1.27 1.27)
+				)
+			)
+		)
+		(property "MPN" "0603WAF1501T5E"
+			(at 264.16 45.72 0)
+			(hide yes)
+			(show_name no)
+			(do_not_autoplace no)
+			(effects
+				(font
+					(size 1.27 1.27)
+				)
+			)
+		)
+		(property "LCSC" "C22843"
+			(at 264.16 45.72 0)
+			(hide yes)
+			(show_name no)
+			(do_not_autoplace no)
+			(effects
+				(font
+					(size 1.27 1.27)
+				)
+			)
+		)
+		(property "Note_Sourcing" "SOURCING D-615 LIVE_RECORD. JLCPCB record read 2026-09-05T00:59:59Z: base library, stock 3722075, land 0603, Operating Temperature -55℃~+155℃; Power(Watts) 100mW; Resistance 1.5kΩ; Temperature Coefficient ±100ppm/℃; Tolerance ±1%; Type Thick Film Resistor; Voltage-Supply(Max) 75V. Gates: land working voltage vs the highest node; 2x the strict over-bound."
+			(at 264.16 45.72 0)
+			(hide yes)
+			(show_name no)
+			(do_not_autoplace no)
+			(effects
+				(font
+					(size 1.27 1.27)
+				)
+			)
+		)
 		(property "Description" ""
 			(at 264.16 45.72 0)
@@
 			)
 		)
+		(property "LCSC" "C160404"
+			(at 176.53 133.35 0)
+			(hide yes)
+			(show_name no)
+			(do_not_autoplace no)
+			(effects
+				(font
+					(size 1.27 1.27)
+				)
+			)
+		)
 		(property "Manufacturer" "JST"
 			(at 176.53 133.35 0)
@@
 			)
 		)
-		(property "Note_Sourcing" "SOURCING D-614. REFERENCE_RULING from the beta-dm audit line 'J8' (SOURCING-LEDGER); manufacturer named with the part in SOURCING_LEDGER; D-238, recorded in docs/full-beta-v2/assembly/SOURCING_LEDGER.md s.2 (JST SH, 1.0 mm, 4 circuit, side entry, SMT, 1.0 A, 50 V) and in DEVICE_SPEC s.10.2, which also lists the absent schematic property as an open item.  The plating-suffixed string is the one D-096 requires: the bare order code resolves to a zero-stock listing."
+		(property "Note_Sourcing" "SOURCING D-615 LIVE_RECORD, SUPERSEDING THE D-614 REFERENCE_RULING. The MPN was grafted at D-614 from D-238 and SOURCING_LEDGER; the LCSC code was the half DEVICE_SPEC s.16 item 8 still listed as OPEN. JLCPCB record read 2026-09-05: JST SM04B-SRSS-TB(LF)(SN), LCSC C160404, stock 69510, SH series, pitch 1 mm, 4P 1x4P, 1 A, 50 V, -25..+85 C, UL94V-0, surface mount right angle, board footprint 6 mm x 4.32 mm -- every field corroborates D-238 and the land Connector_JST:JST_SH_SM04B-SRSS-TB_1x04-1MP_P1.00mm_Horizontal. The bare order code SM04B-SRSS-TB resolves only to ZERO-STOCK JLCPCB Assembly entries, which is why the plating-suffixed string is the one D-096 requires."
 			(at 176.53 133.35 0)
 			(hide yes)

Commit message: demo: D-750 and D-751 -- the external first-spin review found four real defects, and finishing its repairs found two more.
An external first-spin review (Fable 5.1 + Astra) reopened DEMO_READY_FOR_FAB at
b593b97 and named thirteen items.  Four were real defects on the frozen package:
J5's BOM identity still named the 2x12 BCS-112-S-D-HE that D-237 superseded eight
months ago, U14.6 QSTRT was physically floating behind a deliberate no_connect,
audit_rail_ampacity.py computed at 0.0174 mm inner copper against a board that
declares 0.0152 mm, and neither boost converter had a local input capacitor --
the nearest was 36.6 mm and the *named* input part 93.5 mm away.  A fifth,
item 7, is a design-condition failure: TI guarantees the TPS61169 OFF only when
the LED array's minimum Vf exceeds the maximum VIN, this panel is 2.9-3.2 V on a
3.3 V rail, and the shutdown DC path converges at about 25 mA -- a fifth of full
brightness, with no firmware mitigation because +3V3 is switched by SW9.

D-750 closed all of them and dispositioned the other nine, item by item, with
FIRST-ARTICLE and PROCUREMENT work explicitly separated from pre-order blockers.
The charger input was re-laid 250.8 -> 189.8 mm and 440 -> 216 mOhm, which is
what buys the 360 min tMAXCHG its margin; C83 and C84 were fitted on the existing
C33/C64 BOM line; Q11, the backlight true-off disconnect, was fitted on Q1's line.

D-751 FINISHED THE TRANSACTION, AND EACH THING IT TOUCHED HELD ANOTHER DEFECT.

* Q11 was on the board as a symbol and a BOM line and NOT as a circuit: three
  unapproved open edges, all three of them its own pins.  Routed with three
  --tap-first taps, 16.26 mm and four barrels.  The first run was REFUSED for a
  0.44 mm dangling In2 stub the tap left past its T; trimmed, re-run clean.
* placement_contract.py HAD NO WORD FOR AN ADDED PART, so the whole standing
  suite read "placement FAIL" for a legitimate act.  --add exists; PL7 now holds
  an ADDED pad to the same foreign-copper clearance a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
Parts:
- J5: Alternate BCS-112-L-D-HE (10 uin gold, 100 mating cycles - plating-on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 -> SSQ-124-02-F-S-RA (LCSC C6686579, verified live 2026-09-18 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; LCSC C5575816 -> C3323671; MPN BCS-112-S-D-HE -> SSQ-124-02-G-S-RA; Note AQROOT FBV2-S1-008... superseded; FBV2-S1-009 final lock. S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 -> AQROOT J5 COMMUNITY PORT. FBV2-S1-008/S1-009 locked a Samte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; Note2 SOURCING 2026-08-23 (FBV2-S2-002) (B-71). Samtec BCS-112-S-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 -> SOURCING 2026-09-18 (D-750). Samtec SSQ-124-02-G-S-RA is LC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; Note_Sourcing (none) -> SOURCING D-750 2026-09-18. CORRECTION, not a selection: D-2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
Changed lines of the file:
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@@
 			)
 		)
-		(property "Description" "Samtec BCS-112-S-D-HE 2x12 24-contact 2.54 mm female horizontal pass-through socket strip"
+		(property "Note_Sourcing" "SOURCING D-750 2026-09-18. CORRECTION, not a selection: D-237 (FBV2-EXP-002) replaced the 2x12 Samtec BCS-112-S-D-HE with the 1x24 Samtec SSQ-124-02-G-S-RA and moved the Footprint and Datasheet properties, but left MPN, LCSC, Description, Alternate, Note and Note2 on the superseded part, so every released BOM named a 2x12 2-row socket against a PCB carrying one row of 24 pads at x = 65.900. Re-verified live 2026-09-18 per D-096 through the JLCPCB parts API: SSQ-124-02-G-S-RA = LCSC C3323671, Samtec, 1 row, 24P, 2.54 mm, right angle, square hole, gold, stock 0, expand library."
 			(at 120.65 140.97 0)
 			(hide yes)
@@
 			)
 		)
-		(property "Note2" "SOURCING 2026-08-23 (FBV2-S2-002) (B-71). Samtec BCS-112-S-D-HE is LCSC C5575816 with STOCK 0 at $15.54. It is a 24-contact through-hole strip and was already MANUAL/SECONDARY ASSEMBLY by CTO ruling at FBV2-S1-009; buy direct from Samtec or a broadline distributor. The connector architecture is NOT compromised for SMT assembly. LCSC/JLC library state verified live on 2026-08-23 through the JLCPCB parts API (D-096). Stock is a snapshot, not a guarantee."
+		(property "Description" "Samtec SSQ-124-02-G-S-RA 1x24 24-contact 2.54 mm female right-angle square-post socket strip, 20 uin gold, through-hole"
 			(at 120.65 140.97 0)
 			(hide yes)
@@
 			)
 		)
-		(property "LCSC" "C5575816"
+		(property "Note2" "SOURCING 2026-09-18 (D-750). Samtec SSQ-124-02-G-S-RA is LCSC C3323671, expand library, STOCK 0. It is a 24-contact through-hole strip and is MANUAL/SECONDARY ASSEMBLY by CTO ruling at FBV2-S1-009; buy direct from Samtec or a broadline distributor. The connector architecture is NOT compromised for SMT assembly. LCSC/JLC library state verified live on 2026-09-18 through the JLCPCB parts API (D-096); the record is committed at evidence/jlc-live/ssq-124-02-g-s-ra-b06f80e6.json. Stock is a snapshot, not a guarantee. THIS LINE SUPERSEDES THE FBV2-S2-002 BCS-112-S-D-HE SOURCING: D-237 replaced the 2x12 BCS with the 1x24 SSQ and moved the footprint and the datasheet URL, but the MPN, the LCSC code, the Description, the Alternate and this note were left on the superseded part, so the released BOM named a 2x12 against a 1x24 PCB."
+			(at 120.65 140.97 0)
+			(hide yes)
+			(show_name no)
+			(do_not_autoplace no)
+			(effects
+				(font
+					(size 1.27 1.27)
+				)
+			)
+		)
+		(property "LCSC" "C3323671"
 			(at 120.65 140.97 0)
 			(hide yes)
@@
 			)
 		)
-		(property "MPN" "BCS-112-S-D-HE"
+		(property "MPN" "SSQ-124-02-G-S-RA"
 			(at 0 0 0)
 			(hide yes)
@@
 			)
 		)
-		(property "Alternate" "BCS-112-L-D-HE (10 uin gold, 100 mating cycles - plating-only alternate)"
+		(property "Alternate" "SSQ-124-02-F-S-RA (LCSC C6686579, verified live 2026-09-18 per D-096: Samtec, 1 row, 24P, 2.54 mm, right angle, stock 0, expand library). SAME BODY AND SAME FOOTPRINT - it differs only in the plating suffix. Samtec's own scheme makes -F gold flash on contact with matte tin on tail, while the LCSC record lists contact plating as Tin; that disagreement is NOT resolved here, so -F is a plating-only fallback that must be confirmed with Samtec before it is substituted. SSQ-124-02-L-S-RA (10 uin gold) is a valid datasheet configuration but has NO distributor record (0 rows, 2026-09-18) and is therefore NOT baselined - D-096."
 			(at 0 0 0)
 			(hide yes)
@@
 			)
 		)
-		(property "Note" "AQROOT FBV2-S1-008... superseded; FBV2-S1-009 final lock. Samtec BCS-112-S-D-HE, verified live 2026-08-23 per D-096: ACTIVE, 385 pieces ship tomorrow, $7.314 @1 / $5.667 @100, UL E111594, RoHS, halogen free, MSL 1, probable COO Malaysia. 2 x 12 = 24 ACTIVE CONTACTS, .100 in / 2.54 mm pitch, FEMALE Tiger Claw dual-beam pass-through socket strip, HORIZONTAL (right-angle) entry, through-hole, 30 uin selective gold in the contact area. FOOTPRINT RE-VERIFIED AGAINST THE SAMTEC RECOMMENDED PCB LAYOUT DRAWING, REVISION B, FIG 3 (BCS-1XX-XXX-D-HE-XXX): 2.54 mm within a row, ROW-TO-ROW .310 +/-.002 in = 7.87 +/-0.05 mm, hole .028 in = 0.71 mm PTH, pin field 27.94 mm for 12 positions. NOT INTERCHANGEABLE with a vertical 2x12 pattern, whose rows are 2.54 mm apart. ODD = ROW A, EVEN = ROW B (D-084). EVERY POWER CONTACT IS VERTICALLY PAIRED WITH GND - 3/4, 9/10, 15/16, 21/22 - so a row-swap mis-insertion can only make a current-limited rail-to-ground short, never 5 V on a logic pin; ALL 3.3 V IS IN ROW A AND ALL 5 V IN ROW B. NO NC CONTACT, NO KEY CONTACT: the enclosure supplies polarisation and keying (D-097) with a >= 1.5 mm recess, an asymmetric upper rib and CLOSED ENDS that make a one-column offset mechanically impossible. Mates with any 0.64 mm square-post header whose mating post is 4.34-6.35 mm; reference TSW-112-07-L-D. BCS-112-L-D-HE is a plating-only cost-down alternate with an identical footprint but only 100 mating cycles against 2500 for -S (Samtec 187544 Rev 1), which is why -S is locked. THE HARWIN M20-7881242 IS REJECTED AS OBSOLETE AND MUST NEVER REAPPEAR (D-083 struck by D-093). ASSEMBLY: if the JLC service cannot place this through-hole part automatically, it is a MANUAL/SECONDARY assembly operation for the first five boards - the connector architecture is not compromised for SMT convenience."
+		(property "Note" "AQROOT J5 COMMUNITY PORT. FBV2-S1-008/S1-009 locked a Samtec BCS-112-S-D-HE 2 x 12; FBV2-EXP-002 / D-237 SUPERSEDED it with the Samtec SSQ-124-02-G-S-RA, a 1 x 24, 2.54 mm, FEMALE, RIGHT-ANGLE square-post socket strip presenting one pin per line down the right wall and mating an ordinary male header or Dupont jumper. VERIFIED LIVE 2026-09-18 per D-096 (JLCPCB parts API, record committed at evidence/jlc-live/ssq-124-02-g-s-ra-b06f80e6.json): LCSC C3323671, Samtec, Number of Rows 1, Number of Positions 24P, pitch 2.54 mm, Circular/Square Hole = Square Hole, Mounting Type = Right Angle, contact plating Gold, contact material phosphor bronze, -55 to +125 C, insulation height 2.41 mm, expand library, stock 0. CONFIGURATION per the Samtec SSW/SSQ through-hole datasheet held at vendor/Samtec/samtec-ssw-ssq-through-hole.pdf: SSQ = square tail, 124 = 24 positions per row, 02 = standard-insertion-force lead style, G = 20 uin gold on contact, S = single row, RA = right angle. Body 61.47 mm = 24 x 2.54 + 0.51; pin 1 to pin 24 span 58.42 mm; mates .025 in (0.635 mm) square post; 6.3 A per pin with 2 pins powered; 465 VAC / 655 VDC; 100 mating cycles at 10 uin Au. FOOTPRINT AQROOT_Beta:Samtec_SSQ-124-02-G-S-RA, hole pattern 1.02 mm on 2.54 mm, tail row 6.53 mm inboard of the mating face - that 6.53 mm is the dimension the whole right-wall fit turns on. ORDER-B pin order is SAFE UNDER 180 DEGREE REVERSAL BY CONSTRUCTION: 5V to 5V, GND to GND, 3V3 to 3V3, 3.3 V logic to 3.3 V logic everywhere else - power-to-signal maps under reversal: ZERO (D-238/D-240). The enclosure supplies polarisation: a closed-end 62.5 mm recess against a 60.96 mm male body leaves 1.54 mm of play against a 2.54 mm pitch, so a one-position lateral shift is physically impossible; no electrical key contact and no proprietary shroud. J5.9-12 and J5.15-18 are INTENTIONALLY NC on AQROOT Demo by approved scope. ASSEMBLY: through-hole, MANUAL / SECONDARY assembly for the first five boards - the connector architecture is not compromised for SMT convenience. THE HARWIN M20-7881242 IS REJECTED AS OBSOLETE AND MUST NEVER REAPPEAR (D-083 struck by D-093). The BCS-112-S-D-HE footprint is RETAINED in the library, not deleted, because Beta-DM still uses it."
 			(at 0 0 0)
 			(hide yes)

Commit message: demo: D-791 close Round-10 — a floor the node could never reach, a loss model that was only a conduction model, and a gate that was holding a stale procedure in place
Round-10 external review REJECTED D-790.  Fable passed the design for CAM/order
closure with 3 medium / 16 low plus residuals; Astra BLOCKED the order with 15
findings (0 critical, 4 high, 8 medium, 3 low) plus a procurement item, and
established no unconditional PCB respin.

All of D790-A01..A14 and S01 are closed here, plus every Fable complementary
item (F-N01..F-N04, F-V04, F-V05, F-C01, F-C03), plus five this closeout found
itself: R10-N01, R10-N02, R10-N03, and at the verification pass R10-N04 and
R10-N05.

THE THEME IS A NUMBER THAT IS RIGHT ABOUT A STATE THE BOARD CANNOT OCCUPY.

* A03: the firmware's VCELL floors were node voltages BAT_PROTECTED_P cannot
  reach -- 3.85 V there needs >4.3 V upstream and the charger's regulation
  maximum on the pack is 4.221 V -- so the accessory rails this product
  publishes would have been authorised and shed again 400 ms later, on a full
  pack.  New F12 solves the complete cell-to-load network as one fixed point
  and DERIVES three floors: retention 3.20 V, first-rail enable 3.55 V,
  second-rail enable 3.65 V.  Attainability is a clause.
* A02: one electrical network for every sustained mode, states named in
  OBSERVABLE modes, NFC/microSD/IR returned as bounded-duty allowances, TREG
  split into the half it regulates and the half it cannot, and a derived
  30.0 C charge-ambient ceiling.
* A01: the AO4800 conduction row is a ceiling and is now printed, with a 2x
  sensitivity on the declared hot ratio; AO4806 re-examined and re-rejected on
  stock, for the right reason.
* A04: the backlight model gains the four loss terms it was missing,
  211.58 -> 233.13 mA.
* A12 + A10 + A11: the ILIM bound returns to the widest published ratio
  (R97 1.78 -> 1.87 kOhm so U12 stays inside its 2 A rating), BQ OCP and
  TPS22950 RON are read at their own conditions.
* A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
Parts:
- Q10: Manufacturer onsemi -> Jiangsu Changjing Electronics Technology
Changed lines of the file:
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@@
 			)
 		)
-		(property "Manufacturer" "onsemi"
+		(property "Manufacturer" "Jiangsu Changjing Electronics Technology"
 			(at 0 0 0)
 			(hide yes)
