File: hardware/demo/kicad/aqroot-demo/aqroot-Beta-v2.kicad_pcb (KiCad board)
At the start: 6 copper layers, 72 x 148 mm, 311 parts, among them J1 FH69-50S-0.5SH, J2 Molex_5025700893, J3 USB_C_Receptacle_USB2.0_16P, J4 JST-PH-2 BATTERY, J5 COMMUNITY_PORT_1x24, J6 JST-PH-2 SPEAKER, J7 BM02B-ACHSS-GAN-ETF, J8 QWIIC_STEMMA_QT, Q1 AO3400A, Q10 2N7002, Q2 NTMD4820N, Q3 NTMD4820N, Q4 BSS138, Q5 AO3401A, Q6 BSS138, Q7 BSS138, Q8 BSS138, Q9 BSS138, SW1 BOOT, SW2 UP, SW3 DOWN, SW4 LEFT, SW5 RIGHT, SW6 A_SELECT, SW7 B_BACK, SW9 SW_SPDT, U1 ESP32-S3-WROOM-1, U10 USBLC6-2SC6, U11 BQ25185, U12 TPS63020, U13 TPS61023, U14 MAX17048, U16 TCA4307DGKR, U17 TPS61169DCKR, U18 LTC4368-1, U19 TLV7032, U2 PCAL9535APW, U20 TPS22950C, U21 TPS61023, U22 TPS22950C, U3 PCAL9535APW, U4 BMI270, U5 MAX98357A, U6 TSOP38238, U7 E07-400M10S, U8 E22-900M22S, U9 ST25R3916-AQET, Y1 27.12MHz 10pF 3225-4P

Commit message: demo: route NFC AGDC tree
Routing:
- net /04_SPI_B_RADIOS_NFC/NFC_AGDC: track 0.00 -> 40.6 mm
Changed lines of the file:
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@@
+	)
+	(segment
+		(start 23.95 30.2)
+		(end 27 26.95)
+		(width 0.3)
+		(layer "B.Cu")
+		(net "/04_SPI_B_RADIOS_NFC/NFC_AGDC")
+	)
+	(segment
+		(start 34.225 22.5)
+		(end 33.225 22.5)
+		(width 0.3)
+		(layer "B.Cu")
+		(net "/04_SPI_B_RADIOS_NFC/NFC_AGDC")
+	)
+	(segment
+		(start 37.2 31.75)
+		(end 35.875 33.2)
+		(width 0.3)
+		(layer "B.Cu")
+		(net "/04_SPI_B_RADIOS_NFC/NFC_AGDC")
+	)
+	(segment
+		(start 33.6 34.475)
+		(end 32.8 35.5)
+		(width 0.3)
+		(layer "B.Cu")
+		(net "/04_SPI_B_RADIOS_NFC/NFC_AGDC")
+	)
+	(segment
+		(start 37.2 31.75)
+		(end 35.875 33.2)
+		(width 0.3)
+		(layer "B.Cu")
+		(net "/04_SPI_B_RADIOS_NFC/NFC_AGDC")
+	)
+	(segment
+		(start 32.8 35.5)
+		(end 33.225 37.5)
+		(width 0.3)
+		(layer "B.Cu")
+		(net "/04_SPI_B_RADIOS_NFC/NFC_AGDC")
+	)
+	(segment
+		(start 27.525 33.95)
+		(end 23.95 30.2)
+		(width 0.3)
+		(layer "B.Cu")
+		(net "/04_SPI_B_RADIOS_NFC/NFC_AGDC")
+	)
+	(segment
+		(start 34.225 37.5)
+		(end 33.225 37.5)
+		(width 0.3)
+		(layer "B.Cu")
+		(net "/04_SPI_B_RADIOS_NFC/NFC_AGDC")
+	)
+	(segment
+		(start 36.275 31.75)
+		(end 37.2 31.75)
+		(width 0.3)
+		(layer "B.Cu")
+		(net "/04_SPI_B_RADIOS_NFC/NFC_AGDC")
+	)
+	(segment
+		(start 36.275 31.75)
+		(end 37.2 31.75)
+		(width 0.3)
+		(layer "B.Cu")
+		(net "/04_SPI_B_RADIOS_NFC/NFC_AGDC")
+	)
+	(segment
+		(start 27.025 26.4)
+		(end 29.85 23.6)
+		(width 0.3)
+		(layer "B.Cu")
+		(net "/04_SPI_B_RADIOS_NFC/NFC_AGDC")
+	)
+	(segment
+		(start 27 26.95)
+		(end 27.025 26.4)
+		(width 0.3)
+		(layer "B.Cu")
+		(net "/04_SPI_B_RADIOS_NFC/NFC_AGDC")
+	)
+	(segment
+		(start 33.475 22.75)
+		(end 33.225 22.5)
+		(width 0.3)
+		(layer "B.Cu")
+		(net "/04_SPI_B_RADIOS_NFC/NFC_AGDC")
+	)
+	(segment
+		(start 35.875 33.2)
+		(end 27.525 33.95)
+		(width 0.3)
+		(layer "B.Cu")
+		(net "/04_SPI_B_RADIOS_NFC/NFC_AGDC")
+	)
+	(segment
+		(start 32.675 23.6)
+		(end 33.475 22.75)
+		(width 0.3)
+		(layer "B.Cu")
+		(net "/04_SPI_B_RADIOS_NFC/NFC_AGDC")
+	)
+	(segment
+		(start 35.875 33.2)
+		(end 33.6 34.475)
+		(width 0.3)
+		(layer "B.Cu")
+		(net "/04_SPI_B_RADIOS_NFC/NFC_AGDC")
+	)
+	(segment
+		(start 29.85 23.6)
+		(end 32.675 23.6)
+		(width 0.3)
+		(layer "B.Cu")
+		(net "/04_SPI_B_RADIOS_NFC/NFC_AGDC")
 	)
 	(segment

Commit message: demo: route NFC modulator supply tree
Routing:
- net /04_SPI_B_RADIOS_NFC/NFC_VDD_AM: track 0.00 -> 60.9 mm
Changed lines of the file:
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@@
+	)
+	(segment
+		(start 36.275 23.35)
+		(end 37.1 22.475)
+		(width 0.3)
+		(layer "B.Cu")
+		(net "/04_SPI_B_RADIOS_NFC/NFC_VDD_AM")
+	)
+	(segment
+		(start 21.525 29.55)
+		(end 29.475 37.5)
+		(width 0.3)
+		(layer "B.Cu")
+		(net "/04_SPI_B_RADIOS_NFC/NFC_VDD_AM")
+	)
+	(segment
+		(start 36.275 23.35)
+		(end 37.1 22.475)
+		(width 0.3)
+		(layer "B.Cu")
+		(net "/04_SPI_B_RADIOS_NFC/NFC_VDD_AM")
+	)
+	(segment
+		(start 33.925 23.35)
+		(end 36.275 23.35)
+		(width 0.3)
+		(layer "B.Cu")
+		(net "/04_SPI_B_RADIOS_NFC/NFC_VDD_AM")
+	)
+	(segment
+		(start 33.775 19.25)
+		(end 30.9 22.15)
+		(width 0.3)
+		(layer "B.Cu")
+		(net "/04_SPI_B_RADIOS_NFC/NFC_VDD_AM")
+	)
+	(segment
+		(start 33.25 27.725)
+		(end 33.25 26.85)
+		(width 0.3)
+		(layer "B.Cu")
+		(net "/04_SPI_B_RADIOS_NFC/NFC_VDD_AM")
+	)
+	(segment
+		(start 37.1 22.475)
+		(end 32.775 18.3)
+		(width 0.3)
+		(layer "B.Cu")
+		(net "/04_SPI_B_RADIOS_NFC/NFC_VDD_AM")
+	)
+	(segment
+		(start 30.425 37.5)
+		(end 29.475 37.5)
+		(width 0.3)
+		(layer "B.Cu")
+		(net "/04_SPI_B_RADIOS_NFC/NFC_VDD_AM")
+	)
+	(segment
+		(start 33.25 27.725)
+		(end 33.25 26.85)
+		(width 0.3)
+		(layer "B.Cu")
+		(net "/04_SPI_B_RADIOS_NFC/NFC_VDD_AM")
+	)
+	(segment
+		(start 33.125 24.1)
+		(end 33.925 23.35)
+		(width 0.3)
+		(layer "B.Cu")
+		(net "/04_SPI_B_RADIOS_NFC/NFC_VDD_AM")
+	)
+	(segment
+		(start 30.25 22.5)
+		(end 31.25 22.5)
+		(width 0.3)
+		(layer "B.Cu")
+		(net "/04_SPI_B_RADIOS_NFC/NFC_VDD_AM")
+	)
+	(segment
+		(start 37.1 22.475)
+		(end 33.775 19.25)
+		(width 0.3)
+		(layer "B.Cu")
+		(net "/04_SPI_B_RADIOS_NFC/NFC_VDD_AM")
+	)
+	(segment
+		(start 32.775 18.3)
+		(end 21.525 29.55)
+		(width 0.3)
+		(layer "B.Cu")
+		(net "/04_SPI_B_RADIOS_NFC/NFC_VDD_AM")
+	)
+	(segment
+		(start 33.25 26.85)
+		(end 33.125 24.1)
+		(width 0.3)
+		(layer "B.Cu")
+		(net "/04_SPI_B_RADIOS_NFC/NFC_VDD_AM")
+	)
+	(segment
+		(start 33.125 24.1)
+		(end 33.925 23.35)
+		(width 0.3)
+		(layer "B.Cu")
+		(net "/04_SPI_B_RADIOS_NFC/NFC_VDD_AM")
+	)
+	(segment
+		(start 33.25 26.85)
+		(end 33.125 24.1)
+		(width 0.3)
+		(layer "B.Cu")
+		(net "/04_SPI_B_RADIOS_NFC/NFC_VDD_AM")
+	)
+	(segment
+		(start 30.9 22.15)
+		(end 31.25 22.5)
+		(width 0.3)
+		(layer "B.Cu")
+		(net "/04_SPI_B_RADIOS_NFC/NFC_VDD_AM")
+	)
+	(segment
+		(start 33.925 23.35)
+		(end 36.275 23.35)
+		(width 0.3)
+		(layer "B.Cu")
+		(net "/04_SPI_B_RADIOS_NFC/NFC_VDD_AM")
 	)
 	(segment
