File: hardware/demo/kicad/aqroot-demo/02_mcu_core.kicad_sch (KiCad schematic)
At the start: 14 parts, among them SW1 BOOT, U1 ESP32-S3-WROOM-1

Commit message: demo: the BOM is THREE QUARTERS orderable -- 122 part identities grafted from prior CTO audits, every one re-read off the PART instead of the line, and four gates that had never been run (D-614)
NO COPPER CHANGED.  The authoritative board is byte-identical at
c8e421aa50144fe396aedb5e226aaabeb815bd69ffaf6e04f549ded43831d103 and 26 of the
package's 28 artifacts are normalised-sha-identical to D-613's; the two that
moved are the two BOM views.

FAB7 coverage 25.9% -> 75.3%, orderable references 64 -> 186 of 247.
36 BOM lines / 122 references gained Manufacturer / MPN / LCSC -- 487 properties
across nine schematic sheets, replayable to byte-identical sheets.

Four things the mechanical answer would have got wrong: a REJECTED audit row's
JLC Manufacturer column names the match that was THROWN OUT (16 of 31 grafts);
the rating belongs to the PART, not the line; the designator is not the
identity; and the beta-dm 0 ohm current gate had never been run on five of the
Demo's eight links.

Two defects in the instruments fixed: the value parser could not read 15mR, and
MANIFEST.json hashed only the ROOT schematic sheet while nine child sheets
changed.

Re-proved on this tree: verify_promotion.py 14/14, FAB1-FAB6 + FAB8 PASS,
POP1-POP4, P1-P4, protected copper 15 nets / 393 objects IDENTICAL.
FAB7 still FAILS and is partitioned: 8 lines / 16 parts TUNE, 26 lines /
45 parts genuinely open.

Co-Authored-By: Claude Opus 5 <noreply@anthropic.com>
Parts:
- C1: LCSC (none) -> C15849; MPN (none) -> CL10A105KB8NNNC; Manufacturer (none) -> Samsung Electro-Mechanics; Note_Sourcing (none) -> SOURCING D-614. EXACT_PRIOR from the beta-dm audit line '1u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
- C2: LCSC (none) -> C14663; MPN (none) -> CC0603KRX7R9BB104; Manufacturer (none) -> YAGEO; Note_Sourcing (none) -> SOURCING D-614. EXACT_PRIOR from the beta-dm audit line '10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
- C3: LCSC (none) -> C440198; MPN (none) -> GRM21BR61H106KE43L; Manufacturer (none) -> Murata Electronics; Note_Sourcing (none) -> SOURCING D-614. EXACT_PRIOR from the beta-dm audit line '10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
- R1, R108, R110, R111, R2: LCSC (none) -> C25804; MPN (none) -> 0603WAF1002T5E; Manufacturer (none) -> UNI-ROYAL(Uniroyal Elec); Note_Sourcing (none) -> SOURCING D-614. EXACT_PRIOR from the beta-dm audit line '10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
- R109: LCSC (none) -> C21189; MPN (none) -> 0603WAF0000T5E; Manufacturer (none) -> UNI-ROYAL(Uniroyal Elec); Note_Sourcing (none) -> SOURCING D-614. CONTAINED_PRIOR from the beta-dm audit line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
