File: hardware/demo/kicad/aqroot-demo/05_i2c_devices.kicad_sch (KiCad schematic)
At the start: 11 parts, among them U4 BMI270

Commit message: demo: the BOM is THREE QUARTERS orderable -- 122 part identities grafted from prior CTO audits, every one re-read off the PART instead of the line, and four gates that had never been run (D-614)
NO COPPER CHANGED.  The authoritative board is byte-identical at
c8e421aa50144fe396aedb5e226aaabeb815bd69ffaf6e04f549ded43831d103 and 26 of the
package's 28 artifacts are normalised-sha-identical to D-613's; the two that
moved are the two BOM views.

FAB7 coverage 25.9% -> 75.3%, orderable references 64 -> 186 of 247.
36 BOM lines / 122 references gained Manufacturer / MPN / LCSC -- 487 properties
across nine schematic sheets, replayable to byte-identical sheets.

Four things the mechanical answer would have got wrong: a REJECTED audit row's
JLC Manufacturer column names the match that was THROWN OUT (16 of 31 grafts);
the rating belongs to the PART, not the line; the designator is not the
identity; and the beta-dm 0 ohm current gate had never been run on five of the
Demo's eight links.

Two defects in the instruments fixed: the value parser could not read 15mR, and
MANIFEST.json hashed only the ROOT schematic sheet while nine child sheets
changed.

Re-proved on this tree: verify_promotion.py 14/14, FAB1-FAB6 + FAB8 PASS,
POP1-POP4, P1-P4, protected copper 15 nets / 393 objects IDENTICAL.
FAB7 still FAILS and is partitioned: 8 lines / 16 parts TUNE, 26 lines /
45 parts genuinely open.

Co-Authored-By: Claude Opus 5 <noreply@anthropic.com>
Parts:
- C6, C7: LCSC (none) -> C14663; MPN (none) -> CC0603KRX7R9BB104; Manufacturer (none) -> YAGEO; Note_Sourcing (none) -> SOURCING D-614. EXACT_PRIOR from the beta-dm audit line '10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
- R118: LCSC (none) -> C21189; MPN (none) -> 0603WAF0000T5E; Manufacturer (none) -> UNI-ROYAL(Uniroyal Elec); Note_Sourcing (none) -> SOURCING D-614. EXACT_PRIOR from the beta-dm audit line '0R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
- R18: LCSC (none) -> C22962; MPN (none) -> 0603WAF2200T5E; Manufacturer (none) -> UNI-ROYAL(Uniroyal Elec); Note_Sourcing (none) -> SOURCING D-614. EXACT_PRIOR from the beta-dm audit line '22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
Changed lines of the file:
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@@
+			)
+		)
+		(property "Manufacturer" "YAGEO"
+			(at 104.14 58.42 0)
+			(hide yes)
+			(show_name no)
+			(do_not_autoplace no)
+			(effects
+				(font
+					(size 1.27 1.27)
+				)
+			)
+		)
+		(property "MPN" "CC0603KRX7R9BB104"
+			(at 104.14 58.42 0)
+			(hide yes)
+			(show_name no)
+			(do_not_autoplace no)
+			(effects
+				(font
+					(size 1.27 1.27)
+				)
+			)
+		)
+		(property "LCSC" "C14663"
+			(at 104.14 58.42 0)
+			(hide yes)
+			(show_name no)
+			(do_not_autoplace no)
+			(effects
+				(font
+					(size 1.27 1.27)
+				)
+			)
+		)
+		(property "Note_Sourcing" "SOURCING D-614. EXACT_PRIOR from the beta-dm audit line '100nF' (ACCEPTED); manufacturer derived from the YAGEO part-number family and corroborated by the audit text; identical specification."
+			(at 104.14 58.42 0)
+			(hide yes)
+			(show_name no)
+			(do_not_autoplace no)
+			(effects
+				(font
+					(size 1.27 1.27)
+				)
 			)
 		)
@@
 			)
 		)
+		(property "Manufacturer" "YAGEO"
+			(at 73.66 58.42 0)
+			(hide yes)
+			(show_name no)
+			(do_not_autoplace no)
+			(effects
+				(font
+					(size 1.27 1.27)
+				)
+			)
+		)
+		(property "MPN" "CC0603KRX7R9BB104"
+			(at 73.66 58.42 0)
+			(hide yes)
+			(show_name no)
+			(do_not_autoplace no)
+			(effects
+				(font
+					(size 1.27 1.27)
+				)
+			)
+		)
+		(property "LCSC" "C14663"
+			(at 73.66 58.42 0)
+			(hide yes)
+			(show_name no)
+			(do_not_autoplace no)
+			(effects
+				(font
+					(size 1.27 1.27)
+				)
+			)
+		)
+		(property "Note_Sourcing" "SOURCING D-614. EXACT_PRIOR from the beta-dm audit line '100nF' (ACCEPTED); manufacturer derived from the YAGEO part-number family and corroborated by the audit text; identical specification."
+			(at 73.66 58.42 0)
+			(hide yes)
+			(show_name no)
+			(do_not_autoplace no)
+			(effects
+				(font
+					(size 1.27 1.27)
+				)
+			)
+		)
 		(property "Description" "Unpolarized capacitor"
 			(at 73.66 58.42 0)
@@
 		)
 		(property "Datasheet" ""
+			(at 69.85 127 0)
+			(hide yes)
+			(show_name no)
+			(do_not_autoplace no)
+			(effects
+				(font
+					(size 1.27 1.27)
+				)
+			)
+		)
+		(property "Manufacturer" "UNI-ROYAL(Uniroyal Elec)"
+			(at 69.85 127 0)
+			(hide yes)
+			(show_name no)
+			(do_not_autoplace no)
+			(effects
+				(font
+					(size 1.27 1.27)
+				)
+			)
+		)
+		(property "MPN" "0603WAF2200T5E"
+			(at 69.85 127 0)
+			(hide yes)
+			(show_name no)
+			(do_not_autoplace no)
+			(effects
+				(font
+					(size 1.27 1.27)
+				)
+			)
+		)
+		(property "LCSC" "C22962"
+			(at 69.85 127 0)
+			(hide yes)
+			(show_name no)
+			(do_not_autoplace no)
+			(effects
+				(font
+					(size 1.27 1.27)
+				)
+			)
+		)
+		(property "Note_Sourcing" "SOURCING D-614. EXACT_PRIOR from the beta-dm audit line '220R' (ACCEPTED); manufacturer derived from the UNI-ROYAL(Uniroyal Elec) part-number family and corroborated by the audit text; identical specification."
 			(at 69.85 127 0)
 			(hide yes)
@@
 			(at 55.88 93.98 0)
 			(hide yes)
+			(show_name no)
+			(do_not_autoplace no)
+			(effects
+				(font
+					(size 1.27 1.27)
+				)
+			)
+		)
+		(property "Manufacturer" "UNI-ROYAL(Uniroyal Elec)"
+			(at 55.88 93.98 0)
+			(hide yes)
+			(show_name no)
+			(do_not_autoplace no)
+			(effects
+				(font
+					(size 1.27 1.27)
+				)
+			)
+		)
+		(property "MPN" "0603WAF0000T5E"
+			(at 55.88 93.98 0)
+			(hide yes)
+			(show_name no)
+			(do_not_autoplace no)
+			(effects
+				(font
+					(size 1.27 1.27)
+				)
+			)
+		)
+		(property "LCSC" "C21189"
+			(at 55.88 93.98 0)
+			(hide yes)
+			(show_name no)
+			(do_not_autoplace no)
+			(effects
+				(font
+					(size 1.27 1.27)
+				)
+			)
+		)
+		(property "Note_Sourcing" "SOURCING D-614. EXACT_PRIOR from the beta-dm audit line '0R' (ACCEPTED); manufacturer derived from the UNI-ROYAL(Uniroyal Elec) part-number family and corroborated by the audit text; identical specification."
+			(at 55.88 93.98 0)
+			(hide yes)

Commit message: demo: the BOM is 100% ORDERABLE and the safety part was ordered in the WRONG PACKAGE -- 61 identities ruled against a live distributor record, and a screen that asks the C26 question of every line at once (D-615)
D-614 named this task and named what stopped it: D-096 binds -- a part number
configured from an ordering scheme is a hypothesis until a distributor record
confirms lifecycle and stock, and that session had none to read.  This one read
the JLCPCB catalogue 225 times and KEPT every answer, each stamped with the UTC
minute it was read.

NO COPPER CHANGED.  The authoritative board is byte-identical at
c8e421aa50144fe396aedb5e226aaabeb815bd69ffaf6e04f549ded43831d103.

FAB7 IS CLOSED.  Coverage 75.3% -> 100.0%, orderable 186 -> 247 of 247,
needs_a_sourcing_decision ZERO lines, and fab_package_contract.py reads
FAB1-FAB8 PASS for the first time.

THE FINDING.  screen_part_land_parity.py asks D-613's C26 question of every
sourced line at once against the catalogue's own package field: 119 lines carry
a code, 75 are comparable, 74 MATCH and U18 did not.  The land is MSOP-10; the
BOM ordered LTC4368IDD-1#PBF, and DD is DFN-10-EP(3x3) -- against D-099, which
locked LTC4368IMS-1#PBF under FBV2-PWR-002's "no bottom-terminated parts" on
the single most safety-critical component.  The cached library symbol AND the
project .kicad_sym both still carried it, with a Package field describing a DFN
beside a Footprint field already reading MSOP-10.  Corrected to
LTC4368IMS-1#TRPBF, LCSC C688401 -- the tape-and-reel order code of the
identical device, D-210's precedent, not an electrical change.

Three things the obvious answer would have got wrong: R69 is 1.87 ohm and its
part is 0603WAF187KT5E while 0603WAF1873T5E is 187 kOhm; R95's node over-bound
UNDERSTATES its dissipation because a reversed cell adds in series (154 mW vs
54 mW); and R24/C12's Value strings are looser than their own symbol notes.
NET_MAX_DC grew 17 -> 48 established nodes to give the new dissipation gate
nu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
Parts:
- R19, R20: LCSC (none) -> C4190; MPN (none) -> 0603WAF2201T5E; Manufacturer (none) -> UNI-ROYAL(Uniroyal Elec); Note_Sourcing (none) -> SOURCING D-615 LIVE_RECORD. JLCPCB record read 2026-09-05T0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
Changed lines of the file:
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@@
+			)
+		)
+		(property "Manufacturer" "UNI-ROYAL(Uniroyal Elec)"
+			(at 138.43 78.74 0)
+			(hide yes)
+			(show_name no)
+			(do_not_autoplace no)
+			(effects
+				(font
+					(size 1.27 1.27)
+				)
+			)
+		)
+		(property "MPN" "0603WAF2201T5E"
+			(at 138.43 78.74 0)
+			(hide yes)
+			(show_name no)
+			(do_not_autoplace no)
+			(effects
+				(font
+					(size 1.27 1.27)
+				)
+			)
+		)
+		(property "LCSC" "C4190"
+			(at 138.43 78.74 0)
+			(hide yes)
+			(show_name no)
+			(do_not_autoplace no)
+			(effects
+				(font
+					(size 1.27 1.27)
+				)
+			)
+		)
+		(property "Note_Sourcing" "SOURCING D-615 LIVE_RECORD. JLCPCB record read 2026-09-05T00:59:59Z: base library, stock 7045544, land 0603, Operating Temperature -55℃~+155℃; Power(Watts) 100mW; Resistance 2.2kΩ; Temperature Coefficient ±100ppm/℃; Tolerance ±1%; Type Thick Film Resistor; Voltage-Supply(Max) 75V. Gates: land working voltage vs the highest node; 2x the strict over-bound."
+			(at 138.43 78.74 0)
+			(hide yes)
+			(show_name no)
+			(do_not_autoplace no)
+			(effects
+				(font
+					(size 1.27 1.27)
+				)
 			)
 		)
@@
 			(at 181.61 78.74 0)
 			(hide yes)
+			(show_name no)
+			(do_not_autoplace no)
+			(effects
+				(font
+					(size 1.27 1.27)
+				)
+			)
+		)
+		(property "Manufacturer" "UNI-ROYAL(Uniroyal Elec)"
+			(at 181.61 78.74 0)
+			(hide yes)
+			(show_name no)
+			(do_not_autoplace no)
+			(effects
+				(font
+					(size 1.27 1.27)
+				)
+			)
+		)
+		(property "MPN" "0603WAF2201T5E"
+			(at 181.61 78.74 0)
+			(hide yes)
+			(show_name no)
+			(do_not_autoplace no)
+			(effects
+				(font
+					(size 1.27 1.27)
+				)
+			)
+		)
+		(property "LCSC" "C4190"
+			(at 181.61 78.74 0)
+			(hide yes)
+			(show_name no)
+			(do_not_autoplace no)
+			(effects
+				(font
+					(size 1.27 1.27)
+				)
+			)
+		)
+		(property "Note_Sourcing" "SOURCING D-615 LIVE_RECORD. JLCPCB record read 2026-09-05T00:59:59Z: base library, stock 7045544, land 0603, Operating Temperature -55℃~+155℃; Power(Watts) 100mW; Resistance 2.2kΩ; Temperature Coefficient ±100ppm/℃; Tolerance ±1%; Type Thick Film Resistor; Voltage-Supply(Max) 75V. Gates: land working voltage vs the highest node; 2x the strict over-bound."
+			(at 181.61 78.74 0)
+			(hide yes)
