File: hardware/demo/kicad/aqroot-demo/08_buttons_expanders.kicad_sch (KiCad schematic)
At the start: 30 parts, among them SW2 UP, SW3 DOWN, SW4 LEFT, SW5 RIGHT, SW6 A_SELECT, SW7 B_BACK, U2 PCAL9535APW, U3 PCAL9535APW

Commit message: demo: the BOM is THREE QUARTERS orderable -- 122 part identities grafted from prior CTO audits, every one re-read off the PART instead of the line, and four gates that had never been run (D-614)
NO COPPER CHANGED.  The authoritative board is byte-identical at
c8e421aa50144fe396aedb5e226aaabeb815bd69ffaf6e04f549ded43831d103 and 26 of the
package's 28 artifacts are normalised-sha-identical to D-613's; the two that
moved are the two BOM views.

FAB7 coverage 25.9% -> 75.3%, orderable references 64 -> 186 of 247.
36 BOM lines / 122 references gained Manufacturer / MPN / LCSC -- 487 properties
across nine schematic sheets, replayable to byte-identical sheets.

Four things the mechanical answer would have got wrong: a REJECTED audit row's
JLC Manufacturer column names the match that was THROWN OUT (16 of 31 grafts);
the rating belongs to the PART, not the line; the designator is not the
identity; and the beta-dm 0 ohm current gate had never been run on five of the
Demo's eight links.

Two defects in the instruments fixed: the value parser could not read 15mR, and
MANIFEST.json hashed only the ROOT schematic sheet while nine child sheets
changed.

Re-proved on this tree: verify_promotion.py 14/14, FAB1-FAB6 + FAB8 PASS,
POP1-POP4, P1-P4, protected copper 15 nets / 393 objects IDENTICAL.
FAB7 still FAILS and is partitioned: 8 lines / 16 parts TUNE, 26 lines /
45 parts genuinely open.

Co-Authored-By: Claude Opus 5 <noreply@anthropic.com>
Parts:
- C4, C5: LCSC (none) -> C14663; MPN (none) -> CC0603KRX7R9BB104; Manufacturer (none) -> YAGEO; Note_Sourcing (none) -> SOURCING D-614. EXACT_PRIOR from the beta-dm audit line '10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
- R12, R129, R13, R14, R15, R16, R17: LCSC (none) -> C25803; MPN (none) -> 0603WAF1003T5E; Manufacturer (none) -> UNI-ROYAL(Uniroyal Elec); Note_Sourcing (none) -> SOURCING D-614. EXACT_PRIOR from the beta-dm audit line '10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
- R124: LCSC (none) -> C21190; MPN (none) -> 0603WAF1001T5E; Manufacturer (none) -> UNI-ROYAL(Uniroyal Elec); Note_Sourcing (none) -> SOURCING D-614. CONTAINED_PRIOR from the beta-dm audit line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
- R127, R128, R3, R4, R5, R6, R7, R8, R9: LCSC (none) -> C25804; MPN (none) -> 0603WAF1002T5E; Manufacturer (none) -> UNI-ROYAL(Uniroyal Elec); Note_Sourcing (none) -> SOURCING D-614. EXACT_PRIOR from the beta-dm audit line '10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

Commit message: demo: the BOM is 100% ORDERABLE and the safety part was ordered in the WRONG PACKAGE -- 61 identities ruled against a live distributor record, and a screen that asks the C26 question of every line at once (D-615)
D-614 named this task and named what stopped it: D-096 binds -- a part number
configured from an ordering scheme is a hypothesis until a distributor record
confirms lifecycle and stock, and that session had none to read.  This one read
the JLCPCB catalogue 225 times and KEPT every answer, each stamped with the UTC
minute it was read.

NO COPPER CHANGED.  The authoritative board is byte-identical at
c8e421aa50144fe396aedb5e226aaabeb815bd69ffaf6e04f549ded43831d103.

FAB7 IS CLOSED.  Coverage 75.3% -> 100.0%, orderable 186 -> 247 of 247,
needs_a_sourcing_decision ZERO lines, and fab_package_contract.py reads
FAB1-FAB8 PASS for the first time.

THE FINDING.  screen_part_land_parity.py asks D-613's C26 question of every
sourced line at once against the catalogue's own package field: 119 lines carry
a code, 75 are comparable, 74 MATCH and U18 did not.  The land is MSOP-10; the
BOM ordered LTC4368IDD-1#PBF, and DD is DFN-10-EP(3x3) -- against D-099, which
locked LTC4368IMS-1#PBF under FBV2-PWR-002's "no bottom-terminated parts" on
the single most safety-critical component.  The cached library symbol AND the
project .kicad_sym both still carried it, with a Package field describing a DFN
beside a Footprint field already reading MSOP-10.  Corrected to
LTC4368IMS-1#TRPBF, LCSC C688401 -- the tape-and-reel order code of the
identical device, D-210's precedent, not an electrical change.

Three things the obvious answer would have got wrong: R69 is 1.87 ohm and its
part is 0603WAF187KT5E while 0603WAF1873T5E is 187 kOhm; R95's node over-bound
UNDERSTATES its dissipation because a reversed cell adds in series (154 mW vs
54 mW); and R24/C12's Value strings are looser than their own symbol notes.
NET_MAX_DC grew 17 -> 48 established nodes to give the new dissipation gate
nu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
Parts:
- R125: LCSC (none) -> C23228; MPN (none) -> 0603WAF6800T5E; Manufacturer (none) -> UNI-ROYAL(Uniroyal Elec); Note_Sourcing (none) -> SOURCING D-615 LIVE_RECORD. JLCPCB record read 2026-09-05T0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
- R126: LCSC (none) -> C23151; MPN (none) -> 0603WAF3900T5E; Manufacturer (none) -> UNI-ROYAL(Uniroyal Elec); Note_Sourcing (none) -> SOURCING D-615 LIVE_RECORD. JLCPCB record read 2026-09-05T0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
Changed lines of the file:
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@@
+			)
+		)
+		(property "Manufacturer" "UNI-ROYAL(Uniroyal Elec)"
+			(at 307.34 245.11 0)
+			(hide yes)
+			(show_name no)
+			(do_not_autoplace no)
+			(effects
+				(font
+					(size 1.27 1.27)
+				)
+			)
+		)
+		(property "MPN" "0603WAF6800T5E"
+			(at 307.34 245.11 0)
+			(hide yes)
+			(show_name no)
+			(do_not_autoplace no)
+			(effects
+				(font
+					(size 1.27 1.27)
+				)
+			)
+		)
+		(property "LCSC" "C23228"
+			(at 307.34 245.11 0)
+			(hide yes)
+			(show_name no)
+			(do_not_autoplace no)
+			(effects
+				(font
+					(size 1.27 1.27)
+				)
+			)
+		)
+		(property "Note_Sourcing" "SOURCING D-615 LIVE_RECORD. JLCPCB record read 2026-09-05T00:59:59Z: base library, stock 2802834, land 0603, Operating Temperature -55℃~+155℃; Power(Watts) 100mW; Resistance 680Ω; Temperature Coefficient ±100ppm/℃; Tolerance ±1%; Type Thick Film Resistor; Voltage-Supply(Max) 75V. Gates: land working voltage vs the highest node; 2x operating and survives single fault."
+			(at 307.34 245.11 0)
+			(hide yes)
+			(show_name no)
+			(do_not_autoplace no)
+			(effects
+				(font
+					(size 1.27 1.27)
+				)
 			)
 		)
@@
 			(at 307.34 250.19 0)
 			(hide yes)
+			(show_name no)
+			(do_not_autoplace no)
+			(effects
+				(font
+					(size 1.27 1.27)
+				)
+			)
+		)
+		(property "Manufacturer" "UNI-ROYAL(Uniroyal Elec)"
+			(at 307.34 250.19 0)
+			(hide yes)
+			(show_name no)
+			(do_not_autoplace no)
+			(effects
+				(font
+					(size 1.27 1.27)
+				)
+			)
+		)
+		(property "MPN" "0603WAF3900T5E"
+			(at 307.34 250.19 0)
+			(hide yes)
+			(show_name no)
+			(do_not_autoplace no)
+			(effects
+				(font
+					(size 1.27 1.27)
+				)
+			)
+		)
+		(property "LCSC" "C23151"
+			(at 307.34 250.19 0)
+			(hide yes)
+			(show_name no)
+			(do_not_autoplace no)
+			(effects
+				(font
+					(size 1.27 1.27)
+				)
+			)
+		)
+		(property "Note_Sourcing" "SOURCING D-615 LIVE_RECORD. JLCPCB record read 2026-09-05T00:59:59Z: base library, stock 456712, land 0603, Operating Temperature -55℃~+155℃; Power(Watts) 100mW; Resistance 390Ω; Temperature Coefficient ±100ppm/℃; Tolerance ±1%; Type Thick Film Resistor; Voltage-Supply(Max) 75V. Gates: land working voltage vs the highest node; 2x operating and survives single fault."
+			(at 307.34 250.19 0)
+			(hide yes)

Commit message: demo: D-712 -- THE U2 CHANNEL SWAP IS PROMOTED AND /BQ25185_STAT1 IS CLOSED, AND THE TPS63020's PS/SYNC STRAP COMES HOME FROM FIFTY MILLIMETRES AWAY: 15 -> 13 RETAINED OPEN EDGES.
COPPER PROMOTED.  Authority 4414da31 -> 2e8ef9ed; 15 -> 13 retained open
edges over 9 nets.  hardware/beta-v2 UNTOUCHED.

1. D-711's U2 CHANNEL SWAP, SPENT.  P05 <-> P17 and P06 <-> P16 on the
   PCAL9535A, schematic and PCB together.  /BQ25185_STAT1 and /BQ25185_STAT2
   were landed on U2's WEST column with their partners at x 59..70, and
   /SX1262_DIO1 and /TOUCH_INT_N on its EAST column with their partners at
   x 3 and x 22; all four crossed the package.  The netlist diff is exactly
   four nets plus GND, ERC drops 4 (the two removed parts' library links) and
   gains nothing, and /BQ25185_STAT1 now ROUTES: 1 -> 0 open edges.
   /TOUCH_INT_N was evicted whole and comes back closed.

2. THE PS/SYNC STRAP.  R42 is a 0R tying U12.13 (PS/SYNC on the TPS63020) to
   GND and it sat at (16.665, 120.335) -- FIFTY MILLIMETRES from the pin --
   with TP14 on the way, hauling 33 B.Cu objects across the board.  Its last
   two segments lay in the C24/C26 gate, which D-649 measured as a SINGLE-FILE
   corridor the /01_POWER_TREE/BQ25185_SYS pour and that net cannot share --
   which is why C26.2, a 10 uF bulk capacitor on the system rail, was an
   ISLAND.  A 0R to GND and a tie to GND are the same circuit, so U12.13 is
   tied to U12.15, U12's own thermal ground pad, 0.610 mm away, and R42 and
   TP14 come off the board.  BQ25185_SYS 5 -> 4 open edges, and a switching
   converter's mode pin stops being a 50 mm antenna.

3. TP7 OUT OF THE POWER POUR.  /BQ25185_STAT2's test point sat at
   (62.750, 98.500), inside the B.Cu BQ25185_SYS pour, in the 0.4 mm neck that
   is the rail's only north-south conductor.  Every STAT2 re-route through it
   severed the pour.  TP7 moves to (57.500, 97.500), clear of the pour.

4. THE SYS SPINE IS RESERVED DURING THE RUN.  evidence/d712-guard-spine.json
   sample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
Connections:
- net BQ25185_STAT1: now also U2.20 (P17); no longer U2.9 (P05)
- net BQ25185_STAT2: now also U2.19 (P16); no longer U2.10 (P06)
- net SX1262_DIO1: now also U2.9 (P05); no longer U2.20 (P17)
- net TOUCH_INT_N: now also U2.10 (P06); no longer U2.19 (P16)
Changed lines of the file:
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@@
 	(hierarchical_label "TOUCH_INT_N"
 		(shape input)
+		(at 101.6 69.85 0)
+		(effects
+			(font
+				(size 1.27 1.27)
+			)
+			(justify left)
+		)
+	)
+	(label "BQ25185_STAT1"
+		(at 101.6 95.25 0)
+		(effects
+			(font
+				(size 1.27 1.27)
+			)
+			(justify left bottom)
+		)
+	)
+	(label "BQ25185_STAT2"
 		(at 101.6 92.71 0)
 		(effects
@@
 				(size 1.27 1.27)
 			)
-			(justify left)
+			(justify left bottom)
 		)
 	)
 	(hierarchical_label "SX1262_DIO1"
 		(shape input)
-		(at 101.6 95.25 0)
+		(at 101.6 67.31 0)
 		(effects
 			(font
@@
 		)
 	)
-	(wire
-		(pts
-			(xy 101.6 67.31) (xy 113.03 67.31)
-		)
-		(stroke
-			(width 0)
-			(type default)
-		)
-	)
 	(hierarchical_label "BQ25185_STAT1"
 		(shape input)
@@
 		)
 	)
-	(wire
-		(pts
-			(xy 101.6 69.85) (xy 129.54 69.85)
-		)
-		(stroke
-			(width 0)
-			(type default)
-		)
-	)

Commit message: demo: D-732 -- the D-pad defect is closed for ZERO COPPER. D-731 measured it right and priced the wrong repair: the wiring was never wrong, only the declaration of which expander bit carries which function. All eight PCAL9535A port-1 pins are inputs, all interrupt-capable, all masked at power-up, so the function-to-pin map is a free variable and a 5-cycle of five NET NAMES corrects the defect with zero copper, zero part moves, zero BOM lines and no enclosure/aperture decision. It maps exactly, because the placement error was a clean off-by-one in the SW2..SW6 seat order. The same note also named P05/P06/P16/P17 inverted, which would have masked the TOUCH interrupt and left STAT2 waking the MCU forever -- rewritten pin by pin from the board. 4->4 edges, DRC {lib_footprint_issues:199} and nothing else, parity 246/0 errors, 14/14 contracts PASS, fab package re-exported with zero geometry delta.
Co-Authored-By: Claude Opus 5 <noreply@anthropic.com>
Parts:
- SW2: value UP -> A_SELECT
- SW3: value DOWN -> UP
- SW4: value LEFT -> DOWN
- SW5: value RIGHT -> LEFT
- SW6: value A_SELECT -> RIGHT
Connections:
- net BTN_A_N: now also R4.2, SW2.1, U2.13 (P10); no longer R8.2, SW6.1, U2.17 (P14)
- net BTN_DOWN_N: now also R6.2, SW4.1, U2.15 (P12); no longer R5.2, SW3.1, U2.14 (P11)
- net BTN_LEFT_N: now also R7.2, SW5.1, U2.16 (P13); no longer R6.2, SW4.1, U2.15 (P12)
- net BTN_RIGHT_N: now also R8.2, SW6.1, U2.17 (P14); no longer R7.2, SW5.1, U2.16 (P13)
- net BTN_UP_N: now also R5.2, SW3.1, U2.14 (P11); no longer R4.2, SW2.1, U2.13 (P10)
Other:
- note added: "U2 INTERNAL EXPANDER - MIGRATED FBV2-S1-008 NXP PCAL9535APW,118 I2C ADDRESS 0x20 A0 = A1 = A2 = GND PORT 0 = P00-P04 OUT, P05-P07 IN (06h = E0h) PORT 1 = 8 INPUTS (07h = FFh) 16 / 16 USED - ZERO SPARE P00 TOUCH_RST_N OUT ACTIVE LOW P01 SX1262_RST_N OUT ACTIVE LOW P02 NFC_5V_EN OUT ACTIVE HIGH P03 AMP_SD_MODE OUT ACTIVE HIGH P04 DISP_RST_N OUT ACTIVE LOW P05 SX1262_DIO1 IN ACTIVE HIGH P06 TOUCH_IN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"
- note removed: "U2 INTERNAL EXPANDER - MIGRATED FBV2-S1-008 NXP PCAL9535APW,118 I2C ADDRESS 0x20 A0 = A1 = A2 = GND PORT 0 = P00-P04 OUT, P05-P07 IN (06h = E0h) PORT 1 = 8 INPUTS (07h = FFh) 16 / 16 USED - ZERO SPARE P00 TOUCH_RST_N OUT ACTIVE LOW P01 SX1262_RST_N OUT ACTIVE LOW P02 NFC_5V_EN OUT ACTIVE HIGH P03 AMP_SD_MODE OUT ACTIVE HIGH P04 DISP_RST_N OUT ACTIVE LOW P05 BQ25185_STAT1 IN R127 10k UP P06 BQ2518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"
Changed lines of the file:
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@@
 		)
 	)
-	(label "BTN_UP_N"
+	(label "BTN_A_N"
 		(at 36.83 144.78 180)
 		(effects
@@
 		)
 	)
-	(label "BTN_A_N"
+	(label "BTN_RIGHT_N"
 		(at 124.46 144.78 180)
 		(effects
@@
 		)
 	)
-	(label "BTN_DOWN_N"
+	(label "BTN_UP_N"
 		(at 58.42 144.78 180)
 		(effects
@@
 		)
 	)
-	(label "BTN_LEFT_N"
+	(label "BTN_DOWN_N"
 		(at 81.28 144.78 180)
 		(effects
@@
 		)
 	)
-	(label "BTN_RIGHT_N"
+	(label "BTN_LEFT_N"
 		(at 101.6 144.78 180)
 		(effects
@@
 		)
 	)
-	(label "BTN_UP_N"
+	(label "BTN_A_N"
 		(at 101.6 77.47 0)
 		(effects
@@
 		)
 	)
-	(label "BTN_RIGHT_N"
+	(label "BTN_LEFT_N"
 		(at 101.6 85.09 0)
 		(effects
@@
 		)
 	)
-	(label "BTN_LEFT_N"
+	(label "BTN_DOWN_N"
 		(at 101.6 82.55 0)
 		(effects
@@
 		)
 	)
-	(label "BTN_DOWN_N"
+	(label "BTN_UP_N"
 		(at 101.6 80.01 0)
 		(effects
@@
 		)
 	)
-	(label "BTN_A_N"
+	(label "BTN_RIGHT_N"
 		(at 101.6 87.63 0)
 		(effects
@@
 			)
 		)
-		(property "Value" "A_SELECT"
+		(property "Value" "RIGHT"
 			(at 129.54 154.9399 90)
 			(show_name no)
@@
 			)
 		)
-		(property "Value" "RIGHT"
+		(property "Value" "LEFT"
 			(at 106.68 154.9399 90)
 			(show_name no)
@@
 			)
 		)
-		(property "Value" "LEFT"
+		(property "Value" "DOWN"
 			(at 86.36 154.9399 90)
 			(show_name no)
@@
 			)
 		)
-		(property "Value" "UP"
+		(property "Value" "A_SELECT"
 			(at 41.91 154.9399 90)
 			(show_name no)
@@
 			)
 		)
-		(property "Value" "DOWN"
+		(property "Value" "UP"
 			(at 63.5 154.9399 90)
 			(show_name no)
@@
 		)
 	)
-	(text "U2 INTERNAL EXPANDER - MIGRATED FBV2-S1-008\nNXP PCAL9535APW,118   I2C ADDRESS 0x20\nA0 = A1 = A2 = GND\n\nPORT 0 = P00-P04 OUT, P05-P07 IN  (06h = E0h)\nPORT 1 = 8 INPUTS                 (07h = FFh)\n16 / 16 USED - ZERO SPARE\n\nP00 TOUCH_RST_N       OUT  ACTIVE LOW\nP01 SX1262_RST_N      OUT  ACTIVE LOW\nP02 NFC_5V_EN         OUT  ACTIVE HIGH\nP03 AMP_SD_MODE       OUT  ACTIVE HIGH\nP04 DISP_RST_N        OUT  ACTIVE LOW\nP05 BQ25185_STAT1     IN   R127 10k UP\nP06 BQ25185_STAT2     IN   R128 10k UP\nP07 SD_CARD_DETECT_N  IN   R113 100k UP, SHEET 03\nP10-P13 D-PAD UP/DOWN/LEFT/RIGHT  IN  10k UP\nP14 BTN_A_N   P15 BTN_B_N         IN  10k UP\nP16 TOUCH_INT_N       IN   FT6236, ACTIVE LOW\nP17 SX1262_DIO1       IN   ACTIVE HIGH\n\nEVERY P05-P17 INPUT IS INTERRUPT-CAPABLE AND EVERY\nONE POWERS UP MASKED (4Ah/4Bh = FFh). FIRMWARE\nUNMASKS THE SIX BUTTONS, TOUCH_INT_N, SX1262_DIO1\nAND SD_CARD_DETECT_N, AND LEAVES BQ25185_STAT2\nMASKED - IT TOGGLES CONTINUOUSLY WHEN NO BATTERY IS\nFITTED AND WOULD OTHERWISE WAKE THE MCU FOREVER."
+	(text "U2 INTERNAL EXPANDER - MIGRATED FBV2-S1-008\nNXP PCAL9535APW,118   I2C ADDRESS 0x20\nA0 = A1 = A2 = GND\n\nPORT 0 = P00-P04 OUT, P05-P07 IN  (06h = E0h)\nPORT 1 = 8 INPUTS                 (07h = FFh)\n16 / 16 USED - ZERO SPARE\n\nP00 TOUCH_RST_N       OUT  ACTIVE LOW\nP01 SX1262_RST_N      OUT  ACTIVE LOW\nP02 NFC_5V_EN         OUT  ACTIVE HIGH\nP03 AMP_SD_MODE       OUT  ACTIVE HIGH\nP04 DISP_RST_N        OUT  ACTIVE LOW\nP05 SX1262_DIO1       IN   ACTIVE HIGH\nP06 TOUCH_INT_N       IN   FT6236, ACTIVE LOW\nP07 SD_CARD_DETECT_N  IN   R113 100k UP, SHEET 03\nP10 BTN_A_N           IN   R4  10k UP\nP11 BTN_UP_N          IN   R5  10k UP\nP12 BTN_DOWN_N        IN   R6  10k UP\nP13 BTN_LEFT_N        IN   R7  10k UP\nP14 BTN_RIGHT_N       IN   R8  10k UP\nP15 BTN_B_N           IN   R9  10k UP\nP16 BQ25185_STAT2     IN   R128 10k UP\nP17 BQ25185_STAT1     IN   R127 10k UP\n\n*** D-732 CORRECTED THIS MAP TWICE. ***  (1) THE PORT-1\nD-PAD / A ASSIGNMENT WAS CYCLED ONE SEAT SO EACH EXPANDER\nBIT MATCHES THE SWITCH ACTUALLY SEATED UNDER ITS ENCLOSURE\nAPERTURE.  THE PCB PLACED SW2..SW6 ONE POSITION OUT AND\nTHE COPPER IS CORRECT AS BUILT, SO THE PIN ASSIGNMENT\nMOVED, NOT THE PARTS.  THE D-PAD IS P11..P14, NOT\nP10..P13.  (2) P05 / P06 / P16 / P17 WERE NAMED WRONG IN\nTHE PREVIOUS NOTE: STAT1 AND STAT2 ARE ON PORT 1, NOT\nPORT 0.  FIRMWARE MUST USE THIS TABLE, NOT ANY EARLIER\nONE.\n\nEVERY P05-P17 INPUT IS INTERRUPT-CAPABLE AND EVERY\nONE POWERS UP MASKED (4Ah/4Bh = FFh). FIRMWARE\nUNMASKS THE SIX BUTTONS, TOUCH_INT_N, SX1262_DIO1\nAND SD_CARD_DETECT_N, AND LEAVES BQ25185_STAT2\nMASKED - IT IS 4Bh BIT 6 (P16), NOT 4Ah BIT 6.  IT\nTOGGLES CONTINUOUSLY WHEN NO BATTERY IS FITTED AND\nWOULD OTHERWISE WAKE THE MCU FOREVER."
 		(exclude_from_sim no)
 		(at 82.804 33.782 0)
