File: hardware/demo/kicad/aqroot-demo/07_ir.kicad_sch (KiCad schematic)
At the start: 12 parts, among them Q1 AO3400A, U6 TSOP38238

Commit message: demo: the BOM is THREE QUARTERS orderable -- 122 part identities grafted from prior CTO audits, every one re-read off the PART instead of the line, and four gates that had never been run (D-614)
NO COPPER CHANGED.  The authoritative board is byte-identical at
c8e421aa50144fe396aedb5e226aaabeb815bd69ffaf6e04f549ded43831d103 and 26 of the
package's 28 artifacts are normalised-sha-identical to D-613's; the two that
moved are the two BOM views.

FAB7 coverage 25.9% -> 75.3%, orderable references 64 -> 186 of 247.
36 BOM lines / 122 references gained Manufacturer / MPN / LCSC -- 487 properties
across nine schematic sheets, replayable to byte-identical sheets.

Four things the mechanical answer would have got wrong: a REJECTED audit row's
JLC Manufacturer column names the match that was THROWN OUT (16 of 31 grafts);
the rating belongs to the PART, not the line; the designator is not the
identity; and the beta-dm 0 ohm current gate had never been run on five of the
Demo's eight links.

Two defects in the instruments fixed: the value parser could not read 15mR, and
MANIFEST.json hashed only the ROOT schematic sheet while nine child sheets
changed.

Re-proved on this tree: verify_promotion.py 14/14, FAB1-FAB6 + FAB8 PASS,
POP1-POP4, P1-P4, protected copper 15 nets / 393 objects IDENTICAL.
FAB7 still FAILS and is partitioned: 8 lines / 16 parts TUNE, 26 lines /
45 parts genuinely open.

Co-Authored-By: Claude Opus 5 <noreply@anthropic.com>
Parts:
- C11: LCSC (none) -> C1779; MPN (none) -> CL21A475KAQNNNE; Manufacturer (none) -> Samsung Electro-Mechanics; Note_Sourcing (none) -> SOURCING D-614. EXACT_PRIOR from the beta-dm audit line '4.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
- R21, R22: LCSC (none) -> C22775; MPN (none) -> 0603WAF1000T5E; Manufacturer (none) -> UNI-ROYAL(Uniroyal Elec); Note_Sourcing (none) -> SOURCING D-614. CONTAINED_PRIOR from the beta-dm audit line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
- R23: LCSC (none) -> C25803; MPN (none) -> 0603WAF1003T5E; Manufacturer (none) -> UNI-ROYAL(Uniroyal Elec); Note_Sourcing (none) -> SOURCING D-614. EXACT_PRIOR from the beta-dm audit line '10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
Changed lines of the file:
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@@
+			)
+		)
+		(property "Manufacturer" "UNI-ROYAL(Uniroyal Elec)"
+			(at 175.26 35.56 0)
+			(hide yes)
+			(show_name no)
+			(do_not_autoplace no)
+			(effects
+				(font
+					(size 1.27 1.27)
+				)
+			)
+		)
+		(property "MPN" "0603WAF1000T5E"
+			(at 175.26 35.56 0)
+			(hide yes)
+			(show_name no)
+			(do_not_autoplace no)
+			(effects
+				(font
+					(size 1.27 1.27)
+				)
+			)
+		)
+		(property "LCSC" "C22775"
+			(at 175.26 35.56 0)
+			(hide yes)
+			(show_name no)
+			(do_not_autoplace no)
+			(effects
+				(font
+					(size 1.27 1.27)
+				)
+			)
+		)
+		(property "Note_Sourcing" "SOURCING D-614. CONTAINED_PRIOR from the beta-dm audit line '100R 1%' (REJECTED - JLC match wrong); manufacturer derived from the UNI-ROYAL(Uniroyal Elec) part-number family and corroborated by the audit text; identical specification."
+			(at 175.26 35.56 0)
+			(hide yes)
+			(show_name no)
+			(do_not_autoplace no)
+			(effects
+				(font
+					(size 1.27 1.27)
+				)
 			)
 		)
@@
 			)
 		)
+		(property "Manufacturer" "UNI-ROYAL(Uniroyal Elec)"
+			(at 173.99 58.42 0)
+			(hide yes)
+			(show_name no)
+			(do_not_autoplace no)
+			(effects
+				(font
+					(size 1.27 1.27)
+				)
+			)
+		)
+		(property "MPN" "0603WAF1003T5E"
+			(at 173.99 58.42 0)
+			(hide yes)
+			(show_name no)
+			(do_not_autoplace no)
+			(effects
+				(font
+					(size 1.27 1.27)
+				)
+			)
+		)
+		(property "LCSC" "C25803"
+			(at 173.99 58.42 0)
+			(hide yes)
+			(show_name no)
+			(do_not_autoplace no)
+			(effects
+				(font
+					(size 1.27 1.27)
+				)
+			)
+		)
+		(property "Note_Sourcing" "SOURCING D-614. EXACT_PRIOR from the beta-dm audit line '100K' (ACCEPTED); manufacturer derived from the UNI-ROYAL(Uniroyal Elec) part-number family and corroborated by the audit text; identical specification."
+			(at 173.99 58.42 0)
+			(hide yes)
+			(show_name no)
+			(do_not_autoplace no)
+			(effects
+				(font
+					(size 1.27 1.27)
+				)
+			)
+		)
 		(property "Description" "Resistor"
 			(at 173.99 58.42 0)
@@
 			)
 		)
+		(property "Manufacturer" "Samsung Electro-Mechanics"
+			(at 154.94 71.12 0)
+			(hide yes)
+			(show_name no)
+			(do_not_autoplace no)
+			(effects
+				(font
+					(size 1.27 1.27)
+				)
+			)
+		)
+		(property "MPN" "CL21A475KAQNNNE"
+			(at 154.94 71.12 0)
+			(hide yes)
+			(show_name no)
+			(do_not_autoplace no)
+			(effects
+				(font
+					(size 1.27 1.27)
+				)
+			)
+		)
+		(property "LCSC" "C1779"
+			(at 154.94 71.12 0)
+			(hide yes)
+			(show_name no)
+			(do_not_autoplace no)
+			(effects
+				(font
+					(size 1.27 1.27)
+				)
+			)
+		)
+		(property "Note_Sourcing" "SOURCING D-614. EXACT_PRIOR from the beta-dm audit line '4.7uF' (ACCEPTED); manufacturer derived from the Samsung Electro-Mechanics part-number family and corroborated by the audit text; identical specification."
+			(at 154.94 71.12 0)
+			(hide yes)
+			(show_name no)
+			(do_not_autoplace no)
+			(effects
+				(font
+					(size 1.27 1.27)
+				)
+			)
+		)
 		(property "Description" "Unpolarized capacitor"
 			(at 154.94 71.12 0)
@@
 			(at 138.43 60.96 0)
 			(hide yes)
+			(show_name no)
+			(do_not_autoplace no)
+			(effects
+				(font
+					(size 1.27 1.27)
+				)
+			)
+		)
+		(property "Manufacturer" "UNI-ROYAL(Uniroyal Elec)"
+			(at 138.43 60.96 0)
+			(hide yes)
+			(show_name no)
+			(do_not_autoplace no)
+			(effects
+				(font
+					(size 1.27 1.27)
+				)
+			)
+		)
+		(property "MPN" "0603WAF1000T5E"
+			(at 138.43 60.96 0)
+			(hide yes)
+			(show_name no)
+			(do_not_autoplace no)
+			(effects
+				(font
+					(size 1.27 1.27)
+				)
+			)
+		)
+		(property "LCSC" "C22775"
+			(at 138.43 60.96 0)
+			(hide yes)
+			(show_name no)
+			(do_not_autoplace no)
+			(effects
+				(font
+					(size 1.27 1.27)
+				)
+			)
+		)
+		(property "Note_Sourcing" "SOURCING D-614. CONTAINED_PRIOR from the beta-dm audit line '100R 1%' (REJECTED - JLC match wrong); manufacturer derived from the UNI-ROYAL(Uniroyal Elec) part-number family and corroborated by the audit text; identical specification."
+			(at 138.43 60.96 0)
+			(hide yes)

Commit message: demo: the BOM is 100% ORDERABLE and the safety part was ordered in the WRONG PACKAGE -- 61 identities ruled against a live distributor record, and a screen that asks the C26 question of every line at once (D-615)
D-614 named this task and named what stopped it: D-096 binds -- a part number
configured from an ordering scheme is a hypothesis until a distributor record
confirms lifecycle and stock, and that session had none to read.  This one read
the JLCPCB catalogue 225 times and KEPT every answer, each stamped with the UTC
minute it was read.

NO COPPER CHANGED.  The authoritative board is byte-identical at
c8e421aa50144fe396aedb5e226aaabeb815bd69ffaf6e04f549ded43831d103.

FAB7 IS CLOSED.  Coverage 75.3% -> 100.0%, orderable 186 -> 247 of 247,
needs_a_sourcing_decision ZERO lines, and fab_package_contract.py reads
FAB1-FAB8 PASS for the first time.

THE FINDING.  screen_part_land_parity.py asks D-613's C26 question of every
sourced line at once against the catalogue's own package field: 119 lines carry
a code, 75 are comparable, 74 MATCH and U18 did not.  The land is MSOP-10; the
BOM ordered LTC4368IDD-1#PBF, and DD is DFN-10-EP(3x3) -- against D-099, which
locked LTC4368IMS-1#PBF under FBV2-PWR-002's "no bottom-terminated parts" on
the single most safety-critical component.  The cached library symbol AND the
project .kicad_sym both still carried it, with a Package field describing a DFN
beside a Footprint field already reading MSOP-10.  Corrected to
LTC4368IMS-1#TRPBF, LCSC C688401 -- the tape-and-reel order code of the
identical device, D-210's precedent, not an electrical change.

Three things the obvious answer would have got wrong: R69 is 1.87 ohm and its
part is 0603WAF187KT5E while 0603WAF1873T5E is 187 kOhm; R95's node over-bound
UNDERSTATES its dissipation because a reversed cell adds in series (154 mW vs
54 mW); and R24/C12's Value strings are looser than their own symbol notes.
NET_MAX_DC grew 17 -> 48 established nodes to give the new dissipation gate
nu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
Parts:
- C12: LCSC (none) -> C309062; MPN (none) -> CL32B226KAJNNNE; Manufacturer (none) -> Samsung Electro-Mechanics; Note_Sourcing (none) -> SOURCING D-615 LIVE_RECORD. JLCPCB record read 2026-09-05T0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
- R24: LCSC (none) -> C26080556; MPN (none) -> SR0805FR-4712RL; Manufacturer (none) -> YAGEO; Note_Sourcing (none) -> SOURCING D-615 LIVE_RECORD. JLCPCB record read 2026-09-05T0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
Changed lines of the file:
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@@
+			)
+		)
+		(property "Manufacturer" "Samsung Electro-Mechanics"
+			(at 218.44 92.71 0)
+			(hide yes)
+			(show_name no)
+			(do_not_autoplace no)
+			(effects
+				(font
+					(size 1.27 1.27)
+				)
+			)
+		)
+		(property "MPN" "CL32B226KAJNNNE"
+			(at 218.44 92.71 0)
+			(hide yes)
+			(show_name no)
+			(do_not_autoplace no)
+			(effects
+				(font
+					(size 1.27 1.27)
+				)
+			)
+		)
+		(property "LCSC" "C309062"
+			(at 218.44 92.71 0)
+			(hide yes)
+			(show_name no)
+			(do_not_autoplace no)
+			(effects
+				(font
+					(size 1.27 1.27)
+				)
+			)
+		)
+		(property "Note_Sourcing" "SOURCING D-615 LIVE_RECORD. JLCPCB record read 2026-09-05T00:59:59Z: expand library, stock 280611, land 1210, Capacitance 22uF; Temperature Coefficient X7R; Tolerance ±10%; Voltage Rating 25V. Gates: 2x operating and survives absolute; not a resistor."
+			(at 218.44 92.71 0)
+			(hide yes)
+			(show_name no)
+			(do_not_autoplace no)
+			(effects
+				(font
+					(size 1.27 1.27)
+				)
 			)
 		)
@@
 			(at 175.26 92.71 0)
 			(hide yes)
+			(show_name no)
+			(do_not_autoplace no)
+			(effects
+				(font
+					(size 1.27 1.27)
+				)
+			)
+		)
+		(property "Manufacturer" "YAGEO"
+			(at 175.26 92.71 0)
+			(hide yes)
+			(show_name no)
+			(do_not_autoplace no)
+			(effects
+				(font
+					(size 1.27 1.27)
+				)
+			)
+		)
+		(property "MPN" "SR0805FR-4712RL"
+			(at 175.26 92.71 0)
+			(hide yes)
+			(show_name no)
+			(do_not_autoplace no)
+			(effects
+				(font
+					(size 1.27 1.27)
+				)
+			)
+		)
+		(property "LCSC" "C26080556"
+			(at 175.26 92.71 0)
+			(hide yes)
+			(show_name no)
+			(do_not_autoplace no)
+			(effects
+				(font
+					(size 1.27 1.27)
+				)
+			)
+		)
+		(property "Note_Sourcing" "SOURCING D-615 LIVE_RECORD. JLCPCB record read 2026-09-05T00:59:59Z: expand library, stock 1504, land 0805, Operating Temperature -55℃~+155℃; Power(Watts) 500mW; Resistance 12Ω; Temperature Coefficient ±100ppm/℃; Tolerance ±1%; Type Thick Film Resistor; Voltage-Supply(Max) 500V. Gates: land working voltage vs the highest node; 2x operating and survives single fault."
+			(at 175.26 92.71 0)
+			(hide yes)

Commit message: demo: D-750 and D-751 -- the external first-spin review found four real defects, and finishing its repairs found two more.
An external first-spin review (Fable 5.1 + Astra) reopened DEMO_READY_FOR_FAB at
b593b97 and named thirteen items.  Four were real defects on the frozen package:
J5's BOM identity still named the 2x12 BCS-112-S-D-HE that D-237 superseded eight
months ago, U14.6 QSTRT was physically floating behind a deliberate no_connect,
audit_rail_ampacity.py computed at 0.0174 mm inner copper against a board that
declares 0.0152 mm, and neither boost converter had a local input capacitor --
the nearest was 36.6 mm and the *named* input part 93.5 mm away.  A fifth,
item 7, is a design-condition failure: TI guarantees the TPS61169 OFF only when
the LED array's minimum Vf exceeds the maximum VIN, this panel is 2.9-3.2 V on a
3.3 V rail, and the shutdown DC path converges at about 25 mA -- a fifth of full
brightness, with no firmware mitigation because +3V3 is switched by SW9.

D-750 closed all of them and dispositioned the other nine, item by item, with
FIRST-ARTICLE and PROCUREMENT work explicitly separated from pre-order blockers.
The charger input was re-laid 250.8 -> 189.8 mm and 440 -> 216 mOhm, which is
what buys the 360 min tMAXCHG its margin; C83 and C84 were fitted on the existing
C33/C64 BOM line; Q11, the backlight true-off disconnect, was fitted on Q1's line.

D-751 FINISHED THE TRANSACTION, AND EACH THING IT TOUCHED HELD ANOTHER DEFECT.

* Q11 was on the board as a symbol and a BOM line and NOT as a circuit: three
  unapproved open edges, all three of them its own pins.  Routed with three
  --tap-first taps, 16.26 mm and four barrels.  The first run was REFUSED for a
  0.44 mm dangling In2 stub the tap left past its T; trimmed, re-run clean.
* placement_contract.py HAD NO WORD FOR AN ADDED PART, so the whole standing
  suite read "placement FAIL" for a legitimate act.  --add exists; PL7 now holds
  an ADDED pad to the same foreign-copper clearance a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
Parts:
- Q1: LCSC (none) -> C20917; Note_Sourcing (none) -> SOURCING D-751 2026-09-18. The AO3400A was the ONLY line on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
Changed lines of the file:
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@@
+			)
+		)
+		(property "LCSC" "C20917"
+			(at 196.85 46.99 0)
+			(hide yes)
+			(show_name no)
+			(do_not_autoplace no)
+			(effects
+				(font
+					(size 1.27 1.27)
+				)
+			)
+		)
+		(property "Note_Sourcing" "SOURCING D-751 2026-09-18. The AO3400A was the ONLY line on the assembly BOM with no distributor identity (121 of 122 rows carried one), and D-750 made it a two-piece line by adding Q11, the display-backlight true-off disconnect. Verified live 2026-09-18 per D-096 through the JLCPCB parts API; record committed at evidence/jlc-live/ao3400a-568c27aa.json: LCSC C20917, Alpha & Omega Semicon, AO3400A, SOT-23, componentLibraryType = BASE (no extended-part fee, no feeder setup), stock 812570, 0.0847 USD at 1 / 0.0479 at 6000, 30 V, Id 5.7 A continuous, RDS(on) 48 mOhm at VGS 2.5 V, VGS(th) 1.45 V, Pd 1.4 W, -55 to +150 C, RoHS. BOTH FITTED USES ARE FAR INSIDE THAT ENVELOPE: Q1 sinks the IR LED and Q11 carries the 109 mA panel backlight cathode return, where even the worst-case 48 mOhm at a 2.5 V gate costs 5.2 mV. Stock is a snapshot, not a guarantee."
+			(at 196.85 46.99 0)
+			(hide yes)
+			(show_name no)
+			(do_not_autoplace no)
+			(effects
+				(font
+					(size 1.27 1.27)
+				)
 			)
 		)
