File: hardware/demo/kicad/aqroot-demo/03_spi_a_display_sd.kicad_sch (KiCad schematic)
At the start: 25 parts, among them J1 FH69-50S-0.5SH, J2 Molex_5025700893, Q11 AO3400A, U17 TPS61169DCKR

Commit message: demo: D-766 -- a 30 V part on a 39 V node this board publishes, a via where the manufacturer prints "no vias", a warm reset that outlived its own safe state, and a power audit that answered differently every other time it was asked
authority 9e4728ae -> 5849b658; objects_added 0, objects_removed 3 (all GND).

D-752 wrote "THE AO3400A IS A 30 V PART" in bold, in three files, and shipped
the 30 V part -- while this board's own .kicad_dru says an open-LED fault puts
up to 39 V on LED_BOOST, and the entire LED_BOOST clearance regime exists
because of it.  Q11's drain is the panel cathode.  D-752's D14/C85/R132
ordering is sound and is retained in full, but any one of those three failing
re-creates the state it removed, and a protection element must survive the
fault it exists to prevent.  Q11 -> AO3422: BVDSS 55 V min, 41 % margin, same
SOT-23, same 1=G/2=S/3=D, so no land pattern moved.  Conduction is guaranteed
by the threshold spec itself -- VGS(th) is specified at 250 mA and this circuit
needs 109 mA -- and RDS(on) cannot move the LED current because U17's FB senses
Q11's SOURCE.  The one number that gets worse is named: VGS(th) max
1.45 -> 2.00 V cuts the ordering margin 4.6x -> 2.06x, accepted because a 55 V
part turns a violation from avalanche into a recoverable U17 open-LED latch.
F5 gained the clause it never had: it PARSES the 39 V ceiling out of the
.kicad_dru, refuses a FET with no published rating, and measures VDS, held-gate
enhancement and decay-to-threshold against the FITTED part -- four more live
controls, one of which is the board D-752 shipped, refused by the rating clause
alone.

Wurth 74438357010 prints "No vias and traces underneath the inductor" under
both recommended land patterns, and the board carried a 0.8 mm GND barrel
0.200 mm from L4's centre with 0.6 mm of track feeding it.  All three objects
removed; LAND8 added, deriving the restricted strip from L4's own fitted pads
and refusing the previous board by coordinate.  The relocation was ME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
Parts:
- C85: Note D-752 GATE-HOLD RESERVOIR. Holds Q11's gate up through every TPS61169 PWM low phase. Worst droop over the longest low phase the part specifies (5 kHz, 1 % duty = 199 us) is 26 mV on a 2.6 V worst-case gate. With R132 the fall time constant is 22 ms, and the gate is still at 2.29 V at the 2.5 ms by which U17 is guaranteed to be in shutdown. 50 V X7R: the DC bias here is under 3 V, so the derating is negligible and tau is tolerance-bounded to 19.6-24.4 ms. -> D-752 GATE-HOLD RESERVOIR. Holds Q11's gate up through every TPS61169 PWM low phase. Worst droop over the longest low phase the part specifies (5 kHz, 1 % duty = 199 us) is 26 mV on a 2.6 V worst-case gate. With R132 the fall time constant is 22 ms, and the gate is still at 2.29 V at the 2.5 ms by which U17 is guaranteed to be in shutdown. 50 V X7R: the DC bias here is under 3 V, so the derating is negligible and tau is tolerance-bounded to 19.6-24.4 ms. || D-766: 100 nF RETAINED. 220 nF would restore D-752's 4.6x ordering margin after the AO3422's higher VGS(th) max cut it to 2.06x, but it would open a new single-piece BOM line, and the margin now guards only a recoverable converter latch rather than an over-stressed 30 V FET. Droop over the longest low phase the TPS61169 specifies (5 kHz, 1 % duty, 199 us) is unchanged at 26 mV, and the gate is still 2.29 V at the 2.5 ms by which U17 is guaranteed in shutdown - above the AO3422's 2.00 V worst-case threshold.
- D14: Note D-752 BACKLIGHT-DISCONNECT GATE HOLD, AND WHY Q11 MAY NOT SHARE U17 CTRL. D-750/D-751 tied Q11's gate to /DISP_BL_CTL, the same net as U17 CTRL, on the premise that PWM would shut the converter down and open Q11 together. TI SNVSA40B section 6.3.5 says the opposite: the TPS61169 CHOPS ITS INTERNAL 204 mV REFERENCE at the CTRL duty cycle and filters it, so 'only the WLED DC current is modulated, which is often referred as analog dimming' -- THE CONVERTER KEEPS SWITCHING THROUGH EVERY PWM LOW PHASE. Shutdown is entered only after CTRL is low for more than tSD (2.5 ms max, EC table). With the gate shared, every PWM low phase therefore opened the LED string while U17 was actively regulating: FB collapses below 30 mV, SW ramps to VOVP_SW (36/37.5/39 V), open-LED protection (6.3.2) latches the device off after three switching cycles, and Q11's DRAIN -- the panel cathode -- follows the anode to about 36 V while R69 holds its SOURCE at 0 V. THE AO3400A IS A 30 V PART (AOS Rev 3.1). Firmware a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 -> D-752 BACKLIGHT-DISCONNECT GATE HOLD, AND WHY Q11 MAY NOT SHARE U17 CTRL. D-750/D-751 tied Q11's gate to /DISP_BL_CTL, the same net as U17 CTRL, on the premise that PWM would shut the converter down and open Q11 together. TI SNVSA40B section 6.3.5 says the opposite: the TPS61169 CHOPS ITS INTERNAL 204 mV REFERENCE at the CTRL duty cycle and filters it, so 'only the WLED DC current is modulated, which is often referred as analog dimming' -- THE CONVERTER KEEPS SWITCHING THROUGH EVERY PWM LOW PHASE. Shutdown is entered only after CTRL is low for more than tSD (2.5 ms max, EC table). With the gate shared, every PWM low phase therefore opened the LED string while U17 was actively regulating: FB collapses below 30 mV, SW ramps to VOVP_SW (36/37.5/39 V), open-LED protection (6.3.2) latches the device off after three switching cycles, and Q11's DRAIN -- the panel cathode -- follows the anode to about 36 V while R69 holds its SOURCE at 0 V. THE AO3400A IS A 30 V PART (AOS Rev 3.1). Firmware a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
- Q11: value AO3400A -> AO3422; LCSC C20917 -> C37130; MPN AO3400A -> AO3422; Note D-750 BACKLIGHT TRUE-OFF DISCONNECT. TPS61169 (U17) shutdown does NOT make the panel dark: TI states a DC path remains from VIN through L3 and D8 to the LED string and guarantees OFF only when the LED array MINIMUM forward voltage exceeds the MAXIMUM VIN. This board boosts from +3V3 and the EastRising ER-TFT035IPS-6 backlight is SIX LEDs IN PARALLEL at 2.9-3.2 V (D-079), so Vf(min) 2.9 V is BELOW the 3.3 V rail and the condition FAILS. Solving the as-built network (+3V3 - L3 - D8 - R70..R73 8.25 R - six parallel LEDs - R69 1.87 R - GND) with a white-LED forward curve converges at about 25 mA: roughly a fifth of full brightness, plainly visible in a dark room, and about 82 mW of continuous drain whenever +3V3 is up and the backlight is commanded off. +3V3 is switched by SW9, not by firmware, so there is no software mitigation: the screen would never go dark while the device is on. Q11 breaks that DC path in the PANEL CATHODE RETURN, between J1 and the LED_K sense node. IT IS OUTSIDE TH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 -> D-750 BACKLIGHT TRUE-OFF DISCONNECT. TPS61169 (U17) shutdown does NOT make the panel dark: TI states a DC path remains from VIN through L3 and D8 to the LED string and guarantees OFF only when the LED array MINIMUM forward voltage exceeds the MAXIMUM VIN. This board boosts from +3V3 and the EastRising ER-TFT035IPS-6 backlight is SIX LEDs IN PARALLEL at 2.9-3.2 V (D-079), so Vf(min) 2.9 V is BELOW the 3.3 V rail and the condition FAILS. Solving the as-built network (+3V3 - L3 - D8 - R70..R73 8.25 R - six parallel LEDs - R69 1.87 R - GND) with a white-LED forward curve converges at about 25 mA: roughly a fifth of full brightness, plainly visible in a dark room, and about 82 mW of continuous drain whenever +3V3 is up and the backlight is commanded off. +3V3 is switched by SW9, not by firmware, so there is no software mitigation: the screen would never go dark while the device is on. Q11 breaks that DC path in the PANEL CATHODE RETURN, between J1 and the LED_K sense node. IT IS OUTSIDE TH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; Note_Sourcing SOURCING D-751 2026-09-18. The AO3400A was the ONLY line on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 -> SOURCING D-766 2026-09-18. Verified live per D-096 through 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; Package SOT-23-3, pin 1 = G, 2 = S, 3 = D (confirmed from the AOS d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 -> SOT-23-3, pin 1 = G, 2 = S, 3 = D (AOS rev 2.1 top/bottom v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
- R132: Note D-752 GATE-HOLD DISCHARGE. Sets the fall time of Q11's gate with C85: tau = 220 k * 100 nF = 22 ms, against the TPS61169's 2.5 ms max CTRL-low-to-shutdown. Q11 cannot open before U17 has stopped switching. ALSO SETS THE TRUE-OFF FLOOR: D14's worst published reverse leakage (1 uA) plus Q11's 100 nA IGSS across 220 k is 0.242 V, below the AO3400A's 0.65 V minimum VGS(th), so the OFF state is held by a published number rather than an assumption. A larger value would raise that floor; a smaller one would need a larger capacitor for the same tau. Steady-state cost when the backlight is ON is 12.5 uA. -> D-752 GATE-HOLD DISCHARGE. Sets the fall time of Q11's gate with C85: tau = 220 k * 100 nF = 22 ms, against the TPS61169's 2.5 ms max CTRL-low-to-shutdown. Q11 cannot open before U17 has stopped switching. ALSO SETS THE TRUE-OFF FLOOR: D14's worst published reverse leakage (1 uA) plus Q11's 100 nA IGSS across 220 k is 0.242 V, below the AO3400A's 0.65 V minimum VGS(th), so the OFF state is held by a published number rather than an assumption. A larger value would raise that floor; a smaller one would need a larger capacitor for the same tau. Steady-state cost when the backlight is ON is 12.5 uA. || D-766: tau is unchanged at 22 ms, but the AO3422's VGS(th) max of 2.00 V (the AO3400A's was 1.45 V) shortens the worst-case decay-to-threshold from 11.4 ms to 5.14 ms, so the ordering margin against the TPS61169's 2.5 ms tSD is now 2.06x. Retained deliberately: with a 55 V Q11 a lost ordering costs a recoverable U17 open-LED latch, not avalanche in a 30 V part.

Commit message: demo: D-767 -- the same two defect classes, asked of the whole board: a second inductor nobody checked, a second semiconductor on the 39 V node, and an arithmetic error in D-766 itself
authority 5849b658, UNCHANGED.  No PCB change.  Every Gerber, drill, CPL and BOM
file is identical once the embedded CreationDate is normalised; the only
semantic change in MANIFEST.json is the sha256 of 03_spi_a_display_sd.kicad_sch,
the sheet carrying the corrected Q11 note -- and FAB1 refused the package until
that entry was regenerated, which is the provenance clause working as intended.

D-766 fixed four specific defects; each was an INSTANCE of something general,
and a fix that closes one instance and leaves the class open is half a fix.

LAND8 tested L4 BY NAME, and this board carries six inductors -- one of which,
L2, is the SAME Wurth 74438357010, with two /NFC_5V_EN segments running the full
length of its restricted strip.  L2 is DNP, so no fabricated board has a part
over that copper; rerouting a live net through a 1.39 mm channel bracketed by
L2's own pads, and re-certifying the release, to cure a defect on an unpopulated
part was DECLINED.  The gate carries it instead: LAND8 now enumerates every
instance of an explicit table of restricted footprints, FAILS on a fitted one,
REPORTS a DNP one with coordinates, and states its own coverage limit.

And D-766's LAND8 had a bug.  It read the strip from pad.GetSize(), which is in
the PAD's own frame, so a ROTATED instance was measured across the wrong axis
and returned a negative-height rectangle that collided with nothing and passed.
L1 -- the TPS63020 inductor, the highest-current one on this board -- sits at
90 degrees and returned 0.980 x -1.030 mm.  Measured from pad bounding boxes its
strip is 3.400 x 1.390 mm and CLEAN, as are L3, L5 and L6.  A second live
control derives L1's strip every run.

The 39 V node has TWO semiconductors.  D8 stands off the same ceiling in
reverse.  It is RETAINED and is not a defect -- NSR0240, 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
Parts:
- Q11: Note D-750 BACKLIGHT TRUE-OFF DISCONNECT. TPS61169 (U17) shutdown does NOT make the panel dark: TI states a DC path remains from VIN through L3 and D8 to the LED string and guarantees OFF only when the LED array MINIMUM forward voltage exceeds the MAXIMUM VIN. This board boosts from +3V3 and the EastRising ER-TFT035IPS-6 backlight is SIX LEDs IN PARALLEL at 2.9-3.2 V (D-079), so Vf(min) 2.9 V is BELOW the 3.3 V rail and the condition FAILS. Solving the as-built network (+3V3 - L3 - D8 - R70..R73 8.25 R - six parallel LEDs - R69 1.87 R - GND) with a white-LED forward curve converges at about 25 mA: roughly a fifth of full brightness, plainly visible in a dark room, and about 82 mW of continuous drain whenever +3V3 is up and the backlight is commanded off. +3V3 is switched by SW9, not by firmware, so there is no software mitigation: the screen would never go dark while the device is on. Q11 breaks that DC path in the PANEL CATHODE RETURN, between J1 and the LED_K sense node. IT IS OUTSIDE TH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 -> D-750 BACKLIGHT TRUE-OFF DISCONNECT. TPS61169 (U17) shutdown does NOT make the panel dark: TI states a DC path remains from VIN through L3 and D8 to the LED string and guarantees OFF only when the LED array MINIMUM forward voltage exceeds the MAXIMUM VIN. This board boosts from +3V3 and the EastRising ER-TFT035IPS-6 backlight is SIX LEDs IN PARALLEL at 2.9-3.2 V (D-079), so Vf(min) 2.9 V is BELOW the 3.3 V rail and the condition FAILS. Solving the as-built network (+3V3 - L3 - D8 - R70..R73 8.25 R - six parallel LEDs - R69 1.87 R - GND) with a white-LED forward curve converges at about 25 mA: roughly a fifth of full brightness, plainly visible in a dark room, and about 82 mW of continuous drain whenever +3V3 is up and the backlight is commanded off. +3V3 is switched by SW9, not by firmware, so there is no software mitigation: the screen would never go dark while the device is on. Q11 breaks that DC path in the PANEL CATHODE RETURN, between J1 and the LED_K sense node. IT IS OUTSIDE TH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
