File: hardware/demo/kicad/aqroot-demo/03_spi_a_display_sd.kicad_sch (KiCad schematic)
At the start: 25 parts, among them J1 FH69-50S-0.5SH, J2 Molex_5025700893, Q11 AO3422, U17 TPS61169DCKR

Commit message: demo: D-777 · D-778 · D-779 -- the battery connector had no rating in this repository, the derating rule was run against the specification instead of the part, and an extracted datasheet changed a unit that a proof was built on
Closes the round-3 external review hold on D-776.  All six reproduced items
are closed by measurement.  NO COPPER MOVED: every copper Gerber, both drill
files and Edge_Cuts are byte-identical to the D-776 package apart from
timestamps.  One BOM row changed -- C85 100nF -> 1uF, onto a line this board
already buys.  Board 8c548ece -> 880a2ece.

D-777  J4 is a JST B2B-PH-K-S(LF)(SN), published at 2 A AC/DC (AWG #24) --
       the LOWEST number in the battery path, below the BQ25185's 2.5625 A
       IBAT_OCP minimum, D-771's 3.960 A breaker and F1's 5 A fuse.  D-775's
       published simultaneous envelope sat at 2.2715 A, 13.6 % OVER, and
       D-776 passed in that state.  Holding it under 2 A by VCELL alone needs
       a 4.16 V pack, so the bounded term is the internal one: while BOTH
       accessory rails are enabled firmware RESERVES the sub-GHz TX path, the
       NFC field and the IR transmitter, enforced in SpiBusB::beginTransmit.
       The connection carries 1.8797 A, 6.0 % inside its rating; D-098's
       400/300 mA are both still guaranteed.  Rating, rated gauge, applicable
       wire range and the pack's lead gauge are all PARSED from archived
       vendor text.  The JST B2B-XH-A 3 A upgrade is confirmed live, costed
       and deferred to REV-B (needs an owner protected-copper exception on
       BAT_CONNECTOR_P); a first-article J4 temperature-rise measurement is
       added instead.

D-778  Twenty-four value strings UNDERSTATE the part the BOM buys, so three
       of D-774's five derating exceptions were against a rating this board
       does not have.  Ratings now come from the part, joined reference ->
       LCSC -> the committed live distributor record; all 76 fitted
       capacitors covered, a missing record is a re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
Parts:
- C85: value 100nF X7R -> 1uF 10V X7R; LCSC C14663 -> C106858; MPN CC0603KRX7R9BB104 -> CC0603KRX7R8BB105; Note D-752 GATE-HOLD RESERVOIR. Holds Q11's gate up through ever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 -> D-752 GATE-HOLD RESERVOIR, RESIZED AT D-779. Holds Q11's ga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; Package Existing 100nF X7R 50 V 0603 line -- no new purchasing iden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 -> Existing 1uF 10V X7R 0603 line (C25/C37/C38/C62/C63/C67) --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
- Q11: Note D-750 BACKLIGHT TRUE-OFF DISCONNECT. TPS61169 (U17) shutdown does NOT make the panel dark: TI states a DC path remains from VIN through L3 and D8 to the LED string and guarantees OFF only when the LED array MINIMUM forward voltage exceeds the MAXIMUM VIN. This board boosts from +3V3 and the EastRising ER-TFT035IPS-6 backlight is SIX LEDs IN PARALLEL at 2.9-3.2 V (D-079), so Vf(min) 2.9 V is BELOW the 3.3 V rail and the condition FAILS. Solving the as-built network (+3V3 - L3 - D8 - R70..R73 8.25 R - six parallel LEDs - R69 1.87 R - GND) with a white-LED forward curve converges at about 25 mA: roughly a fifth of full brightness, plainly visible in a dark room, and about 82 mW of continuous drain whenever +3V3 is up and the backlight is commanded off. +3V3 is switched by SW9, not by firmware, so there is no software mitigation: the screen would never go dark while the device is on. Q11 breaks that DC path in the PANEL CATHODE RETURN, between J1 and the LED_K sense node. IT IS OUTSIDE TH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 -> D-750 BACKLIGHT TRUE-OFF DISCONNECT. TPS61169 (U17) shutdown does NOT make the panel dark: TI states a DC path remains from VIN through L3 and D8 to the LED string and guarantees OFF only when the LED array MINIMUM forward voltage exceeds the MAXIMUM VIN. This board boosts from +3V3 and the EastRising ER-TFT035IPS-6 backlight is SIX LEDs IN PARALLEL at 2.9-3.2 V (D-079), so Vf(min) 2.9 V is BELOW the 3.3 V rail and the condition FAILS. Solving the as-built network (+3V3 - L3 - D8 - R70..R73 8.25 R - six parallel LEDs - R69 1.87 R - GND) with a white-LED forward curve converges at about 25 mA: roughly a fifth of full brightness, plainly visible in a dark room, and about 82 mW of continuous drain whenever +3V3 is up and the backlight is commanded off. +3V3 is switched by SW9, not by firmware, so there is no software mitigation: the screen would never go dark while the device is on. Q11 breaks that DC path in the PANEL CATHODE RETURN, between J1 and the LED_K sense node. IT IS OUTSIDE TH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
- R132: Note D-752 GATE-HOLD DISCHARGE. Sets the fall time of Q11's gate with C85: tau = 220 k * 100 nF = 22 ms, against the TPS61169's 2.5 ms max CTRL-low-to-shutdown. Q11 cannot open before U17 has stopped switching. ALSO SETS THE TRUE-OFF FLOOR: D14's worst published reverse leakage (1 uA) plus Q11's 100 nA IGSS across 220 k is 0.242 V, below the AO3400A's 0.65 V minimum VGS(th), so the OFF state is held by a published number rather than an assumption. A larger value would raise that floor; a smaller one would need a larger capacitor for the same tau. Steady-state cost when the backlight is ON is 12.5 uA. || D-766: tau is unchanged at 22 ms, but the AO3422's VGS(th) max of 2.00 V (the AO3400A's was 1.45 V) shortens the worst-case decay-to-threshold from 11.4 ms to 5.14 ms, so the ordering margin against the TPS61169's 2.5 ms tSD is now 2.06x. Retained deliberately: with a 55 V Q11 a lost ordering costs a recoverable U17 open-LED latch, not avalanche in a 30 V part. -> D-752 GATE-HOLD DISCHARGE. Sets the fall time of Q11's gate with C85: tau = 220 k * 100 nF = 22 ms, against the TPS61169's 2.5 ms max CTRL-low-to-shutdown. Q11 cannot open before U17 has stopped switching. ALSO SETS THE TRUE-OFF FLOOR: D14's worst published reverse leakage (1 uA) plus Q11's 100 nA IGSS across 220 k is 0.242 V, below the AO3400A's 0.65 V minimum VGS(th), so the OFF state is held by a published number rather than an assumption. A larger value would raise that floor; a smaller one would need a larger capacitor for the same tau. Steady-state cost when the backlight is ON is 12.5 uA. || D-766: the AO3422's VGS(th) max of 2.00 V (the AO3400A's was 1.45 V) shortened the worst-case decay-to-threshold from 11.4 ms to 5.14 ms, an ordering margin of 2.06x against the TPS61169's 2.5 ms tSD. || D-779: R132 STAYS AT 220 k and C85 moves 100 nF -> 1 uF instead. R132 is the wrong knob - it also sets the TRUE-OFF FLOOR, and at 470 k D14's 1 uA plus Q11's 100 nA would reach 0.517 V agai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
