File: hardware/demo/kicad/aqroot-demo/03_spi_a_display_sd.kicad_sch (KiCad schematic)
At the start: 25 parts, among them J1 FH69-50S-0.5SH, J2 Molex_5025700893, Q11 AO3422, U17 TPS61169DCKR

Commit message: demo: D-780/D-781 close Round-3 Q11 and battery blockers
Parts:
- C85: Note D-752 GATE-HOLD RESERVOIR, RESIZED AT D-779. Holds Q11's gate up through every TPS61169 PWM low phase, and sets the CTRL-low decay with R132. || D-779: 100 nF -> 1 uF, ON THE EXISTING 1 uF 0603 X7R LINE, because D-766's conduction proof for Q11 was read off a CORRUPTED UNIT. The archived AO3422 text extraction renders Symbol-font glyphs as Latin -- Ohm as W, micro as m -- so its EC table reads 'VGS(th) ... ID=250mA' when the datasheet says 250 uA (the same file reads 'RDS(ON) 160mW', which the committed JLCPCB record for C37130 independently gives as 160 mOhm, and 'IDSS 1 mA at VDS=44 V', which would be 44 mW standing in a SOT-23). D-766 concluded from the wrong unit that 109 mA is 'LESS THAN HALF the threshold test current'; it is 436 times MORE, so that argument is deleted rather than softened. WHAT IS ACTUALLY PUBLISHED: RDS(on) <= 200 mOhm at VGS = 2.5 V and ID = 1.5 A, which is 13.8x this string's 109 mA and only 104 mV above the held VGS of 2.396 V. Between VGS(th) max 2.0 V and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 -> D-752 GATE-HOLD RESERVOIR, RESIZED AT D-779. Holds Q11's gate up through every TPS61169 PWM low phase, and sets the CTRL-low decay with R132. || D-779: 100 nF -> 1 uF, ON THE EXISTING 1 uF 0603 X7R LINE, because D-766's conduction proof for Q11 was read off a CORRUPTED UNIT. The archived AO3422 text extraction renders Symbol-font glyphs as Latin -- Ohm as W, micro as m -- so its EC table reads 'VGS(th) ... ID=250mA' when the datasheet says 250 uA (the same file reads 'RDS(ON) 160mW', which the committed JLCPCB record for C37130 independently gives as 160 mOhm, and 'IDSS 1 mA at VDS=44 V', which would be 44 mW standing in a SOT-23). D-766 concluded from the wrong unit that 109 mA is 'LESS THAN HALF the threshold test current'; it is 436 times MORE, so that argument is deleted rather than softened. WHAT IS ACTUALLY PUBLISHED: RDS(on) <= 200 mOhm at VGS = 2.5 V and ID = 1.5 A, which is 13.8x this string's 109 mA and only 104 mV above the held VGS of 2.396 V. Between VGS(th) max 2.0 V and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
- Q11: value AO3422 -> SQ2364EES-T1_BE3; LCSC C37130 -> C5758702; MPN AO3422 -> SQ2364EES-T1_BE3; Manufacturer Alpha & Omega Semiconductor -> Vishay Siliconix; Note D-750 BACKLIGHT TRUE-OFF DISCONNECT. TPS61169 (U17) shutdown does NOT make the panel dark: TI states a DC path remains from VIN through L3 and D8 to the LED string and guarantees OFF only when the LED array MINIMUM forward voltage exceeds the MAXIMUM VIN. This board boosts from +3V3 and the EastRising ER-TFT035IPS-6 backlight is SIX LEDs IN PARALLEL at 2.9-3.2 V (D-079), so Vf(min) 2.9 V is BELOW the 3.3 V rail and the condition FAILS. Solving the as-built network (+3V3 - L3 - D8 - R70..R73 8.25 R - six parallel LEDs - R69 1.87 R - GND) with a white-LED forward curve converges at about 25 mA: roughly a fifth of full brightness, plainly visible in a dark room, and about 82 mW of continuous drain whenever +3V3 is up and the backlight is commanded off. +3V3 is switched by SW9, not by firmware, so there is no software mitigation: the screen would never go dark while the device is on. Q11 breaks that DC path in the PANEL CATHODE RETURN, between J1 and the LED_K sense node. IT IS OUTSIDE TH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 -> D-750 BACKLIGHT TRUE-OFF DISCONNECT. TPS61169 (U17) shutdown does NOT make the panel dark: TI states a DC path remains from VIN through L3 and D8 to the LED string and guarantees OFF only when the LED array MINIMUM forward voltage exceeds the MAXIMUM VIN. This board boosts from +3V3 and the EastRising ER-TFT035IPS-6 backlight is SIX LEDs IN PARALLEL at 2.9-3.2 V (D-079), so Vf(min) 2.9 V is BELOW the 3.3 V rail and the condition FAILS. Solving the as-built network (+3V3 - L3 - D8 - R70..R73 8.25 R - six parallel LEDs - R69 1.87 R - GND) with a white-LED forward curve converges at about 25 mA: roughly a fifth of full brightness, plainly visible in a dark room, and about 82 mW of continuous drain whenever +3V3 is up and the backlight is commanded off. +3V3 is switched by SW9, not by firmware, so there is no software mitigation: the screen would never go dark while the device is on. Q11 breaks that DC path in the PANEL CATHODE RETURN, between J1 and the LED_K sense node. IT IS OUTSIDE TH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; Note_Sourcing SOURCING D-766 2026-09-18. Verified live per D-096 through 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 -> SOURCING D-780 2026-09-19. JLCPCB live API record committed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; Package SOT-23-3, pin 1 = G, 2 = S, 3 = D (AOS rev 2.1 top/bottom v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 -> SOT-23 (TO-236), pin 1=G, pin 2=S, pin 3=D; drop-in land/pi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
- R132: Note D-752 GATE-HOLD DISCHARGE. Sets the fall time of Q11's gate with C85: tau = 220 k * 100 nF = 22 ms, against the TPS61169's 2.5 ms max CTRL-low-to-shutdown. Q11 cannot open before U17 has stopped switching. ALSO SETS THE TRUE-OFF FLOOR: D14's worst published reverse leakage (1 uA) plus Q11's 100 nA IGSS across 220 k is 0.242 V, below the AO3400A's 0.65 V minimum VGS(th), so the OFF state is held by a published number rather than an assumption. A larger value would raise that floor; a smaller one would need a larger capacitor for the same tau. Steady-state cost when the backlight is ON is 12.5 uA. || D-766: the AO3422's VGS(th) max of 2.00 V (the AO3400A's was 1.45 V) shortened the worst-case decay-to-threshold from 11.4 ms to 5.14 ms, an ordering margin of 2.06x against the TPS61169's 2.5 ms tSD. || D-779: R132 STAYS AT 220 k and C85 moves 100 nF -> 1 uF instead. R132 is the wrong knob - it also sets the TRUE-OFF FLOOR, and at 470 k D14's 1 uA plus Q11's 100 nA would reach 0.517 V agai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 -> D-752 GATE-HOLD DISCHARGE. Sets the fall time of Q11's gate with C85: tau = 220 k * 100 nF = 22 ms, against the TPS61169's 2.5 ms max CTRL-low-to-shutdown. Q11 cannot open before U17 has stopped switching. ALSO SETS THE TRUE-OFF FLOOR: D14's worst published reverse leakage (1 uA) plus Q11's 100 nA IGSS across 220 k is 0.242 V, below the AO3400A's 0.65 V minimum VGS(th), so the OFF state is held by a published number rather than an assumption. A larger value would raise that floor; a smaller one would need a larger capacitor for the same tau. Steady-state cost when the backlight is ON is 12.5 uA. || D-766: the AO3422's VGS(th) max of 2.00 V (the AO3400A's was 1.45 V) shortened the worst-case decay-to-threshold from 11.4 ms to 5.14 ms, an ordering margin of 2.06x against the TPS61169's 2.5 ms tSD. || D-779: R132 STAYS AT 220 k and C85 moves 100 nF -> 1 uF instead. R132 is the wrong knob - it also sets the TRUE-OFF FLOOR, and at 470 k D14's 1 uA plus Q11's 100 nA would reach 0.517 V agai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
