File: hardware/demo/kicad/aqroot-demo/aqroot-Beta-v2.kicad_sch (KiCad schematic)
At the start: 0 parts

Commit message: demo: D-788 close Round-7 and centre the +3V3 rail inside the display's absolute maximum
Round-7 external review REJECTED D-787.  Astra reproduced 20 observed release
defects (6 high, 6 medium, 8 low) and Fable reproduced a subset plus a sourcing
concern.  All twenty are closed.  Auditing the candidate against its own primary
sources found SIX MORE, R7-N01..R7-N06, and the first two moved the board.

THE HIGH ONE.  The fitted ER-TFT035IPS-6 is an ILI9488 panel whose own datasheet
(archived vendor/ILITEK/ilitek-ili9488-v100.pdf, Table 41) makes 3.3 V the
ABSOLUTE MAXIMUM on both VCI and IOVCC.  D-787's power-save corner stood 242 mV
over it and its NOMINAL stood 9 mV over it.  Closed with two objects and no new
component: U12's PS/SYNC moves GND -> EN (forced fixed-frequency PWM, so TI's
VFB_PS +5 % excursion cannot occur) and the feedback divider moves down.

R7-N01/R7-N02, FOUND HERE.  A DC bound is not the whole high side -- ripple and
load-transient overshoot ride on top of it -- and the low side had NO MCU clause
at all: the rail minimum was checked against the panel's VCI 2.5 V and the
Community Port's published minimum, never against the ESP32-S3-WROOM-1's own
3.0 V VDD33 row.  The first D-788 draft's 187 kOhm left 47.97 mV under a DAMAGE
limit against 86.36 mV over a RECOVERABLE one, which is the wrong way round.
F6 now computes the ripple (1.68 mV pp from SLVS916I's minimum oscillator
frequency and L1's minimum inductance), charges it to both ends, adds the module
floor and the +3V3 plane's bounded distribution drop, and ENUMERATES every
purchasable E192 0.1 % R40 value -- requiring the fitted one to maximise the
smaller of the two headrooms.  R40 is therefore 189 kOhm (YAGEO
RT0603BRD07189KL, C861174, live stock 339), splitting it 76.99 / 58.78 mV.
Load-transient overshoot is deliberately given NO analytic bound, because TI
publishes it only as 50 mV/div plots; it is measured at first article as the new
C-PWR-TRANSIENT-01, and the lever if it fails is C29-C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
Other:
- title: AQROOT Full Beta v2 Main Board -> AQROOT Demo Main Board
Changed lines of the file:
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@@
 	(paper "A3")
 	(title_block
-		(title "AQROOT Full Beta v2 Main Board")
-		(date "2026-07-27")
-		(rev "v2.0-S1-power-tree")
+		(title "AQROOT Demo Main Board")
+		(date "2026-09-20")
+		(rev "D-788")
 		(company "AQROOT Open Hardware")
-		(comment 1 "FULL BETA v2 - FBV2-S1 POWER TREE - DO NOT ROUTE")
-		(comment 2 "PCB FREEZE BLOCKED UNTIL ERC, FOOTPRINT, RF AND DFM REVIEW")
+		(comment 1 "AQROOT DEMO - EXTERNAL REVIEW TARGET D-788 - ROUTED, DRC-CLEAN, NOT AUTHORIZED FOR FABRICATION")
+		(comment 2 "Manufacturer CAM acceptance and first-article acceptance remain outstanding; see docs/full-beta-v2/AQROOT_DEMO_FAB_HANDOFF.md")
+		(comment 3 "D-787 title block read \"Full Beta v2 ... v2.0-S1-power-tree ... 2026-07-27 ... DO NOT ROUTE\" and was corrected at D-788 / R7-D787-17")
 	)
 	(wire
